File: KiCad/Elliott.sch (KiCad schematic (older format))
At the start: 52 parts, among them P1 CONN_01X08, SW1 Reset, SW10 Trace 1, SW11 Interrupt 1, SW12 Interrupt 2, SW13 Interrupt 3, SW14 Obey, SW15 Enter, SW16 Cycle Repeat, SW17 Cycle / Order Stop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

Commit message: 23 April
Parts:
- SW4: footprint Connectors_Molex:Molex_KK-6410-03_03x2.54mm_Straight -> Elliott:C&K_Keyswitch
Changed lines of the file:
@@
 $Descr A3 16535 11693
 encoding utf-8
-Sheet 1 1
+Sheet 1 2
 Title ""
 Date "2017-03-07"
@@
 F 0 "SW4" H 5700 1450 50  0000 C CNN
 F 1 "Key Switch" H 5700 1050 50  0000 C CNN
-F 2 "Connectors_Molex:Molex_KK-6410-03_03x2.54mm_Straight" H 5075 1425 50  0001 C CNN
+F 2 "Elliott:C&K_Keyswitch" H 5075 1425 50  0001 C CNN
 F 3 "" H 5075 1425 50  0000 C CNN
 	1    5700 1250
@@
 Wire Wire Line
 	5725 7025 5725 6175
+$Sheet
+S 13650 975  1825 800
+U 58FC28C7
+F0 "Punch" 60
+F1 "Punch.sch" 60
+$EndSheet
 $EndSCHEMATC
