File: KiCad/CPU.sch (KiCad schematic (older format))
At the start: 29 parts, among them J1 DB9, P1.1 Control Panel, P1.2 Display Unit, P1.3 Tape Punch, P1.4 Tape Reader, P1.5 CONN_01X02, P1.6 Plotter, U1.1 Raspberry_Pi_2_3, U1.2 PCA9516, U1.3 MCP23017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

Commit message: Circuit design updates
Parts:
- removed R1.7, R1.8: 10k, Discret:R5, symbol R
- removed U1.2: PCA9516, Housings_DIP:DIP-16_W7.62mm, symbol PCA9516
- added P1.7: Misc GPIO, Connectors_Terminal_Blocks:TerminalBlock_Pheonix_PT-3.5mm_4pol, symbol CONN_01X04
- R1, R2, R3, R4, R5, R6: value 10k -> 4k7
- U1.2: renamed from U?; footprint (none) -> Ada
Connections:
- net labels added: +5V, SC6, SD6
- net labels removed: +3.3V, DisplayEnable, IOEnable, PanelEnable
- wire segments 153 -> 160
- no-connect marks 43 -> 54
Other:
- moved on the sheet: R5, R6
