File: KiCad/Display.sch (KiCad schematic (older format))
At the start: 110 parts, among them Q1 Q_NPN_BCE, Q2 Q_NPN_BCE, Q3 TIP141, Q4 Q_NPN_BCE

Commit message: Circuit design updates
Parts:
- removed C1: 2200uf 50V, symbol CP
- removed C2: C, symbol CP
- removed C3: 10uf, symbol CP
- removed C5: 1uf, symbol CP
- removed D10, D?: D, symbol D
- removed D1234, D5678: D, symbol D_Bridge_+-AA
- removed D? (x20): LED, symbol LED
- removed F1, F2, F3: Fuse, symbol Fuse
- removed Front, Middle, Rear, SW? (x2): SW_SP3T_Elliott, symbol SW_SP3T_Elliott
- removed P?: CONN_01X05, symbol CONN_01X05
- removed P?: CONN_01X03, symbol CONN_01X03
- removed Q1, Q2, Q4: Q_NPN_BCE, symbol Q_NPN_BCE
- removed Q3: TIP141, TO-220, symbol TIP121
- removed R1, R10, R11, R4, R5, R6, R8, R? (x36): R, symbol R
- removed R15: 236R, symbol R
- removed R3: 1k5, symbol R
- removed R7: 850R, symbol R
- removed R9: 1k, symbol R
- removed RLY1: RLY1, symbol Electromagnetic_Actor
- removed RLY2: Relay 2, symbol Electromagnetic_Actor
- removed T?: Transformer_1P_SS, symbol Transformer_1P_SS
- removed U? (x2): MCP23017, symbol MCP23017
- added C1, C2, C3, C4, DA17, DA18, DB1, DB10, DB11, DB12, DB13, DB14, DB15, DB16, DB17, DB18, DB2, DB3, DB4, DB5, DB6, DB7, DB8, DB9, DQ1, DQ10, DQ11, DQ12, DQ13, DQ14, DQ15, DQ16, DQ17, DQ18, DQ2, DQ3, DQ4, DQ5, DQ6, DQ7, DQ8, DQ9, DS1, DS10, DS11, DS12, DS13, DS14, DS15, DS16, DS17, DS18, DS2, DS3, DS4, DS5, DS6, DS7, DS8, DS9, I1, I2, I3, I4: LED, LEDs:LED_D5.0mm, symbol LED
- added J1: CONN_01X04, Pin_Headers:Pin_Header_Angled_1x04_Pitch2.54mm, symbol CONN_01X04
- added R1, R10, R2, R3, R4, R5, R6, R7, R8, R9: 470R, Connectors_Terminal_Blocks:TerminalBlock_Pheonix_MPT-2.54mm_9pol, symbol ResistorNetwork
- added U1, U2, U3, U4, U6: MCP23017, Elliott:Mirror-DIP-28_W7.62mm, symbol MCP23017
- DA1, DA10, DA11, DA12, DA13, DA14, DA15, DA16, DA2, DA3, DA4, DA5, DA6, DA7, DA8, DA9: renamed from D?; footprint (none) -> LEDs:LED_D5.0mm
Connections:
- net labels added: +5v, 0v, SCL, SDA
- net labels removed: GNDPWR, P4.10, PPC1, PPC4, PPC7PPC10, V+
- wire segments 232 -> 236
- no-connect marks 0 -> 10

Commit message: Finalise display board
Parts:
- renumbered I3 to C1, I4 to C2, DS17 to DA17, DS18 to DA18, DA17 to DS17, DA18 to DS18, C1 to I2, I2 to I3, C2 to I4
Connections:
- wire segments 236 -> 246
Changed lines of the file:
@@
 $EndComp
 $Comp
-L LED DS17
+L LED DA17
 U 1 1 598D9056
 P 8075 2250
-F 0 "DS17" H 7850 2300 50  0000 C CNN
+F 0 "DA17" H 7850 2300 50  0000 C CNN
 F 1 "LED" H 8075 2150 50  0001 C CNN
 F 2 "LEDs:LED_D5.0mm" H 8075 2250 50  0001 C CNN
@@
 $EndComp
 $Comp
-L LED DS18
+L LED DA18
 U 1 1 598D905C
 P 8175 2700
-F 0 "DS18" H 7950 2750 50  0000 C CNN
+F 0 "DA18" H 7950 2750 50  0000 C CNN
 F 1 "LED" H 8175 2600 50  0001 C CNN
 F 2 "LEDs:LED_D5.0mm" H 8175 2700 50  0001 C CNN
@@
 $EndComp
 $Comp
-L LED I2
+L LED I3
 U 1 1 598D9068
 P 8575 2250
-F 0 "I2" H 8350 2300 50  0000 C CNN
+F 0 "I3" H 8350 2300 50  0000 C CNN
 F 1 "LED" H 8575 2150 50  0001 C CNN
 F 2 "LEDs:LED_D5.0mm" H 8575 2250 50  0001 C CNN
@@
 $EndComp
 $Comp
-L LED I3
+L LED C1
 U 1 1 598D906E
 P 8775 2250
-F 0 "I3" H 8550 2300 50  0000 C CNN
+F 0 "C1" H 8550 2300 50  0000 C CNN
 F 1 "LED" H 8775 2150 50  0001 C CNN
 F 2 "LEDs:LED_D5.0mm" H 8775 2250 50  0001 C CNN
@@
 $EndComp
 $Comp
-L LED I4
+L LED C2
 U 1 1 598D9074
 P 8975 2250
-F 0 "I4" H 8750 2300 50  0000 C CNN
+F 0 "C2" H 8750 2300 50  0000 C CNN
 F 1 "LED" H 8975 2150 50  0001 C CNN
 F 2 "LEDs:LED_D5.0mm" H 8975 2250 50  0001 C CNN
@@
 $EndComp
 $Comp
-L LED C2
+L LED I4
 U 1 1 598D9086
 P 8675 2700
-F 0 "C2" H 8450 2750 50  0000 C CNN
+F 0 "I4" H 8450 2750 50  0000 C CNN
 F 1 "LED" H 8675 2600 50  0001 C CNN
 F 2 "LEDs:LED_D5.0mm" H 8675 2700 50  0001 C CNN
@@
 $EndComp
 $Comp
-L LED C1
+L LED I2
 U 1 1 598D908C
 P 8475 2700
-F 0 "C1" H 8250 2750 50  0000 C CNN
+F 0 "I2" H 8250 2750 50  0000 C CNN
 F 1 "LED" H 8475 2600 50  0001 C CNN
 F 2 "LEDs:LED_D5.0mm" H 8475 2700 50  0001 C CNN
@@
 L ResistorNetwork R9
 U 1 1 598D9092
-P 7725 3150
-F 0 "R9" H 7075 3350 60  0000 C CNN
-F 1 "470R" H 7625 3600 60  0000 C CNN
-F 2 "Connectors_Terminal_Blocks:TerminalBlock_Pheonix_MPT-2.54mm_9pol" H 8425 3150 60  0001 C CNN
-F 3 "" H 8425 3150 60  0001 C CNN
-	1    7725 3150
-	-1   0    0    1
-$EndComp
-$Comp
-L LED DA18
+P 7125 3500
+F 0 "R9" H 6475 3700 60  0000 C CNN
+F 1 "470R" H 7025 3950 60  0000 C CNN
+F 2 "Connectors_Terminal_Blocks:TerminalBlock_Pheonix_MPT-2.54mm_9pol" H 7825 3500 60  0001 C CNN
+F 3 "" H 7825 3500 60  0001 C CNN
+	1    7125 3500
+	0    -1   -1   0
+$EndComp
+$Comp
+L LED DS18
 U 1 1 598D9098
 P 7575 2700
-F 0 "DA18" H 7350 2750 50  0000 C CNN
+F 0 "DS18" H 7350 2750 50  0000 C CNN
 F 1 "LED" H 7575 2600 50  0001 C CNN
 F 2 "LEDs:LED_D5.0mm" H 7575 2700 50  0001 C CNN
@@
 $EndComp
 $Comp
-L LED DA17
+L LED DS17
 U 1 1 598D909E
 P 7475 2250
-F 0 "DA17" H 7250 2300 50  0000 C CNN
+F 0 "DS17" H 7250 2300 50  0000 C CNN
 F 1 "LED" H 7475 2150 50  0001 C CNN
 F 2 "LEDs:LED_D5.0mm" H 7475 2250 50  0001 C CNN
@@
 	8175 2050 8175 2550
 Wire Wire Line
-	7475 2400 7475 3000
-Wire Wire Line
-	7575 2850 7575 3000
-Wire Wire Line
-	7675 2400 7675 3000
-Wire Wire Line
-	7775 2850 7775 3000
-Wire Wire Line
-	7875 2400 7875 3000
-Wire Wire Line
-	7975 2850 7975 3000
-Wire Wire Line
-	8075 2400 8075 3000
-Wire Wire Line
-	8175 2850 8175 3000
-Wire Wire Line
-	7825 3850 7825 3900
-Wire Wire Line
-	7825 3900 9425 3900
-Wire Wire Line
 	9425 3900 9425 1550
 Wire Wire Line
@@
 Wire Wire Line
 	7850 5075 7600 5075
+Wire Wire Line
+	6425 3600 6425 4400
+Wire Wire Line
+	6425 4400 8525 4400
+Wire Wire Line
+	8525 4400 8525 3900
+Wire Wire Line
+	8525 3900 9425 3900
+Wire Wire Line
+	8075 2400 8075 3950
+Wire Wire Line
+	8075 3950 7275 3950
+Wire Wire Line
+	8175 2850 8175 3850
+Wire Wire Line
+	8175 3850 7275 3850
+Wire Wire Line
+	7875 2400 7875 3750
+Wire Wire Line
+	7875 3750 7275 3750
+Wire Wire Line
+	7975 2850 7975 3650
+Wire Wire Line
+	7975 3650 7275 3650
+Wire Wire Line
+	7675 2400 7675 3550
+Wire Wire Line
+	7675 3550 7275 3550
+Wire Wire Line
+	7775 2850 7775 3450
+Wire Wire Line
+	7775 3450 7275 3450
+Wire Wire Line
+	7475 2400 7475 3350
+Wire Wire Line
+	7475 3350 7275 3350
+Wire Wire Line
+	7575 2850 7575 3250
+Wire Wire Line
+	7575 3250 7275 3250
 $EndSCHEMATC
