File: KiCad/CPU/CPU.kicad_pcb (KiCad board)
At the start: 2 copper layers, 265.4 x 95.2 mm, 32 parts, among them P1.1 Control Panel, P1.2 Display Unit, P1.3 Tape Punch, P1.4 Tape Reader, P1.5 CONN_01X02, P1.6 Plotter, P1.7 Misc GPIO, P1.8 IO Control, P1.9 RS232, U1.1 Raspberry_Pi_2_3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

Commit message: Update CPU and TTY Interface board
Parts:
- P1.7: value Misc GPIO -> MISC GPIO; footprint lib_fp:PhoenixContact_MC-G_04x3.50mm_Angled -> lib_fp:PhoenixContact_MC-G_06x3.50mm_Angled
- P1.8: footprint lib_fp:PhoenixContact_MC-G_04x3.50mm_Angled -> lib_fp:PhoenixContact_MC-G_05x3.50mm_Angled
- P1.9: footprint lib_fp:PhoenixContact_MC-G_04x3.50mm_Angled -> lib_fp:PhoenixContact_MC-G_03x3.50mm_Angled
- moved R5 0.08 mm to (66.7, 34.4)
Connections:
- C9 pad 1: Net-(C9-Pad1) -> +5V
- P1.7 pad 4: 0v -> Net-(P1.7-Pad4)
- P1.8 pad 1: Net-(C9-Pad1) -> +5V
- P1.9 pad 1: Net-(P1.9-Pad1) -> 0v
- U1.1 pad 11: Net-(P1.7-Pad3) -> Net-(P1.7-Pad4)
- U1.1 pad 12: Net-(P1.7-Pad2) -> Net-(P1.7-Pad3)
- U1.1 pad 29: Net-(U1.1-Pad29) -> Net-(P1.2-Pad5)
- U1.1 pad 31: Net-(U1.1-Pad31) -> Net-(P1.8-Pad5)
- U1.1 pad 35: Net-(P1.7-Pad1) -> Net-(P1.7-Pad2)
- U1.1 pad 36: Net-(U1.1-Pad36) -> Net-(P1.7-Pad5)
- U1.1 pad 37: Net-(U1.1-Pad37) -> Net-(P1.7-Pad1)
- U1.4 pad 13: Net-(P1.9-Pad2) -> Net-(P1.9-Pad3)
- U1.4 pad 14: Net-(P1.9-Pad3) -> Net-(P1.9-Pad2)
Routing:
- net Net-(P1.7-Pad4): track 0.00 -> 120.0 mm
- net Net-(P1.8-Pad5): track 0.00 -> 111.0 mm, vias 0 -> 5
- net Net-(P1.7-Pad5): track 0.00 -> 90.0 mm
- net Net-(P1.2-Pad5): track 0.00 -> 77.0 mm, vias 0 -> 3
- net Net-(P1.7-Pad2): track 111.3 -> 78.6 mm, vias 1 -> 0
- net +5V: track 639.3 -> 658.6 mm
- net Net-(P1.7-Pad1): track 80.8 -> 71.9 mm
- net Net-(C9-Pad1): track 5.62 -> 0.00 mm
- net 0v: track 850.6 -> 846.0 mm
- net Net-(P1.9-Pad2): track 23.4 -> 26.1 mm
- net Net-(P1.7-Pad3): track 113.0 -> 115.6 mm, vias 2 -> 0
- net Net-(P1.8-Pad3): track 150.6 -> 152.3 mm
- net Net-(P1.9-Pad3): track 18.8 -> 19.9 mm
- net PunchA: track 250.9 -> 250.2 mm
Other:
- board text added: "26|19|18|17|16|+0V"
- board text added: "D7|D6|D5|D4|D3|D2|D1|D0|20|21|+5|+0"
- board text added: "Display ________________ 05|0V|SD|SC|5V"
- board text added: "Panel ________________ 04|0V|SD|SC|5V"
- board text added: "RS232 ________ I|O|0V"
- board text removed: "04|0V|SD|SC|5V"
- board text removed: "0V|SD|SC|5V"
- board text removed: "19|18|17|+0V"

Commit message: New CPU Design
Parts:
- added REF**: MountingHole_3mm_Pad, Mounting_Holes:MountingHole_3mm_Pad, F.Cu at (300.0, 27.0)
- added REF**: MountingHole_3mm_Pad, Mounting_Holes:MountingHole_3mm_Pad, F.Cu at (43.0, 27.0)
- added REF**: MountingHole_3mm_Pad, Mounting_Holes:MountingHole_3mm_Pad, F.Cu at (43.0, 114.0)
- added REF**: MountingHole_3mm_Pad, Mounting_Holes:MountingHole_3mm_Pad, F.Cu at (300.0, 114.0)
- P1.1, P1.2, P1.8: footprint lib_fp:PhoenixContact_MC-G_05x3.50mm_Angled -> lib_fp:Harwin_LTek-Male_05_P2.00mm_Vertical_StrainRelief
- P1.3, P1.4, P1.6: footprint lib_fp:PhoenixContact_MC-G_12x3.50mm_Angled -> lib_fp:Harwin_LTek-Male_2x06_P2.00mm_Vertical_StrainRelief
- P1.5: footprint lib_fp:PhoenixContact_MC-G_02x3.50mm_Angled -> lib_fp:Harwin_LTek-Male_02_P2.00mm_Vertical_StrainRelief
- P1.7: footprint lib_fp:PhoenixContact_MC-G_06x3.50mm_Angled -> lib_fp:Harwin_LTek-Male_06_P2.00mm_Vertical_StrainRelief
- P1.9: footprint lib_fp:PhoenixContact_MC-G_03x3.50mm_Angled -> lib_fp:Harwin_LTek-Male_03_P2.00mm_Vertical_StrainRelief
- moved P1.6 78.9 mm to (263.9, 33.7), turned to 0 degrees
- moved U1.5 69.8 mm to (213.0, 64.6), turned to 0 degrees
- moved R2 66.5 mm to (174.9, 102.9)
- moved U1.3 57.5 mm to (189.0, 64.6)
- moved R1 55.0 mm to (181.4, 102.9)
- moved R8 25.5 mm to (198.6, 41.9)
- moved R9 25.1 mm to (184.1, 41.9)
- moved P1.3 22.8 mm to (237.1, 33.7)
- moved P1.7 20.1 mm to (150.1, 103.9), turned to 90 degrees
- moved P1.9 19.2 mm to (172.9, 33.2)
- moved P1.8 18.6 mm to (195.1, 33.5)
- moved C9 17.3 mm to (183.9, 46.6), turned to 180 degrees
- moved P1.4 12.3 mm to (209.4, 34.0)
- moved P1.1 7.00 mm to (59.4, 33.0)
- moved P1.2 6.18 mm to (108.4, 33.1)
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Connections:
- P1.1 pad 2: SC6 -> SC7
- P1.1 pad 3: SD6 -> SD7
- R5 pad 1: SD6 -> SD7
- R6 pad 1: SC6 -> SC7
- U1.2 pad 21: SD6 -> Net-(P1.2-Pad3)
- U1.2 pad 22: SC6 -> Net-(P1.2-Pad2)
- U1.2 pad 23: Net-(P1.2-Pad3) -> SD7
- U1.2 pad 24: Net-(P1.2-Pad2) -> SC7
Routing:
- net Net-(P1.8-Pad5): track 111.0 -> 339.7 mm, vias 5 -> 2
- net 0v: track 846.0 -> 713.2 mm
- net ReaderB: track 192.8 -> 315.7 mm, vias 0 -> 1
- net /Black: track 45.5 -> 96.3 mm
- net /Mauve: track 37.5 -> 86.3 mm
- net /Blue: track 29.5 -> 77.3 mm
- net SD7: track 0.00 -> 46.3 mm
- net ReaderA: track 181.0 -> 227.1 mm
- net SDA: track 201.5 -> 156.0 mm
- net SCL: track 208.4 -> 162.9 mm
- net /Yellow: track 21.8 -> 64.7 mm
- net SC7: track 0.00 -> 42.1 mm
- net SD6: track 39.7 -> 0.00 mm
- net Net-(P1.7-Pad4): track 120.0 -> 81.0 mm
- net Net-(P1.4-Pad8): track 27.7 -> 66.2 mm
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Other:
- board text added: "D6|D4|D2|D0|21|+0 D7|D5|D3|D1|20|+5"
- board text added: "D6|D4|D2|D0|23|+0 D7|D5|D3|D1|22|+5"
- board text added: "D6|D4|D2|D0|25|+0 D7|D5|D3|D1|24|+5"
- board text added: "IO Control ________________ 06|0V|SD|SC|5V"
- board text added: "Plotter"
- board text added: "Punch"
- board text added: "Reader"
- board text removed: "D7|D6|D5|D4|D3|D2|D1|D0|20|21|+5|+0"
- board text removed: "D7|D6|D5|D4|D3|D2|D1|D0|22|23|+5|+0"
- board text removed: "D7|D6|D5|D4|D3|D2|D1|D0|24|25|+5|+0"
- board text removed: "Plotter ____________________________________"
- board text removed: "Punch ____________________________________"
- board text removed: "Reader ____________________________________"

Commit message: Add footprints and gerber plot
Parts:
- removed the REF** at (300.0, 27.0)
- removed the REF** at (43.0, 27.0)
- removed the REF** at (43.0, 114.0)
- removed the REF** at (300.0, 114.0)
- added REF**: MountingHole_3.5mm, Mounting_Holes:MountingHole_3.5mm, F.Cu at (44.0, 27.0)
- added REF**: MountingHole_3.5mm, Mounting_Holes:MountingHole_3.5mm, F.Cu at (44.0, 114.0)
- added REF**: MountingHole_3.5mm, Mounting_Holes:MountingHole_3.5mm, F.Cu at (300.0, 114.0)
- added REF**: MountingHole_3.5mm, Mounting_Holes:MountingHole_3.5mm, F.Cu at (300.0, 27.0)
Changed lines of the file:
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@@
 (kicad_pcb (version 4) (host pcbnew 4.0.7)
   (general
-    (links 0)
+    (links 128)
     (no_connects 0)
-    (area 39.319999 22.809999 304.850001 118.160001)
+    (area 35.571429 21.225 308.428572 119.875)
     (thickness 1.6)
     (drawings 22)
@@
     (mod_text_size 1 1)
     (mod_text_width 0.15)
-    (pad_size 6 6)
-    (pad_drill 3)
+    (pad_size 3.5 3.5)
+    (pad_drill 3.5)
     (pad_to_mask_clearance 0)
     (aux_axis_origin 36.12 117.11)
@@
       (drillshape 0)
       (scaleselection 1)
-      (outputdirectory "CPU Board/"))
+      (outputdirectory gerber/))
   )
   (net 0 "")
@@
     (add_net 0v)
   )
-  (module Mounting_Holes:MountingHole_3mm_Pad (layer F.Cu)
-    (at 300 27)
-    (descr "Mounting Hole 3mm")
-    (tags "mounting hole 3mm")
-    (attr virtual)
-    (fp_text reference REF** (at 0 -4) (layer F.SilkS)
-      (effects (font (size 1 1) (thickness 0.15)))
-    )
-    (fp_text value MountingHole_3mm_Pad (at 0 4) (layer F.Fab)
-      (effects (font (size 1 1) (thickness 0.15)))
-    )
-    (fp_text user %R (at 0.3 0) (layer F.Fab)
-      (effects (font (size 1 1) (thickness 0.15)))
-    )
-    (fp_circle (center 0 0) (end 3 0) (layer Cmts.User) (width 0.15))
-    (fp_circle (center 0 0) (end 3.25 0) (layer F.CrtYd) (width 0.05))
-    (pad 1 thru_hole circle (at 0 0) (size 6 6) (drill 3) (layers *.Cu *.Mask))
-  )
   (module lib_fp:RASPI_BPLUS_MIRRORED (layer F.Cu)
     (at 82.55 99.06)
@@
     )
   )
-  (module Mounting_Holes:MountingHole_3mm_Pad (layer F.Cu)
-    (at 43 27)
-    (descr "Mounting Hole 3mm")
-    (tags "mounting hole 3mm")
+  (module Mounting_Holes:MountingHole_3.5mm (layer F.Cu)
+    (at 44 27)
+    (descr "Mounting Hole 3.5mm, no annular")
+    (tags "mounting hole 3.5mm no annular")
     (attr virtual)
-    (fp_text reference REF** (at 0 -4) (layer F.SilkS)
-      (effects (font (size 1 1) (thickness 0.15)))
-    )
-    (fp_text value MountingHole_3mm_Pad (at 0 4) (layer F.Fab)
+    (fp_text reference REF** (at 0 -4.5) (layer F.SilkS)
+      (effects (font (size 1 1) (thickness 0.15)))
+    )
+    (fp_text value MountingHole_3.5mm (at 0 4.5) (layer F.Fab)
       (effects (font (size 1 1) (thickness 0.15)))
     )
@@
       (effects (font (size 1 1) (thickness 0.15)))
     )
-    (fp_circle (center 0 0) (end 3 0) (layer Cmts.User) (width 0.15))
-    (fp_circle (center 0 0) (end 3.25 0) (layer F.CrtYd) (width 0.05))
-    (pad 1 thru_hole circle (at 0 0) (size 6 6) (drill 3) (layers *.Cu *.Mask))
-  )
-  (module Mounting_Holes:MountingHole_3mm_Pad (layer F.Cu)
-    (at 43 114)
-    (descr "Mounting Hole 3mm")
-    (tags "mounting hole 3mm")
+    (fp_circle (center 0 0) (end 3.5 0) (layer Cmts.User) (width 0.15))
+    (fp_circle (center 0 0) (end 3.75 0) (layer F.CrtYd) (width 0.05))
+    (pad "" np_thru_hole circle (at 0.06 0) (size 3.5 3.5) (drill 3.5) (layers *.Cu *.Mask))
+  )
+  (module Mounting_Holes:MountingHole_3.5mm (layer F.Cu)
+    (at 44 114)
+    (descr "Mounting Hole 3.5mm, no annular")
+    (tags "mounting hole 3.5mm no annular")
     (attr virtual)
-    (fp_text reference REF** (at 0 -4) (layer F.SilkS)
-      (effects (font (size 1 1) (thickness 0.15)))
-    )
-    (fp_text value MountingHole_3mm_Pad (at 0 4) (layer F.Fab)
+    (fp_text reference REF** (at 0 -4.5) (layer F.SilkS)
+      (effects (font (size 1 1) (thickness 0.15)))
+    )
+    (fp_text value MountingHole_3.5mm (at 0 4.5) (layer F.Fab)
       (effects (font (size 1 1) (thickness 0.15)))
     )
@@
       (effects (font (size 1 1) (thickness 0.15)))
     )
-    (fp_circle (center 0 0) (end 3 0) (layer Cmts.User) (width 0.15))
-    (fp_circle (center 0 0) (end 3.25 0) (layer F.CrtYd) (width 0.05))
-    (pad 1 thru_hole circle (at 0 0) (size 6 6) (drill 3) (layers *.Cu *.Mask))
-  )
-  (module Mounting_Holes:MountingHole_3mm_Pad (layer F.Cu)
+    (fp_circle (center 0 0) (end 3.5 0) (layer Cmts.User) (width 0.15))
+    (fp_circle (center 0 0) (end 3.75 0) (layer F.CrtYd) (width 0.05))
+    (pad 1 np_thru_hole circle (at 0 0) (size 3.5 3.5) (drill 3.5) (layers *.Cu *.Mask))
+  )
+  (module Mounting_Holes:MountingHole_3.5mm (layer F.Cu)
     (at 300 114)
-    (descr "Mounting Hole 3mm")
-    (tags "mounting hole 3mm")
+    (descr "Mounting Hole 3.5mm, no annular")
+    (tags "mounting hole 3.5mm no annular")
     (attr virtual)
-    (fp_text reference REF** (at 0 -4) (layer F.SilkS)
-      (effects (font (size 1 1) (thickness 0.15)))
-    )
-    (fp_text value MountingHole_3mm_Pad (at 0 4) (layer F.Fab)
+    (fp_text reference REF** (at 0 -4.5) (layer F.SilkS)
+      (effects (font (size 1 1) (thickness 0.15)))
+    )
+    (fp_text value MountingHole_3.5mm (at 0 4.5) (layer F.Fab)
       (effects (font (size 1 1) (thickness 0.15)))
     )
@@
       (effects (font (size 1 1) (thickness 0.15)))
     )
-    (fp_circle (center 0 0) (end 3 0) (layer Cmts.User) (width 0.15))
-    (fp_circle (center 0 0) (end 3.25 0) (layer F.CrtYd) (width 0.05))
-    (pad 1 thru_hole circle (at 0 0) (size 6 6) (drill 3) (layers *.Cu *.Mask))
+    (fp_circle (center 0 0) (end 3.5 0) (layer Cmts.User) (width 0.15))
+    (fp_circle (center 0 0) (end 3.75 0) (layer F.CrtYd) (width 0.05))
+    (pad 1 np_thru_hole circle (at 0 0) (size 3.5 3.5) (drill 3.5) (layers *.Cu *.Mask))
+  )
+  (module Mounting_Holes:MountingHole_3.5mm (layer F.Cu)
+    (at 300 27)
+    (descr "Mounting Hole 3.5mm, no annular")
+    (tags "mounting hole 3.5mm no annular")
+    (attr virtual)
+    (fp_text reference REF** (at 0 -4.5) (layer F.SilkS)
+      (effects (font (size 1 1) (thickness 0.15)))
+    )
+    (fp_text value MountingHole_3.5mm (at 0 4.5) (layer F.Fab)
+      (effects (font (size 1 1) (thickness 0.15)))
+    )
+    (fp_text user %R (at 0.3 0) (layer F.Fab)
+      (effects (font (size 1 1) (thickness 0.15)))
+    )
+    (fp_circle (center 0 0) (end 3.5 0) (layer Cmts.User) (width 0.15))
+    (fp_circle (center 0 0) (end 3.75 0) (layer F.CrtYd) (width 0.05))
+    (pad 1 np_thru_hole circle (at 0 0) (size 3.5 3.5) (drill 3.5) (layers *.Cu *.Mask))
   )
   (gr_text "RS232\n________\nI|O|0V" (at 161.37 32.61) (layer F.SilkS)

Commit message: Improvements to PCBs and footprints
Parts:
- U1.2: footprint lib_fp:Ada -> lib_fp:ADAMult
Connections:
- P1.7 pad 1: Net-(P1.7-Pad1) -> +5V
- U1.1 pad 37: Net-(P1.7-Pad1) -> Net-(U1.1-Pad37)
Routing:
- net Net-(P1.7-Pad1): track 51.5 -> 0.00 mm
- net +5V: track 674.7 -> 699.9 mm
- net PunchA: track 231.2 -> 234.0 mm
- net ReaderA: track 227.1 -> 229.4 mm
- net PlotterB: track 226.2 -> 228.1 mm
- net ReaderB: track 315.7 -> 317.4 mm
- net PlotterA: track 222.2 -> 224.0 mm
- net Net-(P1.8-Pad5): track 339.7 -> 341.2 mm
- net PunchB: track 288.3 -> 289.3 mm
- net Net-(P1.7-Pad5): track 74.6 -> 75.2 mm
- net Net-(P1.7-Pad4): track 81.0 -> 81.6 mm
