File: KiCad/IOC/IOC.kicad_pcb (KiCad board)
At the start: 2 copper layers, 32 parts, among them J1 Conn_01x06, SW1 Reader Attach, SW10 Input, SW11 Output, SW2 Reader Detach, SW3 Read, SW4 Stop, SW5 List, SW6 Delete, SW7 Punch Attach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

Commit message: Improvements to PCBs and footprints
Parts:
- moved R1 130.1 mm to (183.3, 36.9), turned to 270 degrees
- moved R12 89.4 mm to (55.2, 82.1), turned to 180 degrees
- moved R5 79.5 mm to (33.4, 36.9), turned to 270 degrees
- moved R11 69.8 mm to (104.8, 81.9), turned to 180 degrees
- moved R9 65.9 mm to (120.5, 36.8)
- moved R3 33.5 mm to (65.7, 36.6)
- moved D10 13.9 mm to (203.3, 58.8)
- moved D11 13.9 mm to (73.3, 58.8)
- moved D12 13.9 mm to (128.3, 58.8)
- moved J1 13.9 mm to (264.1, 37.3)
- moved R10 13.9 mm to (195.7, 36.8)
- moved R13 13.9 mm to (252.3, 55.5)
- moved R14 13.9 mm to (252.3, 50.0)
- moved R15 13.9 mm to (252.3, 44.8)
- moved R2 13.9 mm to (55.5, 116.5)
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Routing:
- net Net-(SW3-Pad2): track 0.00 -> 429.4 mm
- net Net-(SW4-Pad2): track 0.00 -> 206.8 mm
- net Net-(SW1-Pad4): track 0.00 -> 199.0 mm
- net Net-(SW1-Pad2): track 0.00 -> 186.7 mm, vias 0 -> 1
- net Net-(SW5-Pad2): track 0.00 -> 160.9 mm
- net 5v: track 275.8 -> 409.4 mm
- net 0v: track 826.9 -> 869.7 mm
- net Net-(R5-Pad2): track 17.1 -> 4.22 mm
- net Net-(R11-Pad1): track 8.28 -> 17.3 mm
- net Net-(R1-Pad2): track 11.7 -> 4.22 mm
- net Net-(J1-Pad5): track 139.6 -> 144.7 mm
- net Net-(D12-Pad1): track 4.22 -> 8.27 mm
- net Net-(D11-Pad1): track 4.22 -> 8.03 mm
- net Net-(R12-Pad1): track 8.03 -> 11.7 mm
- net Net-(J1-Pad6): track 144.2 -> 147.5 mm
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Other:
- board outline added: 265 x 135 mm

Commit message: New IO Board PCB design
Parts:
- removed R1, R10, R11, R12, R2, R3, R4, R5, R6, R7, R8, R9: R, ioc:R5
- D10, D11, D12: footprint ioc:EAO31 -> ioc:EAO31_Led_Only
- U1, U2: footprint ioc:DIP-28_W7.62mm_Socket -> ioc:DIP-28_W7.62mm_Socket_Mirror
- moved J1 248.2 mm to (23.0, 96.4), turned to 90 degrees
- moved R15 245.8 mm to (24.8, 137.9), turned to 270 degrees
- moved R14 239.0 mm to (30.1, 137.9), turned to 270 degrees
- moved R13 231.8 mm to (35.6, 137.9), turned to 270 degrees
- moved U2 144.1 mm to (91.8, 83.1), turned to 0 degrees
- moved U1 85.0 mm to (146.4, 82.4), turned to 0 degrees
Connections:
- net Net-(SW7-Pad2) renamed Punch_Sw
- net Net-(SW7-Pad4) renamed Punch_Led
- D10 pad 1: Net-(D10-Pad1) -> 0v
- D10 pad 2: Net-(D10-Pad2) -> Reload_Led
- D11 pad 1: Net-(D11-Pad1) -> 0v
- D11 pad 2: Net-(D11-Pad2) -> Holdup_Led
- D12 pad 1: Net-(D12-Pad1) -> 0v
- D12 pad 2: Net-(D12-Pad2) -> Demand_Led
- J1 pad 1: (no net) -> Net-(J1-Pad1)
- SW1 pad 2: Net-(SW1-Pad2) -> Reader_Sw
- SW1 pad 3: Net-(R12-Pad1) -> 0v
- SW1 pad 4: Net-(SW1-Pad4) -> Reader_Led
- SW10 pad 2: Net-(SW10-Pad2) -> Input_RDR
- SW10 pad 4: Net-(SW10-Pad4) -> Input_TTY
- SW11 pad 2: Net-(SW11-Pad2) -> Output_PCH
- SW11 pad 4: Net-(SW11-Pad4) -> Output_TTY
- SW2 pad 2: Net-(SW2-Pad2) -> Reader_Detach_Sw
- SW2 pad 3: Net-(R2-Pad1) -> 0v
- SW2 pad 4: Net-(SW2-Pad4) -> Reader_Detach_Led
- SW3 pad 2: Net-(SW3-Pad2) -> Read_Sw
- SW3 pad 3: Net-(R5-Pad2) -> 0v
- SW3 pad 4: Net-(SW3-Pad4) -> Read_Led
- SW4 pad 2: Net-(SW4-Pad2) -> Stop_Sw
- SW4 pad 3: Net-(R4-Pad2) -> 0v
- SW4 pad 4: Net-(SW4-Pad4) -> Stop_Led
- SW5 pad 2: Net-(SW5-Pad2) -> List_Sw
- SW5 pad 3: Net-(R11-Pad1) -> 0v
- SW5 pad 4: 5v -> List_Led
- SW6 pad 2: Net-(SW6-Pad2) -> Delete_Sw
- SW6 pad 3: Net-(R6-Pad1) -> 0v
- SW6 pad 4: 5v -> Delete_Led
- SW7 pad 3: Net-(R7-Pad2) -> 0v
- SW8 pad 2: Net-(SW8-Pad2) -> Punch_Detach_Sw
- SW8 pad 3: Net-(R8-Pad1) -> 0v
- SW8 pad 4: Net-(SW8-Pad4) -> Punch_Detach_Led
- SW9 pad 2: Net-(SW9-Pad2) -> Runout_Sw
- SW9 pad 3: Net-(R1-Pad2) -> 0v
- SW9 pad 4: Net-(SW9-Pad4) -> Runout_Led
- U1 pad 1: (no net) -> Output_PCH
- U1 pad 2: (no net) -> Runout_Led
- U1 pad 21: Net-(SW3-Pad4) -> Delete_Led
- U1 pad 22: Net-(SW4-Pad2) -> Delete_Sw
- U1 pad 23: Net-(SW4-Pad4) -> List_Led
- U1 pad 24: Net-(D11-Pad2) -> List_Sw
- U1 pad 25: Net-(D12-Pad2) -> Input_TTY
- U1 pad 26: Net-(SW9-Pad2) -> Input_RDR
- U1 pad 27: Net-(SW9-Pad4) -> Demand_Led
- U1 pad 28: Net-(D10-Pad2) -> Output_TTY
- U1 pad 3: (no net) -> Runout_Sw
- U1 pad 4: (no net) -> Reload_Led
- U1 pad 7: (no net) -> Punch_Detach_Sw
- U1 pad 8: Net-(SW3-Pad2) -> Punch_Detach_Led
- U2 pad 1: Net-(SW8-Pad2) -> Holdup_Led
- U2 pad 2: Net-(SW8-Pad4) -> Net-(U2-Pad2)
- U2 pad 21: (no net) -> Reader_Detach_Led
- U2 pad 22: Net-(SW5-Pad2) -> Reader_Detach_Sw
- U2 pad 23: Net-(SW1-Pad2) -> Reader_Led
- U2 pad 24: Net-(SW1-Pad4) -> Reader_Sw
- U2 pad 25: Net-(SW11-Pad2) -> Read_Led
- U2 pad 26: Net-(SW11-Pad4) -> Read_Sw
- U2 pad 27: Net-(SW10-Pad2) -> Stop_Led
- U2 pad 28: Net-(SW10-Pad4) -> Stop_Sw
- U2 pad 3: Net-(SW2-Pad2) -> Net-(U2-Pad3)
- U2 pad 4: Net-(SW2-Pad4) -> Net-(U2-Pad4)
- U2 pad 5: Net-(SW6-Pad2) -> Net-(U2-Pad5)
- U2 pad 6: (no net) -> Net-(U2-Pad6)
- U2 pad 7: (no net) -> Net-(U2-Pad7)
- U2 pad 8: (no net) -> Net-(U2-Pad8)
Routing:
- net Net-(SW3-Pad2): track 429.4 -> 0.00 mm
- net 0v: track 869.7 -> 630.5 mm
- net Net-(SW3-Pad4): track 221.4 -> 0.00 mm
- net Net-(SW4-Pad2): track 206.8 -> 0.00 mm
- net Net-(SW1-Pad4): track 199.0 -> 0.00 mm
- net Net-(SW4-Pad4): track 195.0 -> 0.00 mm
- net 5v: track 409.4 -> 217.0 mm
- net Net-(SW1-Pad2): track 186.7 -> 0.00 mm, vias 1 -> 0
- net Net-(SW2-Pad4): track 183.7 -> 0.00 mm
- net Net-(D11-Pad2): track 180.6 -> 0.00 mm
- net Net-(SW2-Pad2): track 178.7 -> 0.00 mm
- net Net-(SW5-Pad2): track 160.9 -> 0.00 mm
- net Net-(SW10-Pad4): track 151.3 -> 0.00 mm
- net Net-(SW10-Pad2): track 148.8 -> 0.00 mm
- net Net-(SW6-Pad2): track 123.2 -> 0.00 mm
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Other:
- board size 265 x 135 mm -> 200 x 110 mm
