File: KiCad/Real903/A-GJ/A-GJ.sch (KiCad schematic (older format))
At the start: 3 parts, among them J1 J1

Commit message: Update for PCB Design
Parts:
- added D1, D10, D11, D12, D13, D14, D15, D16, D17, D18, D19, D2, D20, D21, D22, D23, D24, D25, D26, D27, D3, D4, D5, D6, D7, D8, D9: D, ELLIOTT:D_DO-35_SOD27_P7.62mm_Horizontal, symbol Device:D
- added U1: LS03, ELLIOTT:LSA, symbol LSA:LS03
- added U2, U3, U4, U5: LS02, ELLIOTT:LSA, symbol LSA:LS02
- added U6: LS01, ELLIOTT:LSA, symbol LSA:LS01
- renumbered C2 to C1, C1 to C2
Connections:
- net labels added: II10m, II11m, II12m, II13m, II14m, II15m, II16m, II17m, II18m, II1m, II2m, II3m, II4m, II5m, II6m, II7m, II8m, II9m, IIG, IIG-, IIS, J1', J10, J11, J12, J13, J14-, J15-, J16-, J2-', J3', J3-', J4-, J5, J6, J7, J8, J9, U3GND
- net labels removed: 1, 10, 3, 5, 6, 7, 8, 9, AA, AB, AC, AD, AE, AF, AH, AJ, C, CA2, CA2-, CB, D, DA, DE, E, F, H, J, K, L, M, N, P, R, S, S0c, S1c, S2b, S3b, T, U, V, W, X, Y, Z
- wire segments 179 -> 246
- no-connect marks 19 -> 34
Other:
- note added: "8180| -3"
- note added: "8181| 0 8180"
- note added: "IIG is TRUE when we are at address\n8180 and above"
