File: KiCad/Real903/LS03/LS03.sch (KiCad schematic (older format))
At the start: 22 parts, among them J1 LSAConnect

Commit message: Update for PCB Design
Parts:
- VT1, VT2, VT3: value BC547 -> BC548; footprint ELLIOTT:TO-92 -> ELLIOTT:TO-92L_Inline
Connections:
- wire segments 69 -> 72
Changed lines of the file:
@@
 P 2950 1450
 F 0 "VT1" H 3150 1500 50  0000 L CNN
-F 1 "BC547" H 3150 1400 50  0000 L CNN
-F 2 "ELLIOTT:TO-92" H 3150 1550 50  0001 C CNN
+F 1 "BC548" H 3150 1400 50  0000 L CNN
+F 2 "ELLIOTT:TO-92L_Inline" H 3150 1550 50  0001 C CNN
 F 3 "" H 2950 1450 50  0001 C CNN
 	1    2950 1450
@@
 P 2950 2475
 F 0 "VT2" H 3150 2525 50  0000 L CNN
-F 1 "BC547" H 3150 2425 50  0000 L CNN
-F 2 "ELLIOTT:TO-92" H 3150 2575 50  0001 C CNN
+F 1 "BC548" H 3150 2425 50  0000 L CNN
+F 2 "ELLIOTT:TO-92L_Inline" H 3150 2575 50  0001 C CNN
 F 3 "" H 2950 2475 50  0001 C CNN
 	1    2950 2475
@@
 P 2950 3500
 F 0 "VT3" H 3150 3550 50  0000 L CNN
-F 1 "BC547" H 3150 3450 50  0000 L CNN
-F 2 "ELLIOTT:TO-92" H 3150 3600 50  0001 C CNN
+F 1 "BC548" H 3150 3450 50  0000 L CNN
+F 2 "ELLIOTT:TO-92L_Inline" H 3150 3600 50  0001 C CNN
 F 3 "" H 2950 3500 50  0001 C CNN
 	1    2950 3500
@@
 Wire Wire Line
 	1525 2175 1850 2175
+$Comp
+L power:PWR_FLAG #FLG0101
+U 1 1 5C75E1D0
+P 4575 4900
+F 0 "#FLG0101" H 4575 4975 50  0001 C CNN
+F 1 "PWR_FLAG" H 4575 5073 50  0000 C CNN
+F 2 "" H 4575 4900 50  0001 C CNN
+F 3 "~" H 4575 4900 50  0001 C CNN
+	1    4575 4900
+	-1   0    0    1
+$EndComp
+$Comp
+L power:PWR_FLAG #FLG0102
+U 1 1 5C75E24A
+P 5100 4900
+F 0 "#FLG0102" H 5100 4975 50  0001 C CNN
+F 1 "PWR_FLAG" H 5100 5073 50  0000 C CNN
+F 2 "" H 5100 4900 50  0001 C CNN
+F 3 "~" H 5100 4900 50  0001 C CNN
+	1    5100 4900
+	-1   0    0    1
+$EndComp
+$Comp
+L power:PWR_FLAG #FLG0103
+U 1 1 5C75E304
+P 5575 4900
+F 0 "#FLG0103" H 5575 4975 50  0001 C CNN
+F 1 "PWR_FLAG" H 5575 5073 50  0000 C CNN
+F 2 "" H 5575 4900 50  0001 C CNN
+F 3 "~" H 5575 4900 50  0001 C CNN
+	1    5575 4900
+	-1   0    0    1
+$EndComp
+Text GLabel 5575 4750 1    50   Input ~ 0
+0v
+Wire Wire Line
+	5575 4750 5575 4900
+Text GLabel 5100 4750 1    50   Input ~ 0
++6v
+Wire Wire Line
+	5100 4750 5100 4900
+Text GLabel 4575 4750 1    50   Input ~ 0
+-6v
+Wire Wire Line
+	4575 4750 4575 4900
 $EndSCHEMATC
