File: KiCad/Real903/LS04/LS04.kicad_pcb (KiCad board)
At the start: 2 copper layers, 50.8 x 22.2 mm, 19 parts, among them J1 LSAConnect

Commit message: Update for PCB Design
Parts:
- VT1, VT2, VT3: value BC547 -> BC548; footprint ELLIOTT:TO-92 -> ELLIOTT:TO-92L_Inline
- moved VT2 2.73 mm to (148.9, 16.1), turned to 270 degrees
- moved VT3 2.67 mm to (174.9, 16.1), turned to 270 degrees
- moved VT1 2.67 mm to (140.6, 16.1), turned to 270 degrees
- moved J1 0.14 mm to (136.2, 19.2)
Connections:
- J1 pad 1: 1 -> (no net)
- J1 pad 3: 3 -> (no net)
- J1 pad 5: 5 -> (no net)
Routing:
- net +6v: track 54.5 -> 55.5 mm
- net Net-(D7-Pad1): track 11.2 -> 12.0 mm
- net Net-(D9-Pad1): track 11.9 -> 12.7 mm
- net 12: track 8.76 -> 9.27 mm
- removed copper zone on B.Cu, net 0v
Other:
- board size 50.8 x 22.2 mm -> 50.8 x 22.4 mm
