File: KiCad/Real903/LS04/LS04.sch (KiCad schematic (older format))
At the start: 19 parts, among them J1 LSAConnect

Commit message: Update for PCB Design
Parts:
- VT1, VT2, VT3: value BC547 -> BC548; footprint ELLIOTT:TO-92 -> ELLIOTT:TO-92L_Inline
Connections:
- net labels removed: 1, 3, 5
- no-connect marks 0 -> 3
Changed lines of the file:
@@
 P 2950 1450
 F 0 "VT1" H 3150 1500 50  0000 L CNN
-F 1 "BC547" H 3150 1400 50  0000 L CNN
-F 2 "ELLIOTT:TO-92" H 3150 1550 50  0001 C CNN
+F 1 "BC548" H 3150 1400 50  0000 L CNN
+F 2 "ELLIOTT:TO-92L_Inline" H 3150 1550 50  0001 C CNN
 F 3 "" H 2950 1450 50  0001 C CNN
 	1    2950 1450
@@
 P 2950 2475
 F 0 "VT2" H 3150 2525 50  0000 L CNN
-F 1 "BC547" H 3150 2425 50  0000 L CNN
-F 2 "ELLIOTT:TO-92" H 3150 2575 50  0001 C CNN
+F 1 "BC548" H 3150 2425 50  0000 L CNN
+F 2 "ELLIOTT:TO-92L_Inline" H 3150 2575 50  0001 C CNN
 F 3 "" H 2950 2475 50  0001 C CNN
 	1    2950 2475
@@
 P 2950 3500
 F 0 "VT3" H 3150 3550 50  0000 L CNN
-F 1 "BC547" H 3150 3450 50  0000 L CNN
-F 2 "ELLIOTT:TO-92" H 3150 3600 50  0001 C CNN
+F 1 "BC548" H 3150 3450 50  0000 L CNN
+F 2 "ELLIOTT:TO-92L_Inline" H 3150 3600 50  0001 C CNN
 F 3 "" H 2950 3500 50  0001 C CNN
 	1    2950 3500
@@
 Text GLabel 2300 4725 2    40   Input ~ 0
 13
-Text GLabel 1550 4525 0    40   Input ~ 0
-1
 Text GLabel 1550 4625 0    40   Input ~ 0
 2
-Text GLabel 1550 4725 0    40   Input ~ 0
-3
 Text GLabel 1550 4825 0    40   Input ~ 0
 4
-Text GLabel 1550 4925 0    40   Input ~ 0
-5
 Text GLabel 1550 5025 0    40   Input ~ 0
 6
@@
 $EndComp
 Wire Wire Line
-	1550 4525 1675 4525
-Wire Wire Line
 	1675 4625 1550 4625
 Wire Wire Line
-	1550 4725 1675 4725
-Wire Wire Line
 	1550 4825 1675 4825
-Wire Wire Line
-	1550 4925 1675 4925
 Wire Wire Line
 	1550 5025 1675 5025
@@
 Wire Wire Line
 	1400 2950 1550 2950
+NoConn ~ 1675 4525
+NoConn ~ 1675 4725
+NoConn ~ 1675 4925
+$Comp
+L power:PWR_FLAG #FLG0101
+U 1 1 5C761014
+P 3250 5025
+F 0 "#FLG0101" H 3250 5100 50  0001 C CNN
+F 1 "PWR_FLAG" H 3250 5198 50  0000 C CNN
+F 2 "" H 3250 5025 50  0001 C CNN
+F 3 "~" H 3250 5025 50  0001 C CNN
+	1    3250 5025
+	-1   0    0    1
+$EndComp
+$Comp
+L power:PWR_FLAG #FLG0102
+U 1 1 5C761072
+P 3625 5025
+F 0 "#FLG0102" H 3625 5100 50  0001 C CNN
+F 1 "PWR_FLAG" H 3625 5198 50  0000 C CNN
+F 2 "" H 3625 5025 50  0001 C CNN
+F 3 "~" H 3625 5025 50  0001 C CNN
+	1    3625 5025
+	-1   0    0    1
+$EndComp
+$Comp
+L power:PWR_FLAG #FLG0103
+U 1 1 5C7610A3
+P 4000 5025
+F 0 "#FLG0103" H 4000 5100 50  0001 C CNN
+F 1 "PWR_FLAG" H 4000 5198 50  0000 C CNN
+F 2 "" H 4000 5025 50  0001 C CNN
+F 3 "~" H 4000 5025 50  0001 C CNN
+	1    4000 5025
+	-1   0    0    1
+$EndComp
+Text GLabel 3250 4925 1    50   Input ~ 0
+0v
+Wire Wire Line
+	3250 4925 3250 5025
+Text GLabel 3625 4925 1    50   Input ~ 0
++6v
+Wire Wire Line
+	3625 4925 3625 5025
+Text GLabel 4000 4925 1    50   Input ~ 0
+-6v
+Wire Wire Line
+	4000 4925 4000 5025
 $EndSCHEMATC
