File: KiCad/Real903/LS05/LS05.kicad_pcb (KiCad board)
At the start: 2 copper layers, 18 parts, among them J1 LSAConnect

Commit message: Update for PCB Design
Parts:
- VT3: value BC547 -> BC548; footprint ELLIOTT:TO-92 -> ELLIOTT:TO-92L_Inline
- moved VT3 2.54 mm to (181.1, 76.1), turned to 270 degrees
Routing:
- net +6v: track 48.7 -> 45.7 mm
- net Net-(D10-Pad1): track 43.6 -> 45.3 mm
- removed copper zone on B.Cu, net 0v
