File: KiCad/Real903/LS05/LS05.sch (KiCad schematic (older format))
At the start: 18 parts, among them J1 LSAConnect

Commit message: Update for PCB Design
Parts:
- VT3: value BC547 -> BC548; footprint ELLIOTT:TO-92 -> ELLIOTT:TO-92L_Inline
Changed lines of the file:
@@
 P 2950 3500
 F 0 "VT3" H 3150 3550 50  0000 L CNN
-F 1 "BC547" H 3150 3450 50  0000 L CNN
-F 2 "ELLIOTT:TO-92" H 3150 3600 50  0001 C CNN
+F 1 "BC548" H 3150 3450 50  0000 L CNN
+F 2 "ELLIOTT:TO-92L_Inline" H 3150 3600 50  0001 C CNN
 F 3 "" H 2950 3500 50  0001 C CNN
 	1    2950 3500
