File: KiCad/Real903/LS06/LS06.kicad_pcb (KiCad board)
At the start: 2 copper layers, 20 parts, among them J1 LSAConnect

Commit message: Update for PCB Design
Parts:
- VT1, VT2: value BC547 -> BC548; footprint ELLIOTT:TO-92 -> ELLIOTT:TO-92L_Inline
- moved VT1 2.54 mm to (152.4, 62.5), turned to 270 degrees
- moved VT2 2.54 mm to (162.2, 62.5), turned to 270 degrees
Routing:
- net Net-(D10-Pad1): track 34.3 -> 35.6 mm
- net Net-(D12-Pad1): track 32.5 -> 33.8 mm
- removed copper zone on B.Cu, net 0v
