File: KiCad/Real903/A-GA/A-GA.kicad_pcb (KiCad board)
At the start: 2 copper layers, 233.3 x 160 mm, 645 parts, among them J1 J1, U1 LS_Gen, U2 LS_Gen, U3 LS_Gen, U4 LS_Gen, U5 LS_Gen, U6 LS_Gen

Commit message: G Board
Parts:
- added TPLB1: ~, TestPoint:TestPoint_Bridge_Pitch3.81mm_Drill1.3mm, F.Cu at (95.5, 156.5)
- added TPLB11: ~, TestPoint:TestPoint_THTPad_2.0x2.0mm_Drill1.0mm, F.Cu at (90.7, 115.8)
- added TPLB12: ~, TestPoint:TestPoint_THTPad_2.0x2.0mm_Drill1.0mm, F.Cu at (85.6, 115.8)
- added TPLB13: ~, TestPoint:TestPoint_THTPad_2.0x2.0mm_Drill1.0mm, F.Cu at (80.5, 115.8)
- added TPLB2: ~, TestPoint:TestPoint_Bridge_Pitch3.81mm_Drill1.3mm, F.Cu at (95.5, 152.2)
- added TPLB3: ~, TestPoint:TestPoint_Bridge_Pitch3.81mm_Drill1.3mm, F.Cu at (95.5, 148.0)
- added TPLB4: ~, TestPoint:TestPoint_Bridge_Pitch3.81mm_Drill1.3mm, F.Cu at (95.5, 141.8)
- added TPLB5: ~, TestPoint:TestPoint_Bridge_Pitch3.81mm_Drill1.3mm, F.Cu at (95.5, 137.5)
- added TPLB6: ~, TestPoint:TestPoint_Bridge_Pitch3.81mm_Drill1.3mm, F.Cu at (95.5, 133.2)
- added TPLBD13: ~, TestPoint:TestPoint_THTPad_2.0x2.0mm_Drill1.0mm, F.Cu at (141.4, 115.8)
- added TPLC1: ~, TestPoint:TestPoint_Bridge_Pitch3.81mm_Drill1.3mm, F.Cu at (126.0, 156.5)
- added TPLC11: ~, TestPoint:TestPoint_THTPad_2.0x2.0mm_Drill1.0mm, F.Cu at (121.2, 115.8)
- added TPLC12: ~, TestPoint:TestPoint_THTPad_2.0x2.0mm_Drill1.0mm, F.Cu at (116.1, 115.8)
- added TPLC13: ~, TestPoint:TestPoint_THTPad_2.0x2.0mm_Drill1.0mm, F.Cu at (111.0, 115.8)
- added TPLC2: ~, TestPoint:TestPoint_Bridge_Pitch3.81mm_Drill1.3mm, F.Cu at (126.0, 152.2)
- added TPLC3: ~, TestPoint:TestPoint_Bridge_Pitch3.81mm_Drill1.3mm, F.Cu at (126.0, 148.0)
- added TPLC4: ~, TestPoint:TestPoint_Bridge_Pitch3.81mm_Drill1.3mm, F.Cu at (126.0, 141.8)
- added TPLC5: ~, TestPoint:TestPoint_Bridge_Pitch3.81mm_Drill1.3mm, F.Cu at (126.0, 137.5)
- added TPLC6: ~, TestPoint:TestPoint_Bridge_Pitch3.81mm_Drill1.3mm, F.Cu at (126.0, 133.2)
- added TPLD1: ~, TestPoint:TestPoint_Bridge_Pitch3.81mm_Drill1.3mm, F.Cu at (156.5, 156.5)
- added TPLD11: ~, TestPoint:TestPoint_THTPad_2.0x2.0mm_Drill1.0mm, F.Cu at (151.6, 115.8)
- added TPLD12: ~, TestPoint:TestPoint_THTPad_2.0x2.0mm_Drill1.0mm, F.Cu at (146.5, 115.8)
- added TPLD2: ~, TestPoint:TestPoint_Bridge_Pitch3.81mm_Drill1.3mm, F.Cu at (156.5, 152.2)
- added TPLD3: ~, TestPoint:TestPoint_Bridge_Pitch3.81mm_Drill1.3mm, F.Cu at (156.5, 148.0)
- added TPLD4: ~, TestPoint:TestPoint_Bridge_Pitch3.81mm_Drill1.3mm, F.Cu at (156.5, 141.8)
- added TPLD5: ~, TestPoint:TestPoint_Bridge_Pitch3.81mm_Drill1.3mm, F.Cu at (156.5, 137.5)
- added TPLD6: ~, TestPoint:TestPoint_Bridge_Pitch3.81mm_Drill1.3mm, F.Cu at (156.5, 133.2)
- added TPLE1: ~, TestPoint:TestPoint_Bridge_Pitch3.81mm_Drill1.3mm, F.Cu at (187.0, 156.5)
- added TPLE11: ~, TestPoint:TestPoint_THTPad_2.0x2.0mm_Drill1.0mm, F.Cu at (182.1, 115.8)
- added TPLE12: ~, TestPoint:TestPoint_THTPad_2.0x2.0mm_Drill1.0mm, F.Cu at (177.0, 115.8)
- added TPLE13: ~, TestPoint:TestPoint_THTPad_2.0x2.0mm_Drill1.0mm, F.Cu at (171.9, 115.8)
- added TPLE2: ~, TestPoint:TestPoint_Bridge_Pitch3.81mm_Drill1.3mm, F.Cu at (187.0, 152.2)
- added TPLE3: ~, TestPoint:TestPoint_Bridge_Pitch3.81mm_Drill1.3mm, F.Cu at (187.0, 148.0)
- added TPLE4: ~, TestPoint:TestPoint_Bridge_Pitch3.81mm_Drill1.3mm, F.Cu at (187.0, 141.8)
- added TPLE5: ~, TestPoint:TestPoint_Bridge_Pitch3.81mm_Drill1.3mm, F.Cu at (187.0, 137.5)
- added TPLE6: ~, TestPoint:TestPoint_Bridge_Pitch3.81mm_Drill1.3mm, F.Cu at (187.0, 133.2)
- added TPLF1: ~, TestPoint:TestPoint_Bridge_Pitch3.81mm_Drill1.3mm, F.Cu at (217.5, 156.5)
- added TPLF11: ~, TestPoint:TestPoint_THTPad_2.0x2.0mm_Drill1.0mm, F.Cu at (212.6, 115.8)
- added TPLF12: ~, TestPoint:TestPoint_THTPad_2.0x2.0mm_Drill1.0mm, F.Cu at (207.5, 115.8)
- added TPLF13: ~, TestPoint:TestPoint_THTPad_2.0x2.0mm_Drill1.0mm, F.Cu at (202.4, 115.8)
- added TPLF2: ~, TestPoint:TestPoint_Bridge_Pitch3.81mm_Drill1.3mm, F.Cu at (217.5, 152.2)
- added TPLF3: ~, TestPoint:TestPoint_Bridge_Pitch3.81mm_Drill1.3mm, F.Cu at (217.5, 148.0)
- added TPLF4: ~, TestPoint:TestPoint_Bridge_Pitch3.81mm_Drill1.3mm, F.Cu at (217.5, 141.8)
- added TPLF5: ~, TestPoint:TestPoint_Bridge_Pitch3.81mm_Drill1.3mm, F.Cu at (217.5, 137.5)
- added TPLF6: ~, TestPoint:TestPoint_Bridge_Pitch3.81mm_Drill1.3mm, F.Cu at (217.5, 133.2)
Connections:
- U2 pad 1: (no net) -> Net-(TPLB1-Pad1)
- U2 pad 11: (no net) -> Net-(TPLB11-Pad1)
- U2 pad 12: (no net) -> Net-(TPLB12-Pad1)
- U2 pad 13: (no net) -> Net-(TPLB13-Pad1)
- U2 pad 2: (no net) -> Net-(TPLB2-Pad1)
- U2 pad 3: (no net) -> Net-(TPLB3-Pad1)
- U2 pad 4: (no net) -> Net-(TPLB4-Pad1)
- U2 pad 5: (no net) -> Net-(TPLB5-Pad1)
- U2 pad 6: (no net) -> Net-(TPLB6-Pad1)
- U3 pad 1: (no net) -> Net-(TPLC1-Pad1)
- U3 pad 11: (no net) -> Net-(TPLC11-Pad1)
- U3 pad 12: (no net) -> Net-(TPLC12-Pad1)
- U3 pad 13: (no net) -> Net-(TPLC13-Pad1)
- U3 pad 2: (no net) -> Net-(TPLC2-Pad1)
- U3 pad 3: (no net) -> Net-(TPLC3-Pad1)
- U3 pad 4: (no net) -> Net-(TPLC4-Pad1)
- U3 pad 5: (no net) -> Net-(TPLC5-Pad1)
- U3 pad 6: (no net) -> Net-(TPLC6-Pad1)
- U4 pad 1: (no net) -> Net-(TPLD1-Pad1)
- U4 pad 11: (no net) -> Net-(TPLD11-Pad1)
- U4 pad 12: (no net) -> Net-(TPLD12-Pad1)
- U4 pad 13: (no net) -> Net-(TPLBD13-Pad1)
- U4 pad 2: (no net) -> Net-(TPLD2-Pad1)
- U4 pad 3: (no net) -> Net-(TPLD3-Pad1)
- U4 pad 4: (no net) -> Net-(TPLD4-Pad1)
- U4 pad 5: (no net) -> Net-(TPLD5-Pad1)
- U4 pad 6: (no net) -> Net-(TPLD6-Pad1)
- U5 pad 1: (no net) -> Net-(TPLE1-Pad1)
- U5 pad 11: (no net) -> Net-(TPLE11-Pad1)
- U5 pad 12: (no net) -> Net-(TPLE12-Pad1)
- U5 pad 13: (no net) -> Net-(TPLE13-Pad1)
- U5 pad 2: (no net) -> Net-(TPLE2-Pad1)
- U5 pad 3: (no net) -> Net-(TPLE3-Pad1)
- U5 pad 4: (no net) -> Net-(TPLE4-Pad1)
- U5 pad 5: (no net) -> Net-(TPLE5-Pad1)
- U5 pad 6: (no net) -> Net-(TPLE6-Pad1)
- U6 pad 1: (no net) -> Net-(TPLF1-Pad1)
- U6 pad 11: (no net) -> Net-(TPLF11-Pad1)
- U6 pad 12: (no net) -> Net-(TPLF12-Pad1)
- U6 pad 13: (no net) -> Net-(TPLF13-Pad1)
- U6 pad 2: (no net) -> Net-(TPLF2-Pad1)
- U6 pad 3: (no net) -> Net-(TPLF3-Pad1)
- U6 pad 4: (no net) -> Net-(TPLF4-Pad1)
- U6 pad 5: (no net) -> Net-(TPLF5-Pad1)
- U6 pad 6: (no net) -> Net-(TPLF6-Pad1)
Routing:
- net Net-(TPLF11-Pad1): track 0.00 -> 38.9 mm
- net Net-(TPLE11-Pad1): track 0.00 -> 38.9 mm
- net Net-(TPLC11-Pad1): track 0.00 -> 38.9 mm
- net Net-(TPLB11-Pad1): track 0.00 -> 38.9 mm
- net Net-(TPLD11-Pad1): track 0.00 -> 38.9 mm
- net Net-(TPLF12-Pad1): track 0.00 -> 34.2 mm
- net Net-(TPLE12-Pad1): track 0.00 -> 34.2 mm
- net Net-(TPLC12-Pad1): track 0.00 -> 34.2 mm
- net Net-(TPLB12-Pad1): track 0.00 -> 34.2 mm
- net Net-(TPLD12-Pad1): track 0.00 -> 34.2 mm
- net Net-(TPLF13-Pad1): track 0.00 -> 30.3 mm
- net Net-(TPLC13-Pad1): track 0.00 -> 30.3 mm
- net Net-(TPLB13-Pad1): track 0.00 -> 30.3 mm
- net Net-(TPLE13-Pad1): track 0.00 -> 30.3 mm
- net Net-(TPLBD13-Pad1): track 0.00 -> 30.3 mm
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Other:
- board text added: "1"
- board text added: "10"
- board text added: "2"
- board text added: "3"
- board text added: "4"
- board text added: "5"
- board text added: "6"
- board text added: "7"
- board text added: "8"
- board text added: "9"
- board text added: "GND"
- board text added: "Pin 10"
- board text added: "Pin 11"
- board text added: "Pin 14"
- board text added: "Pin 15"
- board text added: "Pin 18"
- board text added: "Pin 7"
- board text added: "Pin 8"
- board text added: "Pin 9"

Commit message: Update Gerbers
Parts:
- added TPI12: ~, TestPoint:TestPoint_Plated_Hole_D2.0mm, F.Cu at (33.0, 60.0)
- added TPI13: ~, TestPoint:TestPoint_Plated_Hole_D2.0mm, F.Cu at (33.0, 66.0)
- added TPI29: ~, TestPoint:TestPoint_Plated_Hole_D2.0mm, F.Cu at (33.0, 54.0)
Connections:
- J1 pad 12: (no net) -> 12
- J1 pad 13: (no net) -> 13
- J1 pad 29: (no net) -> 29
Routing:
- net 13: track 0.00 -> 83.2 mm
- net 12: track 0.00 -> 81.8 mm
- net 29: track 0.00 -> 30.0 mm
Other:
- board text added: "AA"
- board text added: "AB"
- board text added: "AC"
- board text added: "AD"
- board text added: "AE"
- board text added: "AF"
- board text added: "AH"
- board text added: "AJ"
- board text added: "C"
- board text added: "D"
- board text added: "Definitions Change On Initial Instruction Boards"
- board text added: "E"
- board text added: "F"
- board text added: "H"
- board text added: "J"
- board text added: "K"
- board text added: "L"
- board text added: "M"
- board text added: "N"
- board text added: "P"
- board text added: "Pin C"
- board text added: "R"
- board text added: "S"
- board text added: "T"
- board text added: "U"
- board text added: "Used For Initial Instructions Only"
- board text added: "V"
- board text added: "W"
- board text added: "X"
- board text added: "Y"
- board text added: "Z"
