File: KiCad/Real903/A-FA/A-FA.sch (KiCad schematic (older format))
At the start: 35 parts, among them J1 J1, U1 LS06, U10 LS05, U11 LS06, U12 LS05, U13 LS06, U14 LS06, U2 LS03, U3 LS06, U4 LS05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

Commit message: Update for PCB Design
Parts:
- added D1, D10, D11, D2, D3, D4, D5, D6, D7, D8, D9: ~, ELLIOTT:LED_D5.0mm, symbol Device:LED
- added J2: Conn_01x02, ELLIOTT:PinHeader_1x02_P2.54mm_Vertical, symbol Connector_Generic:Conn_01x02
- added R51, R52, R53, R54, R55, R56, R57, R58, R59, R60, R61: 1k, ELLIOTT:R_Axial_DIN0204_L3.6mm_D1.6mm_P7.62mm_Horizontal, symbol Device:R
- TP1, TP2, TP3: footprint Connector_Pin:Pin_D1.0mm_L10.0mm -> ELLIOTT:Pin_D1.0mm_L10.0mm_LooseFit
Connections:
- wire segments 354 -> 443

Commit message: New boards
Parts:
- removed R54, R58: 1k, ELLIOTT:R_Axial_DIN0204_L3.6mm_D1.6mm_P7.62mm_Horizontal, symbol Device:R
- added J3: Conn_01x02, ELLIOTT:PinHeader_1x02_P2.54mm_Vertical, symbol Connector_Generic:Conn_01x02
Connections:
- net labels added: ~A~n, ~G~n, ~IP~n, ~JTG~|NC, ~J~n, ~M~TF, ~M~n, ~OTA, ~OTG, ~OTIP, ~OTJ, ~OTM, ~OTQ, ~Q~n, ~STORE~n, ~STORE~nx, ~X~n, ~Y~n
- net labels removed: 0TA-, 0TG-, 0TIP-, 0TJ-, 0TM-, 0TQ-, An-, Gn-, IPn-, JTG-|NC, Jn-, M-TF, Mn-, Qn-, STOREn-, STOREnx-, Xn-, Yn-
- wire segments 443 -> 438
