File: KiCad/Real903/A-FA/A-FA.kicad_pcb (KiCad board)
At the start: 2 copper layers, 228.6 x 160 mm, 35 parts, among them J1 J1, U1 LS06, U10 LS05, U11 LS06, U12 LS05, U13 LS06, U14 LS06, U2 LS03, U3 LS06, U4 LS05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

Commit message: Update for PCB Design
Parts:
- added D1: ~, ELLIOTT:LED_D5.0mm, F.Cu at (170.2, 181.9)
- added D10: ~, ELLIOTT:LED_D5.0mm, F.Cu at (78.7, 181.9)
- added D11: ~, ELLIOTT:LED_D5.0mm, F.Cu at (68.6, 181.9)
- added D2: ~, ELLIOTT:LED_D5.0mm, F.Cu at (160.0, 181.9)
- added D3: ~, ELLIOTT:LED_D5.0mm, F.Cu at (149.9, 181.9)
- added D4: ~, ELLIOTT:LED_D5.0mm, F.Cu at (139.7, 181.9)
- added D5: ~, ELLIOTT:LED_D5.0mm, F.Cu at (129.5, 181.9)
- added D6: ~, ELLIOTT:LED_D5.0mm, F.Cu at (119.4, 181.9)
- added D7: ~, ELLIOTT:LED_D5.0mm, F.Cu at (109.2, 181.9)
- added D8: ~, ELLIOTT:LED_D5.0mm, F.Cu at (99.1, 181.9)
- added D9: ~, ELLIOTT:LED_D5.0mm, F.Cu at (88.9, 181.9)
- added J2: Conn_01x02, ELLIOTT:PinHeader_1x02_P2.54mm_Vertical, F.Cu at (42.6, 176.3)
- added R51: 1k, ELLIOTT:R_Axial_DIN0204_L3.6mm_D1.6mm_P7.62mm_Horizontal, F.Cu at (162.6, 176.3)
- added R52: 1k, ELLIOTT:R_Axial_DIN0204_L3.6mm_D1.6mm_P7.62mm_Horizontal, F.Cu at (152.4, 176.3)
- added R53: 1k, ELLIOTT:R_Axial_DIN0204_L3.6mm_D1.6mm_P7.62mm_Horizontal, F.Cu at (142.2, 176.3)
- added R54: 1k, ELLIOTT:R_Axial_DIN0204_L3.6mm_D1.6mm_P7.62mm_Horizontal, F.Cu at (132.1, 176.3)
- added R55: 1k, ELLIOTT:R_Axial_DIN0204_L3.6mm_D1.6mm_P7.62mm_Horizontal, F.Cu at (121.9, 176.3)
- added R56: 1k, ELLIOTT:R_Axial_DIN0204_L3.6mm_D1.6mm_P7.62mm_Horizontal, F.Cu at (111.8, 176.3)
- added R57: 1k, ELLIOTT:R_Axial_DIN0204_L3.6mm_D1.6mm_P7.62mm_Horizontal, F.Cu at (101.6, 176.3)
- added R58: 1k, ELLIOTT:R_Axial_DIN0204_L3.6mm_D1.6mm_P7.62mm_Horizontal, F.Cu at (91.4, 176.3)
- added R59: 1k, ELLIOTT:R_Axial_DIN0204_L3.6mm_D1.6mm_P7.62mm_Horizontal, F.Cu at (81.3, 176.3)
- added R60: 1k, ELLIOTT:R_Axial_DIN0204_L3.6mm_D1.6mm_P7.62mm_Horizontal, F.Cu at (71.1, 176.3)
- added R61: 1k, ELLIOTT:R_Axial_DIN0204_L3.6mm_D1.6mm_P7.62mm_Horizontal, F.Cu at (61.0, 176.3)
- TP1, TP2, TP3: footprint Connector_Pin:Pin_D1.0mm_L10.0mm -> ELLIOTT:Pin_D1.0mm_L10.0mm_LooseFit
- moved J1 59.5 mm to (118.3, 30.9)
Routing:
- net Cn-1: track 166.3 -> 415.4 mm
- net Cn: track 76.0 -> 277.1 mm
- net Fn: track 138.5 -> 314.2 mm
- net GND: track 658.1 -> 831.0 mm
- net Qn: track 85.2 -> 233.8 mm
- net Xn: track 46.4 -> 176.8 mm
- net Net-(J2-Pad1): track 0.00 -> 128.6 mm
- net IPn: track 233.0 -> 356.1 mm, vias 0 -> 1
- net Gn: track 248.1 -> 365.9 mm
- net Yn: track 33.4 -> 147.7 mm, vias 0 -> 1
- net Jn: track 121.0 -> 214.7 mm, vias 0 -> 2
- net RTG: track 69.7 -> 153.3 mm
- net Mn: track 205.4 -> 280.2 mm
- net An: track 159.8 -> 222.1 mm
- net JTG-|NC: track 95.3 -> 154.5 mm
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Other:
- board size 228.6 x 160 mm -> 233.3 x 160 mm
- net class 6v added: clearance 0.2, trace_width 0.5, via_dia 1.6, via_drill 0.8
- net class GND added: clearance 0.2, trace_width 0.5, via_dia 1.6, via_drill 0.8
- net class Neg6v added: clearance 0.2, trace_width 0.5, via_dia 1.6, via_drill 0.8
- board text added: "A"
- board text added: "B"
- board text added: "C"
- board text added: "D"
- board text added: "E"
- board text added: "F"
- board text added: "Fit Connector to Underside"
- board text added: "G"
- board text added: "H"
- board text added: "J"
- board text added: "K"
- board text added: "L"
- board text added: "LS01"
- board text added: "LS02"
- board text added: "LS03"
- board text added: "LS05"
- board text added: "LS06"
- board text added: "M"
- board text added: "N"
- board text added: "P"

Commit message: Sept 1
Changed lines of the file:
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@@
   (page A3)
   (layers
-    (0 F.Cu signal)
-    (31 B.Cu signal)
+    (0 F.Cu signal hide)
+    (31 B.Cu signal hide)
     (32 B.Adhes user)
     (33 F.Adhes user)
@@
       (effects (font (size 1 1) (thickness 0.15)))
     )
-    (fp_text value 3k9 (at 3.81 1.92 270) (layer F.Fab)
+    (fp_text value 3k9 (at 3.81 1.92 270) (layer F.SilkS)
       (effects (font (size 1 1) (thickness 0.15)))
     )
@@
       (effects (font (size 1 1) (thickness 0.15)))
     )
-    (fp_text value 3k9 (at 3.81 1.92 270) (layer F.Fab)
+    (fp_text value 3k9 (at 3.81 1.92 270) (layer F.SilkS)
       (effects (font (size 1 1) (thickness 0.15)))
     )
@@
       (effects (font (size 1 1) (thickness 0.15)))
     )
-    (fp_text value 3k9 (at 3.81 1.92 270) (layer F.Fab)
+    (fp_text value 3k9 (at 3.81 1.92 270) (layer F.SilkS)
       (effects (font (size 1 1) (thickness 0.15)))
     )
@@
       (effects (font (size 1 1) (thickness 0.15)))
     )
-    (fp_text value 3k9 (at 3.81 1.92 270) (layer F.Fab)
+    (fp_text value 3k9 (at 3.81 1.92 270) (layer F.SilkS)
       (effects (font (size 1 1) (thickness 0.15)))
     )
@@
       (effects (font (size 1 1) (thickness 0.15)))
     )
-    (fp_text value 3k9 (at 3.81 1.92 270) (layer F.Fab)
+    (fp_text value 3k9 (at 3.81 1.92 270) (layer F.SilkS)
       (effects (font (size 1 1) (thickness 0.15)))
     )
@@
       (effects (font (size 1 1) (thickness 0.15)))
     )
-    (fp_text value 3k9 (at 3.81 1.92 270) (layer F.Fab)
+    (fp_text value 3k9 (at 3.81 1.92 270) (layer F.SilkS)
       (effects (font (size 1 1) (thickness 0.15)))
     )
@@
       (effects (font (size 1 1) (thickness 0.15)))
     )
-    (fp_text value 2k2 (at 3.81 1.92 270) (layer F.Fab)
+    (fp_text value 2k2 (at 3.81 1.92 270) (layer F.SilkS)
       (effects (font (size 1 1) (thickness 0.15)))
     )
@@
       (effects (font (size 1 1) (thickness 0.15)))
     )
-    (fp_text value 1k (at 3.81 1.92 270) (layer F.Fab)
+    (fp_text value 1k (at 3.81 1.92 270) (layer F.SilkS)
       (effects (font (size 1 1) (thickness 0.15)))
     )
@@
       (effects (font (size 1 1) (thickness 0.15)))
     )
-    (fp_text value 1k (at 3.81 1.92 180) (layer F.Fab)
+    (fp_text value 1k (at 3.81 1.92 180) (layer F.SilkS)
       (effects (font (size 1 1) (thickness 0.15)))
     )
@@
       (effects (font (size 1 1) (thickness 0.15)))
     )
-    (fp_text value 1k (at 3.81 1.92 270) (layer F.Fab)
+    (fp_text value 1k (at 3.81 1.92 270) (layer F.SilkS)
       (effects (font (size 1 1) (thickness 0.15)))
     )
@@
       (effects (font (size 1 1) (thickness 0.15)))
     )
-    (fp_text value 1k (at 3.81 1.92 270) (layer F.Fab)
+    (fp_text value 1k (at 3.81 1.92 270) (layer F.SilkS)
       (effects (font (size 1 1) (thickness 0.15)))
     )
@@
       (effects (font (size 1 1) (thickness 0.15)))
     )
-    (fp_text value 1k (at 3.81 1.92 270) (layer F.Fab)
+    (fp_text value 1k (at 3.81 1.92 270) (layer F.SilkS)
       (effects (font (size 1 1) (thickness 0.15)))
     )
@@
       (effects (font (size 1 1) (thickness 0.15)))
     )
-    (fp_text value 2k2 (at 3.81 1.92 90) (layer F.Fab)
+    (fp_text value 2k2 (at 3.81 1.92 90) (layer F.SilkS)
       (effects (font (size 1 1) (thickness 0.15)))
     )
@@
       (effects (font (size 1 1) (thickness 0.15)))
     )
-    (fp_text value 1k (at 3.81 1.92 270) (layer F.Fab)
+    (fp_text value 1k (at 3.81 1.92 270) (layer F.SilkS)
       (effects (font (size 1 1) (thickness 0.15)))
     )
@@
       (effects (font (size 1 1) (thickness 0.15)))
     )
-    (fp_text value 2k2 (at 3.81 1.92 270) (layer F.Fab)
-      (effects (font (size 1 1) (thickness 0.15)))
-    )
+    (fp_text value 2k2 (at 3.81 1.92 270) (layer F.SilkS)
+      (effects (font (size 1 1) (thickness 0.15)))
+    )

Commit message: 23 oct
Parts:
- removed D1, D10, D11, D2, D3, D4, D5, D6, D7, D8, D9: ~, ELLIOTT:LED_D5.0mm
- removed J2: Conn_01x02, ELLIOTT:PinHeader_1x02_P2.54mm_Vertical
- removed R51, R52, R53, R54, R55, R56, R57, R58, R59, R60, R61: 1k, ELLIOTT:R_Axial_DIN0204_L3.6mm_D1.6mm_P7.62mm_Horizontal
- removed TP1: P1, ELLIOTT:Pin_D1.0mm_L10.0mm_LooseFit
- removed TP2: P2, ELLIOTT:Pin_D1.0mm_L10.0mm_LooseFit
- removed TP3: P3, ELLIOTT:Pin_D1.0mm_L10.0mm_LooseFit
- added R99: 1k, ELLIOTT:R_Axial_DIN0204_L3.6mm_D1.6mm_P7.62mm_Horizontal, F.Cu at (219.6, 93.2)
- C1, C2: value 6u8 -> "6u8"
- moved C2 197.9 mm to (30.8, 39.8)
- moved C1 97.0 mm to (144.4, 37.0)
- moved R3 15.0 mm to (252.4, 74.6)
- moved R12 14.7 mm to (128.6, 150.0)
- moved R6 14.5 mm to (128.4, 133.3)
- moved R14 13.7 mm to (158.4, 143.4)
- moved R5 13.4 mm to (97.4, 133.3)
- moved R9 13.2 mm to (128.2, 77.2)
- moved R13 12.6 mm to (97.4, 83.2)
- moved R7 12.6 mm to (97.4, 69.8)
- moved R8 12.6 mm to (66.6, 70.0)
- moved R16 12.6 mm to (66.6, 83.2)
- moved R4 12.3 mm to (158.4, 69.8)
- moved R10 12.1 mm to (158.4, 87.8)
- moved R15 9.58 mm to (97.4, 145.2), turned to 270 degrees
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Connections:
- net 0TA- renamed ~OTA
- net 0TG- renamed ~OTG
- net 0TIP- renamed ~OTIP
- net 0TJ- renamed ~OTJ
- net 0TM- renamed ~OTM
- net 0TQ- renamed ~OTQ
- net An- renamed ~A~n
- net An-7|IPn renamed An-7
- net Gn- renamed ~G~n
- net IPn- renamed ~IP~n
- net JTG-|NC renamed ~JTG~
- net Jn- renamed ~J~n
- net M-TF renamed ~M~TF
- net Mn- renamed ~M~n
- net Qn- renamed ~Q~n
- net STOREn- renamed ~STORE~n
- net STOREnx- renamed ~STORE~nx
- net TP1 renamed Net-(U1-Pad4)
- net TP2 renamed Net-(U3-Pad13)
- net TP3 renamed Net-(U1-Pad2)
- net Xn- renamed ~X~n
- net Yn- renamed ~Y~n
Routing:
- net Cn-1: track 415.4 -> 224.4 mm
- net GND: track 831.0 -> 670.1 mm
- net Qn: track 233.8 -> 84.6 mm
- net Cn: track 277.1 -> 134.1 mm, vias 0 -> 1
- net Xn: track 176.8 -> 42.4 mm
- net Net-(J2-Pad1): track 128.6 -> 0.00 mm
- net Yn: track 147.7 -> 33.3 mm, vias 1 -> 0
- net Fn: track 314.2 -> 203.1 mm
- net Gn: track 365.9 -> 269.2 mm, vias 0 -> 1
- net Neg6v: track 595.8 -> 526.4 mm
- net An: track 222.1 -> 159.5 mm, vias 0 -> 1
- net IPn: track 356.1 -> 293.8 mm, vias 1 -> 0
- net Jn: track 214.7 -> 169.0 mm, vias 2 -> 0
- net Mn: track 280.2 -> 252.3 mm
- net RTG: track 153.3 -> 129.5 mm
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