File: KiCad/Real903/Display/Display.kicad_pcb (KiCad board)
At the start: 2 copper layers, 330 x 150 mm, 428 parts, among them J10 Conn_01x10, J11 Conn_01x10, J12 Conn_01x10, J14 Conn_01x10, J15 Conn_01x10, J16 Conn_01x10, J17 Conn_01x10, J18 Conn_01x10, J19 Conn_01x10, J2 Conn_01x10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

Commit message: Sept 1
Parts:
- added M1: ~, MountingHole:MountingHole_2.7mm_M2.5_ISO14580_Pad, F.Cu at (60.0, 35.0)
- added M2: ~, MountingHole:MountingHole_2.7mm_M2.5_ISO14580_Pad, F.Cu at (380.0, 35.0)
- added M3: ~, MountingHole:MountingHole_2.7mm_M2.5_ISO14580_Pad, F.Cu at (60.0, 175.0)
- added M3: ~, MountingHole:MountingHole_2.7mm_M2.5_ISO14580_Pad, F.Cu at (380.0, 175.0)
- added M5: ~, MountingHole:MountingHole_2.7mm_M2.5_ISO14580_Pad, F.Cu at (225.0, 112.0)
Changed lines of the file:
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@@
     (tracks 2094)
     (zones 0)
-    (modules 428)
+    (modules 433)
     (nets 276)
   )
@@
     )
   )
+  (module MountingHole:MountingHole_2.7mm_M2.5_ISO14580_Pad (layer F.Cu)
+    (at 60 175)
+    (descr "Mounting Hole 2.7mm, M2.5, ISO14580")
+    (tags "mounting hole 2.7mm m2.5 iso14580")
+    (attr virtual)
+    (fp_text reference M3 (at 0 -3.25) (layer F.SilkS)
+      (effects (font (size 1 1) (thickness 0.15)))
+    )
+    (fp_text value ~ (at 0 3.25) (layer F.Fab)
+      (effects (font (size 1 1) (thickness 0.15)))
+    )
+    (fp_circle (center 0 0) (end 2.5 0) (layer F.CrtYd) (width 0.05))
+    (fp_circle (center 0 0) (end 2.25 0) (layer Cmts.User) (width 0.15))
+    (fp_text user %R (at 0.3 0) (layer F.Fab)
+      (effects (font (size 1 1) (thickness 0.15)))
+    )
+    (pad 1 thru_hole circle (at 0 0) (size 4.5 4.5) (drill 2.7) (layers *.Cu *.Mask))
+  )
+  (module MountingHole:MountingHole_2.7mm_M2.5_ISO14580_Pad (layer F.Cu)
+    (at 380 175)
+    (descr "Mounting Hole 2.7mm, M2.5, ISO14580")
+    (tags "mounting hole 2.7mm m2.5 iso14580")
+    (attr virtual)
+    (fp_text reference M3 (at 0 -3.25) (layer F.SilkS)
+      (effects (font (size 1 1) (thickness 0.15)))
+    )
+    (fp_text value ~ (at 0 3.25) (layer F.Fab)
+      (effects (font (size 1 1) (thickness 0.15)))
+    )
+    (fp_circle (center 0 0) (end 2.5 0) (layer F.CrtYd) (width 0.05))
+    (fp_circle (center 0 0) (end 2.25 0) (layer Cmts.User) (width 0.15))
+    (fp_text user %R (at 0.3 0) (layer F.Fab)
+      (effects (font (size 1 1) (thickness 0.15)))
+    )
+    (pad 1 thru_hole circle (at 0 0) (size 4.5 4.5) (drill 2.7) (layers *.Cu *.Mask))
+  )
+  (module MountingHole:MountingHole_2.7mm_M2.5_ISO14580_Pad (layer F.Cu)
+    (at 60 35)
+    (descr "Mounting Hole 2.7mm, M2.5, ISO14580")
+    (tags "mounting hole 2.7mm m2.5 iso14580")
+    (attr virtual)
+    (fp_text reference M1 (at 0 -3.25) (layer F.SilkS)
+      (effects (font (size 1 1) (thickness 0.15)))
+    )
+    (fp_text value ~ (at 0 3.25) (layer F.Fab)
+      (effects (font (size 1 1) (thickness 0.15)))
+    )
+    (fp_circle (center 0 0) (end 2.5 0) (layer F.CrtYd) (width 0.05))
+    (fp_circle (center 0 0) (end 2.25 0) (layer Cmts.User) (width 0.15))
+    (fp_text user %R (at 0.3 0) (layer F.Fab)
+      (effects (font (size 1 1) (thickness 0.15)))
+    )
+    (pad 1 thru_hole circle (at 0 0) (size 4.5 4.5) (drill 2.7) (layers *.Cu *.Mask))
+  )
+  (module MountingHole:MountingHole_2.7mm_M2.5_ISO14580_Pad (layer F.Cu)
+    (at 380 35)
+    (descr "Mounting Hole 2.7mm, M2.5, ISO14580")
+    (tags "mounting hole 2.7mm m2.5 iso14580")
+    (attr virtual)
+    (fp_text reference M2 (at 0 -3.25) (layer F.SilkS)
+      (effects (font (size 1 1) (thickness 0.15)))
+    )
+    (fp_text value ~ (at 0 3.25) (layer F.Fab)
+      (effects (font (size 1 1) (thickness 0.15)))
+    )
+    (fp_circle (center 0 0) (end 2.5 0) (layer F.CrtYd) (width 0.05))
+    (fp_circle (center 0 0) (end 2.25 0) (layer Cmts.User) (width 0.15))
+    (fp_text user %R (at 0.3 0) (layer F.Fab)
+      (effects (font (size 1 1) (thickness 0.15)))
+    )
+    (pad 1 thru_hole circle (at 0 0) (size 4.5 4.5) (drill 2.7) (layers *.Cu *.Mask))
+  )
+  (module MountingHole:MountingHole_2.7mm_M2.5_ISO14580_Pad (layer F.Cu)
+    (at 225 112)
+    (descr "Mounting Hole 2.7mm, M2.5, ISO14580")
+    (tags "mounting hole 2.7mm m2.5 iso14580")
+    (attr virtual)
+    (fp_text reference M5 (at 0 -3.25) (layer F.SilkS)
+      (effects (font (size 1 1) (thickness 0.15)))
+    )
+    (fp_text value ~ (at 0 3.25) (layer F.Fab)
+      (effects (font (size 1 1) (thickness 0.15)))
+    )
+    (fp_circle (center 0 0) (end 2.5 0) (layer F.CrtYd) (width 0.05))
+    (fp_circle (center 0 0) (end 2.25 0) (layer Cmts.User) (width 0.15))
+    (fp_text user %R (at 0.3 0) (layer F.Fab)
+      (effects (font (size 1 1) (thickness 0.15)))
+    )
+    (pad 1 thru_hole circle (at 0 0) (size 4.5 4.5) (drill 2.7) (layers *.Cu *.Mask))
+  )
   (gr_line (start 55 30) (end 55 180) (layer Edge.Cuts) (width 0.1))
