File: KiCad/Real903/A-FP/A-FP.kicad_pcb (KiCad board)
At the start: 2 copper layers, 228.6 x 160 mm, 20 parts, among them J1 J1, U1 LS01, U10 LS01, U11 LS03, U12 LS01, U13 LS07, U14 LS01, U2 LS07, U3 LS01, U5 LS01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

Commit message: August Update
Parts:
- moved J1 59.5 mm to (118.3, 30.9)
- moved C1 7.62 mm to (228.6, 33.0)
Routing:
- net GND: track 657.8 -> 0.00 mm
- net Neg6v: track 597.3 -> 0.00 mm
- net 6v: track 564.5 -> 0.00 mm
- net JTPC: track 343.9 -> 0.00 mm, vias 1 -> 0
- net WFM-: track 299.2 -> 0.00 mm, vias 1 -> 0
- net PC4-: track 290.7 -> 0.00 mm
- net PC2-: track 249.8 -> 0.00 mm
- net PC1-: track 236.2 -> 0.00 mm
- net PC3-: track 196.7 -> 0.00 mm
- net {PC4}: track 168.1 -> 0.00 mm
- net {PC2}: track 141.6 -> 0.00 mm
- net J4-: track 139.3 -> 0.00 mm
- net Net-(U10-Pad6): track 131.7 -> 0.00 mm
- net Net-(U14-Pad6): track 131.7 -> 0.00 mm
- net {PC3}: track 123.9 -> 0.00 mm
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
Commit message: 1 December
Parts:
- added U4: LS08, ELLIOTT:LSA, F.Cu at (137.2, 165.1)
- moved R1 94.0 mm to (159.2, 71.0), turned to 270 degrees
- moved R2 89.6 mm to (219.8, 134.6), turned to 270 degrees
- moved R3 81.8 mm to (35.0, 73.6), turned to 270 degrees
- moved R4 15.1 mm to (97.6, 134.6)
Connections:
- J1 pad 12: (no net) -> PulseGenMargin
- U13 pad 4: (no net) -> 2.4vRef
- U2 pad 4: (no net) -> 2.4vRef
- U6 pad 4: (no net) -> 2.4vRef
- U9 pad 4: (no net) -> 2.4vRef
Routing:
- net GND: track 0.00 -> 701.6 mm
- net 6v: track 0.00 -> 611.0 mm
- net Neg6v: track 0.00 -> 603.6 mm
- net JTPC: track 0.00 -> 336.3 mm, vias 0 -> 1
- net WFM-: track 0.00 -> 309.7 mm, vias 0 -> 1
- net PC4-: track 0.00 -> 285.6 mm
- net 2.4vRef: track 0.00 -> 260.7 mm
- net PC1-: track 0.00 -> 259.8 mm, vias 0 -> 1
- net PC2-: track 0.00 -> 241.3 mm
- net PC3-: track 0.00 -> 208.9 mm
- net {PC1}: track 0.00 -> 189.5 mm, vias 0 -> 1
- net J1-: track 0.00 -> 148.8 mm
- net J2-: track 0.00 -> 141.7 mm
- net PulseGenMargin: track 0.00 -> 135.8 mm
- net 1TPC-: track 0.00 -> 133.5 mm
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Other:
- board size 228.6 x 160 mm -> 233.3 x 160 mm
- board text added: "A-FP"
- board text added: "Board Positions 23, 24, 25"
- board text added: "Place connector on underside"
