File: KiCad/Real903/A-FS/A-FS.sch (KiCad schematic (older format))
At the start: 7 parts, among them J1 J1, U1 LS01, U2 LS12, U3 LS01, U8 LS12

Commit message: 1 December
Parts:
- added U10, U14: LS01, ELLIOTT:LSA, symbol LSA:LS01
- added U11, U12, U4: LS18, ELLIOTT:LSA, symbol LSA:LS18
- added U13, U9: LS12, ELLIOTT:LSA, symbol LSA:LS12
- added unit 3 of U2
- added unit 2 of U2
- added unit 3 of U3
- added unit 2 of U3
- U1, U2, U3, U8: footprint (none) -> ELLIOTT:LSA
Connections:
- wire segments 153 -> 171
- no-connect marks 23 -> 29
