File: KiCad/Real903/Board Tester/Board Tester.kicad_pcb (KiCad board)
At the start: 2 copper layers, 94 parts, among them J0 Conn_01x03

Commit message: 1 December
Parts:
- added J10: ~, TerminalBlock_Phoenix:TerminalBlock_Phoenix_MKDS-1,5-5-5.08_1x05_P5.08mm_Horizontal, F.Cu at (331.2, 186.2)
- added J11: ~, TerminalBlock_Phoenix:TerminalBlock_Phoenix_MKDS-1,5-5-5.08_1x05_P5.08mm_Horizontal, F.Cu at (331.4, 218.8)
- added J12: ~, TerminalBlock_Phoenix:TerminalBlock_Phoenix_MKDS-1,5-5-5.08_1x05_P5.08mm_Horizontal, F.Cu at (273.0, 46.2)
- added J13: ~, TerminalBlock_Phoenix:TerminalBlock_Phoenix_MKDS-1,5-5-5.08_1x05_P5.08mm_Horizontal, F.Cu at (313.0, 46.2)
- added J14: ~, TerminalBlock_Phoenix:TerminalBlock_Phoenix_MKDS-1,5-5-5.08_1x05_P5.08mm_Horizontal, F.Cu at (193.0, 46.2)
- added J15: ~, TerminalBlock_Phoenix:TerminalBlock_Phoenix_MKDS-1,5-5-5.08_1x05_P5.08mm_Horizontal, F.Cu at (233.0, 46.2)
- added J16: ~, TerminalBlock_Phoenix:TerminalBlock_Phoenix_MKDS-1,5-6-5.08_1x06_P5.08mm_Horizontal, F.Cu at (331.2, 155.4)
- added J17: ~, TerminalBlock_Phoenix:TerminalBlock_Phoenix_MKDS-1,5-6-5.08_1x06_P5.08mm_Horizontal, F.Cu at (331.4, 122.0)
- added J18: ~, Connector_PinHeader_2.54mm:PinHeader_2x10_P2.54mm_Vertical, F.Cu at (300.2, 127.2)
- added J19: ~, TerminalBlock_Phoenix:TerminalBlock_Phoenix_MKDS-1,5-4_1x04_P5.00mm_Horizontal, F.Cu at (331.2, 178.4)
- added J20: ~, TerminalBlock_Phoenix:TerminalBlock_Phoenix_MKDS-1,5-4_1x04_P5.00mm_Horizontal, F.Cu at (331.4, 88.6)
- added J21: ~, ELLIOTT:TerminalBlock_5.08_1x08, F.Cu at (190.8, 116.2)
- added J22: ~, ELLIOTT:TerminalBlock_5.08_1x03, F.Cu at (175.0, 238.4)
- added NE1: ~, Resistor_THT:R_Axial_DIN0204_L3.6mm_D1.6mm_P2.54mm_Vertical, F.Cu at (175.2, 148.4)
- added NE2: ~, Resistor_THT:R_Axial_DIN0204_L3.6mm_D1.6mm_P2.54mm_Vertical, F.Cu at (185.2, 148.4)
- added NE3: ~, Resistor_THT:R_Axial_DIN0204_L3.6mm_D1.6mm_P2.54mm_Vertical, F.Cu at (195.2, 148.4)
- added NE4: ~, Resistor_THT:R_Axial_DIN0204_L3.6mm_D1.6mm_P2.54mm_Vertical, F.Cu at (205.2, 148.4)
- added NE5: ~, Resistor_THT:R_Axial_DIN0204_L3.6mm_D1.6mm_P2.54mm_Vertical, F.Cu at (215.2, 148.4)
- added NE6: ~, Resistor_THT:R_Axial_DIN0204_L3.6mm_D1.6mm_P2.54mm_Vertical, F.Cu at (225.2, 148.4)
- added NE7: ~, Resistor_THT:R_Axial_DIN0204_L3.6mm_D1.6mm_P2.54mm_Vertical, F.Cu at (235.2, 148.4)
- added NE8: ~, Resistor_THT:R_Axial_DIN0204_L3.6mm_D1.6mm_P2.54mm_Vertical, F.Cu at (245.2, 148.4)
- added Q1: ~, Package_TO_SOT_THT:TO-92, F.Cu at (172.7, 133.4)
- added Q2: ~, Package_TO_SOT_THT:TO-92, F.Cu at (182.7, 133.4)
- added Q3: ~, Package_TO_SOT_THT:TO-92, F.Cu at (192.7, 133.4)
- added Q4: ~, Package_TO_SOT_THT:TO-92, F.Cu at (202.7, 133.4)
- added Q5: ~, Package_TO_SOT_THT:TO-92, F.Cu at (212.7, 133.4)
- added Q6: ~, Package_TO_SOT_THT:TO-92, F.Cu at (222.7, 133.4)
- added Q7: ~, Package_TO_SOT_THT:TO-92, F.Cu at (232.7, 133.4)
- added Q8: ~, Package_TO_SOT_THT:TO-92, F.Cu at (242.7, 133.4)
- added R43: 82k, ELLIOTT:R_Axial_DIN0204_L3.6mm_D1.6mm_P7.62mm_Horizontal, F.Cu at (175.2, 160.2)
- added R44: 82k, ELLIOTT:R_Axial_DIN0204_L3.6mm_D1.6mm_P7.62mm_Horizontal, F.Cu at (185.2, 160.2)
- added R45: 82k, ELLIOTT:R_Axial_DIN0204_L3.6mm_D1.6mm_P7.62mm_Horizontal, F.Cu at (195.2, 160.2)
- added R46: 82k, ELLIOTT:R_Axial_DIN0204_L3.6mm_D1.6mm_P7.62mm_Horizontal, F.Cu at (205.2, 160.2)
- added R47: 82k, ELLIOTT:R_Axial_DIN0204_L3.6mm_D1.6mm_P7.62mm_Horizontal, F.Cu at (215.2, 160.2)
- added R48: 82k, ELLIOTT:R_Axial_DIN0204_L3.6mm_D1.6mm_P7.62mm_Horizontal, F.Cu at (225.2, 160.2)
- added R49: 82k, ELLIOTT:R_Axial_DIN0204_L3.6mm_D1.6mm_P7.62mm_Horizontal, F.Cu at (235.2, 160.2)
- added R50: 82k, ELLIOTT:R_Axial_DIN0204_L3.6mm_D1.6mm_P7.62mm_Horizontal, F.Cu at (245.2, 160.2)
- moved R33 229.3 mm to (276.6, 147.4), turned to 270 degrees
- moved R35 226.6 mm to (292.0, 147.4), turned to 270 degrees
- moved R32 214.6 mm to (269.4, 147.4), turned to 270 degrees
- moved D3 211.4 mm to (276.4, 135.6), turned to 270 degrees
- moved D8 210.2 mm to (291.4, 116.2), turned to 90 degrees
- moved D7 210.0 mm to (299.0, 116.2), turned to 90 degrees
- moved D6 207.5 mm to (299.0, 135.6), turned to 270 degrees
- moved D5 206.6 mm to (291.4, 135.6), turned to 270 degrees
- moved R36 202.3 mm to (299.4, 147.4), turned to 270 degrees
- moved D4 202.0 mm to (283.8, 135.6), turned to 270 degrees
- moved D2 194.3 mm to (269.0, 135.6), turned to 270 degrees
- moved R31 193.4 mm to (261.6, 147.4), turned to 270 degrees
- moved R37 190.6 mm to (299.0, 104.6), turned to 90 degrees
- moved D9 189.7 mm to (283.8, 116.2), turned to 90 degrees
- moved SW12 185.1 mm to (281.0, 67.8)
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Connections:
- D1 pad 1: (no net) -> Net-(D1-Pad1)
- D10 pad 1: (no net) -> Net-(D10-Pad1)
- D11 pad 1: (no net) -> Net-(D11-Pad1)
- D12 pad 1: (no net) -> Net-(D12-Pad1)
- D2 pad 1: (no net) -> Net-(D2-Pad1)
- D3 pad 1: (no net) -> Net-(D3-Pad1)
- D4 pad 1: (no net) -> Net-(D4-Pad1)
- D5 pad 1: (no net) -> Net-(D5-Pad1)
- D6 pad 1: (no net) -> Net-(D6-Pad1)
- D7 pad 1: (no net) -> Net-(D7-Pad1)
- D8 pad 1: (no net) -> Net-(D8-Pad1)
- D9 pad 1: (no net) -> Net-(D9-Pad1)
- SW1 pad 2: (no net) -> Net-(J10-Pad5)
- SW10 pad 2: (no net) -> Net-(J11-Pad1)
- SW11 pad 2: (no net) -> Net-(J12-Pad5)
- SW12 pad 2: (no net) -> Net-(J13-Pad5)
- SW13 pad 2: (no net) -> Net-(J12-Pad4)
- SW14 pad 2: (no net) -> Net-(J13-Pad4)
- SW15 pad 2: (no net) -> Net-(J12-Pad3)
- SW16 pad 2: (no net) -> Net-(J13-Pad3)
- SW17 pad 2: (no net) -> Net-(J12-Pad2)
- SW18 pad 2: (no net) -> Net-(J13-Pad2)
- SW19 pad 2: (no net) -> Net-(J12-Pad1)
- SW2 pad 2: (no net) -> Net-(J10-Pad4)
- SW20 pad 2: (no net) -> Net-(J13-Pad1)
- SW21 pad 2: (no net) -> Net-(J14-Pad5)
- SW22 pad 2: (no net) -> Net-(J15-Pad5)
- SW23 pad 2: (no net) -> Net-(J14-Pad4)
- SW24 pad 2: (no net) -> Net-(J15-Pad4)
- SW25 pad 2: (no net) -> Net-(J14-Pad3)
- SW26 pad 2: (no net) -> Net-(J15-Pad3)
- SW27 pad 2: (no net) -> Net-(J14-Pad2)
- SW28 pad 2: (no net) -> Net-(J15-Pad2)
- SW29 pad 2: (no net) -> Net-(J14-Pad1)
- SW3 pad 2: (no net) -> Net-(J10-Pad3)
- SW30 pad 2: (no net) -> Net-(J15-Pad1)
- SW4 pad 2: (no net) -> Net-(J10-Pad2)
- SW5 pad 2: (no net) -> Net-(J10-Pad1)
- SW6 pad 2: (no net) -> Net-(J11-Pad5)
- SW7 pad 2: (no net) -> Net-(J11-Pad4)
- SW8 pad 2: (no net) -> Net-(J11-Pad3)
- SW9 pad 2: (no net) -> Net-(J11-Pad2)
Routing:
- net GND: track 0.00 -> 665.4 mm
- net +6v: track 0.00 -> 646.0 mm
- net -6v: track 0.00 -> 234.4 mm
- net 0v: track 0.00 -> 182.3 mm
- net -40v: track 0.00 -> 166.0 mm
- net +70v: track 0.00 -> 148.2 mm
- net Net-(J11-Pad5): track 0.00 -> 116.7 mm
- net Net-(J10-Pad5): track 0.00 -> 116.6 mm
- net Net-(J11-Pad4): track 0.00 -> 99.7 mm
- net Net-(J10-Pad4): track 0.00 -> 99.5 mm
- net Net-(D12-Pad1): track 0.00 -> 90.2 mm
- net Net-(D1-Pad1): track 0.00 -> 88.9 mm
- net Net-(J11-Pad3): track 0.00 -> 82.6 mm
- net Net-(J10-Pad3): track 0.00 -> 82.3 mm
- net Net-(D11-Pad1): track 0.00 -> 77.8 mm
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Other:
- board outline added: 259.1 x 213.4 mm
- net class Default: trace_width 0.25 -> 1
- board text added: "+6v 0v -6v"
- board text added: "-40v 0v +70v"
- board text added: "1"
- board text added: "1 1 1 1 1 1 1 0 1 2 3 4 5 6"
- board text added: "1 1 1 2 2 2 2 7 8 9 0 1 2 3"
- board text added: "10"
- board text added: "10 9 8 7 6"
- board text added: "2"
- board text added: "2 2 2 2 2 2 3 4 5 6 7 8 9 0"
- board text added: "3"
- board text added: "3 4 5 6 7 8 9"
- board text added: "4"
- board text added: "5"
- board text added: "5 4 3 2 1"
- board text added: "6"
- board text added: "7"
- board text added: "8"
- board text added: "9"
- board text added: "A"
- board text added: "A A A A A A A J H F E D C B"
- board text added: "A Z Y X W V U A"
- board text added: "B"
- board text added: "C"
- board text added: "D"
- board text added: "E"
- board text added: "F"
- board text added: "K J H F E D C"
- board text added: "T S R P N M L"

Commit message: July backplane update
Routing:
- added copper zone on B.Cu, net (none)
- added copper zone on F.Cu, net (none)
Changed lines of the file:
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@@
   (segment (start 93.1 48.3) (end 99.8 41.6) (width 1) (layer F.Cu) (net 170))
   (segment (start 99.8 41.6) (end 124.56 41.6) (width 1) (layer F.Cu) (net 170))
+  (zone (net 0) (net_name "") (layer F.Cu) (hatch edge 0.508)
+    (connect_pads (clearance 2.54))
+    (min_thickness 0.254)
+    (fill yes (arc_segments 16) (thermal_gap 0.508) (thermal_bridge_width 0.508))
+    (polygon
+      (pts
+        (xy 86 41) (xy 336 41) (xy 336 245) (xy 86.2 245)
+      )
+    )
+  )
+  (zone (net 0) (net_name "") (layer B.Cu) (hatch edge 0.508)
+    (connect_pads (clearance 2.54))
+    (min_thickness 0.254)
+    (fill yes (arc_segments 16) (thermal_gap 0.508) (thermal_bridge_width 0.508))
+    (polygon
+      (pts
+        (xy 86 41) (xy 336 41) (xy 336 245) (xy 86.2 245)
+      )
+    )
+  )
 )
