File: KiCad/Real903/Control Panel/Control Panel.sch (KiCad schematic (older format))
At the start: 153 parts, among them K3 4PDTRelay, SW101 Cycle Stop, SW102 Order Stop, SW11 Cycle Repeat, SW12 Int1, SW131 Manual 1, SW132 Trace 1, SW14 Int2, SW151 Manual 2, SW152 Trace 2, SW16 Int3, SW171 Manual 3, SW172 Trace 3, SW2 Jump, SW3 Stop, SW4 Restart, SW5 Reset, SW6 On, SW7 Off, SW81 Obey - Single, SW82 Obey - Continuous, SW83 Obey - Continuous, SW91 Enter - Single, SW92 Enter - Continuous, SW93 Enter - Continuous, SW94 Enter - Continuous

Commit message: July backplane update
Parts:
- added J10: ~, ELLIOTT:TerminalBlock_5.08_1x08, symbol Connector_Generic:Conn_01x08
- C121, C141, C161, C51, C52, C53, C54, C55, C56, C57, C58: footprint (none) -> Capacitor_THT:CP_Axial_L10.0mm_D4.5mm_P15.00mm_Horizontal
- D1, D12, D14, D16, D2, D3, D41, D42, D43, D44, D45, D46, D47, D48: footprint (none) -> ELLIOTT:D_DO-35_SOD27_P7.62mm_Horizontal
- J1: footprint (none) -> Connector_PinHeader_2.54mm:PinHeader_2x10_P2.54mm_Vertical
- J2: footprint (none) -> ELLIOTT:TerminalBlock-5.08_1x10
- J3: footprint (none) -> ELLIOTT:TerminalBlock_5.08_1x03
- J4: footprint (none) -> ELLIOTT:TerminalBlock_5.08_1x08; symbol Connector_Generic:Conn_01x14 -> Connector_Generic:Conn_01x08
- J5: footprint (none) -> ELLIOTT:TerminalBlock_5.08_1x08; symbol Connector_Generic:Conn_01x13 -> Connector_Generic:Conn_01x08
- J6: footprint (none) -> ELLIOTT:TerminalBlock-5.08_1x10; symbol Connector_Generic:Conn_01x05 -> Connector_Generic:Conn_01x10
- K1, K2: footprint Relay_THT:Relay_DPDT_FRT5 -> ELLIOTT:Relay55.13
- K3: footprint (none) -> ELLIOTT:JumpRelay
- Q11, Q12, Q13, Q14, Q15, Q16, Q17, Q18, Q21, Q22, Q23, Q24, Q25, Q26, Q27, Q28: footprint (none) -> ELLIOTT:TO-92L_InlineCBE
- R121, R141, R161, R19, R20, R21, R22, R23, R24, R25, R26, R27, R28, R29, R3, R30, R31, R32, R33, R34, R35, R36, R37, R38, R39, R4, R40, R41, R42, R431, R432, R433, R434, R435, R436, R437, R438, R5, R61, R62, R63, R64, R65, R66, R67, R68: footprint (none) -> ELLIOTT:R_Axial_DIN0204_L3.6mm_D1.6mm_P7.62mm_Horizontal
- SW1: footprint (none) -> ELLIOTT:MiniSPDTSwitch
- SW10: renamed from SW101; value Cycle Stop -> O/C Stop; footprint (none) -> ELLIOTT:ElliottCPSwitch; symbol Switch:SW_SPDT -> LSA:ControlPanelSelectors
- SW10: renamed from SW102; value Order Stop -> O/C Stop; footprint (none) -> ELLIOTT:ElliottCPSwitch; symbol Switch:SW_SPDT -> LSA:ControlPanelSelectors
- SW11: footprint (none) -> ELLIOTT:ElliottCPSwitch
- SW12: renamed from LA121; value ~ -> Int1; footprint (none) -> ELLIOTT:Honeywell Sw; symbol Device:Lamp -> LSA:SPDT_Illuminatedx2
- SW12: renamed from LA123; value ~ -> Int1; footprint (none) -> ELLIOTT:Honeywell Sw; symbol Device:Lamp -> LSA:SPDT_Illuminatedx2
- SW12, SW14, SW16: footprint (none) -> ELLIOTT:Honeywell Sw; symbol Switch:SW_SPDT -> LSA:SPDT_Illuminatedx2
- SW13: renamed from SW131; value Manual 1 -> Man/Trace; footprint (none) -> ELLIOTT:ElliottCPSwitch; symbol Switch:SW_SPDT -> LSA:ControlPanelSelectors
- SW13: renamed from SW132; value Trace 1 -> Man/Trace; footprint (none) -> ELLIOTT:ElliottCPSwitch; symbol Switch:SW_SPDT -> LSA:ControlPanelSelectors
- SW14: renamed from LA141; value ~ -> Int2; footprint (none) -> ELLIOTT:Honeywell Sw; symbol Device:Lamp -> LSA:SPDT_Illuminatedx2
- SW14: renamed from LA143; value ~ -> Int2; footprint (none) -> ELLIOTT:Honeywell Sw; symbol Device:Lamp -> LSA:SPDT_Illuminatedx2
- SW15: renamed from SW151; value Manual 2 -> Man/Trace; footprint (none) -> ELLIOTT:ElliottCPSwitch; symbol Switch:SW_SPDT -> LSA:ControlPanelSelectors
- SW15: renamed from SW152; value Trace 2 -> Man/Trace; footprint (none) -> ELLIOTT:ElliottCPSwitch; symbol Switch:SW_SPDT -> LSA:ControlPanelSelectors
- SW16: renamed from LA161; value ~ -> Int3; footprint (none) -> ELLIOTT:Honeywell Sw; symbol Device:Lamp -> LSA:SPDT_Illuminatedx2
- SW16: renamed from LA163; value ~ -> Int3; footprint (none) -> ELLIOTT:Honeywell Sw; symbol Device:Lamp -> LSA:SPDT_Illuminatedx2
- SW17: renamed from SW171; value Manual 3 -> Man/Trace; footprint (none) -> ELLIOTT:ElliottCPSwitch; symbol Switch:SW_SPDT -> LSA:ControlPanelSelectors
- SW17: renamed from SW172; value Trace 3 -> Man/Trace; footprint (none) -> ELLIOTT:ElliottCPSwitch; symbol Switch:SW_SPDT -> LSA:ControlPanelSelectors
- SW18: value ~ -> NG1; footprint (none) -> ELLIOTT:ElliottNGSwitch
- SW19: value ~ -> NG2; footprint (none) -> ELLIOTT:ElliottNGSwitch
- SW2: footprint (none) -> ELLIOTT:EAO31
- SW20: value ~ -> NG3; footprint (none) -> ELLIOTT:ElliottNGSwitch
- SW21: value ~ -> NG4; footprint (none) -> ELLIOTT:ElliottNGSwitch
- SW22: value ~ -> NG5; footprint (none) -> ELLIOTT:ElliottNGSwitch
- SW23: value ~ -> NG6; footprint (none) -> ELLIOTT:ElliottNGSwitch
- SW24: value ~ -> NG7; footprint (none) -> ELLIOTT:ElliottNGSwitch
- SW25: value ~ -> NG8; footprint (none) -> ELLIOTT:ElliottNGSwitch
- SW26: value ~ -> NG9; footprint (none) -> ELLIOTT:ElliottNGSwitch
- SW27: value ~ -> NG10; footprint (none) -> ELLIOTT:ElliottNGSwitch
- SW28: value ~ -> NG11; footprint (none) -> ELLIOTT:ElliottNGSwitch
- SW29: value ~ -> NG12; footprint (none) -> ELLIOTT:ElliottNGSwitch
- SW3: renamed from LA3; value ~ -> Stop; footprint (none) -> ELLIOTT:EAO31; symbol Device:Lamp -> LSA:SPDT_Illuminated
- SW3, SW4, SW5, SW6, SW7: footprint (none) -> ELLIOTT:EAO31; symbol Switch:SW_SPDT -> LSA:SPDT_Illuminated
- SW30: value ~ -> NG13; footprint (none) -> ELLIOTT:ElliottNGSwitch
- SW31: value ~ -> NG14; footprint (none) -> ELLIOTT:ElliottNGSwitch
- SW32: value ~ -> NG15; footprint (none) -> ELLIOTT:ElliottNGSwitch
- SW33: value ~ -> NG16; footprint (none) -> ELLIOTT:ElliottNGSwitch
- SW34: value ~ -> NG17; footprint (none) -> ELLIOTT:ElliottNGSwitch
- SW35: value ~ -> NG18; footprint (none) -> ELLIOTT:ElliottNGSwitch
- SW5: renamed from LA5; value ~ -> Reset; footprint (none) -> ELLIOTT:EAO31; symbol Device:Lamp -> LSA:SPDT_Illuminated
- SW6: renamed from LA6; value ~ -> On; footprint (none) -> ELLIOTT:EAO31; symbol Device:Lamp -> LSA:SPDT_Illuminated
- SW7: renamed from LA7; value ~ -> Off; footprint (none) -> ELLIOTT:EAO31; symbol Device:Lamp -> LSA:SPDT_Illuminated
- SW8: renamed from SW81; value Obey - Single -> Obey; footprint (none) -> ELLIOTT:ElliottCPSwitch; symbol Switch:SW_SPDT -> LSA:ControlPanelSelectors
- SW8: renamed from SW82; value Obey - Continuous -> Obey; footprint (none) -> ELLIOTT:ElliottCPSwitch; symbol Switch:SW_SPDT -> LSA:ControlPanelSelectors
- SW8: renamed from SW83; value Obey - Continuous -> Obey; footprint (none) -> ELLIOTT:ElliottCPSwitch; symbol Switch:SW_SPDT -> LSA:ControlPanelSelectors
- SW9: renamed from SW91; value Enter - Single -> Enter; footprint (none) -> ELLIOTT:ElliottCPSwitch; symbol Switch:SW_SPDT -> LSA:ControlPanelSelectors
- SW9: renamed from SW92; value Enter - Continuous -> Enter; footprint (none) -> ELLIOTT:ElliottCPSwitch; symbol Switch:SW_SPDT -> LSA:ControlPanelSelectors
- SW9: renamed from SW94; value Enter - Continuous -> Enter; footprint (none) -> ELLIOTT:ElliottCPSwitch; symbol Switch:SW_SPDT -> LSA:ControlPanelSelectors
- SW9: renamed from SW93; value Enter - Continuous -> Enter; footprint (none) -> ELLIOTT:ElliottCPSwitch; symbol Switch:SW_SPDT -> LSA:ControlPanelSelectors
Connections:
- no-connect marks 31 -> 33
