File: KiCad/Real903/Backplane1/Backplane1.sch (KiCad schematic (older format))
At the start: 18 parts, among them J37 Conn_02x32, J38 Conn_02x32, J39 Conn_02x32, J40 Conn_02x32, J41 Conn_02x32, J42 Conn_02x32, J43 Conn_02x32, J44 Conn_02x32, J45 Conn_02x32, J48 Conn_02x32, J49 Conn_02x32, J50 Conn_02x32, J51 Conn_02x32, J52 Conn_02x32, J53 Conn_02x32, J54 Conn_02x32, J55 Conn_02x32, J56 Conn_02x32

Commit message: Update for PCB Design
Parts:
- removed J37, J38, J39, J40, J41, J42, J43, J44, J45, J48, J49, J50, J51, J52, J53, J54, J55, J56: Conn_02x32, symbol LSA:Conn_02x32
- added J1: ~, TerminalBlock_Phoenix:TerminalBlock_Phoenix_MKDS-3-3-5.08_1x03_P5.08mm_Horizontal, symbol Connector_Generic:Conn_01x03
- added J135, J136: ~, ELLIOTT:PinHeader_1x06_P2.54mm_Vertical, symbol Connector_Generic:Conn_01x06
- added J34, J35, J36: ~, ELLIOTT:DIN41612_B_2x32_Horizontal, symbol LSA:Conn_02x32
Connections:
- net labels added: II10m, II11m, II12m, II13m, II14m, II15m, II16m, II17m, II18m, II1m, II2m, II3m, II4m, II5m, II6m, II7m, II8m, II9m, IIG, IIG-, IIS, J1', J1-', J2', J2-', J3', J3-'
- net labels removed: 0TM1-, 0TM2-, A10, A11, A2, A3, A4, A5, A6, A7, A8, A9, ATF1, ATF2, An, C1, C10, C11, C12, C13, C14, C15, C16, C17, C18, C2, C3, C4, C5, C6, C7, C8, C9, DTF1-1, DTF1-2, DTF2a, ETJ2-, ETJ3-, F1, F10, F11, F12, F13, F14, F15, F16, F17, F18, F2, F3, F4, F5, F6, F7, F8, F9, FTG1, FTG2, GTA1, GTA2, GTJ1, GTJ2, GTM1, GTM2, GTQ2, IP-1, IP-2, IP-3, IP-4, IP-5, IP-6, IP-7, IP-8, IP1, IP10, IP11, IP12, IP13, IP14, IP15, IP16, IP17, IP18, IP2, IP3, IP4, IP5, IP6, IP7, IP8, IP9, ITF, J1, J1-, J10-, J11-, J12-, J13-, J14, J15, J16, J2, J2-, J3, J3-, J5-, J6-, J7-, J8-, J9-, JTF1, JTF2, JTG14-, JTG15-, JTG16-, KTJ1-, KTJ5-, LTG1, LTG2, M-TF1, M-TF2, MTF1, MTF2, MTI, MTP1, MTP2, OTA1-, OTA2-, OTG1-, OTG2-, OTI-, OTJ1-, OTJ2-, OTP1-, OTP2-, OTQ1-, OTQ2-, PTG1-1, PTG1-2, PTG2-1, PTG2-2, QTF1, QTF2, Qn, RTG1, RTG2, SKT11B, SKT11F, SKT11G, SKT11H, SKT11J, SKT11K, SKT11L, SKT11M, SKT11N, SKT11P, SKT1AA, SKT1B, SKT1BB, SKT1C, SKT1CC, SKT1D, SKT1DD, SKT1E, SKT1EE, SKT1F, SKT1FF, SKT1G, SKT1GG, SKT1H, SKT1HH, SKT1J, SKT1K, SKT1L, SKT1M, SKT1N, SKT1P, SKT1R, SKT1S, SKT1T, SKT1U, SKT1V, SKT1W, SKT1X, SKT1Y, SKT1Z, SKT1a, SKT1b, SKT1c, SKT1d, SKT1e, SKT1f, SKT1g, SKT1h, SKT1i, SKT1j, SKT1k, SKT1m, SKT1n, SKT1p, SKT1q, SKT1r, SKT1s, SKT1t, SKT1u, SKT1v, SKT1w, SKT1x, SKT1y, SKT1z, SKT2B, SKT2C, SKT2D, SKT2E, SKT2F, SKT2G, SKT2H, SKT2J, SKT2K, SKT2L, SKT2M, SKT2N, SKT2P, SKT2R, SKT2S, SKT2T, SKT2U, SKT2V, SKT2W, SKT2X, SKT2Y, SKT2Z, SKT2a, SKT2b, SKT2c, SKT2d, SKT2e, SKT2f, SKT2g, SKT2h, SKT2i, SKT2j, SKT2k, SKT2m, STORE1-, STORE10-, STORE10X-, STORE11-, STORE11X-, STORE12-, STORE12X-, STORE13-, STORE13X-, STORE14-, STORE14X-, STORE15-, STORE15X-, STORE16-, STORE16X-, STORE17-, STORE17X-, STORE18-, STORE18X-, STORE1X-, STORE2-, STORE2X-, STORE3-, STORE3X-, STORE4-, STORE4X-, STORE5-, STORE5X-, STORE6-, STORE6X-, STORE7-, STORE7X-, STORE8-, STORE8X-, STORE9-, STORE9X-, VTG1, VTG2, W14, W15, W16, W17, W18, W2, W3, W4, WTM1, WTM2, X0, X1
- wire segments 879 -> 137
- no-connect marks 123 -> 70
Other:
- note added: "37 38 39 40 41 42 43 44 45"
- note added: "46 47"
- note added: "48 49 50 51 52 53 54 55 56"

Commit message: New boards
Parts:
- added J~2, J~3: ~, ELLIOTT:TerminalBlock_5.08_1x03, symbol Connector_Generic:Conn_01x03
- added TH33, TH35, TH37, TH39, TH41, TH43, TH45: ~, MountingHole:MountingHole_2.7mm, symbol Mechanical:MountingHole
- J135, J136: footprint ELLIOTT:PinHeader_1x06_P2.54mm_Vertical -> ELLIOTT:TerminalBlock_5.08_1x06
- J34, J35, J36: footprint ELLIOTT:DIN41612_B_2x32_Horizontal -> ELLIOTT:DIN41612_B_2x32_Vertical
- J~1: renamed from J1; footprint TerminalBlock_Phoenix:TerminalBlock_Phoenix_MKDS-3-3-5.08_1x03_P5.08mm_Horizontal -> ELLIOTT:TerminalBlock_5.08_1x03
Connections:
- net labels added: ~IIG, ~J14, ~J16, ~J1~', ~J2~'
- net labels removed: IIG-, J1-', J14-, J16-, J2-'
- wire segments 137 -> 143

Commit message: July backplane update
Parts:
- removed J135, J136: ~, ELLIOTT:TerminalBlock_5.08_1x06, symbol Connector_Generic:Conn_01x06
- removed J34, J35, J36: ~, ELLIOTT:DIN41612_B_2x32_Vertical, symbol LSA:Conn_02x32
- renumbered J~1 to J1, J~2 to J2, J~3 to J3
Connections:
- net labels added: #A[1..18], #G[1..18], #I[1..4], #J[1..16], #M[1..18], #P[1..11], #Q[1..18], IP'[1..8], IP[1..18], ~A~[1..18], ~STORE~[1..18]
- net labels removed: II1, II10, II10m, II11, II11m, II12, II12m, II13, II13m, II14, II14m, II15, II15m, II16, II16m, II17, II17m, II18, II18m, II1m, II2, II2m, II3, II3m, II4, II4m, II5, II5m, II6, II6m, II7, II7m, II8, II8m, II9, II9m, IIG, IIS, J1', J10, J11, J12, J13, J15-, J2', J3', J3-', J4, J4-, J5, J6, J7, J8, J9, ~IIG, ~J14, ~J16, ~J1~', ~J2~'
- wire segments 143 -> 78
- no-connect marks 70 -> 0
Other:
- moved on the sheet: J1, J2, J3

Commit message: July 20th
Parts:
- added TH49, TH51, TH53, TH55, TH56: ~, MountingHole:MountingHole_2.7mm, symbol Mechanical:MountingHole
Connections:
- net labels added: II[1..18], J[1..16], M[1..18], W[1..18]
Other:
- moved on the sheet: J1, J2, J3

Commit message: August 2
Connections:
- net labels added: ~P~[1..13]
Changed lines of the file:
@@
 F44 "#P[1..9]" U R 6075 1675 30
 F45 "W[1..9]" U R 6075 1600 30
+F46 "~P~[1..9]" I R 6075 1525 30
 $EndSheet
 Text GLabel 1000 1150 0    25   Input ~ 0
@@
 GND
 $Sheet
-S 4875 3150 1450 2675
+S 4875 3150 1200 1300
 U 5F060A9A
 F0 "Connections" 50
@@
 F8 "#P[1..11]" I L 4875 3475 30
 F9 "#J[1..16]" I L 4875 3175 30
-F10 "#M[1..18]" I L 4875 3625 30
+F10 "#M[1..18]" U L 4875 3625 30
 F11 "IP[1..18]" I L 4875 4150 30
 F12 "IP'[1..8]" I L 4875 4225 30
@@
 F14 "J[1..16]" U L 4875 3925 30
 F15 "W[1..18]" U L 4875 3700 30
+F16 "~P~[1..13]" I L 4875 4300 30
 $EndSheet
 Wire Bus Line
@@
 Wire Bus Line
 	4750 3325 4875 3325
-Text GLabel 6200 1825 2    25   Input ~ 0
+Text GLabel 6200 1825 2    25   UnSpc ~ 0
 #G[1..18]
-Text GLabel 4750 3325 0    25   Input ~ 0
+Text GLabel 4750 3325 0    25   UnSpc ~ 0
 #G[1..18]
-Text GLabel 6200 1750 2    25   Input ~ 0
+Text GLabel 6200 1750 2    25   UnSpc ~ 0
 #A[1..18]
 Wire Bus Line
 	6200 1750 6075 1750
-Text GLabel 6200 2225 2    25   Input ~ 0
+Text GLabel 6200 2225 2    25   UnSpc ~ 0
 ~A~[1..18]
 Wire Bus Line
 	6075 2225 6200 2225
-Text GLabel 1000 2225 0    25   Input ~ 0
+Text GLabel 1000 2225 0    25   UnSpc ~ 0
 ~A~[1..18]
-Text GLabel 4750 4075 0    25   Input ~ 0
+Text GLabel 4750 4075 0    25   UnSpc ~ 0
 ~A~[1..18]
-Text GLabel 4750 3400 0    25   Input ~ 0
+Text GLabel 4750 3400 0    25   UnSpc ~ 0
 #A[1..18]
 Wire Bus Line
@@
 Wire Bus Line
 	4750 4075 4875 4075
-Text GLabel 1000 1825 0    25   Input ~ 0
+Text GLabel 1000 1825 0    25   UnSpc ~ 0
 #G[1..18]
-Text GLabel 1000 1750 0    25   Input ~ 0
+Text GLabel 1000 1750 0    25   UnSpc ~ 0
 #A[1..18]
-Text GLabel 6200 1900 2    25   Input ~ 0
+Text GLabel 6200 1900 2    25   UnSpc ~ 0
 #Q[1..18]
-Text GLabel 1000 1900 0    25   Input ~ 0
+Text GLabel 1000 1900 0    25   UnSpc ~ 0
 #Q[1..18]
-Text GLabel 4750 3250 0    25   Input ~ 0
+Text GLabel 4750 3250 0    25   UnSpc ~ 0
 #Q[1..18]
 Wire Bus Line
@@
 Wire Wire Line
 	2700 675  4575 675
-Text GLabel 4750 4000 0    25   Input ~ 0
+Text GLabel 4750 4000 0    25   UnSpc ~ 0
 ~STORE~[1..18]
 Wire Bus Line
 	4750 4000 4875 4000
-Text GLabel 1000 2300 0    25   Input ~ 0
+Text GLabel 1000 2300 0    25   UnSpc ~ 0
 ~STORE~[1..18]
 Wire Bus Line
 	1000 2300 1175 2300
-Text GLabel 4750 3175 0    25   Input ~ 0
+Text GLabel 4750 3175 0    25   UnSpc ~ 0
 #J[1..16]
-Text GLabel 1000 2050 0    25   Input ~ 0
+Text GLabel 1000 2050 0    25   UnSpc ~ 0
 #P[1..11]
 Wire Bus Line
@@
 Wire Bus Line
 	1000 2050 1175 2050
-Text GLabel 1000 1475 0    25   Input ~ 0
+Text GLabel 1000 1475 0    25   UnSpc ~ 0
 #I[1..4]
 Wire Bus Line
 	1000 1475 1175 1475
-Text GLabel 6200 2300 2    25   Input ~ 0
+Text GLabel 6200 2300 2    25   UnSpc ~ 0
 ~STORE~[1..18]
 Wire Bus Line
 	6200 2300 6075 2300
-Text GLabel 4750 3550 0    25   Input ~ 0
+Text GLabel 4750 3550 0    25   UnSpc ~ 0
 #I[1..4]
 Wire Bus Line
 	4875 3550 4750 3550
-Text GLabel 4750 3475 0    25   Input ~ 0
+Text GLabel 4750 3475 0    25   UnSpc ~ 0
 #P[1..11]
 Wire Bus Line
@@
 Wire Bus Line
 	4875 3175 4750 3175
-Text GLabel 1000 1975 0    25   Input ~ 0
+Text GLabel 1000 1975 0    25   UnSpc ~ 0
 #J[1..16]
-Text GLabel 1000 1675 0    25   Input ~ 0
+Text GLabel 1000 1675 0    25   UnSpc ~ 0
 #M[1..18]
 Wire Bus Line
 	1000 1675 1175 1675
-Text GLabel 4750 3625 0    25   Input ~ 0
+Text GLabel 4750 3625 0    25   UnSpc ~ 0
 #M[1..18]
 Wire Bus Line
@@
 Wire Bus Line
 	1175 2375 1000 2375
-Text GLabel 6200 2150 2    25   Input ~ 0
+Text GLabel 6200 2150 2    25   UnSpc ~ 0
 IP[1..18]
 Wire Bus Line
 	6075 2150 6200 2150
-Text GLabel 1000 2150 0    25   Input ~ 0
+Text GLabel 1000 2150 0    25   UnSpc ~ 0
 IP[1..18]
 Wire Bus Line
 	1000 2150 1175 2150
-Text GLabel 4750 4150 0    25   Input ~ 0
+Text GLabel 4750 4150 0    25   UnSpc ~ 0
 IP[1..18]
 Wire Bus Line
@@
 Text GLabel 4650 2600 0    25   UnSpc ~ 0
 IP'[1..8]
-Text GLabel 4750 4225 0    25   Input ~ 0
+Text GLabel 4750 4225 0    25   UnSpc ~ 0
 IP'[1..8]
 Wire Bus Line
@@
 Wire Wire Line
 	4300 2150 4850 2150
-Text GLabel 6200 1975 2    25   Input ~ 0
+Text GLabel 6200 1975 2    25   UnSpc ~ 0
 #J[1..16]
 Wire Bus Line
@@
 F49 "M[10..18]" U L 1175 2550 30
 F50 "W[10..18]" U L 1175 1600 30
+F51 "~P~[10..13]" I L 1175 2450 30
 $EndSheet
 Wire Bus Line
@@
 Wire Bus Line
 	6200 1675 6075 1675
-Text GLabel 6200 1675 2    25   Input ~ 0
+Text GLabel 6200 1675 2    25   UnSpc ~ 0
 #P[1..11]
 Text GLabel 6200 1600 2    25   UnSpc ~ 0
@@
 	0    -1   -1   0
 $EndComp
+Text GLabel 1000 2450 0    25   UnSpc ~ 0
+~P~[1..13]
+Wire Bus Line
+	1000 2450 1175 2450
+Text GLabel 6200 1525 2    25   UnSpc ~ 0
+~P~[1..13]
+Wire Bus Line
+	6200 1525 6075 1525
+Text GLabel 4750 4300 0    25   UnSpc ~ 0
+~P~[1..13]
+Wire Bus Line
+	4750 4300 4875 4300
 $EndSCHEMATC
