File: KiCad/Real903/Backplane1/RegistersA.sch (KiCad schematic (older format))
At the start: 36 parts

Commit message: New boards
Parts:
- J137, J138, J139, J140, J141: footprint ELLIOTT:PinHeader_1x06_P2.54mm_Vertical -> ELLIOTT:TerminalBlock_5.08_1x07
- J142, J143, J144, J145: footprint ELLIOTT:PinHeader_1x07_P2.54mm_Vertical -> ELLIOTT:TerminalBlock_5.08_1x07
- J237, J238, J239, J240, J241, J242, J243, J244, J245: footprint ELLIOTT:PinHeader_1x03_P2.54mm_Vertical -> ELLIOTT:TerminalBlock_5.08_1x03
Connections:
- net labels added: DT1-2, SKT1~f, SKT1~g, SKT1~h, SKT1~j, SKT1~k, SKT1~m, SKT1~n, SKT1~p, SKT1~z, SKT2~f, SKT2~g, SKT2~h, SKT2~j, SKT2~k, SKT2~m, SKT2~x, SKT2~y, ~J14, ~J16, ~M~TF2, ~OTA~2, ~OTG~2, ~OTJ~2, ~OTM~2, ~OTP~2
- net labels removed: 0TM2-, DTF1-2, J14-, J16-, M-TF2, OTA2-, OTG2-, OTJ2-, OTP2-, SKT1f_, SKT1g_, SKT1h_, SKT1j_, SKT1k_, SKT1m_, SKT1n_, SKT1p_, SKT1z_, SKT2f_, SKT2g_, SKT2h_, SKT2j_, SKT2k_, SKT2m_, SKT2x_, SKT2y_
- wire segments 630 -> 634
- no-connect marks 111 -> 105

Commit message: July backplane update
Parts:
- removed J137, J138, J139, J140, J141, J145: ~, ELLIOTT:TerminalBlock_5.08_1x07, symbol Connector_Generic:Conn_01x07
Connections:
- net labels added: #A10, #A11, #A12, #A13, #A14, #A15, #A16, #A17, #A18, #A[10..18], #G10, #G11, #G12, #G13, #G14, #G15, #G16, #G17, #G18, #G[10..18], #I1, #I2, #I3, #I4, #I[1..4], #J10, #J11, #J12, #J13, #J14, #J15, #J16, #J[10..18], #M10, #M11, #M12, #M13, #M14, #M15, #M16, #M17, #M18, #M[10..18], #P10, #P11, #P[10..11], #Q10, #Q11, #Q12, #Q13, #Q14, #Q15, #Q16, #Q17, #Q18, #Q[10..18], -6v, 0v, A[3..9], C17-5-H, C18-5-8, DTF1-2-5-23, DTF2a-8-26, F18-5-K, I1-22-D, I2-22-F, I3-22-J, I4-22-L, II[10..18], IP[10..18], J[10..16], M18-7-9, MTI-5-17, P12-30-V, P13-30-R, X1-57-11, ~A~10, ~A~11, ~A~12, ~A~13, ~A~14, ~A~15, ~A~16, ~A~17, ~A~18, ~A~[10..18], ~JTG14~, ~JTG15~, ~JTG16~, ~J~14, ~J~14-22-28, ~J~15, ~J~15-22-29, ~J~16, ~J~16-22-26, ~J~[14..16], ~OTI~, ~OTI~-5-18, ~OTQ2~, ~STORE~10, ~STORE~11, ~STORE~12, ~STORE~13, ~STORE~14, ~STORE~15, ~STORE~16, ~STORE~17, ~STORE~18, ~STORE~[10..18]
- net labels removed: A10-, A11-, A12-, A13-, A14-, A15-, A16-, A17-, A18-, An, C18, I1, I2, I3, I4, J10-, J11-, J12-, J13-, J15-, JTG14-, JTG15-, JTG16-, M18, Neg6v, OTI-, OTQ2-, P12, P13, Qn, SKT1AA, SKT1BB, SKT1CC, SKT1DD, SKT1EE, SKT1FF, SKT1GG, SKT1HH, SKT1L, SKT1M, SKT1N, SKT1P, SKT1R, SKT1S, SKT1T, SKT1U, SKT1V, SKT1i, SKT1~f, SKT1~g, SKT1~h, SKT1~j, SKT1~k, SKT1~m, SKT1~n, SKT1~p, SKT1~z, SKT2L, SKT2M, SKT2N, SKT2P, SKT2R, SKT2S, SKT2T, SKT2U, SKT2V, SKT2i, SKT2~f, SKT2~g, SKT2~h, SKT2~j, SKT2~k, SKT2~m, SKT2~x, SKT2~y, SKT3r, SKT3s, SKT3t, SKT3u, STORE10-, STORE11-, STORE12-, STORE13-, STORE14-, STORE15-, STORE16-, STORE17-, STORE18-, X1, ~J14, ~J16
- wire segments 634 -> 163
- no-connect marks 105 -> 191
Other:
- note removed: "21:"
- note removed: "AB: ACCUMULATOR-"
- note removed: "AC: {Q REGISTER}"
- note removed: "AD:"
- note removed: "AJ: STORE-"
- note removed: "M: {G REGISTER}"
- note removed: "Y: {P REGISTER & I REGISTER}"
- note removed: "Z: {ACCUMULATOR}"

Commit message: July 20th
Parts:
- removed J142, J143, J144: ~, ELLIOTT:TerminalBlock_5.08_1x07, symbol Connector_Generic:Conn_01x07
- removed J237, J238, J239, J240, J241, J242, J243, J244, J245: ~, ELLIOTT:TerminalBlock_5.08_1x03, symbol Connector_Generic:Conn_01x03
- removed J337, J338, J339, J340, J341, J342, J343, J344, J345: ~, ELLIOTT:TerminalBlock_5.08_1x08, symbol Connector_Generic:Conn_01x08
Connections:
- net labels added: M10, M11-7-21, M12-6-W, M13-7-6, M14, M15, M16, M17, M18, M[10..18], W10, W11, W12, W13, W[10..18], ~I~1-22-E, ~I~2-22-H, ~I~3-22-K, ~I~4-22-M, ~M~12-6-Y, ~M~13-6-18, ~M~18-7-11, ~P~10-30-X, ~P~11-30-W, ~P~12-30-T, ~P~13-30-18
- net labels removed: I1-, I2-, I3-, I4-, M10-, M11-, M12-, M13-, M14-, M15-, M16-, M17-, M18-, P10-, P11-, P12-, P13-, SKT11L, SKT11M, SKT11N, SKT11P
- wire segments 163 -> 118
- no-connect marks 191 -> 101
Other:
- note removed: "12: PERIPHERAL INPUT"
- note removed: "18: NUMBER GENERATOR"
- note removed: "9: IP TO G"
- note removed: "R: J REGISTER -"
- note removed: "S: {J REGISTER}"
- note removed: "T: J REGISTER"
- note removed: "U: {M REGISTER}"
- note removed: "V: M REGISTER-"
- note removed: "W: P REGISTER-"

Commit message: August 2
Connections:
- net ~J~12-25-27: now reaches J43.R (Pin_R)
- net ~J~11-25-19: now reaches J44.R (Pin_R)
- net ~J~10-25-8: now reaches J45.R (Pin_R)
- net ~P~10-30-X renamed ~P~10
- net ~P~11-30-W renamed ~P~11
- net ~P~12-30-T renamed ~P~12
- net ~P~13-30-18 renamed ~P~13
- no-connect marks 101 -> 98
Changed lines of the file:
@@
 Wire Wire Line
 	7225 3900 7125 3900
-Text GLabel 10225 3900 2    32   UnSpc ~ 0
-~P~13-30-18
-Text GLabel 11725 3900 2    32   UnSpc ~ 0
-~P~12-30-T
-Text GLabel 13225 3900 2    32   UnSpc ~ 0
-~P~11-30-W
-Text GLabel 14725 3900 2    32   UnSpc ~ 0
-~P~10-30-X
-Wire Wire Line
-	14725 3900 14625 3900
-Wire Wire Line
-	13225 3900 13125 3900
-Wire Wire Line
-	11725 3900 11625 3900
-Wire Wire Line
-	10125 3900 10225 3900
 Text GLabel 13225 4600 2    32   UnSpc ~ 0
 M11-7-21
@@
 ~OTI~
 NoConn ~ 10125 3400
-NoConn ~ 11625 3400
-NoConn ~ 13125 3400
-NoConn ~ 14625 3400
 Text Label 5625 3400 0    40   ~ 0
 ~J~16
@@
 Text Label 14125 3800 2    40   ~ 0
 W10
+Text Label 10125 3900 0    40   ~ 0
+~P~13
+Text Label 11625 3900 0    40   ~ 0
+~P~12
+Text Label 13125 3900 0    40   ~ 0
+~P~11
+Text Label 14625 3900 0    40   ~ 0
+~P~10
+Text HLabel 1050 6075 0    40   Input ~ 0
+~P~[10..13]
+Text GLabel 13225 3400 2    32   UnSpc ~ 0
+~J~11-25-19
+Text GLabel 11725 3400 2    32   UnSpc ~ 0
+~J~12-25-27
+Text GLabel 14725 3400 2    32   UnSpc ~ 0
+~J~10-25-8
+Wire Wire Line
+	14725 3400 14625 3400
+Wire Wire Line
+	13225 3400 13125 3400
+Wire Wire Line
+	11725 3400 11625 3400
 $EndSCHEMATC
