File: KiCad/Real903/Backplane1/RegistersB.sch (KiCad schematic (older format))
At the start: 36 parts

Commit message: New boards
Parts:
- added TP1: Q1-, TestPoint:TestPoint_Plated_Hole_D2.0mm, symbol Connector:TestPoint
- J148, J149, J150, J151, J152, J155, J156: footprint ELLIOTT:PinHeader_1x07_P2.54mm_Vertical -> ELLIOTT:TerminalBlock_5.08_1x07
- J153, J154: footprint ELLIOTT:PinHeader_1x06_P2.54mm_Vertical -> ELLIOTT:TerminalBlock_5.08_1x07
- J248, J249, J250, J251, J252, J253, J254, J255, J256: footprint ELLIOTT:PinHeader_1x03_P2.54mm_Vertical -> ELLIOTT:TerminalBlock_5.08_1x03
Connections:
- net labels added: DT1-1, DT1-2, SKT1~b, SKT1~c, SKT1~d, SKT1~e, SKT1~r, SKT1~s, SKT1~t, SKT1~u, SKT1~v, SKT1~w, SKT1~x, SKT1~y, SKT2~b, SKT2~c, SKT2~d, SKT2~e, SKT2~n, SKT2~p, SKT2~r, SKT2~s, SKT2~t, SKT2~u, SKT2~v, SKT2~w, ~A1, ~A2, ~A3, ~A4, ~A5, ~A6, ~A7, ~A8, ~A9, ~J1~, ~J2~, ~M~TF1, ~OTA~1, ~OTG~1, ~OTJ~1, ~OTM~1, ~OTP~1, ~OTP~2, ~PTG1~1, ~PTG2~1, ~Q1, ~STORE1, ~STORE2, ~STORE3, ~STORE4, ~STORE5
- net labels removed: 0TM1-, 0TM2-, A1-, A2-, A3-, A4-, A5-, A6-, A7-, A8-, A9-, DTF1-1, DTF1-2, J1-, J2-, M-TF1, OTA1-, OTG1-, OTJ1-, OTP1-, OTP2-, PTG1-1, PTG2-1, SKT1b_, SKT1c_, SKT1d_, SKT1e_, SKT1r_, SKT1s_, SKT1t_, SKT1u_, SKT1v_, SKT1w_, SKT1x_, SKT1y_, SKT2b_, SKT2c_, SKT2d_, SKT2e_, SKT2n_, SKT2p_, SKT2r_, SKT2s_, SKT2t_, SKT2u_, SKT2v_, SKT2w_, STORE1-, STORE2-, STORE3-, STORE4-, STORE5-
- wire segments 646 -> 647
- no-connect marks 97 -> 93

Commit message: July backplane update
Parts:
- removed J148, J149, J150, J151, J152, J153, J154, J155, J156: ~, ELLIOTT:TerminalBlock_5.08_1x07, symbol Connector_Generic:Conn_01x07
- J254, J255, J256: footprint ELLIOTT:TerminalBlock_5.08_1x03 -> ELLIOTT:TerminalBlock_5.08_1x03+1
Connections:
- net labels added: #A1, #A2, #A3, #A4, #A5, #A6, #A7, #A8, #A9, #A[1..9], #G1, #G2, #G3, #G4, #G5, #G6, #G7, #G8, #G9, #G[1..9], #J1, #J2, #J3, #J4, #J5, #J6, #J7, #J8, #J9, #J[1..9], #Q1, #Q2, #Q3, #Q4, #Q5, #Q6, #Q7, #Q8, #Q9, #Q[1..9], 0v, A[3..9], DTF1-1, DTF1-1-5-22, DTF1-2, DTF1-2-5-23, F1-57-7, FTG1-57-4, II[1..9], IP'[1..8], IP[1..9], ITF-8-12, J[1..9], LTG1-57-8, PTG1-1, PTG2-1, RTG1-57-6, X0-57-5, ~A~1, ~A~2, ~A~3, ~A~4, ~A~5, ~A~6, ~A~7, ~A~8, ~A~9, ~A~[1..9], ~ETJ2~-6-27, ~ETJ3~-6-28, ~J~4-23-27, ~J~5-24-3, ~J~6-24-8, ~J~7-24-19, ~J~8-24-27, ~J~9-25-3, ~KTJ1~-6-21, ~KTJ5~-6-22, ~OTG1~-57-M, ~OTQ1~, ~STORE~1, ~STORE~2, ~STORE~3, ~STORE~4, ~STORE~5, ~STORE~6, ~STORE~7, ~STORE~8, ~STORE~9, ~STORE~[1..9]
- net labels removed: DT1-1, DT1-2, ETJ2-, ETJ3-, ITF, J3-, J4-, J5-, J6-, J7-, J8-, J9-, KTJ1-, KTJ5-, OTQ1-, SKT1B, SKT1C, SKT1D, SKT1E, SKT1F, SKT1G, SKT1H, SKT1J, SKT1K, SKT1W, SKT1X, SKT1Y, SKT1Z, SKT1a, SKT1q, SKT1~b, SKT1~c, SKT1~d, SKT1~e, SKT1~r, SKT1~s, SKT1~t, SKT1~u, SKT1~v, SKT1~w, SKT1~x, SKT1~y, SKT2W, SKT2X, SKT2Y, SKT2Z, SKT2a, SKT2~b, SKT2~c, SKT2~d, SKT2~e, STORE6-, STORE7-, STORE8-, STORE9-, X0, ~A1, ~A2, ~A3, ~A4, ~A5, ~A6, ~A7, ~A8, ~A9, ~J1~, ~J2~, ~PTG1~1, ~PTG2~1, ~STORE1, ~STORE2, ~STORE3, ~STORE4, ~STORE5
- wire segments 647 -> 214
- no-connect marks 93 -> 143
Other:
- note removed: "12: PERIPHERAL INPUT"
- note removed: "9: IP TO G"
- note removed: "AB: ACCUMULATOR-"
- note removed: "AC: {Q REGISTER}"
- note removed: "C: D: 6: OTHER"
- note removed: "M: {G REGISTER}"
- note removed: "N: J REGISTER SET"
- note removed: "R: J REGISTER -"
- note removed: "S: {J REGISTER}"
- note removed: "Z: {ACCUMULATOR}"

Commit message: July 20th
Parts:
- removed J248, J249, J250, J251, J252, J253: ~, ELLIOTT:TerminalBlock_5.08_1x03, symbol Connector_Generic:Conn_01x03
- removed J254, J255, J256: ~, ELLIOTT:TerminalBlock_5.08_1x03+1, symbol Connector_Generic:Conn_01x03
- removed J348, J349, J350, J351, J352, J353, J354, J355, J356: ~, ELLIOTT:TerminalBlock_5.08_1x08, symbol Connector_Generic:Conn_01x08
- removed TP1: Q1-, TestPoint:TestPoint_Plated_Hole_D2.0mm, symbol Connector:TestPoint
Connections:
- net labels added: #M1, #M2, #M3, #M4, #M5, #M6, #M7, #M8, #M9, #M[1..9], #P1, #P2, #P3, #P4, #P5, #P6, #P7, #P8, #P9, #P[1..9], J1-20-C, J2-20-E, J3-20-H, M1, M2, M3, M4, M5, M6, M7, M8, M9, M[1..9], W1, W5, W6, W7, W8, W9, W[1..9], ~P~1-32-C, ~P~2-32-D, ~P~3-32-E, ~P~4-32-F, ~P~5-30-AC, ~P~6-30-24, ~P~7-30-AA, ~P~8-30-22, ~P~9-30-Y, ~Q~1-7-15
- net labels removed: M1-, M2-, M3-, M4-, M5-, M6-, M7-, M8-, M9-, P1-, P2-, P3-, P4-, P5-, P6-, P7-, P8-, P9-, SKT11B, SKT11F, SKT11G, SKT11H, SKT11J, SKT11K, SKT2B, SKT2C, SKT2D, SKT2E, SKT2F, SKT2G, SKT2H, SKT2J, SKT2K, SKT2q, SKT2~n, SKT2~p, SKT2~r, SKT2~s, SKT2~t, SKT2~u, SKT2~v, SKT2~w, ~Q1
- wire segments 214 -> 145
- no-connect marks 143 -> 89
Other:
- note removed: "18: NUMBER GENERATOR"
- note removed: "AJ: STORE-"
- note removed: "T: J REGISTER"
- note removed: "U: {M REGISTER}"
- note removed: "V: M REGISTER-"
- note removed: "W: P REGISTER-"
- note removed: "Y: {P REGISTER}"

Commit message: August 2
Connections:
- net ~J~3'-20-7: now reaches J54.R (Pin_R)
- net ~J~2'-20-5: now reaches J55.R (Pin_R)
- net ~J~1'-20-3: now reaches J56.R (Pin_R)
- net ~P~1-32-C renamed ~P~1
- net ~P~2-32-D renamed ~P~2
- net ~P~3-32-E renamed ~P~3
- net ~P~4-32-F renamed ~P~4
- net ~P~5-30-AC renamed ~P~5
- net ~P~6-30-24 renamed ~P~6
- net ~P~7-30-AA renamed ~P~7
- net ~P~8-30-22 renamed ~P~8
- net ~P~9-30-Y renamed ~P~9
- no-connect marks 89 -> 86
Changed lines of the file:
@@
 NoConn ~ 13850 1875
 NoConn ~ 13850 2175
-Text GLabel 13950 1775 2    40   Input ~ 0
+Text GLabel 13950 1775 2    32   UnSpc ~ 0
 F1-57-7
 Wire Wire Line
@@
 Wire Wire Line
 	11850 4475 11750 4475
-Text GLabel 13950 1575 2    40   Input ~ 0
+Text GLabel 13950 1575 2    32   UnSpc ~ 0
 ITF-8-12
 Wire Wire Line
 	13950 1575 13850 1575
-Text GLabel 13950 1675 2    40   Input ~ 0
+Text GLabel 13950 1675 2    32   UnSpc ~ 0
 X0-57-5
 Wire Wire Line
@@
 Wire Wire Line
 	1250 2275 1350 2275
-Text GLabel 13950 2475 2    30   Input ~ 0
+Text GLabel 13950 2475 2    32   UnSpc ~ 0
 ~KTJ1~-6-21
-Text GLabel 12450 2475 2    30   Input ~ 0
+Text GLabel 12450 2475 2    32   UnSpc ~ 0
 ~ETJ2~-6-27
 Wire Wire Line
@@
 	10950 2475 10850 2475
 NoConn ~ 9350 2475
-Text GLabel 7950 2475 2    30   Input ~ 0
+Text GLabel 7950 2475 2    32   UnSpc ~ 0
 ~KTJ5~-6-22
 Wire Wire Line
@@
 Text GLabel 1100 4175 0    40   Input ~ 0
 DTF1-2-5-23
-Text GLabel 4100 4175 0    40   Input ~ 0
+Text GLabel 4100 4175 0    32   UnSpc ~ 0
 DTF1-1-5-22
 Wire Wire Line
@@
 Text GLabel 6450 2675 2    30   Input ~ 0
 ~J~6-24-8
-Text GLabel 7950 2675 2    30   Input ~ 0
+Text GLabel 7950 2675 2    32   UnSpc ~ 0
 ~J~5-24-3
 Wire Wire Line
@@
 Wire Wire Line
 	7950 2675 7850 2675
-Text GLabel 9450 2675 2    30   Input ~ 0
+Text GLabel 9450 2675 2    32   UnSpc ~ 0
 ~J~4-23-27
 Wire Wire Line
@@
 Wire Wire Line
 	1850 3075 1950 3075
-Text GLabel 1950 3175 2    32   UnSpc ~ 0
-~P~9-30-Y
-Text GLabel 3450 3175 2    32   UnSpc ~ 0
-~P~8-30-22
-Text GLabel 4950 3175 2    32   UnSpc ~ 0
-~P~7-30-AA
-Text GLabel 6450 3175 2    32   UnSpc ~ 0
-~P~6-30-24
-Text GLabel 7950 3175 2    32   UnSpc ~ 0
-~P~5-30-AC
-Text GLabel 9450 3175 2    32   UnSpc ~ 0
-~P~4-32-F
-Text GLabel 10950 3175 2    32   UnSpc ~ 0
-~P~3-32-E
-Text GLabel 12450 3175 2    32   UnSpc ~ 0
-~P~2-32-D
-Text GLabel 13950 3175 2    32   UnSpc ~ 0
-~P~1-32-C
-Wire Wire Line
-	13950 3175 13850 3175
-Wire Wire Line
-	12450 3175 12350 3175
-Wire Wire Line
-	10950 3175 10850 3175
-Wire Wire Line
-	9350 3175 9450 3175
-Wire Wire Line
-	7850 3175 7950 3175
-Wire Wire Line
-	6350 3175 6450 3175
-Wire Wire Line
-	4850 3175 4950 3175
-Wire Wire Line
-	3450 3175 3350 3175
-Wire Wire Line
-	1950 3175 1850 3175
 NoConn ~ 12350 4175
 NoConn ~ 10850 4175
@@
 NoConn ~ 3350 4175
 NoConn ~ 1850 4175
-Text GLabel 13125 1975 0    40   Input ~ 0
+Text GLabel 13125 1975 0    32   UnSpc ~ 0
 RTG1-57-6
-Text GLabel 14050 1975 2    40   Input ~ 0
+Text GLabel 14050 1975 2    32   UnSpc ~ 0
 LTG1-57-8
 Text GLabel 13975 4175 2    32   UnSpc ~ 0
@@
 Text Label 9350 2875 0    40   ~ 0
 J4
-NoConn ~ 13850 2675
-NoConn ~ 12350 2675
-NoConn ~ 10850 2675
 Text GLabel 10950 2875 2    32   UnSpc ~ 0
 J3-20-H
@@
 Text HLabel 2625 9300 0    40   UnSpc ~ 0
 W[1..9]
+Text Label 1850 3175 0    40   ~ 0
+~P~9
+Text Label 3350 3175 0    40   ~ 0
+~P~8
+Text Label 4850 3175 0    40   ~ 0
+~P~7
+Text Label 6350 3175 0    40   ~ 0
+~P~6
+Text Label 7850 3175 0    40   ~ 0
+~P~5
+Text Label 9350 3175 0    40   ~ 0
+~P~4
+Text Label 10850 3175 0    40   ~ 0
+~P~3
+Text Label 12350 3175 0    40   ~ 0
+~P~2
+Text Label 13850 3175 0    40   ~ 0
+~P~1
+Text HLabel 3000 9300 0    40   Input ~ 0
+~P~[1..9]
+Text GLabel 10950 2675 2    32   UnSpc ~ 0
+~J~3'-20-7
+Text GLabel 12450 2675 2    32   UnSpc ~ 0
+~J~2'-20-5
+Text GLabel 13950 2675 2    32   UnSpc ~ 0
+~J~1'-20-3
+Wire Wire Line
+	13950 2675 13850 2675
+Wire Wire Line
+	12450 2675 12350 2675
+Wire Wire Line
+	10950 2675 10850 2675
 $EndSCHEMATC
