File: KiCad/Real903/Backplane1/WaveformDrivers.sch (KiCad schematic (older format))
At the start: 4 parts

Commit message: New boards
Parts:
- J146, J147: footprint ELLIOTT:PinHeader_1x16_P2.54mm_Vertical -> ELLIOTT:TerminalBlock-5.08_1x18; symbol Connector_Generic:Conn_01x16 -> Connector_Generic:Conn_01x18
Connections:
- net labels added: ~M~TF1, ~M~TF2, ~M~TFa, ~OTA~', ~OTA~1, ~OTA~2, ~OTG~1, ~OTG~2, ~OTJ, ~OTJ~1, ~OTJ~2, ~OTM~1, ~OTM~2, ~OTP~1, ~OTP~2, ~PTG1~1, ~PTG2~1, ~RESET~2, ~VTG
- net labels removed: 0TM1-, 0TM2-, M-TF1, M-TF2, M-TFa, OTA-', OTA1-, OTA2-, OTG1-, OTG2-, OTJ-, OTJ1-, OTJ2-, OTP1-, OTP2-, PTG1-1, PTG2-1, RESET2-
- wire segments 135 -> 138
- no-connect marks 25 -> 26

Commit message: July backplane update
Connections:
- net ~OTG~1: no longer J146.17 (Pin_17), J46.29 (Pin_29)
- net ~OTG~2: no longer J46.AB (Pin_AB)
- net JTG14- renamed ~JTG14~
- net JTG15- renamed ~JTG15~
- net JTG16- renamed ~JTG16~
- net ~PTG1~1 renamed PTG1-1
- net ~PTG2~1 renamed PTG2-1
- new net ~OTQ~1: J46.29 (Pin_29)
- new net ~OTQ~2: J46.AB (Pin_AB)
- no-connect marks 26 -> 27
Changed lines of the file:
@@
 $Descr A4 11693 8268
 encoding utf-8
-Sheet 3 4
+Sheet 2 6
 Title ""
 Date ""
@@
 	1    0    0    -1
 $EndComp
-Text GLabel 4375 3475 2    40   Input ~ 0
-JTG16-
-Text GLabel 4375 4775 2    40   Input ~ 0
-JTG15-
 Wire Wire Line
 	4200 4775 4375 4775
-Text GLabel 4375 4575 2    40   Input ~ 0
-JTG14-
 Wire Wire Line
 	4375 4575 4200 4575
@@
 Text GLabel 4375 3775 2    40   Input ~ 0
 ~M~TFa
-Text GLabel 4375 4075 2    40   Input ~ 0
-J14
-Text GLabel 4375 3875 2    40   Input ~ 0
-MTI
-Text GLabel 3525 4775 0    40   Input ~ 0
-J15
-Text GLabel 4375 3675 2    40   Input ~ 0
-J16
 Text GLabel 4375 4275 2    40   Input ~ 0
 QTFa
@@
 	3700 5075 3525 5075
 Wire Wire Line
-	3525 4775 3700 4775
-Wire Wire Line
 	3525 1975 3700 1975
 Wire Wire Line
@@
 	4200 3175 4375 3175
 Wire Wire Line
-	4375 3675 4200 3675
-Wire Wire Line
 	4200 3775 4375 3775
 Wire Wire Line
@@
 	4200 3975 4375 3975
 Wire Wire Line
-	4375 4075 4200 4075
-Wire Wire Line
 	4200 4175 4375 4175
 Wire Wire Line
@@
 Wire Wire Line
 	4200 4675 4375 4675
-Text GLabel 3525 3375 0    40   Input ~ 0
-JTF1
-Text GLabel 3525 3475 0    40   Input ~ 0
-JTF2
-Text GLabel 3525 3575 0    40   Input ~ 0
-MTF1
-Text GLabel 3525 3675 0    40   Input ~ 0
-MTF2
-Text GLabel 3525 3775 0    40   Input ~ 0
-~M~TF1
-Text GLabel 3525 3875 0    40   Input ~ 0
-~M~TF2
-Text GLabel 3525 4375 0    40   Input ~ 0
-QTF1
-Text GLabel 3525 4475 0    40   Input ~ 0
-QTF2
-Text GLabel 3525 4575 0    40   Input ~ 0
-ATF1
-Text GLabel 3525 4675 0    40   Input ~ 0
-ATF2
-Text GLabel 3525 2275 0    40   Input ~ 0
-FTG1
-Text GLabel 3525 2175 0    40   Input ~ 0
-FTG2
-Text GLabel 3525 2575 0    40   Input ~ 0
-LTG1
-Text GLabel 3525 2675 0    40   Input ~ 0
-LTG2
-Text GLabel 3525 2475 0    40   Input ~ 0
-RTG1
-Text GLabel 3525 2375 0    40   Input ~ 0
-RTG2
-Text GLabel 3525 3275 0    40   Input ~ 0
-VTG1
-Text GLabel 3525 3175 0    40   Input ~ 0
-VTG2
-Text GLabel 3525 3975 0    40   Input ~ 0
-MTP1
-Text GLabel 3525 4075 0    40   Input ~ 0
-MTP2
-Text GLabel 3525 2875 0    40   Input ~ 0
-~PTG1~1
-Text GLabel 3525 2775 0    40   Input ~ 0
-PTG1-2
-Text GLabel 3525 2975 0    40   Input ~ 0
-~PTG2~1
-Text GLabel 3525 3075 0    40   Input ~ 0
-PTG2-2
 Text GLabel 3525 4175 0    40   Input ~ 0
 JTPC
@@
 Wire Wire Line
 	2025 2075 2200 2075
-Text GLabel 2025 4775 0    40   Input ~ 0
-~OTG~1
 Wire Wire Line
 	2025 4775 2200 4775
-Text GLabel 2875 4275 2    40   Input ~ 0
-~OTG~2
 Wire Wire Line
 	2875 4275 2700 4275
-Text GLabel 2025 4475 0    40   Input ~ 0
-~OTA~2
-Text GLabel 2025 4375 0    40   Input ~ 0
-~OTA~1
-Text GLabel 2025 3075 0    40   Input ~ 0
-~OTJ~2
-Text GLabel 2025 2975 0    40   Input ~ 0
-~OTJ~1
-Text GLabel 2025 3475 0    40   Input ~ 0
-~OTM~2
-Text GLabel 2025 3375 0    40   Input ~ 0
-~OTM~1
-Text GLabel 2025 4075 0    40   Input ~ 0
-~OTP~2
-Text GLabel 2025 3975 0    40   Input ~ 0
-~OTP~1
-Text GLabel 2025 2875 0    40   Input ~ 0
-~OTG~2
-Text GLabel 2025 2775 0    40   Input ~ 0
-~OTG~1
-Text GLabel 2025 4175 0    40   Input ~ 0
-GTA1
-Text GLabel 2025 4275 0    40   Input ~ 0
-GTA2
-Text GLabel 2025 3275 0    40   Input ~ 0
-GTJ2
-Text GLabel 2025 3175 0    40   Input ~ 0
-GTJ1
-Text GLabel 2025 3875 0    40   Input ~ 0
-GTM2
-Text GLabel 2025 3775 0    40   Input ~ 0
-GTM1
-Text GLabel 2025 4575 0    40   Input ~ 0
-GTQ1
-Text GLabel 2025 4675 0    40   Input ~ 0
-GTQ2
-Text GLabel 2025 3675 0    40   Input ~ 0
-WTM2
-Text GLabel 2025 3575 0    40   Input ~ 0
-WTM1
 Text GLabel 2025 2375 0    40   Input ~ 0
 CRS
@@
 Text GLabel 2875 4075 2    40   Input ~ 0
 ~OTA~'
-Text GLabel 2875 2975 2    40   Input ~ 0
-~OTJ
 Text GLabel 2875 3375 2    40   Input ~ 0
 OTMa
@@
 Wire Wire Line
 	2300 6950 2150 6950
-Text GLabel 2150 7150 0    40   Input ~ 0
-~OTG~1
-Wire Wire Line
-	2150 7150 2300 7150
 NoConn ~ 2300 7250
 Text GLabel 4375 3275 2    40   Input ~ 0
@@
 	3600 7150 3800 7150
 NoConn ~ 3800 7250
+Text HLabel 3525 2175 0    40   Input ~ 0
+FTG2
+Text HLabel 3525 3175 0    40   Input ~ 0
+VTG2
+Text HLabel 3525 2275 0    40   Input ~ 0
+FTG1
+Text HLabel 3525 3275 0    40   Input ~ 0
+VTG1
+Text HLabel 4375 4575 2    40   Input ~ 0
+~JTG14~
+Text HLabel 4375 3475 2    40   Input ~ 0
+~JTG16~
+Text HLabel 4375 4775 2    40   Input ~ 0
+~JTG15~
+Text HLabel 3525 2475 0    40   Input ~ 0
+RTG1
+Text HLabel 3525 2575 0    40   Input ~ 0
+LTG1
+Text HLabel 3525 2375 0    40   Input ~ 0
+RTG2
+Text HLabel 3525 2675 0    40   Input ~ 0
+LTG2
+Text HLabel 3525 2775 0    40   Input ~ 0
+PTG1-2
+Text HLabel 3525 2875 0    40   Input ~ 0
+PTG1-1
+Text HLabel 3525 3075 0    40   Input ~ 0
+PTG2-2
+Text HLabel 3525 2975 0    40   Input ~ 0
+PTG2-1
+Text HLabel 2025 2775 0    40   Input ~ 0
+~OTG~1
+Text HLabel 2025 2875 0    40   Input ~ 0
+~OTG~2
+Text HLabel 2025 3275 0    40   Input ~ 0
+GTJ2
+Text HLabel 2025 3175 0    40   Input ~ 0
+GTJ1
+Text HLabel 2025 2975 0    40   Input ~ 0
+~OTJ~1
+Text HLabel 2025 3075 0    40   Input ~ 0
+~OTJ~2
+Text HLabel 3525 3575 0    40   Input ~ 0
+MTF1
+Text HLabel 3525 3675 0    40   Input ~ 0
+MTF2
+Text HLabel 2025 3375 0    40   Input ~ 0
+~OTM~1
+Text HLabel 2025 3475 0    40   Input ~ 0
+~OTM~2
+Text HLabel 2025 3575 0    40   Input ~ 0
+WTM1
+Text HLabel 2025 3675 0    40   Input ~ 0
+WTM2
+Text HLabel 3525 3375 0    40   Input ~ 0
+JTF1
+Text HLabel 3525 3475 0    40   Input ~ 0
+JTF2
+Text HLabel 3525 3775 0    40   Input ~ 0
+~M~TF1
+Text HLabel 3525 3875 0    40   Input ~ 0
+~M~TF2
+Text HLabel 2025 3775 0    40   Input ~ 0
+GTM1
+Text HLabel 2025 3875 0    40   Input ~ 0
+GTM2
+Text GLabel 2875 2975 2    40   Input ~ 0
+~OTJ
+Text HLabel 2025 4175 0    40   Input ~ 0
+GTA1
+Text HLabel 2025 4275 0    40   Input ~ 0
+GTA2
+Text HLabel 2025 4375 0    40   Input ~ 0
+~OTA~1
+Text HLabel 2025 4475 0    40   Input ~ 0
+~OTA~2
+Text HLabel 3525 4475 0    40   Input ~ 0
+QTF2
+Text HLabel 3525 4375 0    40   Input ~ 0
+QTF1
+Text HLabel 3525 4575 0    40   Input ~ 0
+ATF1
+Text HLabel 3525 4675 0    40   Input ~ 0
+ATF2
+Text HLabel 2025 4575 0    40   Input ~ 0
+GTQ1
+Text HLabel 2025 4675 0    40   Input ~ 0
+GTQ2
+Text HLabel 2025 4775 0    40   Input ~ 0
+~OTQ~1
+NoConn ~ 2300 7150
+Text HLabel 3525 3975 0    40   Input ~ 0
+MTP1
+Text HLabel 3525 4075 0    40   Input ~ 0
+MTP2
+Text HLabel 4375 3875 2    40   Input ~ 0
+MTI
+Text HLabel 2875 4275 2    40   Input ~ 0
+~OTQ~2
+Text HLabel 2025 3975 0    40   Input ~ 0
+~OTP~1
+Text HLabel 2025 4075 0    40   Input ~ 0
+~OTP~2
+Text Label 4200 4075 0    40   ~ 0
+J14
+Text Label 4200 3675 0    40   ~ 0
+J16
+Text HLabel 4025 5200 0    40   Input ~ 0
+J[14..16]
+Text Label 3700 4775 2    40   ~ 0
+J15
 $EndSCHEMATC

Commit message: July 20th
Parts:
- removed J146, J147: ~, ELLIOTT:TerminalBlock-5.08_1x18, symbol Connector_Generic:Conn_01x18
Connections:
- net ATFa renamed ATFa-9-21
- net CRS renamed CRS-7-AF
- net CRSm renamed CRSm-11-AC
- net FTGa renamed FTGa-8-6
- net GTAa renamed GTAa-8-27
- net GTJa renamed GTJa-8-28
- net GTMa renamed GTMa-8-23
- net GTQa renamed GTQa-8-24
- net JTFa renamed JTFa-9-24
- net JTPCa renamed JTPCa-9-7
- net LTGa renamed LTGa-9-25
- net MTFa renamed MTFa-8-30
- net MTPa renamed MTPa-9-22
- net Neg6v renamed -6v
- net OTMa renamed OTMa-9-23
- net PTG1-a renamed PTG1-a-9-6
- net PTG2-a renamed PTG2-a-9-12
- net QTFa renamed QTFa-9-30
- net RTGa renamed RTGa-9-14
- net SFD renamed SFD-6-R
- net SFDm renamed SFDm-19-V
- net VTGa renamed VTGa-8-7
- net WTMa renamed WTMa-8-21
- net t1 renamed t1-5-27
- net t2-2 renamed t2-2-5-20
- net t3-2 renamed t3-2-5-29
- net t4 renamed t4-5-26
- net t5 renamed t5-5-25
- net ~M~TFa renamed ~M~TFa-9-13
- net ~OTA~' renamed ~OTA~'-5-7
- net ~OTJ renamed ~OTJ~'-5-11
- net ~RESET~2 renamed ~RESET~2-2-Y
- net ~VTG renamed ~VTG~-32-R
- no-connect marks 27 -> 24

Commit message: August 2
Connections:
- net JTPC renamed JTPC-23-L
Changed lines of the file:
@@
 Wire Wire Line
 	4200 4675 4375 4675
-Text GLabel 3525 4175 0    40   Input ~ 0
-JTPC
-Text GLabel 3525 4275 0    40   Input ~ 0
-JTPC
+Text GLabel 3525 4275 0    40   UnSpc ~ 0
+JTPC-23-L
 Wire Wire Line
 	3525 2175 3700 2175
@@
 	3700 4075 3525 4075
 Wire Wire Line
-	3525 4175 3700 4175
-Wire Wire Line
-	3700 4275 3525 4275
+	3700 4275 3625 4275
 Wire Wire Line
 	3525 4375 3700 4375
@@
 Text Label 4200 5075 0    40   ~ 0
 GND
+Wire Wire Line
+	3700 4175 3625 4175
+Wire Wire Line
+	3625 4175 3625 4275
+Connection ~ 3625 4275
+Wire Wire Line
+	3625 4275 3525 4275
 $EndSCHEMATC
