File: KiCad/Real903/Backplane1/Backplane1.kicad_pcb (KiCad board)
At the start: 2 copper layers, 365.8 x 266.7 mm, 118 parts

Commit message: August Update
Parts:
- moved J1 192.1 mm to (214.8, 257.9)
Routing:
- net J11: track 269.0 -> 370.7 mm
- net II10: track 394.3 -> 489.8 mm, vias 1 -> 0
- net J14: track 239.1 -> 333.4 mm, vias 1 -> 2
- net II11: track 469.5 -> 390.3 mm, vias 0 -> 1
- net J12: track 363.1 -> 284.0 mm
- net II3: track 541.7 -> 616.7 mm, vias 1 -> 0
- net II9: track 471.0 -> 541.2 mm, vias 1 -> 0
- net II8: track 484.3 -> 553.6 mm, vias 1 -> 0
- net II1: track 631.2 -> 569.1 mm
- net J15-: track 194.6 -> 256.5 mm, vias 2 -> 1
- net A11: track 307.8 -> 249.9 mm
- net 0TM2-: track 333.9 -> 391.4 mm
- net II7: track 496.3 -> 553.4 mm, vias 1 -> 0
- net II6: track 510.6 -> 566.5 mm, vias 1 -> 0
- net J10: track 315.3 -> 369.8 mm, vias 2 -> 1
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Other:
- board text added: "1/W"
- board text added: "11/AC"
- board text added: "19/V"
- board text added: "2/Y"
- board text added: "20/3"
- board text added: "20/4"
- board text added: "20/5"
- board text added: "20/6"
- board text added: "20/7"
- board text added: "20/8"
- board text added: "22/E"
- board text added: "22/H"
- board text added: "22/K"
- board text added: "22/M"
- board text added: "23/L 47/24 47/23"
- board text added: "27/21 64/S"
- board text added: "27/22 64/K"
- board text added: "27/23 64/AA"
- board text added: "28/10"
- board text added: "28/11"
- board text added: "28/14"
- board text added: "28/15"
- board text added: "28/16"
- board text added: "28/17"
- board text added: "28/18"
- board text added: "28/19"
- board text added: "28/24"
- board text added: "28/25"
- board text added: "28/26"
- board text added: "28/3"
- board text added: "28/4"
- board text added: "28/5"
- board text added: "28/6"
- board text added: "28/7"
- board text added: "28/8"
- board text added: "28/9"
- board text added: "29/10"
- board text added: "29/12"
- board text added: "29/13"
- board text added: "29/14"
- board text added: "29/15"
- board text added: "29/16"
- board text added: "29/17"
- board text added: "29/20"
- board text added: "29/3"
- board text added: "29/4"
- board text added: "29/5"
- board text added: "29/6"
- board text added: "29/7"
- board text added: "29/8"
- board text added: "29/9"
- board text added: "30/18"
- board text added: "30/T"
- board text added: "30/W 32/P"
- board text added: "30/X 32/N"
- board text added: "31/AB"
- board text added: "31/AC 31/H"
- board text added: "31/AD 31/J"
- board text added: "31/AE 31/K"
- board text added: "31/AF 31/L"
- board text added: "31/C 31/Y 29/AJ"
- board text added: "31/D 31/Z"
- board text added: "31/E 31/AA"
- board text added: "31/M"
- board text added: "31/N"
- board text added: "31/P"
- board text added: "31/R"
- board text added: "31/S"
- board text added: "31/T"
- board text added: "31/U"
- board text added: "31/V"
- board text added: "31/W"
- board text added: "31/X"
- board text added: "34/12"
- board text added: "34/13"
- board text added: "34/14"
- board text added: "34/15"
- board text added: "34/16"
- board text added: "34/17"
- board text added: "34/18"
- board text added: "34/19"
- board text added: "34/20"
- board text added: "34/21"
- board text added: "34/22"
- board text added: "34/23"
- board text added: "34/24"
- board text added: "34/25"
- board text added: "34/26"
- board text added: "34/27"
- board text added: "34/28"
- board text added: "34/30"
- board text added: "35/13 63/K"
- board text added: "35/14 63/S"
- board text added: "36/14 63/AA"
- board text added: "36/15 61/S"
- board text added: "36/18 61/K"
- board text added: "36/19 61/AA"
- board text added: "36/20 60/S"
- board text added: "36/21 60/K"
- board text added: "36/22 60/AA"
- board text added: "36/23 60/T"
- board text added: "47/29 26/13"
- board text added: "47/V 26/12"
- board text added: "47/Z 26/19"
- board text added: "5/11"
- board text added: "5/20"
- board text added: "5/25 7/23 57/13"
- board text added: "5/26 6/AD"
- board text added: "5/27 6/AH"
- board text added: "5/29"
- board text added: "5/7"
- board text added: "56"
- board text added: "57/11"
- board text added: "57/15"
- board text added: "57/4"
- board text added: "57/5"
- board text added: "57/7"
- board text added: "59/38"
- board text added: "6/21"
- board text added: "6/22"
- board text added: "6/27"
- board text added: "6/28"
- board text added: "6/R"
- board text added: "6/W 7/13"
- board text added: "6/X 7/6"
- board text added: "7/21"
- board text added: "7/9"
- board text added: "7/AF"
- board text added: "8/12"
- board text added: "8/21"
- board text added: "8/23"
- board text added: "8/24"
- board text added: "8/27"
- board text added: "8/28"
- board text added: "8/30"
- board text added: "8/6"
- board text added: "8/7"
- board text added: "9/12"
- board text added: "9/13"
- board text added: "9/14"
- board text added: "9/21"
- board text added: "9/22"
- board text added: "9/23"
- board text added: "9/24"
- board text added: "9/25"
- board text added: "9/30"
- board text added: "9/6"
- board text added: "9/7 5/4"
- board text added: "J1-"
- board text added: "J10-"
- board text added: "J11-"
- board text added: "J12-"
- board text added: "J13-"
- board text added: "J14-"
- board text added: "J15-"
- board text added: "J16-"
- board text added: "J17-"
- board text added: "J18-"
- board text added: "J2-"
- board text added: "J3-"
- board text added: "J4-"
- board text added: "J5-"
- board text added: "J6-"
- board text added: "J7-"
- board text added: "J8-"
- board text added: "J9-"
- board text added: "M12-"
- board text added: "M13-"
- board text added: "M14-"
- board text added: "M15-"
- board text added: "M16-"
- board text added: "M17-"
- board text added: "SKT 11B"
- board text added: "SKT 11F"
- board text added: "SKT 11G"
- board text added: "SKT 11H"
- board text added: "SKT 11J"
- board text added: "SKT 11K"
- board text added: "SKT 11L"
- board text added: "SKT 11M"
- board text added: "SKT 11N"
- board text added: "SKT 11P"
- board text added: "SKT1AA"
- board text added: "SKT1B"
- board text added: "SKT1BB"
- board text added: "SKT1C"
- board text added: "SKT1CC"
- board text added: "SKT1D"
- board text added: "SKT1DD"
- board text added: "SKT1E"
- board text added: "SKT1EE"
- board text added: "SKT1F"
- board text added: "SKT1FF"
- board text added: "SKT1G"
- board text added: "SKT1GG"
- board text added: "SKT1H"
- board text added: "SKT1HH"
- board text added: "SKT1J"
- board text added: "SKT1K"
- board text added: "SKT1L"
- board text added: "SKT1M"
- board text added: "SKT1N"
- board text added: "SKT1P"
- board text added: "SKT1R"
- board text added: "SKT1S"
- board text added: "SKT1T"
- board text added: "SKT1U"
- board text added: "SKT1V"
- board text added: "SKT1f"
- board text added: "SKT1g"
- board text added: "SKT1h"
- board text added: "SKT1i"
- board text added: "SKT1j"
- board text added: "SKT1k"
- board text added: "SKT1m"
- board text added: "SKT1n"
- board text added: "SKT1p"
- board text added: "SKT1q"
- board text added: "SKT1r"
- board text added: "SKT1s"
- board text added: "SKT1t"
- board text added: "SKT1u"
- board text added: "SKT1v"
- board text added: "SKT1w"
- board text added: "SKT1x"
- board text added: "SKT1y"
- board text added: "SKT1z"
- board text added: "SKT2B"
- board text added: "SKT2C"
- board text added: "SKT2D"
- board text added: "SKT2E"
- board text added: "SKT2F"
- board text added: "SKT2G"
- board text added: "SKT2H"
- board text added: "SKT2J"
- board text added: "SKT2K"
- board text added: "SKT2L"
- board text added: "SKT2M"
- board text added: "SKT2N"
- board text added: "SKT2P"
- board text added: "SKT2R"
- board text added: "SKT2S"
- board text added: "SKT2T"
- board text added: "SKT2U"
- board text added: "SKT2V"
- board text added: "SKT2W"
- board text added: "SKT2X"
- board text added: "SKT2Y"
- board text added: "SKT2Z"
- board text added: "SKT2a"
- board text added: "SKT2b"
- board text added: "SKT2c"
- board text added: "SKT2d"
- board text added: "SKT2e"
- board text added: "SKT2f"
- board text added: "SKT2g"
- board text added: "SKT2h"
- board text added: "SKT2i"
- board text added: "SKT2j"
- board text added: "SKT2k"
- board text added: "SKT2m"
- board text added: "SKT2x"
- board text added: "SKT2y"
- board text added: "SKT3r"
- board text added: "SKT3s"
- board text added: "SKT3t"
- board text added: "SKT3u"
- board text added: "STORE 10"
- board text added: "STORE 11"
- board text added: "STORE 12"
- board text added: "STORE 13"
- board text added: "STORE 14"
- board text added: "STORE 15"
- board text added: "STORE 16"
- board text added: "STORE 17"
- board text added: "STORE 18"
- board text added: "XXX"
- board text removed: "33"

Commit message: Sept 1
Parts:
- moved TH33 1.78 mm to (19.1, 30.8)
- moved TH333 1.78 mm to (19.1, 286.7)
Changed lines of the file:
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@@
   )
   (module MountingHole:MountingHole_2.7mm (layer F.Cu)
-    (at 17.272 30.83)
+    (at 19.05 30.83)
     (descr "Mounting Hole 2.7mm, no annular")
     (tags "mounting hole 2.7mm no annular")
@@
   )
   (module MountingHole:MountingHole_2.7mm (layer F.Cu)
-    (at 17.272 286.68)
+    (at 19.05 286.68)
     (descr "Mounting Hole 2.7mm, no annular")
     (tags "mounting hole 2.7mm no annular")

Commit message: New boards
Parts:
- added J~2: ~, ELLIOTT:TerminalBlock_5.08_1x03, F.Cu at (29.8, 40.8)
- added J~3: ~, ELLIOTT:TerminalBlock_5.08_1x03, F.Cu at (336.9, 40.2)
- added TP1: Q1-, TestPoint:TestPoint_Plated_Hole_D2.0mm, F.Cu at (375.0, 40.2)
- J135, J136: footprint TerminalBlock_Phoenix:TerminalBlock_Phoenix_MKDS-3-6-5.08_1x06_P5.08mm_Horizontal -> ELLIOTT:TerminalBlock_5.08_1x06
- J146, J147: footprint ELLIOTT:TerminalBlock-5.08_1x16 -> ELLIOTT:TerminalBlock-5.08_1x18
- J254, J255, J256: footprint ELLIOTT:TerminalBlock_5.08_1x03 -> ELLIOTT:TerminalBlock_5.08_1x03+1
- TH151, TH156, TH2, TH251, TH256, TH3, TH33, TH35, TH37, TH39, TH41, TH43, TH45: value MountingHole_2.7mm -> ~
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- renumbered J1 to J~1
Connections:
- net A1- renamed ~A1
- net A2- renamed ~A2
- net A3- renamed ~A3
- net A4- renamed ~A4
- net A5- renamed ~A5
- net A6- renamed ~A6
- net A7- renamed ~A7
- net A8- renamed ~A8
- net A9- renamed ~A9
- net IIG- renamed ~IIG
- net J1- renamed ~J1~
- net J1-' renamed ~J1~'
- net J14- renamed ~J14
- net J16- renamed ~J16
- net J2- renamed ~J2~
- net J2-' renamed ~J2~'
- net M-TF1 renamed ~M~TF1
- net M-TF2 renamed ~M~TF2
- net M-TFa renamed ~M~TFa
- net OTA-' renamed ~OTA~'
- net OTA1- renamed ~OTA~1
- net OTA2- renamed ~OTA~2
- net OTG2- renamed ~OTG~2
- net OTJ- renamed ~OTJ
- net OTJ1- renamed ~OTJ~1
- net OTJ2- renamed ~OTJ~2
- net OTP1- renamed ~OTP~1
- net OTP2- renamed ~OTP~2
- net PTG1-1 renamed ~PTG1~1
- net PTG2-1 renamed ~PTG2~1
- net RESET2- renamed ~RESET~2
- net SKT1b_ renamed SKT1~b
- net SKT1c_ renamed SKT1~c
- net SKT1d_ renamed SKT1~d
- net SKT1e_ renamed SKT1~e
- net SKT1f_ renamed SKT1~f
- net SKT1g_ renamed SKT1~g
- net SKT1h_ renamed SKT1~h
- net SKT1j_ renamed SKT1~j
- net SKT1k_ renamed SKT1~k
- net SKT1m_ renamed SKT1~m
- net SKT1n_ renamed SKT1~n
- net SKT1p_ renamed SKT1~p
- net SKT1r_ renamed SKT1~r
- net SKT1s_ renamed SKT1~s
- net SKT1t_ renamed SKT1~t
- net SKT1u_ renamed SKT1~u
- net SKT1v_ renamed SKT1~v
- net SKT1w_ renamed SKT1~w
- net SKT1x_ renamed SKT1~x
- net SKT1y_ renamed SKT1~y
- net SKT1z_ renamed SKT1~z
- net SKT2b_ renamed SKT2~b
- net SKT2c_ renamed SKT2~c
- net SKT2d_ renamed SKT2~d
- net SKT2e_ renamed SKT2~e
- net SKT2f_ renamed SKT2~f
- net SKT2g_ renamed SKT2~g
- net SKT2h_ renamed SKT2~h
- net SKT2j_ renamed SKT2~j
- net SKT2k_ renamed SKT2~k
- net SKT2m_ renamed SKT2~m
- net SKT2n_ renamed SKT2~n
- net SKT2p_ renamed SKT2~p
- net SKT2r_ renamed SKT2~r
- net SKT2s_ renamed SKT2~s
- net SKT2t_ renamed SKT2~t
- net SKT2u_ renamed SKT2~u
- net SKT2v_ renamed SKT2~v
- net SKT2w_ renamed SKT2~w
- net SKT2x_ renamed SKT2~x
- net SKT2y_ renamed SKT2~y
- net STORE1- renamed ~STORE1
- net STORE2- renamed ~STORE2
- net STORE3- renamed ~STORE3
- net STORE4- renamed ~STORE4
- net STORE5- renamed ~STORE5
- J138 pad 1: (no net) -> MTI
- J140 pad 1: (no net) -> OTI-
- J141 pad 1: (no net) -> DTF2a
- J145 pad 1: (no net) -> DT1-2
- J150 pad 1: (no net) -> LTG1
- J151 pad 1: (no net) -> RTG1
- J152 pad 1: (no net) -> DT1-1
- J237 pad 1: (no net) -> F18
- J337 pad 2: (no net) -> M18-
- J37 pad 20: 0TM2- -> ~OTM~2
- J38 pad 20: 0TM2- -> ~OTM~2
- J39 pad 20: 0TM2- -> ~OTM~2
- J40 pad 20: 0TM2- -> ~OTM~2
- J41 pad 20: 0TM2- -> ~OTM~2
- J42 pad 20: 0TM2- -> ~OTM~2
- J42 pad 29: DTF1-2 -> DT1-2
- J43 pad 20: 0TM2- -> ~OTM~2
- J43 pad 29: DTF1-2 -> DT1-2
- J44 pad 20: 0TM2- -> ~OTM~2
- J44 pad 29: DTF1-2 -> DT1-2
- J45 pad 20: 0TM2- -> ~OTM~2
- J45 pad 29: DTF1-2 -> DT1-2
- J46 pad 15: 0TM1- -> ~OTM~1
- J46 pad 16: 0TM2- -> ~OTM~2
- J46 pad 29: OTG1- -> ~OTG~1
- J46 pad 9: OTG1- -> ~OTG~1
- J47 pad R: (no net) -> ~VTG
- J48 pad 10: OTG1- -> ~OTG~1
- J48 pad 20: 0TM1- -> ~OTM~1
- J48 pad 29: DTF1-2 -> DT1-2
- J49 pad 10: OTG1- -> ~OTG~1
- J49 pad 20: 0TM1- -> ~OTM~1
- J49 pad 29: DTF1-2 -> DT1-2
- J50 pad 10: OTG1- -> ~OTG~1
- J50 pad 20: 0TM1- -> ~OTM~1
- J50 pad 29: DTF1-1 -> DT1-1
- J51 pad 10: OTG1- -> ~OTG~1
- J51 pad 20: 0TM1- -> ~OTM~1
- J51 pad 29: DTF1-1 -> DT1-1
- J52 pad 10: OTG1- -> ~OTG~1
- J52 pad 20: 0TM1- -> ~OTM~1
- J52 pad 29: DTF1-1 -> DT1-1
- J53 pad 10: OTG1- -> ~OTG~1
- J53 pad 20: 0TM1- -> ~OTM~1
- J53 pad 29: DTF1-1 -> DT1-1
- J54 pad 10: OTG1- -> ~OTG~1
- J54 pad 20: 0TM1- -> ~OTM~1
- J54 pad 29: DTF1-1 -> DT1-1
- J55 pad 10: OTG1- -> ~OTG~1
- J55 pad 20: 0TM1- -> ~OTM~1
- J55 pad 29: DTF1-1 -> DT1-1
- J56 pad 10: OTG1- -> ~OTG~1
- J56 pad 20: 0TM2- -> ~OTM~1
- J56 pad 29: DTF1-1 -> DT1-1
- J56 pad AH: (no net) -> ~Q1
Routing:
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- added copper zone on B.Cu, net (none)
- added copper zone on F.Cu, net (none)
Other:
- board size 365.8 x 266.7 mm -> 386.1 x 266.7 mm
- board text added: "35/10 > 20/5"
- board text added: "35/11 > 20/8"
- board text added: "35/12 > 20/7"
- board text added: "35/7 > 20/4"
- board text added: "35/8 > 20/3"
- board text added: "35/9 > 20/6"
- board text added: "36/8 > 57/15"
- board text added: "37/18 > 29/14"
- board text added: "37/3 > 5/8"
- board text added: "37/5 > 57/11"
- board text added: "37/9 > 28/26"
- board text added: "37/AB > 31/X"
- board text added: "37/AD > 7/9"
- board text added: "37/E > 5/K"
- board text added: "37/V > 7/11"
- board text added: "38/18 > 1/W"
- board text added: "38/21 > 22/L"
- board text added: "38/22 > 5/17"
- board text added: "38/3 > 5/H"
- board text added: "38/9 > 28/25"
- board text added: "38/AB > 31/W"
- board text added: "38/W > 22/M"
- board text added: "39/18 > 29/12"
- board text added: "39/21 > 22/J"
- board text added: "39/9 > 28/24"
- board text added: "39/AB > 31/V"
- board text added: "39/R > 22/26"
- board text added: "39/W > 22/K"
- board text added: "40/18 > 29/20"
- board text added: "40/21 > 22/F"
- board text added: "40/9 > 28/19"
- board text added: "40/AB > 31/U"
- board text added: "40/R > 22/29"
- board text added: "40/W > 22/H"
- board text added: "40/X > 5/18"
- board text added: "41/18 > 29/13"
- board text added: "41/21 > 22/D"
- board text added: "41/29 > 8/26"
- board text added: "41/9 > 28/18"
- board text added: "41/AB > 31/T"
- board text added: "41/R > 22/28"
- board text added: "41/W > 22/E"
- board text added: "42/21 > 31/R"
- board text added: "42/9 > 28/17"
- board text added: "42/AB > 31/S"
- board text added: "42/AD > 7/6"
- board text added: "42/W > 30/18"
- board text added: "43/21 > 30/V"
- board text added: "43/9 > 28/16"
- board text added: "43/AB > 31/R"
- board text added: "43/AD > 7/13"
- board text added: "43/R > 25/27"
- board text added: "43/W > 30/T"
- board text added: "44/9 > 28/15"
- board text added: "44/AB > 31/P"
- board text added: "44/AD > 7/21"
- board text added: "44/R > 25/19"
- board text added: "44/W > 30/W"
- board text added: "45/29 > 5/23"
- board text added: "45/9 > 28/14"
- board text added: "45/AB > 31/N"
- board text added: "45/R > 25/8"
- board text added: "45/W > 30/X"
- board text added: "46/6 > 6/R"
- board text added: "46/8 > 7/AF"
- board text added: "46/9 > 57/M"
- board text added: "46/AA > 8/27"
- board text added: "46/AC > 8/24"
- board text added: "46/AD > 6/AD"
- board text added: "46/AE > 5/29"
- board text added: "46/AF > 6/AH"
- board text added: "46/AH > 2/Y"
- board text added: "46/E > 11/AC"
- board text added: "46/F > 19/V"
- board text added: "46/M > 5/11"
- board text added: "46/P > 8/28"
- board text added: "46/S > 9/23"
- board text added: "46/U > 8/21"
- board text added: "46/W > 8/23"
- board text added: "46/Y > 9/22"
- board text added: "46/Z > 5/7"
- board text added: "47/23 > 23/L"
- board text added: "47/4 > 57/4"
- board text added: "47/5 > 9/24"
- board text added: "47/6 > 57/6"
- board text added: "47/7 > 57/8"
- board text added: "47/AA > 9/7"
- board text added: "47/AB > 9/30"
- board text added: "47/AC > 9/21"
- board text added: "47/AD > 5/25"
- board text added: "47/AF > 5/20"
- board text added: "47/C > 8/6"
- board text added: "47/E > 9/14"
- board text added: "47/H > 9/25"
- board text added: "47/K > 9/6"
- board text added: "47/M > 9/12"
- board text added: "47/P > 8/7"
- board text added: "47/R > 32/R"
- board text added: "47/U > 8/30"
- board text added: "47/W > 9/13"
- board text added: "48/9 > 28/11"
- board text added: "48/AB > 31/M"
- board text added: "48/R > 25/3"
- board text added: "48/W > 30/Y"
- board text added: "49/12 > 29/9"
- board text added: "49/9 > 28/10"
- board text added: "49/AB > 31/L"
- board text added: "49/R > 24/27"
- board text added: "49/W > 30/22"
- board text added: "50/12 > 29/8"
- board text added: "50/9 > 28/9"
- board text added: "50/AB > 31/K"
- board text added: "50/R > 24/19"
- board text added: "50/W > 30/AA"
- board text added: "51/12 > 29/7"
- board text added: "51/9 > 28/8"
- board text added: "51/AB > 31/J"
- board text added: "51/R > 24/8"
- board text added: "51/W > 30/24"
- board text added: "52/12 > 29/10"
- board text added: "52/29 > 5/22"
- board text added: "52/9 > 28/7"
- board text added: "52/AB > 31/H"
- board text added: "52/N > 6/22"
- board text added: "52/R > 24/3"
- board text added: "52/W > 30/AC"
- board text added: "53/12 > 29/6"
- board text added: "53/18 > 29/17"
- board text added: "53/9 > 28/6"
- board text added: "53/AB > 31/F"
- board text added: "53/R > 23/27"
- board text added: "53/W > 32/F"
- board text added: "54/12 > 29/5"
- board text added: "54/18 > 29/16"
- board text added: "54/9 > 28/5"
- board text added: "54/AB > 31/E"
- board text added: "54/N > 6/28"
- board text added: "54/T > 20/H"
- board text added: "54/W > 32/E"
- board text added: "55/12 > 29/4"
- board text added: "55/18 > 29/15"
- board text added: "55/9 > 28/4"
- board text added: "55/AB > 31/D"
- board text added: "55/N > 6/27"
- board text added: "55/T > 20/E"
- board text added: "55/W > 32/D"
- board text added: "56/12 > 29/3"
- board text added: "56/9 > 28/3"
- board text added: "56/AB > 31/C"
- board text added: "56/AH > 7/15"
- board text added: "56/C > 8/12"
- board text added: "56/D > 57/5"
- board text added: "56/E > 57/7"
- board text added: "56/N > 6/21"
- board text added: "56/T > 20/C"
- board text added: "56/W > 32/C"
- board text added: "SKT11B NG1k"
- board text added: "SKT11F NG5k"
- board text added: "SKT11G NG6k"
- board text added: "SKT11H NG7k"
- board text added: "SKT11J NG8k"
- board text added: "SKT11K NG9k"
- board text added: "SKT11L NG10k"
- board text added: "SKT1AA {Q11}"
- board text added: "SKT1B {G1}"
- board text added: "SKT1BB {Q12}"
- board text added: "SKT1C {G2}"
- board text added: "SKT1CC {Q13}"
- board text added: "SKT1D {G3}"
- board text added: "SKT1DD {Q14}"
- board text added: "SKT1E {G4}"
- board text added: "SKT1EE {Q15}"
- board text added: "SKT1F {G5}"
- board text added: "SKT1FF {Q16}"
- board text added: "SKT1G {G6}"
- board text added: "SKT1GG {Q17}"
- board text added: "SKT1H {G7}"
- board text added: "SKT1HH {Q18}"
- board text added: "SKT1J {G8}"
- board text added: "SKT1K {G9}"
- board text added: "SKT1L {G10}"
- board text added: "SKT1M {G11}"
- board text added: "SKT1N {G12}"
- board text added: "SKT1P {G13}"
- board text added: "SKT1R {G14}"
- board text added: "SKT1S {G15}"
- board text added: "SKT1T {G16}"
- board text added: "SKT1U {G17}"
- board text added: "SKT1V {G18}"
- board text added: "SKT1W {A1}"
- board text added: "SKT1X {A2}"
- board text added: "SKT1Y {A3}"
- board text added: "SKT1Z {A4}"
- board text added: "SKT1a {A5}"
- board text added: "SKT1b {A6}"
- board text added: "SKT1c {A7}"
- board text added: "SKT1d {A8}"
- board text added: "SKT1e {A9}"
- board text added: "SKT1f {A10}"
- board text added: "SKT1g {A11}"
- board text added: "SKT1h {A12}"
- board text added: "SKT1i {A13}"
- board text added: "SKT1j {A14}"
- board text added: "SKT1k {A15}"
- board text added: "SKT1m {A16}"
- board text added: "SKT1n {A17}"
- board text added: "SKT1p {A18}"
- board text added: "SKT1q {Q1}"
- board text added: "SKT1r {Q2}"
- board text added: "SKT1s {Q3}"
- board text added: "SKT1t {Q4}"
- board text added: "SKT1u {Q5}"
- board text added: "SKT1v {Q6}"
- board text added: "SKT1w {Q7}"
- board text added: "SKT1x {Q8}"
- board text added: "SKT1y {Q9}"
- board text added: "SKT1z {Q10}"
- board text added: "SKT2B {M1}"
- board text added: "SKT2C {M2}"
- board text added: "SKT2D {M3}"
- board text added: "SKT2E {M4}"
- board text added: "SKT2F {M5}"
- board text added: "SKT2G {M6}"
- board text added: "SKT2H {M7}"
- board text added: "SKT2J {M8}"
- board text added: "SKT2K {M9}"
- board text added: "SKT2L {M10}"
- board text added: "SKT2M {M11}"
- board text added: "SKT2N {M12}"
- board text added: "SKT2P {M13}"
- board text added: "SKT2R {M14}"
- board text added: "SKT2S {M15}"
- board text added: "SKT2T {M16}"
- board text added: "SKT2U {M17}"
- board text added: "SKT2V {M18}"
- board text added: "SKT2W {J1}"
- board text added: "SKT2X {J2}"
- board text added: "SKT2Y {J3}"
- board text added: "SKT2Z {J4}"
- board text added: "SKT2a {J5}"
- board text added: "SKT2b {J6}"
- board text added: "SKT2c {J7}"
- board text added: "SKT2d {J8}"
- board text added: "SKT2e {J9}"
- board text added: "SKT2f {J10}"
- board text added: "SKT2g {J11}"
- board text added: "SKT2h {J12}"
- board text added: "SKT2i {J13}"
- board text added: "SKT2j {J14}"
- board text added: "SKT2k {J15}"
- board text added: "SKT2m {J16}"
- board text added: "SKT2n {P1}"
- board text added: "SKT2p {P2}"
- board text added: "SKT2q {P3}"
- board text added: "SKT2r {P4}"
- board text added: "SKT2s {P5}"
- board text added: "SKT2t {P6}"
- board text added: "SKT2u {P7}"
- board text added: "SKT2v {P8}"
- board text added: "SKT2w {P9}"
- board text added: "SKT2x {P10}"
- board text added: "SKT2y {P11}"
- board text added: "xxx"
- board text added: "~IIG"
- board text added: "~J1"
- board text added: "~J13"
- board text added: "~J2"
- board text added: "~J3"
- board text added: "~M1"
- board text added: "~M10"
- board text added: "~M11"
- board text added: "~M12"
- board text added: "~M13"
- board text added: "~M14"
- board text added: "~M15"
- board text added: "~M16"
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
Commit message: 23 oct
Other:
- board text added: "46/5 > 7/AF"
- board text added: "47/S > 9/24"
- board text removed: "46/8 > 7/AF"
- board text removed: "47/5 > 9/24"
Changed lines of the file:
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@@
     (effects (font (size 1 1) (thickness 0.25)) (justify left))
   )
-  (gr_text "46/8 >\n7/AF" (at 205.74 175.26) (layer F.SilkS)
+  (gr_text "46/5 >\n7/AF" (at 205.74 175.26) (layer F.SilkS)
     (effects (font (size 1 1) (thickness 0.25)) (justify left))
   )
@@
     (effects (font (size 1 1) (thickness 0.25)) (justify left))
   )
-  (gr_text "47/5 >\n9/24" (at 236.22 205.74) (layer F.SilkS)
+  (gr_text "47/S >\n9/24" (at 236.22 205.74) (layer F.SilkS)
     (effects (font (size 1 1) (thickness 0.25)) (justify left))
   )

Commit message: July backplane update
Parts:
- added J5: ~, Connector_IDC:IDC-Header_2x10_P2.54mm_Vertical_Lock, F.Cu at (113.8, 275.7)
- renumbered J~1 to J1, J~2 to J2, J~3 to J3
Connections:
- J337 pad 5: A18- -> (no net)
- J338 pad 5: A17- -> (no net)
- J339 pad 5: A16- -> (no net)
- J340 pad 5: A15- -> (no net)
- J341 pad 5: A14- -> (no net)
- J342 pad 5: A13- -> (no net)
- J343 pad 5: A12- -> (no net)
- J344 pad 5: A11- -> (no net)
- J345 pad 5: A10- -> (no net)
- J348 pad 5: ~A9 -> (no net)
- J349 pad 5: ~A8 -> (no net)
- J350 pad 5: ~A7 -> (no net)
- J351 pad 5: ~A6 -> (no net)
- J352 pad 5: ~A5 -> (no net)
- J353 pad 5: ~A4 -> (no net)
- J354 pad 5: ~A3 -> (no net)
- J355 pad 5: ~A2 -> (no net)
- J356 pad 5: ~A1 -> (no net)
- J37 pad AB: A18- -> /Connections/~A~18
- J38 pad AB: A17- -> /Connections/~A~17
- J39 pad AB: A16- -> /Connections/~A~16
- J40 pad AB: A15- -> /Connections/~A~15
- J41 pad AB: A14- -> /Connections/~A~14
- J42 pad AB: A13- -> /Connections/~A~13
- J43 pad AB: A12- -> /Connections/~A~12
- J44 pad AB: A11- -> /Connections/~A~11
- J45 pad AB: A10- -> /Connections/~A~10
- J48 pad AB: ~A9 -> /Connections/~A~9
- J49 pad AB: ~A8 -> /Connections/~A~8
- J50 pad AB: ~A7 -> /Connections/~A~7
- J51 pad AB: ~A6 -> /Connections/~A~6
- J52 pad AB: ~A5 -> /Connections/~A~5
- J53 pad AB: ~A4 -> /Connections/~A~4
- J54 pad AB: ~A3 -> /Connections/~A~3
- J55 pad AB: ~A2 -> /Connections/~A~2
- J56 pad AB: ~A1 -> /Connections/~A~1
Routing:
- net A11-: track 182.8 -> 0.00 mm
- net /Connections/~A~11: track 0.00 -> 182.8 mm
- net ~A9: track 182.6 -> 0.00 mm
- net /Connections/~A~9: track 0.00 -> 182.6 mm
- net A10-: track 182.6 -> 0.00 mm
- net /Connections/~A~10: track 0.00 -> 182.6 mm
- net A16-: track 181.5 -> 0.00 mm
- net /Connections/~A~16: track 0.00 -> 181.5 mm
- net ~A8: track 181.2 -> 0.00 mm
- net /Connections/~A~8: track 0.00 -> 181.2 mm
- net ~A4: track 180.8 -> 0.00 mm
- net /Connections/~A~4: track 0.00 -> 180.8 mm
- net A14-: track 180.7 -> 0.00 mm
- net /Connections/~A~14: track 0.00 -> 180.7 mm
- net A12-: track 180.5 -> 0.00 mm
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
Commit message: July 20th
Parts:
- removed J135, J136: ~, ELLIOTT:TerminalBlock_5.08_1x06
- removed J137, J138, J139, J140, J141, J142, J143, J144, J145, J148, J149, J150, J151, J152, J153, J154, J155, J156: ~, ELLIOTT:TerminalBlock_5.08_1x07
- removed J146, J147: ~, ELLIOTT:TerminalBlock-5.08_1x18
- removed J237, J238, J239, J240, J241, J242, J243, J244, J245, J248, J249, J250, J251, J252, J253: ~, ELLIOTT:TerminalBlock_5.08_1x03
- removed J254, J255, J256: ~, ELLIOTT:TerminalBlock_5.08_1x03+1
- removed J337, J338, J339, J340, J341, J342, J343, J344, J345, J348, J349, J350, J351, J352, J353, J354, J355, J356: ~, ELLIOTT:TerminalBlock_5.08_1x08
- removed J5: ~, Connector_IDC:IDC-Header_2x10_P2.54mm_Vertical_Lock
- removed TP1: Q1-, TestPoint:TestPoint_Plated_Hole_D2.0mm
- added JBP1-BP2-1: ~, Connector_IDC:IDC-Header_2x10_P2.54mm_Horizontal_Lock, F.Cu at (110.0, 180.0)
- added JBP1-BP2-2: ~, Connector_IDC:IDC-Header_2x10_P2.54mm_Horizontal_Lock, F.Cu at (110.0, 215.0)
- added JBP1-BP2-3: ~, Connector_IDC:IDC-Header_2x10_P2.54mm_Horizontal_Lock, F.Cu at (235.0, 180.0)
- added JBP1-BP2-4: ~, Connector_IDC:IDC-Header_2x10_P2.54mm_Horizontal_Lock, F.Cu at (165.0, 215.0)
- added JBP1-BP2-5: ~, Connector_IDC:IDC-Header_2x10_P2.54mm_Horizontal_Lock, F.Cu at (370.0, 250.0)
- added JBP1-BP3-1: ~, Connector_IDC:IDC-Header_2x10_P2.54mm_Horizontal_Lock, F.Cu at (310.0, 250.0)
- added JIP1: ~, Connector_IDC:IDC-Header_2x10_P2.54mm_Horizontal_Lock, F.Cu at (165.3, 180.0)
- added JJ1: ~, Connector_IDC:IDC-Header_2x10_P2.54mm_Horizontal_Lock, F.Cu at (56.0, 180.0)
- added JM1: ~, Connector_IDC:IDC-Header_2x10_P2.54mm_Horizontal_Lock, F.Cu at (56.0, 215.0)
- added JSKT1-1: ~, Connector_IDC:IDC-Header_2x10_P2.54mm_Horizontal_Lock, F.Cu at (370.0, 180.0)
- added JSKT1-2: ~, Connector_IDC:IDC-Header_2x10_P2.54mm_Horizontal_Lock, F.Cu at (235.0, 250.0)
- added JSKT1-3: ~, Connector_IDC:IDC-Header_2x10_P2.54mm_Horizontal_Lock, F.Cu at (110.0, 250.0)
- added JSKT2-1: ~, Connector_IDC:IDC-Header_2x10_P2.54mm_Horizontal_Lock, F.Cu at (165.0, 250.0)
- added JSKT2-2: ~, Connector_IDC:IDC-Header_2x10_P2.54mm_Horizontal_Lock, F.Cu at (370.0, 215.0)
- added JSKT2-3: ~, Connector_IDC:IDC-Header_2x10_P2.54mm_Horizontal_Lock, F.Cu at (310.0, 180.0)
- added JW1: ~, Connector_IDC:IDC-Header_2x10_P2.54mm_Horizontal_Lock, F.Cu at (235.0, 215.0)
- added J~A~1: ~, Connector_IDC:IDC-Header_2x10_P2.54mm_Horizontal_Lock, F.Cu at (310.0, 215.0)
- added J~STORE~1: ~, Connector_IDC:IDC-Header_2x10_P2.54mm_Horizontal_Lock, F.Cu at (56.0, 250.0)
- TH49, TH51, TH53, TH55, TH56: value MountingHole_2.7mm -> ~
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Connections:
- net A10 renamed /RegistersA/A10
- net A11 renamed /RegistersA/A11
- net A2 renamed /RegistersB/A2
- net A3 renamed /RegistersA/A3
- net A4 renamed /RegistersA/A4
- net A5 renamed /RegistersA/A5
- net A6 renamed /RegistersA/A6
- net A7 renamed /RegistersA/A7
- net A8 renamed /RegistersA/A8
- net A9 renamed /RegistersA/A9
- net ATF1 renamed /RegistersB/ATF1
- net ATF2 renamed /RegistersA/ATF2
- net C17 renamed C17-5-H
- net C9 renamed /RegistersA/C9
- net DT1-1 renamed DTF1-1-5-22
- net DT1-2 renamed DTF1-2-5-23
- net DTF2a renamed DTF2a-8-26
- net F1 renamed F1-57-7
- net F10 renamed /RegistersA/F10
- net F11 renamed /RegistersA/F11
- net F12 renamed /RegistersA/F12
- net F13 renamed /RegistersA/F13
- net F14 renamed /RegistersA/F14
- net F15 renamed /RegistersA/F15
- net F16 renamed /RegistersA/F16
- net F17 renamed /RegistersA/F17
- net F18 renamed F18-5-K
- net F2 renamed /RegistersB/F2
- net F3 renamed /RegistersB/F3
- net F4 renamed /RegistersB/F4
- net F5 renamed /RegistersB/F5
- net F6 renamed /RegistersB/F6
- net F7 renamed /RegistersB/F7
- net F8 renamed /RegistersB/F8
- net F9 renamed /RegistersA/F9
- net FTG1 renamed FTG1-57-4
- net FTG2 renamed /RegistersA/FTG2
- net GTA1 renamed /RegistersB/GTA1
- net GTA2 renamed /RegistersA/GTA2
- net GTJ1 renamed /RegistersB/GTJ1
- net GTJ2 renamed /RegistersA/GTJ2
- net GTM1 renamed /RegistersB/GTM1
- net GTM2 renamed /RegistersA/GTM2
- net GTQ1 renamed /RegistersB/GTQ1
- net GTQ2 renamed /RegistersA/GTQ2
- net II10m renamed /InitInstructions/II10m
- net II11m renamed /InitInstructions/II11m
- net II12m renamed /InitInstructions/II12m
- net II13m renamed /InitInstructions/II13m
- net II14m renamed /InitInstructions/II14m
- net II15m renamed /InitInstructions/II15m
- net II16m renamed /InitInstructions/II16m
- net II17m renamed /InitInstructions/II17m
- net II18m renamed /InitInstructions/II18m
- net II1m renamed /InitInstructions/II1m
- net II2m renamed /InitInstructions/II2m
- net II3m renamed /InitInstructions/II3m
- net II4m renamed /InitInstructions/II4m
- net II5m renamed /InitInstructions/II5m
- net II6m renamed /InitInstructions/II6m
- net II7m renamed /InitInstructions/II7m
- net II8m renamed /InitInstructions/II8m
- net II9m renamed /InitInstructions/II9m
- net IIG renamed /InitInstructions/IIG
- net IIS renamed IIS-57-15
- net J1' renamed J1'-20-4
- net J15- renamed ~J~15-22-29
- net J3' renamed J3'-20-8
- net J3-' renamed ~J~3'-20-7
- net JTF1 renamed /RegistersB/JTF1
- net JTF2 renamed /RegistersA/JTF2
- net JTG14- renamed /RegistersA/~JTG14~
- net JTG15- renamed /RegistersA/~JTG15~
- net JTG16- renamed /RegistersA/~JTG16~
- net LTG1 renamed LTG1-57-8
- net LTG2 renamed /RegistersA/LTG2
- net MTF1 renamed /RegistersB/MTF1
- net MTF2 renamed /RegistersA/MTF2
- net MTI renamed MTI-5-17
- net MTP1 renamed /RegistersB/MTP1
- net MTP2 renamed /RegistersA/MTP2
- net MTPa renamed MTPa-9-22
- net OTI- renamed ~OTI~-5-18
- net PTG1-2 renamed /RegistersA/PTG1-2
- net PTG2-2 renamed /RegistersA/PTG2-2
- net QTF1 renamed /RegistersB/QTF1
- net QTF2 renamed /RegistersA/QTF2
- net RTG1 renamed RTG1-57-6
- net RTG2 renamed /RegistersA/RTG2
- net VTG1 renamed /RegistersB/VTG1
- net VTG2 renamed /RegistersA/VTG2
- net WTM1 renamed /RegistersB/WTM1
- net WTM2 renamed /RegistersA/WTM2
- net ~J14 renamed ~J~14-22-28
- net ~J16 renamed ~J~16-22-26
- net ~J2~' renamed ~J~2'-20-5
- net ~OTA~1 renamed /RegistersB/~OTA~1
- net ~OTA~2 renamed /RegistersA/~OTA~2
- net ~OTJ~1 renamed /RegistersB/~OTJ~1
- net ~OTJ~2 renamed /RegistersA/~OTJ~2
- net ~OTM~1 renamed /RegistersB/~OTM~1
- net ~OTM~2 renamed /RegistersA/~OTM~2
- net ~OTP~1 renamed /RegistersB/~OTP~1
- net ~PTG1~1 renamed /RegistersB/PTG1-1
- net ~PTG2~1 renamed /RegistersB/PTG2-1
- J34 pad 1: GND -> /InitInstructions/GND
- J34 pad 2: 6v -> /InitInstructions/6v
- J34 pad 31: Neg6v -> /InitInstructions/-6v
- J34 pad 32: GND -> /InitInstructions/GND
- J34 pad A: GND -> /InitInstructions/GND
- J34 pad AK: Neg6v -> /InitInstructions/-6v
- J34 pad AL: GND -> /InitInstructions/GND
- J34 pad B: 6v -> /InitInstructions/6v
- J35 pad 1: GND -> /InitInstructions/GND
- J35 pad 13: J4- -> /InitInstructions/~J~4
- J35 pad 2: 6v -> /InitInstructions/6v
- J35 pad 31: Neg6v -> /InitInstructions/-6v
- J35 pad 32: GND -> /InitInstructions/GND
- J35 pad 8: ~J1~' -> ~J~1'-20-3
- J35 pad 9: J2' -> J2'-20-6
- J35 pad A: GND -> /InitInstructions/GND
- J35 pad AK: Neg6v -> /InitInstructions/-6v
- J35 pad AL: GND -> /InitInstructions/GND
- J35 pad B: 6v -> /InitInstructions/6v
- J36 pad 1: GND -> /InitInstructions/GND
- J36 pad 12: J4- -> /InitInstructions/~J~4
- J36 pad 2: 6v -> /InitInstructions/6v
- J36 pad 31: Neg6v -> /InitInstructions/-6v
- J36 pad 32: GND -> /InitInstructions/GND
- J36 pad 9: ~IIG -> ~IIG~
- J36 pad A: GND -> /InitInstructions/GND
- J36 pad AK: Neg6v -> /InitInstructions/-6v
- J36 pad AL: GND -> /InitInstructions/GND
- J36 pad B: 6v -> /InitInstructions/6v
- J37 pad 10: ~OTG~2 -> /RegistersA/~OTG~2
- J37 pad 16: ~M~TF2 -> /WaveformDrivers/~M~TF1
- J37 pad 26: OTQ2- -> /RegistersA/~OTQ2~
- J37 pad 3: C18 -> C18-5-8
- J37 pad 5: X1 -> X1-57-11
- J37 pad AB: /Connections/~A~18 -> ~A~18
- J37 pad AC: SKT1HH -> #Q18
- J37 pad AD: M18 -> M18-7-9
- J37 pad AJ: STORE18- -> ~STORE~18
- J37 pad M: SKT1V -> #G18
- J37 pad U: SKT2V -> #M18
- J37 pad V: M18- -> ~M~18-7-11
- J37 pad Z: SKT1~p -> #A18
- J38 pad 10: ~OTG~2 -> /RegistersA/~OTG~2
- J38 pad 16: ~M~TF2 -> /WaveformDrivers/~M~TF1
- J38 pad 21: I4 -> I4-22-L
- J38 pad 26: OTQ2- -> /RegistersA/~OTQ2~
- J38 pad AB: /Connections/~A~17 -> ~A~17
- J38 pad AC: SKT1GG -> #Q17
- J38 pad AD: (no net) -> M17
- J38 pad AJ: STORE17- -> ~STORE~17
- J38 pad M: SKT1U -> #G17
- J38 pad U: SKT2U -> #M17
- J38 pad V: M17- -> (no net)
- J38 pad W: I4- -> ~I~4-22-M
- J38 pad Y: SKT3u -> #I4
- J38 pad Z: SKT1~n -> #A17
- J39 pad 10: ~OTG~2 -> /RegistersA/~OTG~2
- J39 pad 16: ~M~TF2 -> /WaveformDrivers/~M~TF1
- J39 pad 21: I3 -> I3-22-J
- J39 pad 26: OTQ2- -> /RegistersA/~OTQ2~
- J39 pad AB: /Connections/~A~16 -> ~A~16
- J39 pad AC: SKT1FF -> #Q16
- J39 pad AD: (no net) -> M16
- J39 pad AJ: STORE16- -> ~STORE~16
- J39 pad M: SKT1T -> #G16
- J39 pad S: SKT2~m -> #J16
- J39 pad U: SKT2T -> #M16
- J39 pad V: M16- -> (no net)
- J39 pad W: I3- -> ~I~3-22-K
- J39 pad Y: SKT3t -> #I3
- J39 pad Z: SKT1~m -> #A16
- J40 pad 10: ~OTG~2 -> /RegistersA/~OTG~2
- J40 pad 16: ~M~TF2 -> /WaveformDrivers/~M~TF1
- J40 pad 21: I2 -> I2-22-F
- J40 pad 26: OTQ2- -> /RegistersA/~OTQ2~
- J40 pad AB: /Connections/~A~15 -> ~A~15
- J40 pad AC: SKT1EE -> #Q15
- J40 pad AD: (no net) -> M15
- J40 pad AJ: STORE15- -> ~STORE~15
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Routing:
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- removed copper zone on B.Cu, net (none)
- removed copper zone on F.Cu, net (none)
Other:
- copper layers 2 -> 4
- board text removed: "35/10 > 20/5"
- board text removed: "35/11 > 20/8"
- board text removed: "35/12 > 20/7"
- board text removed: "35/7 > 20/4"
- board text removed: "35/8 > 20/3"
- board text removed: "35/9 > 20/6"
- board text removed: "36/8 > 57/15"
- board text removed: "37/18 > 29/14"
- board text removed: "37/3 > 5/8"
- board text removed: "37/5 > 57/11"
- board text removed: "37/9 > 28/26"
- board text removed: "37/AB > 31/X"
- board text removed: "37/AD > 7/9"
- board text removed: "37/E > 5/K"
- board text removed: "37/V > 7/11"
- board text removed: "38/18 > 1/W"
- board text removed: "38/21 > 22/L"
- board text removed: "38/22 > 5/17"
- board text removed: "38/3 > 5/H"
- board text removed: "38/9 > 28/25"
- board text removed: "38/AB > 31/W"
- board text removed: "38/W > 22/M"
- board text removed: "39/18 > 29/12"
- board text removed: "39/21 > 22/J"
- board text removed: "39/9 > 28/24"
- board text removed: "39/AB > 31/V"
- board text removed: "39/R > 22/26"
- board text removed: "39/W > 22/K"
- board text removed: "40/18 > 29/20"
- board text removed: "40/21 > 22/F"
- board text removed: "40/9 > 28/19"
- board text removed: "40/AB > 31/U"
- board text removed: "40/R > 22/29"
- board text removed: "40/W > 22/H"
- board text removed: "40/X > 5/18"
- board text removed: "41/18 > 29/13"
- board text removed: "41/21 > 22/D"
- board text removed: "41/29 > 8/26"
- board text removed: "41/9 > 28/18"
- board text removed: "41/AB > 31/T"
- board text removed: "41/R > 22/28"
- board text removed: "41/W > 22/E"
- board text removed: "42/21 > 31/R"
- board text removed: "42/9 > 28/17"
- board text removed: "42/AB > 31/S"
- board text removed: "42/AD > 7/6"
- board text removed: "42/W > 30/18"
- board text removed: "43/21 > 30/V"
- board text removed: "43/9 > 28/16"
- board text removed: "43/AB > 31/R"
- board text removed: "43/AD > 7/13"
- board text removed: "43/R > 25/27"
- board text removed: "43/W > 30/T"
- board text removed: "44/9 > 28/15"
- board text removed: "44/AB > 31/P"
- board text removed: "44/AD > 7/21"
- board text removed: "44/R > 25/19"
- board text removed: "44/W > 30/W"
- board text removed: "45/29 > 5/23"
- board text removed: "45/9 > 28/14"
- board text removed: "45/AB > 31/N"
- board text removed: "45/R > 25/8"
- board text removed: "45/W > 30/X"
- board text removed: "46/5 > 7/AF"
- board text removed: "46/6 > 6/R"
- board text removed: "46/9 > 57/M"
- board text removed: "46/AA > 8/27"
- board text removed: "46/AC > 8/24"
- board text removed: "46/AD > 6/AD"
- board text removed: "46/AE > 5/29"
- board text removed: "46/AF > 6/AH"
- board text removed: "46/AH > 2/Y"
- board text removed: "46/E > 11/AC"
- board text removed: "46/F > 19/V"
- board text removed: "46/M > 5/11"
- board text removed: "46/P > 8/28"
- board text removed: "46/S > 9/23"
- board text removed: "46/U > 8/21"
- board text removed: "46/W > 8/23"
- board text removed: "46/Y > 9/22"
- board text removed: "46/Z > 5/7"
- board text removed: "47/23 > 23/L"
- board text removed: "47/4 > 57/4"
- board text removed: "47/6 > 57/6"
- board text removed: "47/7 > 57/8"
- board text removed: "47/AA > 9/7"
- board text removed: "47/AB > 9/30"
- board text removed: "47/AC > 9/21"
- board text removed: "47/AD > 5/25"
- board text removed: "47/AF > 5/20"
- board text removed: "47/C > 8/6"
- board text removed: "47/E > 9/14"
- board text removed: "47/H > 9/25"
- board text removed: "47/K > 9/6"
- board text removed: "47/M > 9/12"
- board text removed: "47/P > 8/7"
- board text removed: "47/R > 32/R"
- board text removed: "47/S > 9/24"
- board text removed: "47/U > 8/30"
- board text removed: "47/W > 9/13"
- board text removed: "48/9 > 28/11"
- board text removed: "48/AB > 31/M"
- board text removed: "48/R > 25/3"
- board text removed: "48/W > 30/Y"
- board text removed: "49/12 > 29/9"
- board text removed: "49/9 > 28/10"
- board text removed: "49/AB > 31/L"
- board text removed: "49/R > 24/27"
- board text removed: "49/W > 30/22"
- board text removed: "50/12 > 29/8"
- board text removed: "50/9 > 28/9"
- board text removed: "50/AB > 31/K"
- board text removed: "50/R > 24/19"
- board text removed: "50/W > 30/AA"
- board text removed: "51/12 > 29/7"
- board text removed: "51/9 > 28/8"
- board text removed: "51/AB > 31/J"
- board text removed: "51/R > 24/8"
- board text removed: "51/W > 30/24"
- board text removed: "52/12 > 29/10"
- board text removed: "52/29 > 5/22"
- board text removed: "52/9 > 28/7"
- board text removed: "52/AB > 31/H"
- board text removed: "52/N > 6/22"
- board text removed: "52/R > 24/3"
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
Commit message: August 2
Parts:
- moved JSKT1-1 322.5 mm to (55.4, 250.8)
- moved J~STORE~1 319.6 mm to (368.3, 182.0)
- moved JM1 183.3 mm to (236.1, 249.5)
- moved JSKT1-2 182.8 mm to (55.4, 215.7)
- moved JJ1 89.0 mm to (110.3, 250.5)
- moved JSKT1-3 87.9 mm to (56.1, 180.6)
Routing:
- net GND: track 768.1 -> 0.00 mm
- net ~STORE~2: track 506.1 -> 0.00 mm, vias 1 -> 0
- net ~STORE~1: track 487.6 -> 0.00 mm, vias 1 -> 0
- net M2: track 477.6 -> 0.00 mm, vias 1 -> 0
- net 6v: track 475.5 -> 0.00 mm, vias 1 -> 0
- net ~STORE~3: track 454.6 -> 0.00 mm, vias 1 -> 0
- net II1: track 450.3 -> 0.00 mm
- net ~STORE~4: track 450.3 -> 0.00 mm, vias 1 -> 0
- net M1: track 449.1 -> 0.00 mm, vias 1 -> 0
- net IIS-57-15: track 448.1 -> 0.00 mm, vias 1 -> 0
- net J4: track 447.4 -> 0.00 mm, vias 2 -> 0
- net X1-57-11: track 425.6 -> 0.00 mm, vias 1 -> 0
- net #Q1: track 424.0 -> 0.00 mm, vias 1 -> 0
- net M3: track 422.7 -> 0.00 mm, vias 2 -> 0
- net ~STORE~5: track 422.3 -> 0.00 mm, vias 2 -> 0
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