File: KiCad/Real903/Backplane1/Backplane1.kicad_pcb (KiCad board)
At the start: 4 copper layers, 386.1 x 266.7 mm, 80 parts

Commit message: September 4
Parts:
- removed JBP1-BP2-1, JBP1-BP2-2, JBP1-BP2-3, JBP1-BP2-4, JBP1-BP2-5, JBP1-BP3-1, JIP1, JJ1, JM1, JSKT1-1, JSKT1-2, JSKT1-3, JSKT2-1, JSKT2-2, JSKT2-3, JW1, J~A~1, J~STORE~1: ~, Connector_IDC:IDC-Header_2x10_P2.54mm_Horizontal_Lock
- added BP1-DSP-1: ~, Connector_IDC:IDC-Header_2x10_P2.54mm_Vertical, F.Cu at (341.6, 185.4)
- added BP1-DSP-2: ~, Connector_IDC:IDC-Header_2x10_P2.54mm_Vertical, F.Cu at (141.0, 185.4)
- added BP1-DSP-3: ~, Connector_IDC:IDC-Header_2x10_P2.54mm_Vertical, F.Cu at (304.8, 185.4)
- added BP1-DSP-4: ~, Connector_IDC:IDC-Header_2x10_P2.54mm_Vertical, F.Cu at (104.1, 185.4)
- added BP1-DSP-5: ~, Connector_IDC:IDC-Header_2x10_P2.54mm_Vertical, F.Cu at (377.2, 185.4)
- added BP1-DSP-6: ~, Connector_IDC:IDC-Header_2x10_P2.54mm_Vertical, F.Cu at (67.3, 185.4)
Connections:
- net JTPC renamed JTPC-23-L
- J34 pad 10: (no net) -> Net-(J34-Pad10)
- J34 pad 11: (no net) -> Net-(J34-Pad11)
- J34 pad 29: (no net) -> Net-(J34-Pad29)
- J34 pad 3: (no net) -> Net-(J34-Pad3)
- J34 pad 4: (no net) -> Net-(J34-Pad4)
- J34 pad 5: (no net) -> Net-(J34-Pad5)
- J34 pad 6: (no net) -> Net-(J34-Pad6)
- J34 pad 7: (no net) -> Net-(J34-Pad7)
- J34 pad 8: (no net) -> Net-(J34-Pad8)
- J34 pad 9: (no net) -> Net-(J34-Pad9)
- J34 pad AH: (no net) -> Net-(J34-PadAH)
- J34 pad C: (no net) -> Net-(J34-PadC)
- J34 pad D: (no net) -> Net-(J34-PadD)
- J34 pad E: (no net) -> Net-(J34-PadE)
- J34 pad F: (no net) -> Net-(J34-PadF)
- J34 pad H: (no net) -> Net-(J34-PadH)
- J34 pad J: (no net) -> Net-(J34-PadJ)
- J34 pad K: (no net) -> Net-(J34-PadK)
- J34 pad L: (no net) -> Net-(J34-PadL)
- J34 pad M: (no net) -> Net-(J34-PadM)
- J35 pad 16: (no net) -> Net-(J35-Pad16)
- J35 pad 17: (no net) -> Net-(J35-Pad17)
- J35 pad 18: (no net) -> Net-(J35-Pad18)
- J35 pad 19: (no net) -> Net-(J35-Pad19)
- J35 pad 20: (no net) -> Net-(J35-Pad20)
- J35 pad 21: (no net) -> Net-(J35-Pad21)
- J35 pad 22: (no net) -> Net-(J35-Pad22)
- J35 pad 23: (no net) -> Net-(J35-Pad23)
- J35 pad 24: (no net) -> Net-(J35-Pad24)
- J35 pad 25: (no net) -> Net-(J35-Pad25)
- J35 pad 27: (no net) -> Net-(J35-Pad27)
- J35 pad 28: (no net) -> Net-(J35-Pad28)
- J35 pad 29: (no net) -> Net-(J35-Pad29)
- J35 pad 3: (no net) -> Net-(J35-Pad3)
- J35 pad 30: (no net) -> Net-(J35-Pad30)
- J35 pad 4: (no net) -> Net-(J35-Pad4)
- J35 pad 5: (no net) -> Net-(J35-Pad5)
- J35 pad 6: (no net) -> Net-(J35-Pad6)
- J35 pad C: (no net) -> Net-(J35-PadC)
- J35 pad D: (no net) -> Net-(J35-PadD)
- J35 pad E: (no net) -> Net-(J35-PadE)
- J35 pad F: (no net) -> Net-(J35-PadF)
- J35 pad H: (no net) -> Net-(J35-PadH)
- J35 pad J: (no net) -> Net-(J35-PadJ)
- J35 pad K: (no net) -> Net-(J35-PadK)
- J35 pad L: (no net) -> Net-(J35-PadL)
- J35 pad M: (no net) -> Net-(J35-PadM)
- J35 pad N: (no net) -> Net-(J35-PadN)
- J36 pad 16: (no net) -> Net-(J36-Pad16)
- J36 pad 17: (no net) -> Net-(J36-Pad17)
- J36 pad 27: (no net) -> Net-(J36-Pad27)
- J36 pad 28: (no net) -> Net-(J36-Pad28)
- J36 pad 3: (no net) -> Net-(J36-Pad3)
- J36 pad 30: (no net) -> Net-(J36-Pad30)
- J36 pad 4: (no net) -> Net-(J36-Pad4)
- J36 pad 5: (no net) -> Net-(J36-Pad5)
- J36 pad 6: (no net) -> Net-(J36-Pad6)
- J36 pad D: (no net) -> Net-(J36-PadD)
- J36 pad E: (no net) -> Net-(J36-PadE)
- J36 pad F: (no net) -> Net-(J36-PadF)
- J36 pad H: (no net) -> Net-(J36-PadH)
- J36 pad J: (no net) -> Net-(J36-PadJ)
- J36 pad K: (no net) -> Net-(J36-PadK)
- J36 pad L: (no net) -> Net-(J36-PadL)
- J36 pad M: (no net) -> Net-(J36-PadM)
- J36 pad N: (no net) -> Net-(J36-PadN)
- J37 pad 21: (no net) -> Net-(J37-Pad21)
- J37 pad 22: (no net) -> Net-(J37-Pad22)
- J37 pad 24: (no net) -> Net-(J37-Pad24)
- J37 pad 27: (no net) -> Net-(J37-Pad27)
- J37 pad 4: (no net) -> Net-(J37-Pad4)
- J37 pad AF: (no net) -> Net-(J37-PadAF)
- J37 pad AH: (no net) -> Net-(J37-PadAH)
- J37 pad F: (no net) -> Net-(J37-PadF)
- J37 pad J: (no net) -> Net-(J37-PadJ)
- J37 pad K: (no net) -> Net-(J37-PadK)
- J37 pad N: (no net) -> Net-(J37-PadN)
- J37 pad R: (no net) -> Net-(J37-PadR)
- J37 pad S: (no net) -> Net-(J37-PadS)
- J37 pad T: (no net) -> Net-(J37-PadT)
- J37 pad W: (no net) -> Net-(J37-PadW)
- J37 pad X: (no net) -> Net-(J37-PadX)
- J37 pad Y: (no net) -> Net-(J37-PadY)
- J38 pad 24: (no net) -> Net-(J38-Pad24)
- J38 pad 27: (no net) -> Net-(J38-Pad27)
- J38 pad 4: (no net) -> Net-(J38-Pad4)
- J38 pad AF: (no net) -> Net-(J38-PadAF)
- J38 pad AH: (no net) -> Net-(J38-PadAH)
- J38 pad F: (no net) -> Net-(J38-PadF)
- J38 pad J: (no net) -> Net-(J38-PadJ)
- J38 pad K: (no net) -> Net-(J38-PadK)
- J38 pad N: (no net) -> Net-(J38-PadN)
- J38 pad R: (no net) -> Net-(J38-PadR)
- J38 pad S: (no net) -> Net-(J38-PadS)
- J38 pad T: (no net) -> Net-(J38-PadT)
- J38 pad V: (no net) -> Net-(J38-PadV)
- J39 pad 24: (no net) -> Net-(J39-Pad24)
- J39 pad 27: (no net) -> Net-(J39-Pad27)
- J39 pad AF: (no net) -> Net-(J39-PadAF)
- J39 pad AH: (no net) -> Net-(J39-PadAH)
- J39 pad F: (no net) -> Net-(J39-PadF)
- J39 pad J: (no net) -> Net-(J39-PadJ)
- J39 pad K: (no net) -> Net-(J39-PadK)
- J39 pad N: (no net) -> Net-(J39-PadN)
- J39 pad V: (no net) -> Net-(J39-PadV)
- J40 pad 24: (no net) -> Net-(J40-Pad24)
- J40 pad 27: (no net) -> Net-(J40-Pad27)
- J40 pad AF: (no net) -> Net-(J40-PadAF)
- J40 pad AH: (no net) -> Net-(J40-PadAH)
- J40 pad F: (no net) -> Net-(J40-PadF)
- J40 pad J: (no net) -> Net-(J40-PadJ)
- J40 pad K: (no net) -> Net-(J40-PadK)
- J40 pad N: (no net) -> Net-(J40-PadN)
- J40 pad V: (no net) -> Net-(J40-PadV)
- J41 pad 24: (no net) -> Net-(J41-Pad24)
- J41 pad 27: (no net) -> Net-(J41-Pad27)
- J41 pad AF: (no net) -> Net-(J41-PadAF)
- J41 pad AH: (no net) -> Net-(J41-PadAH)
- J41 pad F: (no net) -> Net-(J41-PadF)
- J41 pad J: (no net) -> Net-(J41-PadJ)
- J41 pad K: (no net) -> Net-(J41-PadK)
- J41 pad N: (no net) -> Net-(J41-PadN)
- J41 pad V: (no net) -> Net-(J41-PadV)
- J42 pad 24: (no net) -> Net-(J42-Pad24)
- J42 pad 27: (no net) -> Net-(J42-Pad27)
- J42 pad 4: (no net) -> Net-(J42-Pad4)
- J42 pad AF: (no net) -> Net-(J42-PadAF)
- J42 pad AH: (no net) -> Net-(J42-PadAH)
- J42 pad F: (no net) -> Net-(J42-PadF)
- J42 pad J: (no net) -> Net-(J42-PadJ)
- J42 pad K: (no net) -> Net-(J42-PadK)
- J42 pad N: (no net) -> Net-(J42-PadN)
- J42 pad R: (no net) -> Net-(J42-PadR)
- J42 pad W: ~P~13-30-18 -> ~P~13
- J42 pad Y: (no net) -> Net-(J42-PadY)
- J43 pad 24: (no net) -> Net-(J43-Pad24)
- J43 pad 27: (no net) -> Net-(J43-Pad27)
- J43 pad 4: (no net) -> Net-(J43-Pad4)
- J43 pad AF: (no net) -> Net-(J43-PadAF)
- J43 pad AH: (no net) -> Net-(J43-PadAH)
- J43 pad F: (no net) -> Net-(J43-PadF)
- J43 pad J: (no net) -> Net-(J43-PadJ)
- J43 pad K: (no net) -> Net-(J43-PadK)
- J43 pad N: (no net) -> Net-(J43-PadN)
- J43 pad R: (no net) -> ~J~12-25-27
- J43 pad W: ~P~12-30-T -> ~P~12
- J43 pad Y: (no net) -> Net-(J43-PadY)
- J44 pad 21: (no net) -> Net-(J44-Pad21)
- J44 pad 24: (no net) -> Net-(J44-Pad24)
- J44 pad 4: (no net) -> Net-(J44-Pad4)
- J44 pad AF: (no net) -> Net-(J44-PadAF)
- J44 pad AH: (no net) -> Net-(J44-PadAH)
- J44 pad F: (no net) -> Net-(J44-PadF)
- J44 pad J: (no net) -> Net-(J44-PadJ)
- J44 pad K: (no net) -> Net-(J44-PadK)
- J44 pad N: (no net) -> Net-(J44-PadN)
- J44 pad R: (no net) -> ~J~11-25-19
- J44 pad V: (no net) -> Net-(J44-PadV)
- J44 pad W: ~P~11-30-W -> ~P~11
- J45 pad 21: (no net) -> Net-(J45-Pad21)
- J45 pad 24: (no net) -> Net-(J45-Pad24)
- J45 pad 4: (no net) -> Net-(J45-Pad4)
- J45 pad AF: (no net) -> Net-(J45-PadAF)
- J45 pad AH: (no net) -> Net-(J45-PadAH)
- J45 pad F: (no net) -> Net-(J45-PadF)
- J45 pad J: (no net) -> Net-(J45-PadJ)
- J45 pad K: (no net) -> Net-(J45-PadK)
- J45 pad N: (no net) -> Net-(J45-PadN)
- J45 pad R: (no net) -> ~J~10-25-8
- J45 pad V: (no net) -> Net-(J45-PadV)
- J45 pad W: ~P~10-30-X -> ~P~10
- J46 pad 3: (no net) -> Net-(J46-Pad3)
- J46 pad 30: (no net) -> Net-(J46-Pad30)
- J46 pad 4: (no net) -> Net-(J46-Pad4)
- J46 pad 7: (no net) -> Net-(J46-Pad7)
- J46 pad 8: (no net) -> Net-(J46-Pad8)
- J46 pad AJ: (no net) -> Net-(J46-PadAJ)
- J46 pad C: (no net) -> Net-(J46-PadC)
- J46 pad D: (no net) -> Net-(J46-PadD)
- J46 pad H: (no net) -> Net-(J46-PadH)
- J46 pad J: (no net) -> Net-(J46-PadJ)
- J46 pad K: (no net) -> Net-(J46-PadK)
- J46 pad L: (no net) -> Net-(J46-PadL)
- J46 pad N: (no net) -> Net-(J46-PadN)
- J46 pad R: (no net) -> Net-(J46-PadR)
- J46 pad T: (no net) -> Net-(J46-PadT)
- J46 pad V: (no net) -> Net-(J46-PadV)
- J46 pad X: (no net) -> Net-(J46-PadX)
- J47 pad 30: (no net) -> Net-(J47-Pad30)
- J47 pad AJ: (no net) -> Net-(J47-PadAJ)
- J47 pad D: (no net) -> Net-(J47-PadD)
- J47 pad F: (no net) -> Net-(J47-PadF)
- J47 pad J: (no net) -> Net-(J47-PadJ)
- J47 pad L: (no net) -> Net-(J47-PadL)
- J47 pad N: (no net) -> Net-(J47-PadN)
- J48 pad 21: (no net) -> Net-(J48-Pad21)
- J48 pad 24: (no net) -> Net-(J48-Pad24)
- J48 pad 4: (no net) -> Net-(J48-Pad4)
- J48 pad AF: (no net) -> Net-(J48-PadAF)
- J48 pad AH: (no net) -> Net-(J48-PadAH)
- J48 pad F: (no net) -> Net-(J48-PadF)
- J48 pad J: (no net) -> Net-(J48-PadJ)
- J48 pad K: (no net) -> Net-(J48-PadK)
- J48 pad N: (no net) -> Net-(J48-PadN)
- J48 pad V: (no net) -> Net-(J48-PadV)
- J48 pad W: ~P~9-30-Y -> ~P~9
- J49 pad 21: (no net) -> Net-(J49-Pad21)
- J49 pad 24: (no net) -> Net-(J49-Pad24)
- J49 pad 4: (no net) -> Net-(J49-Pad4)
- J49 pad AF: (no net) -> Net-(J49-PadAF)
- J49 pad AH: (no net) -> Net-(J49-PadAH)
- J49 pad F: (no net) -> Net-(J49-PadF)
- J49 pad J: (no net) -> Net-(J49-PadJ)
- J49 pad K: (no net) -> Net-(J49-PadK)
- J49 pad N: (no net) -> Net-(J49-PadN)
- J49 pad V: (no net) -> Net-(J49-PadV)
- J49 pad W: ~P~8-30-22 -> ~P~8
- J50 pad 21: (no net) -> Net-(J50-Pad21)
- J50 pad 24: (no net) -> Net-(J50-Pad24)
- J50 pad 4: (no net) -> Net-(J50-Pad4)
- J50 pad AF: (no net) -> Net-(J50-PadAF)
- J50 pad AH: (no net) -> Net-(J50-PadAH)
- J50 pad F: (no net) -> Net-(J50-PadF)
- J50 pad J: (no net) -> Net-(J50-PadJ)
- J50 pad K: (no net) -> Net-(J50-PadK)
- J50 pad N: (no net) -> Net-(J50-PadN)
- J50 pad V: (no net) -> Net-(J50-PadV)
- J50 pad W: ~P~7-30-AA -> ~P~7
- J51 pad 21: (no net) -> Net-(J51-Pad21)
- J51 pad 24: (no net) -> Net-(J51-Pad24)
- J51 pad 4: (no net) -> Net-(J51-Pad4)
- J51 pad AF: (no net) -> Net-(J51-PadAF)
- J51 pad AH: (no net) -> Net-(J51-PadAH)
- J51 pad F: (no net) -> Net-(J51-PadF)
- J51 pad J: (no net) -> Net-(J51-PadJ)
- J51 pad K: (no net) -> Net-(J51-PadK)
- J51 pad N: (no net) -> Net-(J51-PadN)
- J51 pad V: (no net) -> Net-(J51-PadV)
- J51 pad W: ~P~6-30-24 -> ~P~6
- J52 pad 21: (no net) -> Net-(J52-Pad21)
- J52 pad 24: (no net) -> Net-(J52-Pad24)
- J52 pad 4: (no net) -> Net-(J52-Pad4)
- J52 pad AF: (no net) -> Net-(J52-PadAF)
- J52 pad AH: (no net) -> Net-(J52-PadAH)
- J52 pad F: (no net) -> Net-(J52-PadF)
- J52 pad J: (no net) -> Net-(J52-PadJ)
- J52 pad K: (no net) -> Net-(J52-PadK)
- J52 pad V: (no net) -> Net-(J52-PadV)
- J52 pad W: ~P~5-30-AC -> ~P~5
- J53 pad 21: (no net) -> Net-(J53-Pad21)
- J53 pad 24: (no net) -> Net-(J53-Pad24)
- J53 pad 4: (no net) -> Net-(J53-Pad4)
- J53 pad AF: (no net) -> Net-(J53-PadAF)
- J53 pad AH: (no net) -> Net-(J53-PadAH)
- J53 pad F: (no net) -> Net-(J53-PadF)
- J53 pad J: (no net) -> Net-(J53-PadJ)
- J53 pad K: (no net) -> Net-(J53-PadK)
- J53 pad N: (no net) -> Net-(J53-PadN)
- J53 pad V: (no net) -> Net-(J53-PadV)
- J53 pad W: ~P~4-32-F -> ~P~4
- J54 pad 21: (no net) -> Net-(J54-Pad21)
- J54 pad 24: (no net) -> Net-(J54-Pad24)
- J54 pad 4: (no net) -> Net-(J54-Pad4)
- J54 pad AF: (no net) -> Net-(J54-PadAF)
- J54 pad AH: (no net) -> Net-(J54-PadAH)
- J54 pad F: (no net) -> Net-(J54-PadF)
- J54 pad J: (no net) -> Net-(J54-PadJ)
- J54 pad K: (no net) -> Net-(J54-PadK)
- J54 pad R: (no net) -> ~J~3'-20-7
- J54 pad V: (no net) -> Net-(J54-PadV)
- J54 pad W: ~P~3-32-E -> ~P~3
- J55 pad 21: (no net) -> Net-(J55-Pad21)
- J55 pad 24: (no net) -> Net-(J55-Pad24)
- J55 pad 4: (no net) -> Net-(J55-Pad4)
- J55 pad AF: (no net) -> Net-(J55-PadAF)
- J55 pad AH: (no net) -> Net-(J55-PadAH)
- J55 pad F: (no net) -> Net-(J55-PadF)
- J55 pad J: (no net) -> Net-(J55-PadJ)
- J55 pad K: (no net) -> Net-(J55-PadK)
- J55 pad R: (no net) -> ~J~2'-20-5
- J55 pad V: (no net) -> Net-(J55-PadV)
- J55 pad W: ~P~2-32-D -> ~P~2
- J56 pad 21: (no net) -> Net-(J56-Pad21)
- J56 pad 24: (no net) -> Net-(J56-Pad24)
- J56 pad 27: (no net) -> Net-(J56-Pad27)
- J56 pad 4: (no net) -> Net-(J56-Pad4)
- J56 pad AF: (no net) -> Net-(J56-PadAF)
- J56 pad F: (no net) -> Net-(J56-PadF)
- J56 pad J: (no net) -> Net-(J56-PadJ)
- J56 pad K: (no net) -> Net-(J56-PadK)
- J56 pad R: (no net) -> ~J~1'-20-3
- J56 pad V: (no net) -> Net-(J56-PadV)
- J56 pad W: ~P~1-32-C -> ~P~1
