File: KiCad/Real903/Backplane1/Connections.sch (KiCad schematic (older format))
At the start: 8 parts

Commit message: July 20th
Parts:
- removed BP2: ~, Connector_IDC:IDC-Header_2x10_P2.54mm_Vertical_Lock, symbol Connector_Generic:Conn_01x40
- removed JIP'1: ~, Connector_IDC:IDC-Header_2x10_P2.54mm_Vertical_Lock, symbol Connector_Generic:Conn_01x08
- removed SKT1, SKT2, SKT3: ~, symbol Connector_Generic:Conn_02x31_Counter_Clockwise
- added JBP1-BP2-1, JBP1-BP2-2, JBP1-BP2-3, JBP1-BP2-4, JBP1-BP2-5, JBP1-BP3-1, JSKT2-1, JSKT2-2, JSKT2-3, JW1: ~, Connector_IDC:IDC-Header_2x10_P2.54mm_Horizontal_Lock, symbol Connector_Generic:Conn_01x20
- added JJ1, JM1, JSKT1-1, JSKT1-2, JSKT1-3: ~, Connector_IDC:IDC-Header_2x10_P2.54mm_Horizontal_Lock, symbol Connector_Generic:Conn_01x18
- JIP1, J~A~1, J~STORE~1: footprint Connector_IDC:IDC-Header_2x10_P2.54mm_Vertical_Lock -> Connector_IDC:IDC-Header_2x10_P2.54mm_Horizontal_Lock
Connections:
- net labels added: #M1, #M2, #M3, #M4, #M5, #M6, #M7, #M8, #M9, #P1, #P2, #P3, #P4, #P5, #P6, #P7, #P8, #P9, ATFa-9-21, CRS-7-AF, CRSm-11-AC, FTGa-8-6, GTAa-8-27, GTJa-8-28, GTMa-8-23, GTQa-8-24, J1, J1-20-C, J10, J11, J12, J13, J14, J15, J16, J2, J2-20-E, J3, J3-20-H, J4, J5, J6, J7, J8, J9, JTFa-9-24, JTPCa-9-7, J[1..16], LTGa-9-25, M1, M10, M11, M11-7-21, M12, M12-6-W, M13, M13-7-6, M14, M15, M16, M17, M18, M2, M3, M4, M5, M6, M7, M8, M9, MTFa-8-30, MTPa-9-22, M[1..18], OTMa-9-23, PTG1-a-9-6, PTG2-a-9-12, QTFa-9-30, RTGa-9-14, SFD-6-R, SFDm-19-V, VTGa-8-7, W1, W10, W11, W12, W13, W14, W15, W16, W17, W18, W2, W3, W4, W5, W6, W7, W8, W9, WTMa-8-21, W[1..18], t1-5-27, t2-2-5-20, t3-2-5-29, t4-5-26, t5-5-25, ~IIG~, ~I~1-22-E, ~I~2-22-H, ~I~3-22-K, ~I~4-22-M, ~J~4-23-27, ~J~5-24-3, ~J~6-24-8, ~J~7-24-19, ~J~8-24-27, ~J~9-25-3, ~M~12-6-Y, ~M~13-6-18, ~M~18-7-11, ~M~TFa-9-13, ~OTA~'-5-7, ~OTJ~'-5-11, ~P~1-32-C, ~P~10-30-X, ~P~11-30-W, ~P~12-30-T, ~P~13-30-18, ~P~2-32-D, ~P~3-32-E, ~P~4-32-F, ~P~5-30-AC, ~P~6-30-24, ~P~7-30-AA, ~P~8-30-22, ~P~9-30-Y, ~Q~1-7-15, ~RESET~2-2-Y, ~VTG~-32-R
- no-connect marks 104 -> 24
Other:
- note added: "To Store"
- moved on the sheet: JIP1, J~{A}1, J~{STORE}1

Commit message: August 2
Parts:
- renumbered JW1 to JBP1-BP3-2
Connections:
- net W1: now also JSKT2-1.20 (Pin_20); no longer JSKT2-1.19 (Pin_19)
- net W17: now also JBP1-BP2-4.20 (Pin_20); no longer JBP1-BP3-2.7 (Pin_7)
- net ~J~10-25-8: now reaches JBP1-BP2-5.10 (Pin_10)
- net ~J~11-25-19: now reaches JBP1-BP2-5.11 (Pin_11)
- net ~J~12-25-27: now reaches JBP1-BP2-5.12 (Pin_12)
- net JTPC-23-L: now reaches JBP1-BP2-5.9 (Pin_9)
- net ~P~1-32-C renamed ~P~1
- net ~P~10-30-X renamed ~P~10
- net ~P~11-30-W renamed ~P~11
- net ~P~12-30-T renamed ~P~12
- net ~P~13-30-18 renamed ~P~13
- net ~P~2-32-D renamed ~P~2
- net ~P~3-32-E renamed ~P~3
- net ~P~4-32-F renamed ~P~4
- net ~P~5-30-AC renamed ~P~5
- net ~P~6-30-24 renamed ~P~6
- net ~P~7-30-AA renamed ~P~7
- net ~P~8-30-22 renamed ~P~8
- net ~P~9-30-Y renamed ~P~9
- no-connect marks 24 -> 20
Changed lines of the file:
@@
 Text GLabel 9100 2275 2    32   UnSpc ~ 0
 ~I~1-22-E
-Text GLabel 1950 3475 2    32   UnSpc ~ 0
-~P~13-30-18
-Text GLabel 1950 3575 2    32   UnSpc ~ 0
-~P~12-30-T
-Text GLabel 1950 3675 2    32   UnSpc ~ 0
-~P~11-30-W
-Text GLabel 1350 2875 2    32   UnSpc ~ 0
-~P~10-30-X
-Text GLabel 1350 2675 2    32   UnSpc ~ 0
-~P~9-30-Y
-Text GLabel 1350 2775 2    32   UnSpc ~ 0
-~P~8-30-22
-Text GLabel 1350 2475 2    32   UnSpc ~ 0
-~P~7-30-AA
-Text GLabel 1350 2575 2    32   UnSpc ~ 0
-~P~6-30-24
-Text GLabel 1350 2275 2    32   UnSpc ~ 0
-~P~5-30-AC
-Text GLabel 1350 1875 2    32   UnSpc ~ 0
-~P~4-32-F
-Text GLabel 1350 1975 2    32   UnSpc ~ 0
-~P~3-32-E
-Text GLabel 1350 2075 2    32   UnSpc ~ 0
-~P~2-32-D
-Text GLabel 1350 2175 2    32   UnSpc ~ 0
-~P~1-32-C
 Text Label 5575 2575 0    40   ~ 0
 #P9
@@
 ~Q~1-7-15
 $Comp
-L Connector_Generic:Conn_01x20 JW1
+L Connector_Generic:Conn_01x20 JBP1-BP3-2
 U 1 1 5F2E7A81
 P 1750 2675
-F 0 "JW1" H 1675 3700 50  0000 C CNN
+F 0 "JBP1-BP3-2" H 1675 3700 50  0000 C CNN
 F 1 "~" H 1670 3601 50  0000 C CNN
 F 2 "Connector_IDC:IDC-Header_2x10_P2.54mm_Horizontal_Lock" H 1750 2675 50  0001 C CNN
@@
 Text HLabel 1775 3725 3    30   UnSpc ~ 0
 W[1..18]
-Text Label 4425 3575 0    40   ~ 0
+Text Label 4425 3675 0    40   ~ 0
 W1
-Text Label 1950 1775 0    40   ~ 0
+Text Label 1950 1775 0    35   ~ 0
 W2
-Text Label 1950 1875 0    40   ~ 0
+Text Label 1950 1875 0    35   ~ 0
 W3
 Text Label 1950 1975 0    40   ~ 0
@@
 Text Label 5575 3675 0    40   ~ 0
 W13
-Text Label 1950 2075 0    40   ~ 0
+Text Label 1950 2075 0    35   ~ 0
 W14
-Text Label 1950 2175 0    40   ~ 0
+Text Label 1950 2175 0    35   ~ 0
 W15
-Text Label 1950 2275 0    40   ~ 0
+Text Label 1950 2275 0    35   ~ 0
 W16
-Text Label 1950 2375 0    40   ~ 0
-W17
-Text Label 1950 2475 0    40   ~ 0
+Text Label 1950 2475 0    35   ~ 0
 W18
 Text GLabel 6575 2775 2    32   UnSpc ~ 0
@@
 	-1   0    0    -1
 $EndComp
-NoConn ~ 9100 3675
 $Comp
 L Connector_Generic:Conn_01x20 JBP1-BP2-5
@@
 	-1   0    0    -1
 $EndComp
-NoConn ~ 9925 2575
-NoConn ~ 9925 2675
-NoConn ~ 9925 2775
-NoConn ~ 9925 2875
 NoConn ~ 9925 2975
 NoConn ~ 9925 3075
@@
 	-1   0    0    -1
 $EndComp
-NoConn ~ 4425 3675
 NoConn ~ 1350 3675
 NoConn ~ 1350 3575
@@
 NoConn ~ 1350 3075
 NoConn ~ 1350 2975
+NoConn ~ 4425 3575
+Text HLabel 1175 3725 3    30   Input ~ 0
+~P~[1..13]
+Text Label 1350 1875 0    35   ~ 0
+~P~4
+Text Label 1350 1975 0    35   ~ 0
+~P~3
+Text Label 1350 2075 0    35   ~ 0
+~P~2
+Text Label 1350 2175 0    35   ~ 0
+~P~1
+Text Label 1350 2275 0    35   ~ 0
+~P~5
+Text Label 1350 2575 0    35   ~ 0
+~P~6
+Text Label 1350 2475 0    35   ~ 0
+~P~7
+Text Label 1350 2775 0    35   ~ 0
+~P~8
+Text Label 1350 2675 0    35   ~ 0
+~P~9
+Text Label 1350 2875 0    35   ~ 0
+~P~10
+Text Label 1950 3675 0    35   ~ 0
+~P~11
+Text Label 1950 3575 0    35   ~ 0
+~P~12
+Text Label 1950 3475 0    35   ~ 0
+~P~13
+NoConn ~ 1950 2375
+Text Label 9100 3675 0    32   ~ 0
+W17
+Text GLabel 9925 2575 2    32   UnSpc ~ 0
+JTPC-23-L
+Text GLabel 9925 2675 2    32   UnSpc ~ 0
+~J~10-25-8
+Text GLabel 9925 2775 2    32   UnSpc ~ 0
+~J~11-25-19
+Text GLabel 9925 2875 2    32   UnSpc ~ 0
+~J~12-25-27
 $EndSCHEMATC

Commit message: August 15
Connections:
- net #A1: now also JSKT1-1.10 (Pin_10); no longer JSKT1-2.1 (Pin_1)
- net #A2: now also JSKT1-1.11 (Pin_11); no longer JSKT1-2.2 (Pin_2)
- net #A3: now also JSKT1-1.12 (Pin_12); no longer JSKT1-2.3 (Pin_3)
- net #A4: now also JSKT1-1.13 (Pin_13); no longer JSKT1-2.4 (Pin_4)
- net #A5: now also JSKT1-1.14 (Pin_14); no longer JSKT1-2.5 (Pin_5)
- net #A6: now also JSKT1-1.15 (Pin_15); no longer JSKT1-2.6 (Pin_6)
- net #A7: now also JSKT1-1.16 (Pin_16); no longer JSKT1-2.7 (Pin_7)
- net #A8: now also JSKT1-1.17 (Pin_17); no longer JSKT1-2.8 (Pin_8)
- net #A9: now also JSKT1-1.18 (Pin_18); no longer JSKT1-2.9 (Pin_9)
- net #G10: now also JSKT1-2.1 (Pin_1); no longer JSKT1-1.10 (Pin_10)
- net #G11: now also JSKT1-2.2 (Pin_2); no longer JSKT1-1.11 (Pin_11)
- net #G12: now also JSKT1-2.3 (Pin_3); no longer JSKT1-1.12 (Pin_12)
- net #G13: now also JSKT1-2.4 (Pin_4); no longer JSKT1-1.13 (Pin_13)
- net #G14: now also JSKT1-2.5 (Pin_5); no longer JSKT1-1.14 (Pin_14)
- net #G15: now also JSKT1-2.6 (Pin_6); no longer JSKT1-1.15 (Pin_15)
- net #G16: now also JSKT1-2.7 (Pin_7); no longer JSKT1-1.16 (Pin_16)
- net #G17: now also JSKT1-2.8 (Pin_8); no longer JSKT1-1.17 (Pin_17)
- net #G18: now also JSKT1-2.9 (Pin_9); no longer JSKT1-1.18 (Pin_18)
Changed lines of the file:
@@
 EESchema Schematic File Version 4
-LIBS:Backplane1-cache
-EELAYER 26 0
+EELAYER 30 0
 EELAYER END
 $Descr A4 11693 8268
@@
 Text Label 2600 2575 0    35   ~ 0
 #G9
-Text Label 2600 2675 0    35   ~ 0
+Text Label 3200 1775 0    35   ~ 0
 #G10
-Text Label 2600 2775 0    35   ~ 0
+Text Label 3200 1875 0    35   ~ 0
 #G11
-Text Label 2600 2875 0    35   ~ 0
+Text Label 3200 1975 0    35   ~ 0
 #G12
-Text Label 2600 2975 0    35   ~ 0
+Text Label 3200 2075 0    35   ~ 0
 #G13
-Text Label 2600 3075 0    35   ~ 0
+Text Label 3200 2175 0    35   ~ 0
 #G14
-Text Label 2600 3175 0    35   ~ 0
+Text Label 3200 2275 0    35   ~ 0
 #G15
-Text Label 2600 3275 0    35   ~ 0
+Text Label 3200 2375 0    35   ~ 0
 #G16
-Text Label 2600 3375 0    35   ~ 0
+Text Label 3200 2475 0    35   ~ 0
 #G17
-Text Label 2600 3475 0    35   ~ 0
+Text Label 3200 2575 0    35   ~ 0
 #G18
 Text HLabel 3025 3525 3    32   UnSpc ~ 0
 #A[1..18]
-Text Label 3200 1775 0    35   ~ 0
+Text Label 2600 2675 0    35   ~ 0
 #A1
-Text Label 3200 1875 0    35   ~ 0
+Text Label 2600 2775 0    35   ~ 0
 #A2
-Text Label 3200 1975 0    35   ~ 0
+Text Label 2600 2875 0    35   ~ 0
 #A3
-Text Label 3200 2075 0    35   ~ 0
+Text Label 2600 2975 0    35   ~ 0
 #A4
-Text Label 3200 2175 0    35   ~ 0
+Text Label 2600 3075 0    35   ~ 0
 #A5
-Text Label 3200 2275 0    35   ~ 0
+Text Label 2600 3175 0    35   ~ 0
 #A6
-Text Label 3200 2375 0    35   ~ 0
+Text Label 2600 3275 0    35   ~ 0
 #A7
-Text Label 3200 2475 0    35   ~ 0
+Text Label 2600 3375 0    35   ~ 0
 #A8
-Text Label 3200 2575 0    35   ~ 0
+Text Label 2600 3475 0    35   ~ 0
 #A9
 Text Label 3200 2675 0    35   ~ 0

Commit message: September 4
Parts:
- BP1-BP2-1: renamed from JBP1-BP2-1; footprint Connector_IDC:IDC-Header_2x10_P2.54mm_Horizontal_Lock -> (none)
- BP1-BP2-2: renamed from JBP1-BP2-2; footprint Connector_IDC:IDC-Header_2x10_P2.54mm_Horizontal_Lock -> (none)
- BP1-BP2-3: renamed from JBP1-BP2-3; footprint Connector_IDC:IDC-Header_2x10_P2.54mm_Horizontal_Lock -> (none)
- BP1-BP2-4: renamed from JBP1-BP2-4; footprint Connector_IDC:IDC-Header_2x10_P2.54mm_Horizontal_Lock -> (none)
- BP1-BP2-5: renamed from JBP1-BP2-5; footprint Connector_IDC:IDC-Header_2x10_P2.54mm_Horizontal_Lock -> (none)
- BP1-BP3-1: renamed from JBP1-BP3-1; footprint Connector_IDC:IDC-Header_2x10_P2.54mm_Horizontal_Lock -> (none)
- BP1-BP3-2: renamed from JBP1-BP3-2; footprint Connector_IDC:IDC-Header_2x10_P2.54mm_Horizontal_Lock -> (none)
- BP1-BP3-3: renamed from J~STORE~1; footprint Connector_IDC:IDC-Header_2x10_P2.54mm_Horizontal_Lock -> (none)
- BP1-BP3-4: renamed from JM1; footprint Connector_IDC:IDC-Header_2x10_P2.54mm_Horizontal_Lock -> (none)
- BP1-BP3-5: renamed from JJ1; footprint Connector_IDC:IDC-Header_2x10_P2.54mm_Horizontal_Lock -> (none)
- BP1-BP3-6: renamed from J~A~1; footprint Connector_IDC:IDC-Header_2x10_P2.54mm_Horizontal_Lock -> (none)
- BP1-BP3-7: renamed from JIP1; footprint Connector_IDC:IDC-Header_2x10_P2.54mm_Horizontal_Lock -> (none)
- BP1-DSP-1: renamed from JSKT1-1; footprint Connector_IDC:IDC-Header_2x10_P2.54mm_Horizontal_Lock -> Connector_IDC:IDC-Header_2x10_P2.54mm_Vertical; symbol Connector_Generic:Conn_01x18 -> Connector_Generic:Conn_01x20
- BP1-DSP-2: renamed from JSKT1-2; footprint Connector_IDC:IDC-Header_2x10_P2.54mm_Horizontal_Lock -> Connector_IDC:IDC-Header_2x10_P2.54mm_Vertical; symbol Connector_Generic:Conn_01x18 -> Connector_Generic:Conn_01x20
- BP1-DSP-3: renamed from JSKT1-3; footprint Connector_IDC:IDC-Header_2x10_P2.54mm_Horizontal_Lock -> Connector_IDC:IDC-Header_2x10_P2.54mm_Vertical; symbol Connector_Generic:Conn_01x18 -> Connector_Generic:Conn_01x20
- BP1-DSP-4: renamed from JSKT2-1; footprint Connector_IDC:IDC-Header_2x10_P2.54mm_Horizontal_Lock -> Connector_IDC:IDC-Header_2x10_P2.54mm_Vertical
- BP1-DSP-5: renamed from JSKT2-2; footprint Connector_IDC:IDC-Header_2x10_P2.54mm_Horizontal_Lock -> Connector_IDC:IDC-Header_2x10_P2.54mm_Vertical
- BP1-DSP-6: renamed from JSKT2-3; footprint Connector_IDC:IDC-Header_2x10_P2.54mm_Horizontal_Lock -> Connector_IDC:IDC-Header_2x10_P2.54mm_Vertical
Connections:
- net #A1: now also BP1-DSP-1.2 (Pin_2); no longer BP1-DSP-1.10 (Pin_10)
- net #A10: now also BP1-DSP-2.2 (Pin_2); no longer BP1-DSP-2.10 (Pin_10)
- net #A11: now also BP1-DSP-2.4 (Pin_4); no longer BP1-DSP-2.11 (Pin_11)
- net #A12: now also BP1-DSP-2.6 (Pin_6); no longer BP1-DSP-2.12 (Pin_12)
- net #A13: now also BP1-DSP-2.8 (Pin_8); no longer BP1-DSP-2.13 (Pin_13)
- net #A14: now also BP1-DSP-2.10 (Pin_10); no longer BP1-DSP-2.14 (Pin_14)
- net #A15: now also BP1-DSP-2.12 (Pin_12); no longer BP1-DSP-2.15 (Pin_15)
- net #A16: now also BP1-DSP-2.14 (Pin_14); no longer BP1-DSP-2.16 (Pin_16)
- net #A17: now also BP1-DSP-2.16 (Pin_16); no longer BP1-DSP-2.17 (Pin_17)
- net #A2: now also BP1-DSP-1.4 (Pin_4); no longer BP1-DSP-1.11 (Pin_11)
- net #A3: now also BP1-DSP-1.6 (Pin_6); no longer BP1-DSP-1.12 (Pin_12)
- net #A4: now also BP1-DSP-1.8 (Pin_8); no longer BP1-DSP-1.13 (Pin_13)
- net #A5: now also BP1-DSP-1.10 (Pin_10); no longer BP1-DSP-1.14 (Pin_14)
- net #A6: now also BP1-DSP-1.12 (Pin_12); no longer BP1-DSP-1.15 (Pin_15)
- net #A7: now also BP1-DSP-1.14 (Pin_14); no longer BP1-DSP-1.16 (Pin_16)
- net #A8: now also BP1-DSP-1.16 (Pin_16); no longer BP1-DSP-1.17 (Pin_17)
- net #G11: now also BP1-DSP-2.3 (Pin_3); no longer BP1-DSP-2.2 (Pin_2)
- net #G12: now also BP1-DSP-2.5 (Pin_5); no longer BP1-DSP-2.3 (Pin_3)
- net #G13: now also BP1-DSP-2.7 (Pin_7); no longer BP1-DSP-2.4 (Pin_4)
- net #G14: now also BP1-DSP-2.9 (Pin_9); no longer BP1-DSP-2.5 (Pin_5)
- net #G15: now also BP1-DSP-2.11 (Pin_11); no longer BP1-DSP-2.6 (Pin_6)
- net #G16: now also BP1-DSP-2.13 (Pin_13); no longer BP1-DSP-2.7 (Pin_7)
- net #G17: now also BP1-DSP-2.15 (Pin_15); no longer BP1-DSP-2.8 (Pin_8)
- net #G18: now also BP1-DSP-2.17 (Pin_17); no longer BP1-DSP-2.9 (Pin_9)
- net #G2: now also BP1-DSP-1.3 (Pin_3); no longer BP1-DSP-1.2 (Pin_2)
- net #G3: now also BP1-DSP-1.5 (Pin_5); no longer BP1-DSP-1.3 (Pin_3)
- net #G4: now also BP1-DSP-1.7 (Pin_7); no longer BP1-DSP-1.4 (Pin_4)
- net #G5: now also BP1-DSP-1.9 (Pin_9); no longer BP1-DSP-1.5 (Pin_5)
- net #G6: now also BP1-DSP-1.11 (Pin_11); no longer BP1-DSP-1.6 (Pin_6)
- net #G7: now also BP1-DSP-1.13 (Pin_13); no longer BP1-DSP-1.7 (Pin_7)
- net #G8: now also BP1-DSP-1.15 (Pin_15); no longer BP1-DSP-1.8 (Pin_8)
- net #G9: now also BP1-DSP-1.17 (Pin_17); no longer BP1-DSP-1.9 (Pin_9)
- net #I1: now also BP1-DSP-2.19 (Pin_19); no longer BP1-DSP-5.17 (Pin_17)
- net #I2: now also BP1-DSP-2.20 (Pin_20); no longer BP1-DSP-5.18 (Pin_18)
- net #I3: now also BP1-DSP-4.19 (Pin_19); no longer BP1-DSP-5.19 (Pin_19)
- net #I4: now also BP1-DSP-4.20 (Pin_20); no longer BP1-DSP-5.20 (Pin_20)
- net #J10: now also BP1-DSP-6.1 (Pin_1); no longer BP1-DSP-5.10 (Pin_10)
- net #J11: now also BP1-DSP-6.2 (Pin_2); no longer BP1-DSP-5.11 (Pin_11)
- net #J12: now also BP1-DSP-6.3 (Pin_3); no longer BP1-DSP-5.12 (Pin_12)
- net #J13: now also BP1-DSP-6.4 (Pin_4); no longer BP1-DSP-5.13 (Pin_13)
- net #J14: now also BP1-DSP-6.5 (Pin_5); no longer BP1-DSP-5.14 (Pin_14)
- net #J15: now also BP1-DSP-6.6 (Pin_6); no longer BP1-DSP-5.15 (Pin_15)
- net #J16: now also BP1-DSP-6.7 (Pin_7); no longer BP1-DSP-5.16 (Pin_16)
- net #M1: now also BP1-DSP-3.2 (Pin_2); no longer BP1-DSP-4.1 (Pin_1)
- net #M2: now also BP1-DSP-3.4 (Pin_4); no longer BP1-DSP-4.2 (Pin_2)
- net #M3: now also BP1-DSP-3.6 (Pin_6); no longer BP1-DSP-4.3 (Pin_3)
- net #M4: now also BP1-DSP-3.8 (Pin_8); no longer BP1-DSP-4.4 (Pin_4)
- net #M5: now also BP1-DSP-3.10 (Pin_10); no longer BP1-DSP-4.5 (Pin_5)
- net #M6: now also BP1-DSP-3.12 (Pin_12); no longer BP1-DSP-4.6 (Pin_6)
- net #M7: now also BP1-DSP-3.14 (Pin_14); no longer BP1-DSP-4.7 (Pin_7)
- net #M8: now also BP1-DSP-3.16 (Pin_16); no longer BP1-DSP-4.8 (Pin_8)
- net #M9: now also BP1-DSP-3.18 (Pin_18); no longer BP1-DSP-4.9 (Pin_9)
- net #P1: now also BP1-DSP-5.10 (Pin_10); no longer BP1-DSP-6.1 (Pin_1)
- net #P2: now also BP1-DSP-5.11 (Pin_11); no longer BP1-DSP-6.2 (Pin_2)
- net #P3: now also BP1-DSP-5.12 (Pin_12); no longer BP1-DSP-6.3 (Pin_3)
- net #P4: now also BP1-DSP-5.13 (Pin_13); no longer BP1-DSP-6.4 (Pin_4)
- net #P5: now also BP1-DSP-5.14 (Pin_14); no longer BP1-DSP-6.5 (Pin_5)
- net #P6: now also BP1-DSP-5.15 (Pin_15); no longer BP1-DSP-6.6 (Pin_6)
- net #P7: now also BP1-DSP-5.16 (Pin_16); no longer BP1-DSP-6.7 (Pin_7)
- net #P8: now also BP1-DSP-5.17 (Pin_17); no longer BP1-DSP-6.8 (Pin_8)
- net #P9: now also BP1-DSP-5.18 (Pin_18); no longer BP1-DSP-6.9 (Pin_9)
- net #Q10: now also BP1-DSP-4.1 (Pin_1); no longer BP1-DSP-3.10 (Pin_10)
- net #Q11: now also BP1-DSP-4.2 (Pin_2); no longer BP1-DSP-3.11 (Pin_11)
- net #Q12: now also BP1-DSP-4.3 (Pin_3); no longer BP1-DSP-3.12 (Pin_12)
- net #Q13: now also BP1-DSP-4.4 (Pin_4); no longer BP1-DSP-3.13 (Pin_13)
- net #Q14: now also BP1-DSP-4.5 (Pin_5); no longer BP1-DSP-3.14 (Pin_14)
- net #Q15: now also BP1-DSP-4.6 (Pin_6); no longer BP1-DSP-3.15 (Pin_15)
- net #Q16: now also BP1-DSP-4.7 (Pin_7); no longer BP1-DSP-3.16 (Pin_16)
- net #Q17: now also BP1-DSP-4.8 (Pin_8); no longer BP1-DSP-3.17 (Pin_17)
- net #Q18: now also BP1-DSP-4.9 (Pin_9); no longer BP1-DSP-3.18 (Pin_18)
- net #Q2: now also BP1-DSP-3.3 (Pin_3); no longer BP1-DSP-3.2 (Pin_2)
- net #Q3: now also BP1-DSP-3.5 (Pin_5); no longer BP1-DSP-3.3 (Pin_3)
- net #Q4: now also BP1-DSP-3.7 (Pin_7); no longer BP1-DSP-3.4 (Pin_4)
- net #Q5: now also BP1-DSP-3.9 (Pin_9); no longer BP1-DSP-3.5 (Pin_5)
- net #Q6: now also BP1-DSP-3.11 (Pin_11); no longer BP1-DSP-3.6 (Pin_6)
- net #Q7: now also BP1-DSP-3.13 (Pin_13); no longer BP1-DSP-3.7 (Pin_7)
- net #Q8: now also BP1-DSP-3.15 (Pin_15); no longer BP1-DSP-3.8 (Pin_8)
- net #Q9: now also BP1-DSP-3.17 (Pin_17); no longer BP1-DSP-3.9 (Pin_9)
- net W1: now also BP1-DSP-1.19 (Pin_19); no longer BP1-DSP-4.20 (Pin_20)
- net W10: now also BP1-DSP-6.13 (Pin_13); no longer BP1-DSP-6.17 (Pin_17)
- net W11: now also BP1-DSP-6.14 (Pin_14); no longer BP1-DSP-6.18 (Pin_18)
- net W12: now also BP1-DSP-6.15 (Pin_15); no longer BP1-DSP-6.19 (Pin_19)
- net W13: now also BP1-DSP-6.16 (Pin_16); no longer BP1-DSP-6.20 (Pin_20)
- net W5: now also BP1-DSP-1.20 (Pin_20); no longer BP1-DSP-6.12 (Pin_12)
- net W6: now also BP1-DSP-3.19 (Pin_19); no longer BP1-DSP-6.13 (Pin_13)
- net W7: now also BP1-DSP-3.20 (Pin_20); no longer BP1-DSP-6.14 (Pin_14)
- net W8: now also BP1-DSP-5.19 (Pin_19); no longer BP1-DSP-6.15 (Pin_15)
- net W9: now also BP1-DSP-5.20 (Pin_20); no longer BP1-DSP-6.16 (Pin_16)
- no-connect marks 20 -> 26

Commit message: New Backplanes
Parts:
- BP1-BP2-1, BP1-BP2-2, BP1-BP2-3, BP1-BP2-4, BP1-BP2-5, BP1-BP3-1, BP1-BP3-2: footprint (none) -> Connector_IDC:IDC-Header_2x10_P2.54mm_Vertical
- BP1-BP3-3, BP1-BP3-4, BP1-BP3-5, BP1-BP3-6, BP1-BP3-7: footprint (none) -> Connector_IDC:IDC-Header_2x10_P2.54mm_Vertical; symbol Connector_Generic:Conn_01x18 -> Connector_Generic:Conn_01x20
Connections:
- net #A1: now also BP1-DSP-1.19 (Pin_19); no longer BP1-DSP-1.2 (Pin_2)
- net #A10: now also BP1-DSP-2.8 (Pin_8); no longer BP1-DSP-2.2 (Pin_2)
- net #A11: now also BP1-DSP-2.9 (Pin_9); no longer BP1-DSP-2.4 (Pin_4)
- net #A12: now also BP1-DSP-2.10 (Pin_10); no longer BP1-DSP-2.6 (Pin_6)
- net #A13: now also BP1-DSP-2.11 (Pin_11); no longer BP1-DSP-2.8 (Pin_8)
- net #A14: now also BP1-DSP-2.12 (Pin_12); no longer BP1-DSP-2.10 (Pin_10)
- net #A15: now also BP1-DSP-2.13 (Pin_13); no longer BP1-DSP-2.12 (Pin_12)
- net #A17: now also BP1-DSP-2.15 (Pin_15); no longer BP1-DSP-2.16 (Pin_16)
- net #A18: now also BP1-DSP-2.16 (Pin_16); no longer BP1-DSP-2.18 (Pin_18)
- net #A2: now also BP1-DSP-1.20 (Pin_20); no longer BP1-DSP-1.4 (Pin_4)
- net #A3: now also BP1-DSP-2.1 (Pin_1); no longer BP1-DSP-1.6 (Pin_6)
- net #A4: now also BP1-DSP-2.2 (Pin_2); no longer BP1-DSP-1.8 (Pin_8)
- net #A5: now also BP1-DSP-2.3 (Pin_3); no longer BP1-DSP-1.10 (Pin_10)
- net #A6: now also BP1-DSP-2.4 (Pin_4); no longer BP1-DSP-1.12 (Pin_12)
- net #A7: now also BP1-DSP-2.5 (Pin_5); no longer BP1-DSP-1.14 (Pin_14)
- net #A8: now also BP1-DSP-2.6 (Pin_6); no longer BP1-DSP-1.16 (Pin_16)
- net #A9: now also BP1-DSP-2.7 (Pin_7); no longer BP1-DSP-1.18 (Pin_18)
- net #G10: now also BP1-DSP-1.10 (Pin_10); no longer BP1-DSP-2.1 (Pin_1)
- net #G11: now also BP1-DSP-1.11 (Pin_11); no longer BP1-DSP-2.3 (Pin_3)
- net #G12: now also BP1-DSP-1.12 (Pin_12); no longer BP1-DSP-2.5 (Pin_5)
- net #G13: now also BP1-DSP-1.13 (Pin_13); no longer BP1-DSP-2.7 (Pin_7)
- net #G14: now also BP1-DSP-1.14 (Pin_14); no longer BP1-DSP-2.9 (Pin_9)
- net #G15: now also BP1-DSP-1.15 (Pin_15); no longer BP1-DSP-2.11 (Pin_11)
- net #G16: now also BP1-DSP-1.16 (Pin_16); no longer BP1-DSP-2.13 (Pin_13)
- net #G17: now also BP1-DSP-1.17 (Pin_17); no longer BP1-DSP-2.15 (Pin_15)
- net #G18: now also BP1-DSP-1.18 (Pin_18); no longer BP1-DSP-2.17 (Pin_17)
- net #G2: now also BP1-DSP-1.2 (Pin_2); no longer BP1-DSP-1.3 (Pin_3)
- net #G3: now also BP1-DSP-1.3 (Pin_3); no longer BP1-DSP-1.5 (Pin_5)
- net #G4: now also BP1-DSP-1.4 (Pin_4); no longer BP1-DSP-1.7 (Pin_7)
- net #G5: now also BP1-DSP-1.5 (Pin_5); no longer BP1-DSP-1.9 (Pin_9)
- net #G6: now also BP1-DSP-1.6 (Pin_6); no longer BP1-DSP-1.11 (Pin_11)
- net #G7: now also BP1-DSP-1.7 (Pin_7); no longer BP1-DSP-1.13 (Pin_13)
- net #G8: now also BP1-DSP-1.8 (Pin_8); no longer BP1-DSP-1.15 (Pin_15)
- net #G9: now also BP1-DSP-1.9 (Pin_9); no longer BP1-DSP-1.17 (Pin_17)
- net #I1: now also BP1-DSP-6.1 (Pin_1); no longer BP1-DSP-2.19 (Pin_19)
- net #I2: now also BP1-DSP-6.2 (Pin_2); no longer BP1-DSP-2.20 (Pin_20)
- net #I3: now also BP1-DSP-6.3 (Pin_3); no longer BP1-DSP-4.19 (Pin_19)
- net #I4: now also BP1-DSP-6.4 (Pin_4); no longer BP1-DSP-4.20 (Pin_20)
- net #J1: now also BP1-DSP-4.19 (Pin_19); no longer BP1-DSP-5.1 (Pin_1)
- net #J10: now also BP1-DSP-5.8 (Pin_8); no longer BP1-DSP-6.1 (Pin_1)
- net #J11: now also BP1-DSP-5.9 (Pin_9); no longer BP1-DSP-6.2 (Pin_2)
- net #J12: now also BP1-DSP-5.10 (Pin_10); no longer BP1-DSP-6.3 (Pin_3)
- net #J13: now also BP1-DSP-5.11 (Pin_11); no longer BP1-DSP-6.4 (Pin_4)
- net #J14: now also BP1-DSP-5.12 (Pin_12); no longer BP1-DSP-6.5 (Pin_5)
- net #J15: now also BP1-DSP-5.13 (Pin_13); no longer BP1-DSP-6.6 (Pin_6)
- net #J16: now also BP1-DSP-5.14 (Pin_14); no longer BP1-DSP-6.7 (Pin_7)
- net #J2: now also BP1-DSP-4.20 (Pin_20); no longer BP1-DSP-5.2 (Pin_2)
- net #J3: now also BP1-DSP-5.1 (Pin_1); no longer BP1-DSP-5.3 (Pin_3)
- net #J4: now also BP1-DSP-5.2 (Pin_2); no longer BP1-DSP-5.4 (Pin_4)
- net #J5: now also BP1-DSP-5.3 (Pin_3); no longer BP1-DSP-5.5 (Pin_5)
- net #J6: now also BP1-DSP-5.4 (Pin_4); no longer BP1-DSP-5.6 (Pin_6)
- net #J7: now also BP1-DSP-5.5 (Pin_5); no longer BP1-DSP-5.7 (Pin_7)
- net #J8: now also BP1-DSP-5.6 (Pin_6); no longer BP1-DSP-5.8 (Pin_8)
- net #J9: now also BP1-DSP-5.7 (Pin_7); no longer BP1-DSP-5.9 (Pin_9)
- net #M1: now also BP1-DSP-4.1 (Pin_1); no longer BP1-DSP-3.2 (Pin_2)
- net #M2: now also BP1-DSP-4.2 (Pin_2); no longer BP1-DSP-3.4 (Pin_4)
- net #M3: now also BP1-DSP-4.3 (Pin_3); no longer BP1-DSP-3.6 (Pin_6)
- net #M4: now also BP1-DSP-4.4 (Pin_4); no longer BP1-DSP-3.8 (Pin_8)
- net #M5: now also BP1-DSP-4.5 (Pin_5); no longer BP1-DSP-3.10 (Pin_10)
- net #M6: now also BP1-DSP-4.6 (Pin_6); no longer BP1-DSP-3.12 (Pin_12)
- net #M7: now also BP1-DSP-4.7 (Pin_7); no longer BP1-DSP-3.14 (Pin_14)
- net #M8: now also BP1-DSP-4.8 (Pin_8); no longer BP1-DSP-3.16 (Pin_16)
- net #M9: now also BP1-DSP-4.9 (Pin_9); no longer BP1-DSP-3.18 (Pin_18)
- net #P1: now also BP1-DSP-5.15 (Pin_15); no longer BP1-DSP-5.10 (Pin_10)
- net #P10: now also BP1-DSP-3.18 (Pin_18); no longer BP1-DSP-6.10 (Pin_10)
- net #P11: now also BP1-DSP-3.19 (Pin_19); no longer BP1-DSP-6.11 (Pin_11)
- net #P2: now also BP1-DSP-5.16 (Pin_16); no longer BP1-DSP-5.11 (Pin_11)
- net #P3: now also BP1-DSP-5.17 (Pin_17); no longer BP1-DSP-5.12 (Pin_12)
- net #P4: now also BP1-DSP-5.18 (Pin_18); no longer BP1-DSP-5.13 (Pin_13)
- net #P5: now also BP1-DSP-5.19 (Pin_19); no longer BP1-DSP-5.14 (Pin_14)
- net #P6: now also BP1-DSP-5.20 (Pin_20); no longer BP1-DSP-5.15 (Pin_15)
- net #P7: now also BP1-DSP-3.15 (Pin_15); no longer BP1-DSP-5.16 (Pin_16)
- net #P8: now also BP1-DSP-3.16 (Pin_16); no longer BP1-DSP-5.17 (Pin_17)
- net #P9: now also BP1-DSP-3.17 (Pin_17); no longer BP1-DSP-5.18 (Pin_18)
- net #Q1: now also BP1-DSP-2.17 (Pin_17); no longer BP1-DSP-3.1 (Pin_1)
- net #Q10: now also BP1-DSP-3.6 (Pin_6); no longer BP1-DSP-4.1 (Pin_1)
- net #Q11: now also BP1-DSP-3.7 (Pin_7); no longer BP1-DSP-4.2 (Pin_2)
- net #Q12: now also BP1-DSP-3.8 (Pin_8); no longer BP1-DSP-4.3 (Pin_3)
- net #Q13: now also BP1-DSP-3.9 (Pin_9); no longer BP1-DSP-4.4 (Pin_4)
- net #Q14: now also BP1-DSP-3.10 (Pin_10); no longer BP1-DSP-4.5 (Pin_5)
- net #Q15: now also BP1-DSP-3.11 (Pin_11); no longer BP1-DSP-4.6 (Pin_6)
- net #Q16: now also BP1-DSP-3.12 (Pin_12); no longer BP1-DSP-4.7 (Pin_7)
- net #Q17: now also BP1-DSP-3.13 (Pin_13); no longer BP1-DSP-4.8 (Pin_8)
- net #Q18: now also BP1-DSP-3.14 (Pin_14); no longer BP1-DSP-4.9 (Pin_9)
- net #Q2: now also BP1-DSP-2.18 (Pin_18); no longer BP1-DSP-3.3 (Pin_3)
- net #Q3: now also BP1-DSP-2.19 (Pin_19); no longer BP1-DSP-3.5 (Pin_5)
- net #Q4: now also BP1-DSP-2.20 (Pin_20); no longer BP1-DSP-3.7 (Pin_7)
- net #Q5: now also BP1-DSP-3.1 (Pin_1); no longer BP1-DSP-3.9 (Pin_9)
- net #Q6: now also BP1-DSP-3.2 (Pin_2); no longer BP1-DSP-3.11 (Pin_11)
- net #Q7: now also BP1-DSP-3.3 (Pin_3); no longer BP1-DSP-3.13 (Pin_13)
- net #Q8: now also BP1-DSP-3.4 (Pin_4); no longer BP1-DSP-3.15 (Pin_15)
- net #Q9: now also BP1-DSP-3.5 (Pin_5); no longer BP1-DSP-3.17 (Pin_17)
- net W1: now also BP1-DSP-6.5 (Pin_5); no longer BP1-DSP-1.19 (Pin_19)
- net W10: now also BP1-DSP-6.14 (Pin_14); no longer BP1-DSP-6.13 (Pin_13)
- net W11: now also BP1-DSP-6.15 (Pin_15); no longer BP1-DSP-6.14 (Pin_14)
- net W12: now also BP1-DSP-6.16 (Pin_16); no longer BP1-DSP-6.15 (Pin_15)
- net W13: now also BP1-DSP-6.17 (Pin_17); no longer BP1-DSP-6.16 (Pin_16)
- net W5: now also BP1-DSP-6.9 (Pin_9); no longer BP1-DSP-1.20 (Pin_20)
- net W6: now also BP1-DSP-6.10 (Pin_10); no longer BP1-DSP-3.19 (Pin_19)
- net W7: now also BP1-DSP-6.11 (Pin_11); no longer BP1-DSP-3.20 (Pin_20)
- net W8: now also BP1-DSP-6.12 (Pin_12); no longer BP1-DSP-5.19 (Pin_19)
- net W9: now also BP1-DSP-6.13 (Pin_13); no longer BP1-DSP-5.20 (Pin_20)
- no-connect marks 26 -> 36
Other:
- moved on the sheet: BP1-BP2-1, BP1-BP2-2, BP1-BP2-3, BP1-BP2-4, BP1-BP2-5, BP1-BP3-1, BP1-BP3-2, BP1-DSP-1, BP1-DSP-2, BP1-DSP-3, BP1-DSP-4, BP1-DSP-5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
