File: KiCad/Real903/Backplane1/Connections.kicad_sch (KiCad schematic)
At the start: 18 parts

Commit message: Start new layout with IDC connectors
Parts:
- BP1-BP2-1, BP1-BP2-2, BP1-BP2-3, BP1-BP2-4, BP1-BP2-5, BP1-BP3-1, BP1-BP3-2, BP1-BP3-3, BP1-BP3-4, BP1-BP3-5, BP1-BP3-6, BP1-BP3-7, BP1-CNT-1, BP1-DSP-1, BP1-DSP-2, BP1-DSP-3, BP1-DSP-4, BP1-DSP-5: footprint Connector_IDC:IDC-Header_2x10_P2.54mm_Vertical -> Connector_IDC:IDC-Header_2x10_P2.54mm_Latch_Vertical
Changed lines of the file:
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@@
     (property "Reference" "BP1-BP3-6" (id 0) (at 140.97 187.96 0))
     (property "Value" "~" (id 1) (at 143.002 190.4746 0))
-    (property "Footprint" "Connector_IDC:IDC-Header_2x10_P2.54mm_Vertical" (id 2) (at 140.97 213.995 0)
+    (property "Footprint" "Connector_IDC:IDC-Header_2x10_P2.54mm_Latch_Vertical" (id 2) (at 140.97 213.995 0)
       (effects (font (size 1.27 1.27)) hide)
     )
@@
     (property "Reference" "BP1-BP3-4" (id 0) (at 96.52 188.595 0))
     (property "Value" "~" (id 1) (at 98.552 191.1096 0))
-    (property "Footprint" "Connector_IDC:IDC-Header_2x10_P2.54mm_Vertical" (id 2) (at 96.52 214.63 0)
+    (property "Footprint" "Connector_IDC:IDC-Header_2x10_P2.54mm_Latch_Vertical" (id 2) (at 96.52 214.63 0)
       (effects (font (size 1.27 1.27)) hide)
     )
@@
     (property "Reference" "BP1-BP3-5" (id 0) (at 117.475 187.96 0))
     (property "Value" "~" (id 1) (at 119.507 190.4746 0))
-    (property "Footprint" "Connector_IDC:IDC-Header_2x10_P2.54mm_Vertical" (id 2) (at 117.475 213.995 0)
+    (property "Footprint" "Connector_IDC:IDC-Header_2x10_P2.54mm_Latch_Vertical" (id 2) (at 117.475 213.995 0)
       (effects (font (size 1.27 1.27)) hide)
     )
@@
     (property "Reference" "BP1-DSP-1" (id 0) (at 34.925 44.45 0))
     (property "Value" "~" (id 1) (at 35.052 46.9646 0))
-    (property "Footprint" "Connector_IDC:IDC-Header_2x10_P2.54mm_Vertical" (id 2) (at 33.02 70.485 0)
+    (property "Footprint" "Connector_IDC:IDC-Header_2x10_P2.54mm_Latch_Vertical" (id 2) (at 33.02 70.485 0)
       (effects (font (size 1.27 1.27)) hide)
     )
@@
     (property "Reference" "BP1-DSP-2" (id 0) (at 55.245 44.45 0))
     (property "Value" "~" (id 1) (at 55.372 46.9646 0))
-    (property "Footprint" "Connector_IDC:IDC-Header_2x10_P2.54mm_Vertical" (id 2) (at 53.34 70.485 0)
+    (property "Footprint" "Connector_IDC:IDC-Header_2x10_P2.54mm_Latch_Vertical" (id 2) (at 53.34 70.485 0)
       (effects (font (size 1.27 1.27)) hide)
     )
@@
     (property "Reference" "BP1-DSP-3" (id 0) (at 76.2 44.45 0))
     (property "Value" "~" (id 1) (at 76.327 46.9646 0))
-    (property "Footprint" "Connector_IDC:IDC-Header_2x10_P2.54mm_Vertical" (id 2) (at 74.295 70.485 0)
+    (property "Footprint" "Connector_IDC:IDC-Header_2x10_P2.54mm_Latch_Vertical" (id 2) (at 74.295 70.485 0)
       (effects (font (size 1.27 1.27)) hide)
     )
@@
     (property "Reference" "BP1-DSP-4" (id 0) (at 99.06 44.45 0))
     (property "Value" "~" (id 1) (at 99.187 46.9646 0))
-    (property "Footprint" "Connector_IDC:IDC-Header_2x10_P2.54mm_Vertical" (id 2) (at 97.155 70.485 0)
+    (property "Footprint" "Connector_IDC:IDC-Header_2x10_P2.54mm_Latch_Vertical" (id 2) (at 97.155 70.485 0)
       (effects (font (size 1.27 1.27)) hide)
     )
@@
     (property "Reference" "BP1-DSP-5" (id 0) (at 120.015 44.45 0))
     (property "Value" "~" (id 1) (at 120.142 46.9646 0))
-    (property "Footprint" "Connector_IDC:IDC-Header_2x10_P2.54mm_Vertical" (id 2) (at 118.11 70.485 0)
+    (property "Footprint" "Connector_IDC:IDC-Header_2x10_P2.54mm_Latch_Vertical" (id 2) (at 118.11 70.485 0)
       (effects (font (size 1.27 1.27)) hide)
     )
@@
     (property "Reference" "BP1-CNT-1" (id 0) (at 142.875 44.45 0))
     (property "Value" "~" (id 1) (at 143.002 46.9646 0))
-    (property "Footprint" "Connector_IDC:IDC-Header_2x10_P2.54mm_Vertical" (id 2) (at 140.97 70.485 0)
+    (property "Footprint" "Connector_IDC:IDC-Header_2x10_P2.54mm_Latch_Vertical" (id 2) (at 140.97 70.485 0)
       (effects (font (size 1.27 1.27)) hide)
     )
@@
     (property "Reference" "BP1-BP2-1" (id 0) (at 34.925 120.65 0))
     (property "Value" "~" (id 1) (at 35.052 123.1646 0))
-    (property "Footprint" "Connector_IDC:IDC-Header_2x10_P2.54mm_Vertical" (id 2) (at 33.02 146.685 0)
+    (property "Footprint" "Connector_IDC:IDC-Header_2x10_P2.54mm_Latch_Vertical" (id 2) (at 33.02 146.685 0)
       (effects (font (size 1.27 1.27)) hide)
     )
@@
     (property "Reference" "BP1-BP2-2" (id 0) (at 55.245 120.65 0))
     (property "Value" "~" (id 1) (at 55.372 123.1646 0))
-    (property "Footprint" "Connector_IDC:IDC-Header_2x10_P2.54mm_Vertical" (id 2) (at 53.34 146.685 0)
+    (property "Footprint" "Connector_IDC:IDC-Header_2x10_P2.54mm_Latch_Vertical" (id 2) (at 53.34 146.685 0)
       (effects (font (size 1.27 1.27)) hide)
     )
@@
     (property "Reference" "BP1-BP2-3" (id 0) (at 76.2 120.65 0))
     (property "Value" "~" (id 1) (at 76.327 123.1646 0))
-    (property "Footprint" "Connector_IDC:IDC-Header_2x10_P2.54mm_Vertical" (id 2) (at 74.295 146.685 0)
+    (property "Footprint" "Connector_IDC:IDC-Header_2x10_P2.54mm_Latch_Vertical" (id 2) (at 74.295 146.685 0)
       (effects (font (size 1.27 1.27)) hide)
     )
@@
     (property "Reference" "BP1-BP2-4" (id 0) (at 99.06 120.65 0))
     (property "Value" "~" (id 1) (at 99.187 123.1646 0))
-    (property "Footprint" "Connector_IDC:IDC-Header_2x10_P2.54mm_Vertical" (id 2) (at 97.155 146.685 0)
+    (property "Footprint" "Connector_IDC:IDC-Header_2x10_P2.54mm_Latch_Vertical" (id 2) (at 97.155 146.685 0)
       (effects (font (size 1.27 1.27)) hide)
     )
@@
     (property "Reference" "BP1-BP2-5" (id 0) (at 120.015 120.65 0))
     (property "Value" "~" (id 1) (at 120.142 123.1646 0))
-    (property "Footprint" "Connector_IDC:IDC-Header_2x10_P2.54mm_Vertical" (id 2) (at 118.11 146.685 0)
+    (property "Footprint" "Connector_IDC:IDC-Header_2x10_P2.54mm_Latch_Vertical" (id 2) (at 118.11 146.685 0)
       (effects (font (size 1.27 1.27)) hide)
     )
@@
     (property "Reference" "BP1-BP3-1" (id 0) (at 34.925 187.96 0))
     (property "Value" "~" (id 1) (at 35.052 190.4746 0))
-    (property "Footprint" "Connector_IDC:IDC-Header_2x10_P2.54mm_Vertical" (id 2) (at 33.02 213.995 0)
+    (property "Footprint" "Connector_IDC:IDC-Header_2x10_P2.54mm_Latch_Vertical" (id 2) (at 33.02 213.995 0)
       (effects (font (size 1.27 1.27)) hide)
     )
@@
     (property "Reference" "BP1-BP3-2" (id 0) (at 55.245 187.96 0))
     (property "Value" "~" (id 1) (at 55.372 190.4746 0))
-    (property "Footprint" "Connector_IDC:IDC-Header_2x10_P2.54mm_Vertical" (id 2) (at 53.34 213.995 0)
+    (property "Footprint" "Connector_IDC:IDC-Header_2x10_P2.54mm_Latch_Vertical" (id 2) (at 53.34 213.995 0)
       (effects (font (size 1.27 1.27)) hide)
     )
@@
     (property "Reference" "BP1-BP3-3" (id 0) (at 73.66 188.595 0))
     (property "Value" "~" (id 1) (at 75.692 191.1096 0))
-    (property "Footprint" "Connector_IDC:IDC-Header_2x10_P2.54mm_Vertical" (id 2) (at 73.66 214.63 0)
+    (property "Footprint" "Connector_IDC:IDC-Header_2x10_P2.54mm_Latch_Vertical" (id 2) (at 73.66 214.63 0)
       (effects (font (size 1.27 1.27)) hide)
     )
@@
     (property "Reference" "BP1-BP3-7" (id 0) (at 161.925 187.96 0))
     (property "Value" "~" (id 1) (at 163.957 190.4746 0))
-    (property "Footprint" "Connector_IDC:IDC-Header_2x10_P2.54mm_Vertical" (id 2) (at 161.925 213.995 0)
-      (effects (font (size 1.27 1.27)) hide)
-    )
+    (property "Footprint" "Connector_IDC:IDC-Header_2x10_P2.54mm_Latch_Vertical" (id 2) (at 161.925 213.995 0)
+      (effects (font (size 1.27 1.27)) hide)
+    )
