File: KiCad/Real903/Backplane1/WaveformDrivers.kicad_sch (KiCad schematic)
At the start: 2 parts

Commit message: Update to design
Connections:
- net ATF1 renamed Low.ATF
- net ATF2 renamed High.ATF
- net FTG2 renamed High.FTG
- net GTA2 renamed High.GTA
- net GTJ2 renamed High.GTJ
- net GTM2 renamed High.GTM
- net GTQ1 renamed Low.GTQ
- net GTQ2 renamed High.GTQ
- net JTF2 renamed High.JTF
- net LTG2 renamed High.LTG
- net MTF2 renamed High.MTF
- net MTP2 renamed High.MTP
- net PTG1-2 renamed High.PTG1
- net PTG2-2 renamed High.PTG2
- net QTF1 renamed Low.QTF
- net QTF2 renamed High.QTF
- net RTG2 renamed High.RTG
- net VTG2 renamed High.VTG
- net WTM2 renamed High.WTM
- net ~{JTG14} renamed ~{JTG}14
- net ~{JTG15} renamed ~{JTG}15
- net ~{JTG16} renamed ~{JTG}16
- net ~{M}TF1 renamed Low.~{M}TF
- net ~{M}TF2 renamed High.~{M}TF
- net ~{OTA}1 renamed Low.~{OTA}
- net ~{OTA}2 renamed High.~{OTA}
- net ~{OTG}2 renamed High.~{OTG}
- net ~{OTJ}2 renamed High.~{OTJ}
- net ~{OTM}1 renamed Low.~{OTM}
- net ~{OTM}2 renamed High.~{OTM}
- net ~{OTP}1 renamed Low.~{OTP}
- net ~{OTQ}1 renamed Low.~{OTQ}
- net ~{OTQ}2 renamed High.~{OTQ}
