File: KiCad/Real903/Sockets/Display.sch (KiCad schematic (older format))
At the start: 11 parts

Commit message: New Backplanes
Parts:
- removed J0: ~, Connector_IDC:IDC-Header_2x03_P2.54mm_Vertical, symbol Connector_Generic:Conn_01x03
- removed JSKT2-3, JSKT3-1: ~, Connector_IDC:IDC-Header_2x10_P2.54mm_Vertical, symbol Sockets-rescue:Conn_01x20-Connector_Generic
- added DSP-BP2-1, DSP-BP2-2: ~, Connector_IDC:IDC-Header_2x10_P2.54mm_Vertical, symbol Connector_Generic:Conn_01x20
- renumbered JSKT1-1 to DSP-BP1-1, JSKT1-2 to DSP-BP1-2, JSKT1-3 to DSP-BP1-3, JSKT2-1 to DSP-BP1-4, JSKT2-2 to DSP-BP1-5
Connections:
- net #AA1'-21-K: now also DSP-BP2-2.6 (Pin_6)
- net #AA1-21-M: now also DSP-BP2-2.10 (Pin_10)
- net #AA2'-21-U: now also DSP-BP2-2.7 (Pin_7)
- net #AA2-21-X: now also DSP-BP2-2.11 (Pin_11)
- net #AA3'-21-AF: now also DSP-BP2-2.8 (Pin_8)
- net #AA3-21-AA: now also DSP-BP2-2.12 (Pin_12)
- net #C-6-N: now also DSP-BP2-2.16 (Pin_16)
- net #CA-7-Z: now also DSP-BP2-2.14 (Pin_14)
- net #CB-7-V: now also DSP-BP2-2.15 (Pin_15)
- net #CD-6-V: now also DSP-BP2-2.17 (Pin_17)
- net #FD-6-S: now also DSP-BP2-2.1 (Pin_1)
- net #NOTRDY-2-AC: now also DSP-BP2-2.20 (Pin_20)
- net #PC1: now also DSP-BP2-1.1 (Pin_1)
- net #PC10: now also DSP-BP2-1.10 (Pin_10)
- net #PC11: now also DSP-BP2-1.11 (Pin_11)
- net #PC12: now also DSP-BP2-1.12 (Pin_12)
- net #PC2: now also DSP-BP2-1.2 (Pin_2)
- net #PC3: now also DSP-BP2-1.3 (Pin_3)
- net #PC4: now also DSP-BP2-1.4 (Pin_4)
- net #PC5: now also DSP-BP2-1.5 (Pin_5)
- net #PC6: now also DSP-BP2-1.6 (Pin_6)
- net #PC7: now also DSP-BP2-1.7 (Pin_7)
- net #PC8: now also DSP-BP2-1.8 (Pin_8)
- net #PC9: now also DSP-BP2-1.9 (Pin_9)
- net #RESET-2-Z: now also DSP-BP2-2.18 (Pin_18)
- net #SIP-30-Z: no longer DSP-BP1-3.20 (Pin_20)
- net #SOP-30-P: no longer DSP-BP1-3.19 (Pin_19)
- net #STOP-2-T: now also DSP-BP2-2.19 (Pin_19)
- net #STP-30-L: no longer DSP-BP1-1.1 (Pin_1)
- net #STR-30-H: no longer DSP-BP1-1.2 (Pin_2)
- net #X-57-D: now also DSP-BP2-1.14 (Pin_14); no longer DSP-BP1-3.17 (Pin_17)
- net #Y-57-Z: now also DSP-BP2-1.13 (Pin_13); no longer DSP-BP1-3.18 (Pin_18)
- net A1: now also DSP-BP1-1.19 (Pin_19); no longer DSP-BP1-2.1 (Pin_1)
- net A10: now also DSP-BP1-2.8 (Pin_8); no longer DSP-BP1-2.10 (Pin_10)
- net A11: now also DSP-BP1-2.9 (Pin_9); no longer DSP-BP1-2.11 (Pin_11)
- net A12: now also DSP-BP1-2.10 (Pin_10); no longer DSP-BP1-2.12 (Pin_12)
- net A13: now also DSP-BP1-2.11 (Pin_11); no longer DSP-BP1-2.13 (Pin_13)
- net A14: now also DSP-BP1-2.12 (Pin_12); no longer DSP-BP1-2.14 (Pin_14)
- net A15: now also DSP-BP1-2.13 (Pin_13); no longer DSP-BP1-2.15 (Pin_15)
- net A16: now also DSP-BP1-2.14 (Pin_14); no longer DSP-BP1-2.16 (Pin_16)
- net A17: now also DSP-BP1-2.15 (Pin_15); no longer DSP-BP1-2.17 (Pin_17)
- net A18: now also DSP-BP1-2.16 (Pin_16); no longer DSP-BP1-2.18 (Pin_18)
- net A2: now also DSP-BP1-1.20 (Pin_20); no longer DSP-BP1-2.2 (Pin_2)
- net A3: now also DSP-BP1-2.1 (Pin_1); no longer DSP-BP1-2.3 (Pin_3)
- net A4: now also DSP-BP1-2.2 (Pin_2); no longer DSP-BP1-2.4 (Pin_4)
- net A5: now also DSP-BP1-2.3 (Pin_3); no longer DSP-BP1-2.5 (Pin_5)
- net A6: now also DSP-BP1-2.4 (Pin_4); no longer DSP-BP1-2.6 (Pin_6)
- net A7: now also DSP-BP1-2.5 (Pin_5); no longer DSP-BP1-2.7 (Pin_7)
- net A8: now also DSP-BP1-2.6 (Pin_6); no longer DSP-BP1-2.8 (Pin_8)
- net A9: now also DSP-BP1-2.7 (Pin_7); no longer DSP-BP1-2.9 (Pin_9)
- net G1: now also DSP-BP1-1.1 (Pin_1); no longer DSP-BP1-1.3 (Pin_3)
- net G10: now also DSP-BP1-1.10 (Pin_10); no longer DSP-BP1-1.12 (Pin_12)
- net G11: now also DSP-BP1-1.11 (Pin_11); no longer DSP-BP1-1.13 (Pin_13)
- net G12: now also DSP-BP1-1.12 (Pin_12); no longer DSP-BP1-1.14 (Pin_14)
- net G13: now also DSP-BP1-1.13 (Pin_13); no longer DSP-BP1-1.15 (Pin_15)
- net G14: now also DSP-BP1-1.14 (Pin_14); no longer DSP-BP1-1.16 (Pin_16)
- net G15: now also DSP-BP1-1.15 (Pin_15); no longer DSP-BP1-1.17 (Pin_17)
- net G16: now also DSP-BP1-1.16 (Pin_16); no longer DSP-BP1-1.18 (Pin_18)
- net G17: now also DSP-BP1-1.17 (Pin_17); no longer DSP-BP1-1.19 (Pin_19)
- net G18: now also DSP-BP1-1.18 (Pin_18); no longer DSP-BP1-1.20 (Pin_20)
- net G2: now also DSP-BP1-1.2 (Pin_2); no longer DSP-BP1-1.4 (Pin_4)
- net G3: now also DSP-BP1-1.3 (Pin_3); no longer DSP-BP1-1.5 (Pin_5)
- net G4: now also DSP-BP1-1.4 (Pin_4); no longer DSP-BP1-1.6 (Pin_6)
- net G5: now also DSP-BP1-1.5 (Pin_5); no longer DSP-BP1-1.7 (Pin_7)
- net G6: now also DSP-BP1-1.6 (Pin_6); no longer DSP-BP1-1.8 (Pin_8)
- net G7: now also DSP-BP1-1.7 (Pin_7); no longer DSP-BP1-1.9 (Pin_9)
- net G8: now also DSP-BP1-1.8 (Pin_8); no longer DSP-BP1-1.10 (Pin_10)
- net G9: now also DSP-BP1-1.9 (Pin_9); no longer DSP-BP1-1.11 (Pin_11)
- net P10: now also DSP-BP1-3.18 (Pin_18)
- net P11: now also DSP-BP1-3.19 (Pin_19)
- net P7: now also DSP-BP1-3.15 (Pin_15)
- net P8: now also DSP-BP1-3.16 (Pin_16)
- net P9: now also DSP-BP1-3.17 (Pin_17)
- net Q1: now also DSP-BP1-2.17 (Pin_17); no longer DSP-BP1-2.19 (Pin_19)
- net Q10: now also DSP-BP1-3.6 (Pin_6); no longer DSP-BP1-3.8 (Pin_8)
- net Q11: now also DSP-BP1-3.7 (Pin_7); no longer DSP-BP1-3.9 (Pin_9)
- net Q12: now also DSP-BP1-3.8 (Pin_8); no longer DSP-BP1-3.10 (Pin_10)
- net Q13: now also DSP-BP1-3.9 (Pin_9); no longer DSP-BP1-3.11 (Pin_11)
- net Q14: now also DSP-BP1-3.10 (Pin_10); no longer DSP-BP1-3.12 (Pin_12)
- net Q15: now also DSP-BP1-3.11 (Pin_11); no longer DSP-BP1-3.13 (Pin_13)
- net Q16: now also DSP-BP1-3.12 (Pin_12); no longer DSP-BP1-3.14 (Pin_14)
- net Q17: now also DSP-BP1-3.13 (Pin_13); no longer DSP-BP1-3.15 (Pin_15)
- net Q18: now also DSP-BP1-3.14 (Pin_14); no longer DSP-BP1-3.16 (Pin_16)
- net Q2: now also DSP-BP1-2.18 (Pin_18); no longer DSP-BP1-2.20 (Pin_20)
- net Q3: now also DSP-BP1-2.19 (Pin_19); no longer DSP-BP1-3.1 (Pin_1)
- net Q4: now also DSP-BP1-2.20 (Pin_20); no longer DSP-BP1-3.2 (Pin_2)
- net Q5: now also DSP-BP1-3.1 (Pin_1); no longer DSP-BP1-3.3 (Pin_3)
- net Q6: now also DSP-BP1-3.2 (Pin_2); no longer DSP-BP1-3.4 (Pin_4)
- net Q7: now also DSP-BP1-3.3 (Pin_3); no longer DSP-BP1-3.5 (Pin_5)
- net Q8: now also DSP-BP1-3.4 (Pin_4); no longer DSP-BP1-3.6 (Pin_6)
- net Q9: now also DSP-BP1-3.5 (Pin_5); no longer DSP-BP1-3.7 (Pin_7)
- no-connect marks 46 -> 54
Other:
- note removed: "A Register"
- note removed: "BP1"
- note removed: "BP2"
- note removed: "BP3"
- note removed: "G Register"
- note removed: "J Register"
- note removed: "M Register"
- note removed: "P Register"
- note removed: "Q Register"
- moved on the sheet: DSP-BP1-1, DSP-BP1-2, DSP-BP1-3, DSP-BP1-4, DSP-BP1-5, JSKT2, JSKT3
