File: KiCad/Real903/Sockets/Sockets.kicad_pcb (KiCad board)
At the start: 2 copper layers, 4 parts

Commit message: July 20th
Parts:
- removed J1: ~, ELLIOTT:MC61
- removed J2, J3, J4: ~, Connector_IDC:IDC-Header_2x10_P2.54mm_Horizontal_Lock
- added JSKT1: Circ61, ELLIOTT:MC61, F.Cu at (50.0, 45.0)
- added JSKT1-1: ~, Connector_IDC:IDC-Header_2x10_P2.54mm_Horizontal_Lock, F.Cu at (29.6, 150.1)
- added JSKT1-2: ~, Connector_IDC:IDC-Header_2x10_P2.54mm_Horizontal_Lock, F.Cu at (31.3, 201.4)
- added JSKT1-3: ~, Connector_IDC:IDC-Header_2x10_P2.54mm_Horizontal_Lock, F.Cu at (59.1, 149.9)
- added JSKT10: Circ32, ELLIOTT:MC32, F.Cu at (100.0, 100.0)
- added JSKT11: Circ41, ELLIOTT:MC41, F.Cu at (350.0, 100.0)
- added JSKT13: Circ19, ELLIOTT:MC19, F.Cu at (250.0, 100.0)
- added JSKT2: Circ61, ELLIOTT:MC61, F.Cu at (100.0, 45.0)
- added JSKT2-1: ~, Connector_IDC:IDC-Header_2x10_P2.54mm_Horizontal_Lock, F.Cu at (88.8, 200.8)
- added JSKT2-2: ~, Connector_IDC:IDC-Header_2x10_P2.54mm_Horizontal_Lock, F.Cu at (109.1, 149.8)
- added JSKT2-3: ~, Connector_IDC:IDC-Header_2x10_P2.54mm_Horizontal_Lock, F.Cu at (109.1, 200.9)
- added JSKT3: Circ61, ELLIOTT:MC61, F.Cu at (150.0, 45.0)
- added JSKT4: Circ61, ELLIOTT:MC61, F.Cu at (250.0, 45.0)
- added JSKT4-1: ~, Connector_IDC:IDC-Header_2x10_P2.54mm_Horizontal_Lock, F.Cu at (239.9, 148.8)
- added JSKT5: Circ41, ELLIOTT:MC41, F.Cu at (350.0, 45.0)
- added JSKT6: Circ19, ELLIOTT:MC19, F.Cu at (150.0, 100.0)
- added JSKT7: Circ32, ELLIOTT:MC32, F.Cu at (50.0, 100.0)
Routing:
- net /GND: track 0.00 -> 410.3 mm, vias 0 -> 2
- net /0v: track 0.00 -> 373.9 mm, vias 0 -> 1
- net /On-Light: track 0.00 -> 285.3 mm
- net /Off: track 0.00 -> 254.8 mm
- net /+6v: track 0.00 -> 252.8 mm
- net /Off-Light: track 0.00 -> 244.4 mm
- net /On-Off-Common: track 0.00 -> 241.9 mm
- net /On: track 0.00 -> 239.8 mm
- net Net-(JSKT2-3-Pad5): track 0.00 -> 227.0 mm
- net Net-(JSKT2-3-Pad10): track 0.00 -> 221.1 mm, vias 0 -> 1
- net Net-(JSKT2-3-Pad6): track 0.00 -> 211.6 mm, vias 0 -> 1
- net Net-(JSKT2-1-Pad4): track 0.00 -> 210.5 mm, vias 0 -> 1
- net Net-(JSKT1-2-Pad9): track 0.00 -> 209.9 mm
- net Net-(JSKT1-2-Pad8): track 0.00 -> 207.5 mm
- net Net-(JSKT1-2-Pad13): track 0.00 -> 201.7 mm
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Other:
- board outline added: 380 x 230 mm

Commit message: August 2
Parts:
- added J1: ~, Connector_PinSocket_2.00mm:PinSocket_1x02_P2.00mm_Horizontal, B.Cu at (145.8, 30.9)
- added J2: ~, Connector_PinSocket_2.00mm:PinSocket_1x03_P2.00mm_Horizontal, B.Cu at (186.1, 33.2)
- added J3: ~, Connector_PinSocket_2.00mm:PinSocket_1x03_P2.00mm_Horizontal, B.Cu at (169.4, 33.2)
- added J4: ~, Connector_PinSocket_2.00mm:PinSocket_1x03_P2.00mm_Horizontal, B.Cu at (200.2, 33.6)
- added J5: ~, Connector_PinSocket_2.00mm:PinSocket_1x02_P2.00mm_Horizontal, B.Cu at (131.4, 31.3)
- added JSKT1-4: ~, Connector_IDC:IDC-Header_2x10_P2.54mm_Horizontal_Lock, B.Cu at (32.7, 229.3)
- added JSKT10-1: ~, Connector_IDC:IDC-Header_2x10_P2.54mm_Horizontal_Lock, B.Cu at (138.9, 230.7)
- added JSKT11-1: ~, Connector_IDC:IDC-Header_2x10_P2.54mm_Horizontal_Lock, B.Cu at (336.0, 183.7)
- added JSKT2-4: ~, Connector_IDC:IDC-Header_2x10_P2.54mm_Horizontal_Lock, B.Cu at (87.1, 229.3)
- added JSKT3-1: ~, Connector_IDC:IDC-Header_2x10_P2.54mm_Horizontal_Lock, B.Cu at (184.0, 83.1)
- added JSKT3-2: ~, Connector_IDC:IDC-Header_2x10_P2.54mm_Horizontal_Lock, B.Cu at (361.3, 39.2)
- added JSKT4-2: ~, Connector_IDC:IDC-Header_2x10_P2.54mm_Horizontal_Lock, B.Cu at (239.3, 184.1)
- added JSKT4-3: ~, Connector_IDC:IDC-Header_2x10_P2.54mm_Horizontal_Lock, B.Cu at (287.5, 183.4)
- JSKT1-1, JSKT1-2, JSKT1-3, JSKT2-1, JSKT2-2, JSKT2-3, JSKT4-1: moved to B.Cu
- moved JSKT2-1 164.6 mm to (112.0, 37.8), turned to 90 degrees
- moved JSKT1-1 116.8 mm to (60.5, 37.5), turned to 90 degrees
- moved JSKT4-1 112.2 mm to (258.3, 38.1), turned to 90 degrees
- moved JSKT1-3 49.3 mm to (33.3, 192.0), turned to 270 degrees
- moved JSKT1-2 49.1 mm to (34.0, 152.3), turned to 270 degrees
- moved JSKT2-3 21.9 mm to (88.7, 192.6), turned to 270 degrees
- moved JSKT2-2 20.2 mm to (89.1, 152.3), turned to 270 degrees
- moved JSKT1 20.0 mm to (50.0, 65.0)
- moved JSKT10 20.0 mm to (100.0, 120.0)
- moved JSKT11 20.0 mm to (350.0, 120.0)
- moved JSKT13 20.0 mm to (250.0, 120.0)
- moved JSKT2 20.0 mm to (100.0, 65.0)
- moved JSKT3 20.0 mm to (150.0, 65.0)
- moved JSKT4 20.0 mm to (250.0, 65.0)
- moved JSKT5 20.0 mm to (350.0, 65.0)
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Connections:
- JSKT1 pad JJ: (no net) -> #X-57-D
- JSKT1 pad KK: (no net) -> #Y-57-Z
- JSKT1 pad LL: (no net) -> #SOP-30-P
- JSKT1 pad MM: (no net) -> #SIP-30-Z
- JSKT1 pad NN: (no net) -> #STP-30-L
- JSKT1 pad PP: (no net) -> #STR-30-H
- JSKT10 pad A: (no net) -> Net-(JSKT10-1-Pad1)
- JSKT10 pad B: (no net) -> Net-(JSKT10-1-Pad2)
- JSKT10 pad C: (no net) -> Net-(JSKT10-1-Pad3)
- JSKT10 pad D: (no net) -> Net-(JSKT10-1-Pad4)
- JSKT10 pad E: (no net) -> Net-(JSKT10-1-Pad5)
- JSKT10 pad F: (no net) -> Net-(JSKT10-1-Pad6)
- JSKT10 pad G: (no net) -> Net-(JSKT10-1-Pad7)
- JSKT10 pad H: (no net) -> Net-(JSKT10-1-Pad8)
- JSKT10 pad J: (no net) -> Net-(JSKT10-1-Pad9)
- JSKT10 pad K: (no net) -> Net-(JSKT10-1-Pad10)
- JSKT10 pad L: (no net) -> Net-(JSKT10-1-Pad11)
- JSKT10 pad M: (no net) -> Net-(JSKT10-1-Pad12)
- JSKT10 pad N: (no net) -> Net-(JSKT10-1-Pad13)
- JSKT10 pad P: (no net) -> Net-(JSKT10-1-Pad14)
- JSKT10 pad R: (no net) -> Net-(JSKT10-1-Pad15)
- JSKT10 pad S: (no net) -> Net-(JSKT10-1-Pad16)
- JSKT10 pad T: (no net) -> /GND
- JSKT10 pad U: (no net) -> P3-32-18
- JSKT10 pad V: (no net) -> STR-30-14
- JSKT10 pad W: (no net) -> RTR-30-D
- JSKT10 pad X: (no net) -> P1-32-17
- JSKT10 pad Y: (no net) -> P2-32-15
- JSKT10 pad Z: (no net) -> /AUT
- JSKT10 pad a: (no net) -> /PUNCH-INT
- JSKT10 pad b: (no net) -> P4-32-19
- JSKT10 pad c: (no net) -> /RDR-INT
- JSKT10 pad d: (no net) -> RESET-31-16
- JSKT10 pad e: (no net) -> /0v
- JSKT10 pad f: (no net) -> /+24v
- JSKT10 pad g: (no net) -> /-24v
- JSKT10 pad h: (no net) -> STP_30_15
- JSKT10 pad j: (no net) -> RTP-30-C
- JSKT11 pad A: (no net) -> /GND
- JSKT11 pad B: (no net) -> /W1
- JSKT11 pad C: (no net) -> /~W~2
- JSKT11 pad D: (no net) -> /~W~3
- JSKT11 pad E: (no net) -> /~W~4
- JSKT11 pad F: (no net) -> /W5
- JSKT11 pad G: (no net) -> /W6
- JSKT11 pad H: (no net) -> /W7
- JSKT11 pad J: (no net) -> /W8
- JSKT11 pad K: (no net) -> /W9
- JSKT11 pad L: (no net) -> /W10
- JSKT11 pad M: (no net) -> /W11
- JSKT11 pad N: (no net) -> /W12
- JSKT11 pad P: (no net) -> /W13
- JSKT11 pad R: (no net) -> /~W~14
- JSKT11 pad S: (no net) -> /~W~15
- JSKT11 pad T: (no net) -> /~W~16
- JSKT11 pad U: (no net) -> /~W~17
- JSKT11 pad V: (no net) -> /~W~18
- JSKT11 pad W: (no net) -> INT1-3-9
- JSKT11 pad X: (no net) -> INT2-3-10
- JSKT11 pad Y: (no net) -> INT3-3-11
- JSKT11 pad Z: (no net) -> /AUT
- JSKT11 pad e: (no net) -> /0v
- JSKT11 pad f: (no net) -> ONG-1-7
- JSKT11 pad g: (no net) -> ~ONG~-1-F
- JSKT11 pad h: (no net) -> ENG-1-6
- JSKT11 pad i: (no net) -> ~ENG~-1-4
- JSKT11 pad j: (no net) -> RESET-1-24
- JSKT11 pad m: (no net) -> PS1-3-E
- JSKT11 pad n: (no net) -> PS2-3-L
- JSKT11 pad p: (no net) -> PS3-3-S
- JSKT11 pad q: (no net) -> /W17
- JSKT11 pad r: (no net) -> /Auto-Start
- JSKT11 pad s: (no net) -> /Auto-Start
- JSKT11 pad t: (no net) -> /+6v
- JSKT13 pad A: (no net) -> PI1-29-AE
- JSKT13 pad C: (no net) -> PI2-29-AF
- JSKT13 pad E: (no net) -> PI3-29-AH
- JSKT13 pad G: (no net) -> SOP-30-20
- JSKT13 pad J: (no net) -> SIP-30-21
- JSKT13 pad L: (no net) -> PR-30-E
- JSKT13 pad N: (no net) -> BT-30-U
- JSKT13 pad R: (no net) -> LW-30-13
- JSKT13 pad T: (no net) -> /PUNCH-INT
- JSKT13 pad V: (no net) -> /RDR-INT
- JSKT2 pad AA: (no net) -> /#PC2
- JSKT2 pad BB: (no net) -> /#PC3
- JSKT2 pad CC: (no net) -> /#PC4
- JSKT2 pad DD: (no net) -> /#PC5
- JSKT2 pad EE: (no net) -> /#PC6
- JSKT2 pad FF: (no net) -> /#PC7
- JSKT2 pad GG: (no net) -> /#PC8
- JSKT2 pad HH: (no net) -> /#PC9
- JSKT2 pad JJ: (no net) -> /#PC10
- JSKT2 pad KK: (no net) -> /#PC11
- JSKT2 pad LL: (no net) -> /#PC12
- JSKT2 pad NN: /+6v -> /+5vDisplay
- JSKT2 pad PP: /-6v -> (no net)
- JSKT2 pad ~z~: (no net) -> /#PC1
- JSKT2-1 pad 20: (no net) -> /W1
- JSKT2-3 pad 12: (no net) -> /W5
- JSKT2-3 pad 13: (no net) -> /W6
- JSKT2-3 pad 14: (no net) -> /W7
- JSKT2-3 pad 15: (no net) -> /W8
- JSKT2-3 pad 16: (no net) -> /W9
- JSKT2-3 pad 17: (no net) -> /W10
- JSKT2-3 pad 18: (no net) -> /W11
- JSKT2-3 pad 19: (no net) -> /W12
- JSKT2-3 pad 20: (no net) -> /W13
- JSKT3 pad AA: (no net) -> #AA2-21-X
- JSKT3 pad BB: (no net) -> #AA3-21-AA
- JSKT3 pad DD: (no net) -> #CA-7-Z
- JSKT3 pad EE: (no net) -> #CB-7-V
- JSKT3 pad FF: (no net) -> #C-6-N
- JSKT3 pad GG: (no net) -> #CD-6-V
- JSKT3 pad HH: (no net) -> #RESET-2-Z
- JSKT3 pad JJ: (no net) -> #STOP-2-T
- JSKT3 pad KK: (no net) -> #NOTRDY-2-AC
- JSKT3 pad MM: /+6v -> /+5vDisplay
- JSKT3 pad NN: /-6v -> (no net)
- JSKT3 pad PP: /0v -> /0vDisplay
- JSKT3 pad ~q~: (no net) -> #FD-6-S
- JSKT3 pad ~v~: (no net) -> #AA1'-21-K
- JSKT3 pad ~w~: (no net) -> #AA2'-21-U
- JSKT3 pad ~x~: (no net) -> #AA3'-21-AF
- JSKT3 pad ~z~: (no net) -> #AA1-21-M
- JSKT4 pad AA: (no net) -> Net-(JSKT4-3-Pad11)
- JSKT4 pad BB: (no net) -> Net-(JSKT4-3-Pad12)
- JSKT4 pad CC: (no net) -> Net-(JSKT4-3-Pad13)
- JSKT4 pad DD: (no net) -> Net-(JSKT4-3-Pad14)
- JSKT4 pad EE: (no net) -> Net-(JSKT4-3-Pad15)
- JSKT4 pad FF: (no net) -> Net-(JSKT4-3-Pad16)
- JSKT4 pad GG: (no net) -> Net-(JSKT4-3-Pad17)
- JSKT4 pad HH: (no net) -> Net-(JSKT4-3-Pad18)
- JSKT4 pad PP: (no net) -> RESET-32-20
- JSKT4 pad W: (no net) -> Net-(JSKT4-2-Pad1)
- JSKT4 pad X: (no net) -> Net-(JSKT4-2-Pad2)
- JSKT4 pad Y: (no net) -> Net-(JSKT4-2-Pad3)
- JSKT4 pad Z: (no net) -> Net-(JSKT4-2-Pad4)
- JSKT4 pad ~a~: (no net) -> Net-(JSKT4-2-Pad5)
- JSKT4 pad ~b~: (no net) -> Net-(JSKT4-2-Pad6)
- JSKT4 pad ~c~: (no net) -> Net-(JSKT4-2-Pad7)
- JSKT4 pad ~d~: (no net) -> Net-(JSKT4-2-Pad8)
- JSKT4 pad ~e~: (no net) -> Net-(JSKT4-2-Pad9)
- JSKT4 pad ~f~: (no net) -> Net-(JSKT4-2-Pad10)
- JSKT4 pad ~g~: (no net) -> Net-(JSKT4-2-Pad11)
- JSKT4 pad ~q~: (no net) -> Net-(JSKT4-3-Pad1)
- JSKT4 pad ~r~: (no net) -> Net-(JSKT4-3-Pad2)
- JSKT4 pad ~s~: (no net) -> Net-(JSKT4-3-Pad3)
- JSKT4 pad ~t~: (no net) -> Net-(JSKT4-3-Pad4)
- JSKT4 pad ~u~: (no net) -> Net-(JSKT4-3-Pad5)
- JSKT4 pad ~v~: (no net) -> Net-(JSKT4-3-Pad6)
- JSKT4 pad ~w~: (no net) -> Net-(JSKT4-3-Pad7)
- JSKT4 pad ~x~: (no net) -> Net-(JSKT4-3-Pad8)
- JSKT4 pad ~y~: (no net) -> Net-(JSKT4-3-Pad9)
- JSKT4 pad ~z~: (no net) -> Net-(JSKT4-3-Pad10)
- JSKT5 pad D: (no net) -> ~TEST~-1-5
- JSKT5 pad H: (no net) -> RESET-2-U
- JSKT5 pad P: (no net) -> ~STOP~-1-25
- JSKT5 pad R: (no net) -> #STOP-2-E
- JSKT5 pad T: (no net) -> RESTART-1-C
- JSKT5 pad U: (no net) -> ~RESTART~-1-3
- JSKT5 pad V: (no net) -> JUMP-1-M
- JSKT5 pad W: (no net) -> ~JUMP~-1-11
- JSKT5 pad X: (no net) -> #ACTIVE1-1-Y
- JSKT5 pad Y: (no net) -> #INT1-3-F
- JSKT5 pad Z: (no net) -> #ACTIVE2-1-V
- JSKT5 pad a: (no net) -> #INT2-3-W
- JSKT5 pad b: (no net) -> CINS-1-J
- JSKT5 pad c: (no net) -> ~CINS~-1-8
- JSKT5 pad d: (no net) -> ~TCS~-1-AB
- JSKT5 pad e: (no net) -> ~CS~-1-H
- JSKT5 pad f: (no net) -> ~OS~-1-19
- JSKT5 pad g: (no net) -> #ACTIVE3-1-S
- JSKT5 pad h: (no net) -> #INT3-3-AD
- JSKT5 pad i: (no net) -> ~SMN~-4-7
- JSKT5 pad k: (no net) -> AUTO-1-L
- JSKT5 pad p: (no net) -> AUDIO-32-14
- JSKT5 pad q: (no net) -> /0v
- JSKT5 pad r: (no net) -> /0v
- JSKT5 pad s: (no net) -> /+6v
- JSKT5 pad t: (no net) -> /-6v
- JSKT6 pad B: (no net) -> /Auto-Start
- JSKT6 pad U: (no net) -> /0vDisplay
- JSKT6 pad V: (no net) -> /+5vDisplay
- JSKT7 pad A: (no net) -> /GND
- JSKT7 pad B: (no net) -> /-6v
- JSKT7 pad C: (no net) -> /-6v
- JSKT7 pad D: (no net) -> /-6v
- JSKT7 pad F: (no net) -> /VREF
- JSKT7 pad G: (no net) -> /0v
- JSKT7 pad J: (no net) -> MARGIN-30-10
- JSKT7 pad K: (no net) -> MARGIN-4-3
- JSKT7 pad L: (no net) -> MARGIN-25-12
Routing:
- net /GND: track 410.3 -> 0.00 mm, vias 2 -> 0
- net /0v: track 373.9 -> 0.00 mm, vias 1 -> 0
- net /On-Light: track 285.3 -> 0.00 mm
- net /Off: track 254.8 -> 0.00 mm
- net /+6v: track 252.8 -> 0.00 mm
- net /Off-Light: track 244.4 -> 0.00 mm
- net /On-Off-Common: track 241.9 -> 0.00 mm
- net /On: track 239.8 -> 0.00 mm
- net Net-(JSKT2-3-Pad5): track 227.0 -> 0.00 mm
- net Net-(JSKT2-3-Pad10): track 221.1 -> 0.00 mm, vias 1 -> 0
- net Net-(JSKT2-3-Pad6): track 211.6 -> 0.00 mm, vias 1 -> 0
- net Net-(JSKT2-1-Pad4): track 210.5 -> 0.00 mm, vias 1 -> 0
- net Net-(JSKT1-2-Pad9): track 209.9 -> 0.00 mm
- net Net-(JSKT1-2-Pad8): track 207.5 -> 0.00 mm
- net Net-(JSKT1-2-Pad13): track 201.7 -> 0.00 mm
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
Commit message: August 15
Parts:
- removed J5: ~, Connector_PinSocket_2.00mm:PinSocket_1x02_P2.00mm_Horizontal
- removed JSKT1-4, JSKT2-4, JSKT3-2: ~, Connector_IDC:IDC-Header_2x10_P2.54mm_Horizontal_Lock
- added J0: ~, Connector_IDC:IDC-Header_2x03_P2.54mm_Vertical, F.Cu at (184.2, 48.3)
- added JSKT10-2: ~, Connector_IDC:IDC-Header_2x10_P2.54mm_Vertical, F.Cu at (165.1, 118.1)
- added JSKT11-2: ~, Connector_IDC:IDC-Header_2x10_P2.54mm_Vertical, F.Cu at (379.7, 81.3)
- added JSKT5-1: ~, Connector_IDC:IDC-Header_2x10_P2.54mm_Vertical, F.Cu at (339.1, 16.5)
- J1: footprint Connector_PinSocket_2.00mm:PinSocket_1x02_P2.00mm_Horizontal -> Connector_IDC:IDC-Header_2x07_P2.54mm_Vertical; moved to F.Cu
- J2: footprint Connector_PinSocket_2.00mm:PinSocket_1x03_P2.00mm_Horizontal -> Connector_IDC:IDC-Header_2x07_P2.54mm_Vertical; moved to F.Cu
- J3: footprint Connector_PinSocket_2.00mm:PinSocket_1x03_P2.00mm_Horizontal -> Connector_IDC:IDC-Header_2x03_P2.54mm_Vertical; moved to F.Cu
- J4: footprint Connector_PinSocket_2.00mm:PinSocket_1x03_P2.00mm_Horizontal -> Connector_IDC:IDC-Header_2x06_P2.54mm_Vertical; moved to F.Cu
- JSKT1: value Circ61 -> ~; moved to B.Cu
- JSKT1-1, JSKT1-2, JSKT1-3, JSKT10-1, JSKT11-1, JSKT2-1, JSKT2-2, JSKT2-3, JSKT3-1, JSKT4-1, JSKT4-2, JSKT4-3: footprint Connector_IDC:IDC-Header_2x10_P2.54mm_Horizontal_Lock -> Connector_IDC:IDC-Header_2x10_P2.54mm_Vertical; moved to F.Cu
- JSKT10, JSKT11, JSKT13, JSKT2, JSKT3, JSKT4, JSKT5, JSKT6, JSKT7: moved to B.Cu
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Connections:
- net /~W~17 renamed /Control Unit/~W~17
- net INT2-3-10 renamed /Control Unit/INT2-3-10
- net MARGIN-30-10 renamed /TapePSUMargins/MARGIN-30-10
- net Net-(JSKT1-2-Pad1) renamed /Display/A1
- net Net-(JSKT1-2-Pad10) renamed /Display/A10
- net Net-(JSKT1-2-Pad11) renamed /Display/A11
- net Net-(JSKT1-2-Pad12) renamed /Display/A12
- net Net-(JSKT1-2-Pad13) renamed /Display/A13
- net Net-(JSKT1-2-Pad14) renamed /Display/A14
- net Net-(JSKT1-2-Pad15) renamed /Display/A15
- net Net-(JSKT1-2-Pad16) renamed /Display/A16
- net Net-(JSKT1-2-Pad17) renamed /Display/A17
- net Net-(JSKT1-2-Pad18) renamed /Display/A18
- net Net-(JSKT1-2-Pad2) renamed /Display/A2
- net Net-(JSKT1-2-Pad3) renamed /Display/A3
- net Net-(JSKT1-2-Pad4) renamed /Display/A4
- net Net-(JSKT1-2-Pad5) renamed /Display/A5
- net Net-(JSKT1-2-Pad6) renamed /Display/A6
- net Net-(JSKT1-2-Pad7) renamed /Display/A7
- net Net-(JSKT1-2-Pad8) renamed /Display/A8
- net Net-(JSKT1-2-Pad9) renamed /Display/A9
- net Net-(JSKT2-1-Pad1) renamed /Display/M1
- net Net-(JSKT2-1-Pad10) renamed /Display/M10
- net Net-(JSKT2-1-Pad11) renamed /Display/M11
- net Net-(JSKT2-1-Pad12) renamed /Display/M12
- net Net-(JSKT2-1-Pad13) renamed /Display/M13
- net Net-(JSKT2-1-Pad14) renamed /Display/M14
- net Net-(JSKT2-1-Pad15) renamed /Display/M15
- net Net-(JSKT2-1-Pad16) renamed /Display/M16
- net Net-(JSKT2-1-Pad17) renamed /Display/M17
- net Net-(JSKT2-1-Pad18) renamed /Display/M18
- net Net-(JSKT2-1-Pad2) renamed /Display/M2
- net Net-(JSKT2-1-Pad3) renamed /Display/M3
- net Net-(JSKT2-1-Pad4) renamed /Display/M4
- net Net-(JSKT2-1-Pad5) renamed /Display/M5
- net Net-(JSKT2-1-Pad6) renamed /Display/M6
- net Net-(JSKT2-1-Pad7) renamed /Display/M7
- net Net-(JSKT2-1-Pad8) renamed /Display/M8
- net Net-(JSKT2-1-Pad9) renamed /Display/M9
- net Net-(JSKT4-1-Pad1) renamed /IO/OA1
- net Net-(JSKT4-1-Pad10) renamed /IO/OA10
- net Net-(JSKT4-1-Pad11) renamed /IO/OA11
- net Net-(JSKT4-1-Pad12) renamed /IO/OA12
- net Net-(JSKT4-1-Pad13) renamed /IO/OA13
- net Net-(JSKT4-1-Pad14) renamed /IO/OA14
- net Net-(JSKT4-1-Pad15) renamed /IO/OA15
- net Net-(JSKT4-1-Pad16) renamed /IO/OA16
- net Net-(JSKT4-1-Pad17) renamed /IO/OA17
- net Net-(JSKT4-1-Pad18) renamed /IO/OA18
- net Net-(JSKT4-1-Pad2) renamed /IO/OA2
- net Net-(JSKT4-1-Pad3) renamed /IO/OA3
- net Net-(JSKT4-1-Pad4) renamed /IO/OA4
- net Net-(JSKT4-1-Pad5) renamed /IO/OA5
- net Net-(JSKT4-1-Pad6) renamed /IO/OA6
- net Net-(JSKT4-1-Pad7) renamed /IO/OA7
- net Net-(JSKT4-1-Pad8) renamed /IO/OA8
- net Net-(JSKT4-1-Pad9) renamed /IO/OA9
- net Net-(JSKT4-3-Pad1) renamed /IO/IG1
- net Net-(JSKT4-3-Pad10) renamed /IO/IG10
- net Net-(JSKT4-3-Pad11) renamed /IO/IG11
- net Net-(JSKT4-3-Pad12) renamed /IO/IG12
- net Net-(JSKT4-3-Pad13) renamed /IO/IG13
- net Net-(JSKT4-3-Pad14) renamed /IO/IG14
- net Net-(JSKT4-3-Pad15) renamed /IO/IG15
- net Net-(JSKT4-3-Pad16) renamed /IO/IG16
- net Net-(JSKT4-3-Pad17) renamed /IO/IG17
- net Net-(JSKT4-3-Pad18) renamed /IO/IG18
- net Net-(JSKT4-3-Pad2) renamed /IO/IG2
- net Net-(JSKT4-3-Pad3) renamed /IO/IG3
- net Net-(JSKT4-3-Pad4) renamed /IO/IG4
- net Net-(JSKT4-3-Pad5) renamed /IO/IG5
- net Net-(JSKT4-3-Pad6) renamed /IO/IG6
- net Net-(JSKT4-3-Pad7) renamed /IO/IG7
- net Net-(JSKT4-3-Pad8) renamed /IO/IG8
- net Net-(JSKT4-3-Pad9) renamed /IO/IG9
- J1 pad 1: /+24v -> /TapePSUMargins/+24v
- J1 pad 2: /-24v -> /TapePSUMargins/-24v
- J2 pad 1: /+6v -> /IO/RDR-INT
- J2 pad 2: /0v -> /Display/+5vDisplay
- J2 pad 3: /-6v -> /IO/PUNCH-INT
- J3 pad 1: /+6v -> /IO/RDR-INT
- J3 pad 2: /0v -> GND
- J3 pad 3: /-6v -> /IO/PUNCH-INT
- J4 pad 1: /+6v -> GND
- J4 pad 2: /0v -> /Control Unit/-6v
- J4 pad 3: /-6v -> /Control Unit/On
- JSKT1 pad A: /GND -> GND
- JSKT1 pad AA: Net-(JSKT1-3-Pad11) -> /Display/Q11
- JSKT1 pad B: Net-(JSKT1-1-Pad1) -> /Display/G1
- JSKT1 pad BB: Net-(JSKT1-3-Pad12) -> /Display/Q12
- JSKT1 pad C: Net-(JSKT1-1-Pad2) -> /Display/G2
- JSKT1 pad CC: Net-(JSKT1-3-Pad13) -> /Display/Q13
- JSKT1 pad D: Net-(JSKT1-1-Pad3) -> /Display/G3
- JSKT1 pad DD: Net-(JSKT1-3-Pad14) -> /Display/Q14
- JSKT1 pad E: Net-(JSKT1-1-Pad4) -> /Display/G4
- JSKT1 pad EE: Net-(JSKT1-3-Pad15) -> /Display/Q15
- JSKT1 pad F: Net-(JSKT1-1-Pad5) -> /Display/G5
- JSKT1 pad FF: Net-(JSKT1-3-Pad16) -> /Display/Q16
- JSKT1 pad G: Net-(JSKT1-1-Pad6) -> /Display/G6
- JSKT1 pad GG: Net-(JSKT1-3-Pad17) -> /Display/Q17
- JSKT1 pad H: Net-(JSKT1-1-Pad7) -> /Display/G7
- JSKT1 pad HH: Net-(JSKT1-3-Pad18) -> /Display/Q18
- JSKT1 pad J: Net-(JSKT1-1-Pad8) -> /Display/G8
- JSKT1 pad JJ: #X-57-D -> /Display/#X-57-D
- JSKT1 pad K: Net-(JSKT1-1-Pad9) -> /Display/G9
- JSKT1 pad KK: #Y-57-Z -> /Display/#Y-57-Z
- JSKT1 pad L: Net-(JSKT1-1-Pad10) -> /Display/G10
- JSKT1 pad LL: #SOP-30-P -> /Display/#SOP-30-P
- JSKT1 pad M: Net-(JSKT1-1-Pad11) -> /Display/G11
- JSKT1 pad MM: #SIP-30-Z -> /Display/#SIP-30-Z
- JSKT1 pad N: Net-(JSKT1-1-Pad12) -> /Display/G12
- JSKT1 pad NN: #STP-30-L -> /Display/#STP-30-L
- JSKT1 pad P: Net-(JSKT1-1-Pad13) -> /Display/G13
- JSKT1 pad PP: #STR-30-H -> /Display/#STR-30-H
- JSKT1 pad R: Net-(JSKT1-1-Pad14) -> /Display/G14
- JSKT1 pad S: Net-(JSKT1-1-Pad15) -> /Display/G15
- JSKT1 pad T: Net-(JSKT1-1-Pad16) -> /Display/G16
- JSKT1 pad U: Net-(JSKT1-1-Pad17) -> /Display/G17
- JSKT1 pad V: Net-(JSKT1-1-Pad18) -> /Display/G18
- JSKT1 pad ~q~: Net-(JSKT1-3-Pad1) -> /Display/Q1
- JSKT1 pad ~r~: Net-(JSKT1-3-Pad2) -> /Display/Q2
- JSKT1 pad ~s~: Net-(JSKT1-3-Pad3) -> /Display/Q3
- JSKT1 pad ~t~: Net-(JSKT1-3-Pad4) -> /Display/Q4
- JSKT1 pad ~u~: Net-(JSKT1-3-Pad5) -> /Display/Q5
- JSKT1 pad ~v~: Net-(JSKT1-3-Pad6) -> /Display/Q6
- JSKT1 pad ~w~: Net-(JSKT1-3-Pad7) -> /Display/Q7
- JSKT1 pad ~x~: Net-(JSKT1-3-Pad8) -> /Display/Q8
- JSKT1 pad ~y~: Net-(JSKT1-3-Pad9) -> /Display/Q9
- JSKT1 pad ~z~: Net-(JSKT1-3-Pad10) -> /Display/Q10
- JSKT1-1 pad 1: Net-(JSKT1-1-Pad1) -> /Display/#STP-30-L
- JSKT1-1 pad 10: Net-(JSKT1-1-Pad10) -> /Display/G8
- JSKT1-1 pad 11: Net-(JSKT1-1-Pad11) -> /Display/G9
- JSKT1-1 pad 12: Net-(JSKT1-1-Pad12) -> /Display/G10
- JSKT1-1 pad 13: Net-(JSKT1-1-Pad13) -> /Display/G11
- JSKT1-1 pad 14: Net-(JSKT1-1-Pad14) -> /Display/G12
- JSKT1-1 pad 15: Net-(JSKT1-1-Pad15) -> /Display/G13
- JSKT1-1 pad 16: Net-(JSKT1-1-Pad16) -> /Display/G14
- JSKT1-1 pad 17: Net-(JSKT1-1-Pad17) -> /Display/G15
- JSKT1-1 pad 18: Net-(JSKT1-1-Pad18) -> /Display/G16
- JSKT1-1 pad 19: (no net) -> /Display/G17
- JSKT1-1 pad 2: Net-(JSKT1-1-Pad2) -> /Display/#STR-30-H
- JSKT1-1 pad 20: (no net) -> /Display/G18
- JSKT1-1 pad 3: Net-(JSKT1-1-Pad3) -> /Display/G1
- JSKT1-1 pad 4: Net-(JSKT1-1-Pad4) -> /Display/G2
- JSKT1-1 pad 5: Net-(JSKT1-1-Pad5) -> /Display/G3
- JSKT1-1 pad 6: Net-(JSKT1-1-Pad6) -> /Display/G4
- JSKT1-1 pad 7: Net-(JSKT1-1-Pad7) -> /Display/G5
- JSKT1-1 pad 8: Net-(JSKT1-1-Pad8) -> /Display/G6
- JSKT1-1 pad 9: Net-(JSKT1-1-Pad9) -> /Display/G7
- JSKT1-2 pad 19: (no net) -> /Display/Q1
- JSKT1-2 pad 20: (no net) -> /Display/Q2
- JSKT1-3 pad 1: Net-(JSKT1-3-Pad1) -> /Display/Q3
- JSKT1-3 pad 10: Net-(JSKT1-3-Pad10) -> /Display/Q12
- JSKT1-3 pad 11: Net-(JSKT1-3-Pad11) -> /Display/Q13
- JSKT1-3 pad 12: Net-(JSKT1-3-Pad12) -> /Display/Q14
- JSKT1-3 pad 13: Net-(JSKT1-3-Pad13) -> /Display/Q15
- JSKT1-3 pad 14: Net-(JSKT1-3-Pad14) -> /Display/Q16
- JSKT1-3 pad 15: Net-(JSKT1-3-Pad15) -> /Display/Q17
- JSKT1-3 pad 16: Net-(JSKT1-3-Pad16) -> /Display/Q18
- JSKT1-3 pad 17: Net-(JSKT1-3-Pad17) -> /Display/#X-57-D
- JSKT1-3 pad 18: Net-(JSKT1-3-Pad18) -> /Display/#Y-57-Z
- JSKT1-3 pad 19: (no net) -> /Display/#SOP-30-P
- JSKT1-3 pad 2: Net-(JSKT1-3-Pad2) -> /Display/Q4
- JSKT1-3 pad 20: (no net) -> /Display/#SIP-30-Z
- JSKT1-3 pad 3: Net-(JSKT1-3-Pad3) -> /Display/Q5
- JSKT1-3 pad 4: Net-(JSKT1-3-Pad4) -> /Display/Q6
- JSKT1-3 pad 5: Net-(JSKT1-3-Pad5) -> /Display/Q7
- JSKT1-3 pad 6: Net-(JSKT1-3-Pad6) -> /Display/Q8
- JSKT1-3 pad 7: Net-(JSKT1-3-Pad7) -> /Display/Q9
- JSKT1-3 pad 8: Net-(JSKT1-3-Pad8) -> /Display/Q10
- JSKT1-3 pad 9: Net-(JSKT1-3-Pad9) -> /Display/Q11
- JSKT10 pad T: /GND -> GND
- JSKT10 pad U: P3-32-18 -> /TapePSUMargins/P3-32-18
- JSKT10 pad V: STR-30-14 -> /TapePSUMargins/STR-30-14
- JSKT10 pad W: RTR-30-D -> /TapePSUMargins/RTR-30-D
- JSKT10 pad X: P1-32-17 -> /TapePSUMargins/P1-32-17
- JSKT10 pad Y: P2-32-15 -> /TapePSUMargins/P2-32-15
- JSKT10 pad Z: /AUT -> /Control Unit/AUT
- JSKT10-1 pad 17: P4-32-19 -> /TapePSUMargins/P4-32-19
- JSKT10-1 pad 18: P3-32-18 -> /TapePSUMargins/P3-32-18
- JSKT10-1 pad 20: (no net) -> /TapePSUMargins/MARGIN-4-3
- JSKT11 pad A: /GND -> GND
- JSKT11 pad B: /W1 -> /Control Unit/W1
- JSKT11 pad C: /~W~2 -> /Control Unit/~W~2
- JSKT11 pad D: /~W~3 -> /Control Unit/~W~3
- JSKT11 pad E: /~W~4 -> /Control Unit/~W~4
- JSKT11 pad F: /W5 -> /Control Unit/W5
- JSKT11 pad G: /W6 -> /Control Unit/W6
- JSKT11 pad H: /W7 -> /Control Unit/W7
- JSKT11 pad J: /W8 -> /Control Unit/W8
- JSKT11 pad K: /W9 -> /Control Unit/W9
- JSKT11 pad L: /W10 -> /Control Unit/W10
- JSKT11 pad M: /W11 -> /Control Unit/W11
- JSKT11 pad N: /W12 -> /Control Unit/W12
- JSKT11 pad P: /W13 -> /Control Unit/W13
- JSKT11 pad R: /~W~14 -> /Control Unit/~W~14
- JSKT11 pad S: /~W~15 -> /Control Unit/~W~15
- JSKT11 pad T: /~W~16 -> /Control Unit/~W~16
- JSKT11 pad V: /~W~18 -> /Control Unit/~W~18
- JSKT11 pad W: INT1-3-9 -> /Control Unit/INT1-3-9
- JSKT11 pad Y: INT3-3-11 -> /Control Unit/INT3-3-11
- JSKT11 pad Z: /AUT -> /Control Unit/AUT
- JSKT11-1 pad 1: /~W~2 -> /Control Unit/W1
- JSKT11-1 pad 10: P3-32-18 -> /Control Unit/W13
- JSKT11-1 pad 11: (no net) -> /Control Unit/~W~2
- JSKT11-1 pad 12: (no net) -> /Control Unit/~W~3
- JSKT11-1 pad 13: (no net) -> /Control Unit/~W~4
- JSKT11-1 pad 14: (no net) -> /Control Unit/~W~14
- JSKT11-1 pad 15: (no net) -> /Control Unit/~W~15
- JSKT11-1 pad 16: (no net) -> /Control Unit/~W~16
- JSKT11-1 pad 18: /W17 -> /Control Unit/~W~18
- JSKT11-1 pad 19: INT3-3-11 -> /Control Unit/INT1-3-9
- JSKT11-1 pad 2: /~W~3 -> /Control Unit/W5
- JSKT11-1 pad 3: /~W~4 -> /Control Unit/W6
- JSKT11-1 pad 4: /~W~14 -> /Control Unit/W7
- JSKT11-1 pad 5: /~W~15 -> /Control Unit/W8
- JSKT11-1 pad 6: /~W~16 -> /Control Unit/W9
- JSKT11-1 pad 7: /~W~18 -> /Control Unit/W10
- JSKT11-1 pad 8: (no net) -> /Control Unit/W11
- JSKT11-1 pad 9: P4-32-19 -> /Control Unit/W12
- JSKT13 pad A: PI1-29-AE -> /IO/PI1-29-AE
- JSKT13 pad B: /0v -> /Control Unit/0v
- JSKT13 pad C: PI2-29-AF -> /IO/PI2-29-AF
- JSKT13 pad D: /0v -> /Control Unit/0v
- JSKT13 pad E: PI3-29-AH -> /IO/PI3-29-AH
- JSKT13 pad F: /0v -> /Control Unit/0v
- JSKT13 pad G: SOP-30-20 -> /IO/SOP-30-20
- JSKT13 pad H: /0v -> /Control Unit/0v
- JSKT13 pad J: SIP-30-21 -> /IO/SIP-30-21
- JSKT13 pad K: /0v -> /Control Unit/0v
- JSKT13 pad L: PR-30-E -> /IO/PR-30-E
- JSKT13 pad M: /0v -> /Control Unit/0v
- JSKT13 pad N: BT-30-U -> /IO/BT-30-U
- JSKT13 pad P: /0v -> /Control Unit/0v
- JSKT13 pad R: LW-30-13 -> /IO/LW-30-13
- JSKT13 pad S: /0v -> /Control Unit/0v
- JSKT13 pad T: /PUNCH-INT -> /IO/PUNCH-INT
- JSKT13 pad U: /0v -> /Control Unit/0v
- JSKT13 pad V: /RDR-INT -> /IO/RDR-INT
- JSKT2 pad A: /GND -> GND
- JSKT2 pad AA: /#PC2 -> /Display/#PC2
- JSKT2 pad BB: /#PC3 -> /Display/#PC3
- JSKT2 pad CC: /#PC4 -> /Display/#PC4
- JSKT2 pad DD: /#PC5 -> /Display/#PC5
- JSKT2 pad EE: /#PC6 -> /Display/#PC6
- JSKT2 pad FF: /#PC7 -> /Display/#PC7
- JSKT2 pad GG: /#PC8 -> /Display/#PC8
- JSKT2 pad HH: /#PC9 -> /Display/#PC9
- JSKT2 pad JJ: /#PC10 -> /Display/#PC10
- JSKT2 pad KK: /#PC11 -> /Display/#PC11
- JSKT2 pad LL: /#PC12 -> /Display/#PC12
- JSKT2 pad MM: /0v -> /Display/0vDisplay
- JSKT2 pad NN: /+5vDisplay -> /Display/+5vDisplay
- JSKT2 pad PP: (no net) -> Net-(JSKT2-PadPP)
- JSKT2 pad W: Net-(JSKT2-2-Pad1) -> /Display/J1
- JSKT2 pad X: Net-(JSKT2-2-Pad2) -> /Display/J2
- JSKT2 pad Y: Net-(JSKT2-2-Pad3) -> /Display/J3
- JSKT2 pad Z: Net-(JSKT2-2-Pad4) -> /Display/J4
- JSKT2 pad ~a~: Net-(JSKT2-2-Pad5) -> /Display/J5
- JSKT2 pad ~b~: Net-(JSKT2-2-Pad6) -> /Display/J6
- JSKT2 pad ~c~: Net-(JSKT2-2-Pad7) -> /Display/J7
- JSKT2 pad ~d~: Net-(JSKT2-2-Pad8) -> /Display/J8
- JSKT2 pad ~e~: Net-(JSKT2-2-Pad9) -> /Display/J9
- JSKT2 pad ~f~: Net-(JSKT2-2-Pad10) -> /Display/J10
- JSKT2 pad ~g~: Net-(JSKT2-2-Pad11) -> /Display/J11
- JSKT2 pad ~h~: Net-(JSKT2-2-Pad12) -> /Display/J12
- JSKT2 pad ~i~: Net-(JSKT2-2-Pad13) -> /Display/J13
- JSKT2 pad ~j~: Net-(JSKT2-2-Pad14) -> /Display/J14
- JSKT2 pad ~k~: Net-(JSKT2-2-Pad15) -> /Display/J15
- JSKT2 pad ~m~: Net-(JSKT2-2-Pad16) -> /Display/J16
- JSKT2 pad ~n~: Net-(JSKT2-3-Pad1) -> /Display/P1
- JSKT2 pad ~p~: Net-(JSKT2-3-Pad2) -> /Display/P2
- JSKT2 pad ~q~: Net-(JSKT2-3-Pad3) -> /Display/P3
- JSKT2 pad ~r~: Net-(JSKT2-3-Pad4) -> /Display/P4
- JSKT2 pad ~s~: Net-(JSKT2-3-Pad5) -> /Display/P5
- JSKT2 pad ~t~: Net-(JSKT2-3-Pad6) -> /Display/P6
- JSKT2 pad ~u~: Net-(JSKT2-3-Pad7) -> /Display/P7
- JSKT2 pad ~v~: Net-(JSKT2-3-Pad8) -> /Display/P8
- JSKT2 pad ~w~: Net-(JSKT2-3-Pad9) -> /Display/P9
- JSKT2 pad ~x~: Net-(JSKT2-3-Pad10) -> /Display/P10
- JSKT2 pad ~y~: Net-(JSKT2-3-Pad11) -> /Display/P11
- JSKT2 pad ~z~: /#PC1 -> /Display/#PC1
- JSKT2-1 pad 19: (no net) -> /Display/J1
- JSKT2-1 pad 20: /W1 -> /Display/J2
- JSKT2-2 pad 1: Net-(JSKT2-2-Pad1) -> /Display/J3
- JSKT2-2 pad 10: Net-(JSKT2-2-Pad10) -> /Display/J12
- JSKT2-2 pad 11: Net-(JSKT2-2-Pad11) -> /Display/J13
- JSKT2-2 pad 12: Net-(JSKT2-2-Pad12) -> /Display/J14
- JSKT2-2 pad 13: Net-(JSKT2-2-Pad13) -> /Display/J15
- JSKT2-2 pad 14: Net-(JSKT2-2-Pad14) -> /Display/J16
- JSKT2-2 pad 15: Net-(JSKT2-2-Pad15) -> /Display/P1
- JSKT2-2 pad 16: Net-(JSKT2-2-Pad16) -> /Display/P2
- JSKT2-2 pad 17: /#I1 -> /Display/P3
- JSKT2-2 pad 18: /#I2 -> /Display/P4
- JSKT2-2 pad 19: /#I3 -> /Display/P5
- JSKT2-2 pad 2: Net-(JSKT2-2-Pad2) -> /Display/J4
- JSKT2-2 pad 20: /#I4 -> /Display/P6
- JSKT2-2 pad 3: Net-(JSKT2-2-Pad3) -> /Display/J5
- JSKT2-2 pad 4: Net-(JSKT2-2-Pad4) -> /Display/J6
- JSKT2-2 pad 5: Net-(JSKT2-2-Pad5) -> /Display/J7
- JSKT2-2 pad 6: Net-(JSKT2-2-Pad6) -> /Display/J8
- JSKT2-2 pad 7: Net-(JSKT2-2-Pad7) -> /Display/J9
- JSKT2-2 pad 8: Net-(JSKT2-2-Pad8) -> /Display/J10
- JSKT2-2 pad 9: Net-(JSKT2-2-Pad9) -> /Display/J11
- JSKT2-3 pad 1: Net-(JSKT2-3-Pad1) -> /Display/P7
- JSKT2-3 pad 10: Net-(JSKT2-3-Pad10) -> /Display/#PC5
- JSKT2-3 pad 11: Net-(JSKT2-3-Pad11) -> /Display/#PC6
- JSKT2-3 pad 12: /W5 -> /Display/#PC7
- JSKT2-3 pad 13: /W6 -> /Display/#PC8
- JSKT2-3 pad 14: /W7 -> /Display/#PC9
- JSKT2-3 pad 15: /W8 -> /Display/#PC10
- JSKT2-3 pad 16: /W9 -> /Display/#PC11
- JSKT2-3 pad 17: /W10 -> /Display/#PC12
- JSKT2-3 pad 18: /W11 -> Net-(JSKT2-3-Pad18)
- JSKT2-3 pad 19: /W12 -> Net-(JSKT2-3-Pad19)
- JSKT2-3 pad 2: Net-(JSKT2-3-Pad2) -> /Display/P8
- JSKT2-3 pad 20: /W13 -> Net-(JSKT2-3-Pad20)
- JSKT2-3 pad 3: Net-(JSKT2-3-Pad3) -> /Display/P9
- JSKT2-3 pad 4: Net-(JSKT2-3-Pad4) -> /Display/P10
- JSKT2-3 pad 5: Net-(JSKT2-3-Pad5) -> /Display/P11
- JSKT2-3 pad 6: Net-(JSKT2-3-Pad6) -> /Display/#PC1
- JSKT2-3 pad 7: Net-(JSKT2-3-Pad7) -> /Display/#PC2
- JSKT2-3 pad 8: Net-(JSKT2-3-Pad8) -> /Display/#PC3
- JSKT2-3 pad 9: Net-(JSKT2-3-Pad9) -> /Display/#PC4
- JSKT3 pad A: /GND -> GND
- JSKT3 pad AA: #AA2-21-X -> /Display/#AA2-21-X
- JSKT3 pad B: (no net) -> Net-(JSKT3-PadB)
- JSKT3 pad BB: #AA3-21-AA -> /Display/#AA3-21-AA
- JSKT3 pad C: (no net) -> Net-(JSKT3-PadC)
- JSKT3 pad CC: (no net) -> Net-(JSKT3-PadCC)
- JSKT3 pad D: (no net) -> Net-(JSKT3-PadD)
- JSKT3 pad DD: #CA-7-Z -> /Display/#CA-7-Z
- JSKT3 pad E: (no net) -> Net-(JSKT3-PadE)
- JSKT3 pad EE: #CB-7-V -> /Display/#CB-7-V
- JSKT3 pad F: (no net) -> Net-(JSKT3-PadF)
- JSKT3 pad FF: #C-6-N -> /Display/#C-6-N
- JSKT3 pad G: (no net) -> Net-(JSKT3-PadG)
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Other:
- board outline removed
- copper layers 2 -> 4
- net class Default: clearance 0.2 -> 0.15; trace_width 0.25 -> 0.2
- rule trace_clearance: 0.2 -> 0.15

Commit message: September 4
Parts:
- removed J0: ~, Connector_IDC:IDC-Header_2x03_P2.54mm_Vertical
- removed J2: ~, Connector_IDC:IDC-Header_2x07_P2.54mm_Vertical
- removed JSKT11, JSKT5: Circ41, ELLIOTT:MC41
- removed JSKT11-1, JSKT11-2, JSKT4-1, JSKT4-2, JSKT4-3, JSKT5-1: ~, Connector_IDC:IDC-Header_2x10_P2.54mm_Vertical
- removed JSKT13: Circ19, ELLIOTT:MC19
- removed JSKT4: Circ61, ELLIOTT:MC61
- J1, J3, J4, JSKT1-1, JSKT1-2, JSKT1-3, JSKT10-1, JSKT10-2, JSKT2-1, JSKT2-2, JSKT2-3, JSKT3-1: moved to B.Cu
- JSKT1, JSKT10, JSKT2, JSKT3, JSKT6, JSKT7: moved to F.Cu
- moved J3 259.1 mm to (40.6, 121.9), turned to 90 degrees
- moved JSKT2-2 73.2 mm to (149.9, 73.7), turned to 90 degrees
- moved JSKT3-1 51.1 mm to (193.0, 15.2)
- moved JSKT10-1 38.3 mm to (88.9, 121.9), turned to 90 degrees
- moved JSKT10-2 37.0 mm to (128.3, 121.9), turned to 90 degrees
- moved J1 35.8 mm to (189.2, 121.9), turned to 90 degrees
- moved J4 35.8 mm to (158.8, 121.9), turned to 90 degrees
- moved JSKT2-3 28.4 mm to (154.9, 15.2)
- moved JSKT1-3 24.4 mm to (39.4, 71.1), turned to 270 degrees
- moved JSKT1-2 17.3 mm to (80.0, 15.2)
- moved JSKT2-1 9.92 mm to (116.8, 15.2), turned to 90 degrees
- moved JSKT1-1 7.62 mm to (43.2, 15.2), turned to 90 degrees
Routing:
- net GND: track 0.00 -> 365.5 mm
- net /Control Unit/+6v: track 0.00 -> 184.0 mm
- net /Control Unit/0v: track 0.00 -> 164.8 mm
- net /Control Unit/-6v: track 0.00 -> 163.0 mm
- net /TapePSUMargins/VREF: track 0.00 -> 133.6 mm
- net /Display/0vDisplay: track 0.00 -> 124.3 mm
- net /TapePSUMargins/+24v: track 0.00 -> 104.7 mm
- net /Display/+5vDisplay: track 0.00 -> 103.9 mm
- net /Display/G9: track 0.00 -> 97.3 mm
- net /TapePSUMargins/-24v: track 0.00 -> 96.9 mm
- net /Display/J6: track 0.00 -> 91.6 mm
- net /Display/J3: track 0.00 -> 89.2 mm
- net /Display/J4: track 0.00 -> 85.7 mm
- net /Display/J5: track 0.00 -> 79.7 mm
- net /Display/G8: track 0.00 -> 76.4 mm
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Other:
- board outline added: 210 x 129.5 mm

Commit message: Convert to KiCad 6
Other:
- net class Default removed

Commit message: Start new layout with IDC connectors
Parts:
- removed J3: ~, Connector_IDC:IDC-Header_2x03_P2.54mm_Vertical
- removed J4: ~, Connector_IDC:IDC-Header_2x06_P2.54mm_Vertical
- removed JSKT1-1, JSKT1-2, JSKT1-3, JSKT10-1, JSKT10-2, JSKT2-1, JSKT2-2, JSKT2-3, JSKT3-1: ~, Connector_IDC:IDC-Header_2x10_P2.54mm_Vertical
- added CNT-BP2-1: ~, Connector_IDC:IDC-Header_2x10_P2.54mm_Vertical, F.Cu at (363.1, 40.0)
- added CNT-BP2-2: ~, Connector_IDC:IDC-Header_2x10_P2.54mm_Vertical, F.Cu at (390.9, 132.7)
- added CNT-BP3-1: ~, Connector_IDC:IDC-Header_2x10_P2.54mm_Vertical, F.Cu at (327.4, 114.6)
- added DSP-BP1-1: ~, Connector_IDC:IDC-Header_2x10_P2.54mm_Vertical, F.Cu at (18.9, 53.8)
- added DSP-BP1-2: ~, Connector_IDC:IDC-Header_2x10_P2.54mm_Vertical, F.Cu at (30.0, 53.8)
- added DSP-BP1-3: ~, Connector_IDC:IDC-Header_2x10_P2.54mm_Vertical, F.Cu at (18.2, 92.5)
- added DSP-BP1-4: ~, Connector_IDC:IDC-Header_2x10_P2.54mm_Vertical, F.Cu at (29.5, 91.8)
- added DSP-BP1-5: ~, Connector_IDC:IDC-Header_2x10_P2.54mm_Vertical, F.Cu at (18.5, 129.5)
- added DSP-BP1-6: ~, Connector_IDC:IDC-Header_2x10_P2.54mm_Vertical, F.Cu at (369.4, 151.7)
- added DSP-BP2-1: ~, Connector_IDC:IDC-Header_2x10_P2.54mm_Vertical, F.Cu at (209.0, 88.2)
- added DSP-BP2-2: ~, Connector_IDC:IDC-Header_2x10_P2.54mm_Vertical, F.Cu at (208.9, 39.7)
- added IO-BP3-1: ~, Connector_IDC:IDC-Header_2x10_P2.54mm_Vertical, F.Cu at (120.6, 151.2)
- added IO-BP3-2: ~, Connector_IDC:IDC-Header_2x10_P2.54mm_Vertical, F.Cu at (286.6, 40.0)
- added IO-BP3-3: ~, Connector_IDC:IDC-Header_2x10_P2.54mm_Vertical, F.Cu at (248.4, 40.0)
- added IO-BP3-4: ~, Connector_IDC:IDC-Header_2x10_P2.54mm_Vertical, F.Cu at (325.4, 39.7)
- added IO-BP3-5: ~, Connector_IDC:IDC-Header_2x10_P2.54mm_Vertical, F.Cu at (78.4, 151.0)
- added J2: Conn_01x10, Connector_Wago:Wago_734-140_1x10_P3.50mm_Vertical, F.Cu at (173.0, 150.5)
- added JSKT11: ~, ELLIOTT:MC41, F.Cu at (358.7, 125.5)
- added JSKT13: ~, ELLIOTT:MC19, F.Cu at (258.7, 125.5)
- added JSKT4: ~, ELLIOTT:MC61, F.Cu at (258.7, 75.5)
- added JSKT5: ~, ELLIOTT:MC41, F.Cu at (358.7, 75.5)
- J1: value ~ -> Conn_01x02; footprint Connector_IDC:IDC-Header_2x07_P2.54mm_Vertical -> Connector_Wago:Wago_734-132_1x02_P3.50mm_Vertical
- JSKT10, JSKT7: value Circ32 -> ~
- JSKT2, JSKT3: value Circ61 -> ~
- JSKT6: value Circ19 -> ~
- moved J1 31.7 mm to (197.9, 152.4)
- moved JSKT1 31.7 mm to (58.7, 75.5)
- moved JSKT10 31.7 mm to (108.7, 125.5)
- moved JSKT2 31.7 mm to (108.7, 75.5)
- moved JSKT3 31.7 mm to (158.7, 75.5)
- moved JSKT6 31.7 mm to (158.7, 125.5)
- moved JSKT7 31.7 mm to (58.7, 125.5)
Connections:
- net /Display/+5vDisplay renamed /Control Unit/PW.+5vDisplay
- net /Display/0vDisplay renamed /Control Unit/PW.0vDisplay
- J1 pad 1: /TapePSUMargins/+24v -> /IO/-24v
- J1 pad 2: /TapePSUMargins/-24v -> /IO/+24v
- JSKT1 pad A: GND -> /Control Unit/PW.GND
- JSKT1 pad LL: /Display/#SOP-30-P -> /Display/S4
- JSKT1 pad MM: /Display/#SIP-30-Z -> /Display/S3
- JSKT1 pad NN: /Display/#STP-30-L -> /Display/S2
- JSKT1 pad PP: /Display/#STR-30-H -> /Display/S1
- JSKT10 pad A: Net-(JSKT10-1-Pad1) -> /IO/IR1
- JSKT10 pad B: Net-(JSKT10-1-Pad2) -> /IO/IR2
- JSKT10 pad C: Net-(JSKT10-1-Pad3) -> /IO/IR3
- JSKT10 pad D: Net-(JSKT10-1-Pad4) -> /IO/IR4
- JSKT10 pad E: Net-(JSKT10-1-Pad5) -> /IO/IR5
- JSKT10 pad F: Net-(JSKT10-1-Pad6) -> /IO/IR6
- JSKT10 pad G: Net-(JSKT10-1-Pad7) -> /IO/IR7
- JSKT10 pad H: Net-(JSKT10-1-Pad8) -> /IO/IR8
- JSKT10 pad J: Net-(JSKT10-1-Pad9) -> /IO/OP1
- JSKT10 pad K: Net-(JSKT10-1-Pad10) -> /IO/OP2
- JSKT10 pad L: Net-(JSKT10-1-Pad11) -> /IO/OP3
- JSKT10 pad M: Net-(JSKT10-1-Pad12) -> /IO/OP4
- JSKT10 pad N: Net-(JSKT10-1-Pad13) -> /IO/OP5
- JSKT10 pad P: Net-(JSKT10-1-Pad14) -> /IO/OP6
- JSKT10 pad R: Net-(JSKT10-1-Pad15) -> /IO/OP7
- JSKT10 pad S: Net-(JSKT10-1-Pad16) -> /IO/OP8
- JSKT10 pad T: GND -> /Control Unit/PW.GND
- JSKT10 pad U: /TapePSUMargins/P3-32-18 -> /IO/P3-32-18
- JSKT10 pad V: /TapePSUMargins/STR-30-14 -> /IO/STR-30-14
- JSKT10 pad W: /TapePSUMargins/RTR-30-D -> /IO/RTR-30-D
- JSKT10 pad X: /TapePSUMargins/P1-32-17 -> /IO/P1-32-17
- JSKT10 pad Y: /TapePSUMargins/P2-32-15 -> /IO/P2-32-15
- JSKT2 pad A: GND -> /Control Unit/PW.GND
- JSKT2 pad PP: Net-(JSKT2-PadPP) -> unconnected-(JSKT2-PadPP)
- JSKT3 pad A: GND -> /Control Unit/PW.GND
- JSKT3 pad B: Net-(JSKT3-PadB) -> unconnected-(JSKT3-PadB)
- JSKT3 pad C: Net-(JSKT3-PadC) -> unconnected-(JSKT3-PadC)
- JSKT3 pad CC: Net-(JSKT3-PadCC) -> unconnected-(JSKT3-PadCC)
- JSKT3 pad D: Net-(JSKT3-PadD) -> unconnected-(JSKT3-PadD)
- JSKT3 pad E: Net-(JSKT3-PadE) -> unconnected-(JSKT3-PadE)
- JSKT3 pad F: Net-(JSKT3-PadF) -> unconnected-(JSKT3-PadF)
- JSKT3 pad G: Net-(JSKT3-PadG) -> unconnected-(JSKT3-PadG)
- JSKT3 pad H: Net-(JSKT3-PadH) -> unconnected-(JSKT3-PadH)
- JSKT3 pad J: Net-(JSKT3-PadJ) -> unconnected-(JSKT3-PadJ)
- JSKT3 pad K: Net-(JSKT3-PadK) -> unconnected-(JSKT3-PadK)
- JSKT3 pad L: Net-(JSKT3-PadL) -> unconnected-(JSKT3-PadL)
- JSKT3 pad LL: Net-(JSKT3-PadLL) -> unconnected-(JSKT3-PadLL)
- JSKT3 pad M: Net-(JSKT3-PadM) -> unconnected-(JSKT3-PadM)
- JSKT3 pad N: Net-(JSKT3-PadN) -> unconnected-(JSKT3-PadN)
- JSKT3 pad NN: Net-(JSKT3-PadNN) -> unconnected-(JSKT3-PadNN)
- JSKT3 pad P: Net-(JSKT3-PadP) -> unconnected-(JSKT3-PadP)
- JSKT3 pad R: Net-(JSKT3-PadR) -> unconnected-(JSKT3-PadR)
- JSKT3 pad S: Net-(JSKT3-PadS) -> unconnected-(JSKT3-PadS)
- JSKT3 pad T: Net-(JSKT3-PadT) -> unconnected-(JSKT3-PadT)
- JSKT3 pad U: Net-(JSKT3-PadU) -> unconnected-(JSKT3-PadU)
- JSKT3 pad V: Net-(JSKT3-PadV) -> unconnected-(JSKT3-PadV)
- JSKT3 pad W: Net-(JSKT3-PadW) -> unconnected-(JSKT3-PadW)
- JSKT3 pad X: Net-(JSKT3-PadX) -> unconnected-(JSKT3-PadX)
- JSKT3 pad Y: Net-(JSKT3-PadY) -> unconnected-(JSKT3-PadY)
- JSKT3 pad Z: Net-(JSKT3-PadZ) -> unconnected-(JSKT3-PadZ)
- JSKT6 pad A: GND -> /Control Unit/PW.GND
- JSKT6 pad B: /Control Unit/Auto-Start -> /Control Unit/PW.Auto-Start
- JSKT6 pad C: /TapePSUMargins/PSC -> /Control Unit/PW.PSC
- JSKT6 pad D: /Control Unit/0v -> /Control Unit/PW.0v
- JSKT6 pad E: /TapePSUMargins/0vA -> /Control Unit/PW.0va
- JSKT6 pad F: /TapePSUMargins/0vB -> /Control Unit/PW.0vb
- JSKT6 pad G: /TapePSUMargins/0vC -> /Control Unit/PW.0vc
- JSKT6 pad H: /Control Unit/On-Off-Common -> /Control Unit/PW.On-Off-Common
- JSKT6 pad J: /Control Unit/On -> /Control Unit/PW.On
- JSKT6 pad K: /Control Unit/Off -> /Control Unit/PW.Off
- JSKT6 pad L: /Control Unit/+6v -> /Control Unit/PW.+6vc
- JSKT6 pad M: /TapePSUMargins/+6vB -> /Control Unit/PW.+6vb
- JSKT6 pad N: /TapePSUMargins/+6vA -> /Control Unit/PW.+6va
- JSKT6 pad P: /Control Unit/-6v -> /Control Unit/PW.-6vb
- JSKT6 pad R: /TapePSUMargins/-6vA -> /Control Unit/PW.-6va
- JSKT6 pad S: /Control Unit/On-Light -> /Control Unit/PW.On-Light
- JSKT6 pad T: /Control Unit/Off-Light -> /Control Unit/PW.Off-Light
- JSKT7 pad A: GND -> /Control Unit/PW.GND
- JSKT7 pad B: /Control Unit/-6v -> /Control Unit/PW.-6va
- JSKT7 pad C: /Control Unit/-6v -> /Control Unit/PW.-6va
- JSKT7 pad D: /Control Unit/-6v -> /Control Unit/PW.-6va
- JSKT7 pad E: Net-(JSKT7-PadE) -> unconnected-(JSKT7-PadE)
- JSKT7 pad F: /TapePSUMargins/VREF -> /PSUMargins/VREF
- JSKT7 pad G: /Control Unit/0v -> /Control Unit/PW.0v
- JSKT7 pad H: Net-(JSKT7-PadH) -> unconnected-(JSKT7-PadH)
- JSKT7 pad J: /TapePSUMargins/MARGIN-30-10 -> /PSUMargins/MARGIN-25-12
- JSKT7 pad K: /TapePSUMargins/MARGIN-4-3 -> /Control Unit/MARGIN-4-3
- JSKT7 pad L: /TapePSUMargins/MARGIN-25-12 -> /IO/MARGIN-30-10
- JSKT7 pad M: Net-(JSKT7-PadM) -> unconnected-(JSKT7-PadM)
- JSKT7 pad N: Net-(JSKT7-PadN) -> unconnected-(JSKT7-PadN)
- JSKT7 pad P: Net-(JSKT7-PadP) -> unconnected-(JSKT7-PadP)
- JSKT7 pad R: Net-(JSKT7-PadR) -> unconnected-(JSKT7-PadR)
- JSKT7 pad S: Net-(JSKT7-PadS) -> unconnected-(JSKT7-PadS)
- JSKT7 pad T: Net-(JSKT7-PadT) -> unconnected-(JSKT7-PadT)
- JSKT7 pad U: Net-(JSKT7-PadU) -> unconnected-(JSKT7-PadU)
- JSKT7 pad V: Net-(JSKT7-PadV) -> unconnected-(JSKT7-PadV)
- JSKT7 pad W: Net-(JSKT7-PadW) -> unconnected-(JSKT7-PadW)
- JSKT7 pad X: Net-(JSKT7-PadX) -> unconnected-(JSKT7-PadX)
- JSKT7 pad Y: Net-(JSKT7-PadY) -> unconnected-(JSKT7-PadY)
- JSKT7 pad Z: Net-(JSKT7-PadZ) -> unconnected-(JSKT7-PadZ)
Routing:
- net GND: track 365.5 -> 0.00 mm
- net /Control Unit/+6v: track 184.0 -> 0.00 mm
- net /Control Unit/0v: track 164.8 -> 0.00 mm
- net /Control Unit/-6v: track 163.0 -> 0.00 mm
- net /TapePSUMargins/VREF: track 133.6 -> 0.00 mm
- net /Control Unit/PW.0vDisplay: track 124.3 -> 0.00 mm
- net /TapePSUMargins/+24v: track 104.7 -> 0.00 mm
- net /Control Unit/PW.+5vDisplay: track 103.9 -> 0.00 mm
- net /Display/G9: track 97.3 -> 0.00 mm
- net /TapePSUMargins/-24v: track 96.9 -> 0.00 mm
- net /Display/J6: track 91.6 -> 0.00 mm
- net /Display/J3: track 89.2 -> 0.00 mm
- net /Display/J4: track 85.7 -> 0.00 mm
- net /Display/J5: track 79.7 -> 0.00 mm
- net /Display/G8: track 76.4 -> 0.00 mm
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Other:
- board size 210 x 129.5 mm -> 400 x 130 mm
