File: KiCad/Real903/Sockets/Sockets.kicad_pcb (KiCad board)
At the start: 4 copper layers, 400 x 130 mm, 28 parts, among them J1 Conn_01x02, J2 Conn_01x10

Commit message: Update to design
Parts:
- added H1: MountingHole, ELLIOTT:MC61_Hole, F.Cu at (258.0, 75.0)
- added H10: MountingHole, ELLIOTT:MC19_Hole, F.Cu at (258.0, 125.0)
- added H2: MountingHole, ELLIOTT:MC61_Hole, F.Cu at (108.0, 75.0)
- added H3: MountingHole, ELLIOTT:MC61_Hole, F.Cu at (58.0, 75.0)
- added H4: MountingHole, ELLIOTT:MC61_Hole, F.Cu at (158.0, 75.0)
- added H5: MountingHole, ELLIOTT:MC19_Hole, F.Cu at (158.0, 125.0)
- added H6: MountingHole, ELLIOTT:MC41_Hole, F.Cu at (358.0, 75.0)
- added H7: MountingHole, ELLIOTT:MC41_Hole, F.Cu at (358.0, 125.0)
- added H8: MountingHole, ELLIOTT:MC32_Hole, F.Cu at (57.0, 125.0)
- added H9: MountingHole, ELLIOTT:MC32_Hole, F.Cu at (108.0, 125.0)
- moved IO-BP3-2 298.2 mm to (80.0, 255.0), turned to 90 degrees
- moved DSP-BP1-5 262.5 mm to (230.0, 285.0), turned to 90 degrees
- moved IO-BP3-4 259.7 mm to (180.0, 255.0), turned to 90 degrees
- moved IO-BP3-3 245.4 mm to (130.0, 255.0), turned to 90 degrees
- moved DSP-BP1-4 244.9 mm to (180.0, 285.0), turned to 90 degrees
- moved DSP-BP2-2 241.0 mm to (280.0, 270.0), turned to 90 degrees
- moved DSP-BP1-2 236.5 mm to (80.0, 285.0), turned to 90 degrees
- moved CNT-BP2-1 232.4 mm to (330.0, 270.0), turned to 90 degrees
- moved DSP-BP1-1 231.4 mm to (30.0, 285.0), turned to 90 degrees
- moved DSP-BP1-3 222.6 mm to (130.0, 285.0), turned to 90 degrees
- moved IO-BP3-5 183.9 mm to (230.0, 255.0), turned to 90 degrees
- moved DSP-BP2-1 183.0 mm to (230.0, 270.0), turned to 90 degrees
- moved DSP-BP1-6 160.4 mm to (280.0, 285.0), turned to 90 degrees
- moved JSKT1 149.5 mm to (58.0, 225.0)
- moved JSKT2 149.5 mm to (108.0, 225.0)
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Routing:
- net /Control Unit/PW.GND: track 0.00 -> 363.3 mm, vias 0 -> 1
- net /IO/PR-30-E: track 0.00 -> 278.3 mm, vias 0 -> 2
- net /IO/BT-30-U: track 0.00 -> 276.9 mm, vias 0 -> 2
- net /Control Unit/PW.0v: track 0.00 -> 276.2 mm, vias 0 -> 2
- net /IO/PI1-29-AE: track 0.00 -> 274.2 mm, vias 0 -> 2
- net /IO/LW-30-13: track 0.00 -> 272.3 mm, vias 0 -> 2
- net /IO/PI3-29-AH: track 0.00 -> 268.4 mm, vias 0 -> 2
- net /Control Unit/PW.+6va: track 0.00 -> 265.4 mm
- net /IO/SOP-30-20: track 0.00 -> 263.9 mm, vias 0 -> 2
- net /Control Unit/AUT: track 0.00 -> 263.1 mm
- net /IO/OA1: track 0.00 -> 222.2 mm, vias 0 -> 1
- net /IO/OA4: track 0.00 -> 213.8 mm, vias 0 -> 1
- net /IO/OA3: track 0.00 -> 210.0 mm, vias 0 -> 1
- net /Control Unit/PW.Auto-Start: track 0.00 -> 209.9 mm
- net /IO/OP8: track 0.00 -> 209.2 mm, vias 0 -> 1
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Other:
- board size 400 x 130 mm -> 419.1 x 266.7 mm
