File: KiCad/Real903/Sockets/Sockets.kicad_sch (KiCad schematic)
At the start: 0 parts

Commit message: Update to design
Parts:
- added H1, H2, H3, H4: MountingHole, ELLIOTT:MC61_Hole, symbol Mechanical:MountingHole
- added H10, H5: MountingHole, ELLIOTT:MC19_Hole, symbol Mechanical:MountingHole
- added H6, H7: MountingHole, ELLIOTT:MC41_Hole, symbol Mechanical:MountingHole
- added H8, H9: MountingHole, ELLIOTT:MC32_Hole, symbol Mechanical:MountingHole
Changed lines of the file:
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@@
     (effects (font (size 1.016 1.016)) (justify left bottom))
+  )
+  (symbol (lib_id "Mechanical:MountingHole") (at 66.675 149.225 0) (unit 1)
+    (in_bom yes) (on_board yes) (fields_autoplaced)
+    (property "Reference" "H5" (id 0) (at 69.215 148.3903 0)
+      (effects (font (size 1.27 1.27)) (justify left))
+    )
+    (property "Value" "MountingHole" (id 1) (at 69.215 150.9272 0)
+      (effects (font (size 1.27 1.27)) (justify left))
+    )
+    (property "Footprint" "ELLIOTT:MC19_Hole" (id 2) (at 66.675 149.225 0)
+      (effects (font (size 1.27 1.27)) hide)
+    )
+    (property "Datasheet" "~" (id 3) (at 66.675 149.225 0)
+      (effects (font (size 1.27 1.27)) hide)
+    )
+  )
+  (symbol (lib_id "Mechanical:MountingHole") (at 90.805 149.225 0) (unit 1)
+    (in_bom yes) (on_board yes) (fields_autoplaced)
+    (property "Reference" "H8" (id 0) (at 93.345 148.3903 0)
+      (effects (font (size 1.27 1.27)) (justify left))
+    )
+    (property "Value" "MountingHole" (id 1) (at 93.345 150.9272 0)
+      (effects (font (size 1.27 1.27)) (justify left))
+    )
+    (property "Footprint" "ELLIOTT:MC32_Hole" (id 2) (at 90.805 149.225 0)
+      (effects (font (size 1.27 1.27)) hide)
+    )
+    (property "Datasheet" "~" (id 3) (at 90.805 149.225 0)
+      (effects (font (size 1.27 1.27)) hide)
+    )
+  )
+  (symbol (lib_id "Mechanical:MountingHole") (at 90.805 140.97 0) (unit 1)
+    (in_bom yes) (on_board yes) (fields_autoplaced)
+    (property "Reference" "H7" (id 0) (at 93.345 140.1353 0)
+      (effects (font (size 1.27 1.27)) (justify left))
+    )
+    (property "Value" "MountingHole" (id 1) (at 93.345 142.6722 0)
+      (effects (font (size 1.27 1.27)) (justify left))
+    )
+    (property "Footprint" "ELLIOTT:MC41_Hole" (id 2) (at 90.805 140.97 0)
+      (effects (font (size 1.27 1.27)) hide)
+    )
+    (property "Datasheet" "~" (id 3) (at 90.805 140.97 0)
+      (effects (font (size 1.27 1.27)) hide)
+    )
+  )
+  (symbol (lib_id "Mechanical:MountingHole") (at 43.815 157.48 0) (unit 1)
+    (in_bom yes) (on_board yes) (fields_autoplaced)
+    (property "Reference" "H3" (id 0) (at 46.355 156.6453 0)
+      (effects (font (size 1.27 1.27)) (justify left))
+    )
+    (property "Value" "MountingHole" (id 1) (at 46.355 159.1822 0)
+      (effects (font (size 1.27 1.27)) (justify left))
+    )
+    (property "Footprint" "ELLIOTT:MC61_Hole" (id 2) (at 43.815 157.48 0)
+      (effects (font (size 1.27 1.27)) hide)
+    )
+    (property "Datasheet" "~" (id 3) (at 43.815 157.48 0)
+      (effects (font (size 1.27 1.27)) hide)
+    )
+  )
+  (symbol (lib_id "Mechanical:MountingHole") (at 43.815 149.225 0) (unit 1)
+    (in_bom yes) (on_board yes) (fields_autoplaced)
+    (property "Reference" "H2" (id 0) (at 46.355 148.3903 0)
+      (effects (font (size 1.27 1.27)) (justify left))
+    )
+    (property "Value" "MountingHole" (id 1) (at 46.355 150.9272 0)
+      (effects (font (size 1.27 1.27)) (justify left))
+    )
+    (property "Footprint" "ELLIOTT:MC61_Hole" (id 2) (at 43.815 149.225 0)
+      (effects (font (size 1.27 1.27)) hide)
+    )
+    (property "Datasheet" "~" (id 3) (at 43.815 149.225 0)
+      (effects (font (size 1.27 1.27)) hide)
+    )
+  )
+  (symbol (lib_id "Mechanical:MountingHole") (at 90.805 157.48 0) (unit 1)
+    (in_bom yes) (on_board yes) (fields_autoplaced)
+    (property "Reference" "H9" (id 0) (at 93.345 156.6453 0)
+      (effects (font (size 1.27 1.27)) (justify left))
+    )
+    (property "Value" "MountingHole" (id 1) (at 93.345 159.1822 0)
+      (effects (font (size 1.27 1.27)) (justify left))
+    )
+    (property "Footprint" "ELLIOTT:MC32_Hole" (id 2) (at 90.805 157.48 0)
+      (effects (font (size 1.27 1.27)) hide)
+    )
+    (property "Datasheet" "~" (id 3) (at 90.805 157.48 0)
+      (effects (font (size 1.27 1.27)) hide)
+    )
+  )
+  (symbol (lib_id "Mechanical:MountingHole") (at 43.815 140.97 0) (unit 1)
+    (in_bom yes) (on_board yes) (fields_autoplaced)
+    (property "Reference" "H1" (id 0) (at 46.355 140.1353 0)
+      (effects (font (size 1.27 1.27)) (justify left))
+    )
+    (property "Value" "MountingHole" (id 1) (at 46.355 142.6722 0)
+      (effects (font (size 1.27 1.27)) (justify left))
+    )
+    (property "Footprint" "ELLIOTT:MC61_Hole" (id 2) (at 43.815 140.97 0)
+      (effects (font (size 1.27 1.27)) hide)
+    )
+    (property "Datasheet" "~" (id 3) (at 43.815 140.97 0)
+      (effects (font (size 1.27 1.27)) hide)
+    )
+  )
+  (symbol (lib_id "Mechanical:MountingHole") (at 66.675 157.48 0) (unit 1)
+    (in_bom yes) (on_board yes) (fields_autoplaced)
+    (property "Reference" "H6" (id 0) (at 69.215 156.6453 0)
+      (effects (font (size 1.27 1.27)) (justify left))
+    )
+    (property "Value" "MountingHole" (id 1) (at 69.215 159.1822 0)
+      (effects (font (size 1.27 1.27)) (justify left))
+    )
+    (property "Footprint" "ELLIOTT:MC41_Hole" (id 2) (at 66.675 157.48 0)
+      (effects (font (size 1.27 1.27)) hide)
+    )
+    (property "Datasheet" "~" (id 3) (at 66.675 157.48 0)
+      (effects (font (size 1.27 1.27)) hide)
+    )
+  )
+  (symbol (lib_id "Mechanical:MountingHole") (at 66.675 140.97 0) (unit 1)
+    (in_bom yes) (on_board yes) (fields_autoplaced)
+    (property "Reference" "H4" (id 0) (at 69.215 140.1353 0)
+      (effects (font (size 1.27 1.27)) (justify left))
+    )
+    (property "Value" "MountingHole" (id 1) (at 69.215 142.6722 0)
+      (effects (font (size 1.27 1.27)) (justify left))
+    )
+    (property "Footprint" "ELLIOTT:MC61_Hole" (id 2) (at 66.675 140.97 0)
+      (effects (font (size 1.27 1.27)) hide)
+    )
+    (property "Datasheet" "~" (id 3) (at 66.675 140.97 0)
+      (effects (font (size 1.27 1.27)) hide)
+    )
+  )
+  (symbol (lib_id "Mechanical:MountingHole") (at 111.125 149.225 0) (unit 1)
+    (in_bom yes) (on_board yes) (fields_autoplaced)
+    (property "Reference" "H10" (id 0) (at 113.665 148.3903 0)
+      (effects (font (size 1.27 1.27)) (justify left))
+    )
+    (property "Value" "MountingHole" (id 1) (at 113.665 150.9272 0)
+      (effects (font (size 1.27 1.27)) (justify left))
+    )
+    (property "Footprint" "ELLIOTT:MC19_Hole" (id 2) (at 111.125 149.225 0)
+      (effects (font (size 1.27 1.27)) hide)
+    )
+    (property "Datasheet" "~" (id 3) (at 111.125 149.225 0)
+      (effects (font (size 1.27 1.27)) hide)
+    )
   )
   (sheet (at 82.55 106.68) (size 44.45 17.78) (fields_autoplaced)
@@
       (reference "DSP-BP2-2") (unit 1) (value "~") (footprint "Connector_IDC:IDC-Header_2x10_P2.54mm_Vertical")
     )
+    (path "/774a50bf-2c68-4055-a943-69d485e86b09"
+      (reference "H1") (unit 1) (value "MountingHole") (footprint "ELLIOTT:MC61_Hole")
+    )
+    (path "/6143e413-5497-406c-9968-6e006f8288ed"
+      (reference "H2") (unit 1) (value "MountingHole") (footprint "ELLIOTT:MC61_Hole")
+    )
+    (path "/5bbba885-36e2-49d0-a991-7df613f99c54"
+      (reference "H3") (unit 1) (value "MountingHole") (footprint "ELLIOTT:MC61_Hole")
+    )
+    (path "/d4fec0c6-d634-46b9-a407-4be843b0f212"
+      (reference "H4") (unit 1) (value "MountingHole") (footprint "ELLIOTT:MC61_Hole")
+    )
+    (path "/4ebd502e-a1c2-4e2e-a396-43a35177ec00"
+      (reference "H5") (unit 1) (value "MountingHole") (footprint "ELLIOTT:MC19_Hole")
+    )
+    (path "/b458a265-a7e4-4e40-a44c-434b79fb0220"
+      (reference "H6") (unit 1) (value "MountingHole") (footprint "ELLIOTT:MC41_Hole")
+    )
+    (path "/554bf7de-6331-496d-87c3-648976b0259d"
+      (reference "H7") (unit 1) (value "MountingHole") (footprint "ELLIOTT:MC41_Hole")
+    )
+    (path "/4ef66951-32cc-4618-84ed-ed3e523f67ee"
+      (reference "H8") (unit 1) (value "MountingHole") (footprint "ELLIOTT:MC32_Hole")
+    )
+    (path "/65bb93c0-19d0-45ee-9f1b-b4c76671bc0b"
+      (reference "H9") (unit 1) (value "MountingHole") (footprint "ELLIOTT:MC32_Hole")
+    )
+    (path "/eb134a26-5443-4a01-bd25-2cc40162ff8a"
+      (reference "H10") (unit 1) (value "MountingHole") (footprint "ELLIOTT:MC19_Hole")
+    )
     (path "/00000000-0000-0000-0000-00005f2f538b/00000000-0000-0000-0000-000063ebd7c4"
