File: KiCad/Real903/Backplane2/Backplane2.sch (KiCad schematic (older format))
At the start: 3 parts

Commit message: July 20th
Parts:
- added JBP1-BP2-1, JBP1-BP2-2, JBP1-BP2-3, JBP1-BP2-4, JBP1-BP2-5: ~, Connector_IDC:IDC-Header_2x10_P2.54mm_Horizontal_Lock, symbol Connector_Generic:Conn_01x20
Connections:
- net labels added: ATFa-9-21, C17-5-H, C18-5-8, CRS-7-AF, CRSm-11-AC, DTF1-1-5-22, DTF1-2-5-23, DTF2a-8-26, F1-57-7, F18-5-K, FTG1-57-4, FTGa-8-6, GTAa-8-27, GTJa-8-28, GTMa-8-23, GTQa-8-24, I1-22-D, I2-22-F, I3-22-J, I4-22-L, IIS-57-15, ITF-8-12, J1'-20-4, J1-20-C, J2'-20-6, J2-20-E, J3'-20-8, J3-20-H, JTFa-9-24, JTPCa-9-7, LTG1-57-8, LTGa-9-25, M11-7-21, M12-6-W, M13-7-6, M18-7-9, MTFa-8-30, MTI-5-17, MTPa-9-22, OTMa-9-23, PTG1-a-9-6, PTG2-a-9-12, QTFa-9-30, RTG1-57-6, RTGa-9-14, SFD-6-R, SFDm-19-V, VTGa-8-7, WTMa-8-21, X0-57-5, X1-57-11, t1-5-27, t2-2-5-20, t3-2-5-29, t4-5-26, t5-5-25, ~ETJ2~-6-27, ~ETJ3~-6-28, ~IIG~, ~I~1-22-E, ~I~2-22-H, ~I~3-22-K, ~I~4-22-M, ~J~1'-20-3, ~J~14-22-28, ~J~15-22-29, ~J~16-22-26, ~J~2'-20-5, ~J~3'-20-7, ~J~4-23-27, ~J~5-24-3, ~J~6-24-8, ~J~7-24-19, ~J~8-24-27, ~J~9-25-3, ~KTJ1~-6-21, ~KTJ5~-6-22, ~M~12-6-Y, ~M~13-6-18, ~M~18-7-11, ~M~TFa-9-13, ~OTA~'-5-7, ~OTG1~-57-M, ~OTI~-5-18, ~OTJ~'-5-11, ~Q~1-7-15, ~RESET~2-2-Y
- no-connect marks 0 -> 13
Other:
- note added: "20 21 22 23 24 25"
- note removed: "20 21 22\n23 24 25"

Commit message: August 2
Parts:
- removed JBP1-BP2-1, JBP1-BP2-2, JBP1-BP2-3, JBP1-BP2-4, JBP1-BP2-5: ~, Connector_IDC:IDC-Header_2x10_P2.54mm_Horizontal_Lock, symbol Connector_Generic:Conn_01x20
Connections:
- net labels removed: ATFa-9-21, C17-5-H, C18-5-8, CRS-7-AF, CRSm-11-AC, DTF1-1-5-22, DTF1-2-5-23, DTF2a-8-26, F1-57-7, F18-5-K, FTG1-57-4, FTGa-8-6, GTAa-8-27, GTJa-8-28, GTMa-8-23, GTQa-8-24, I1-22-D, I2-22-F, I3-22-J, I4-22-L, IIS-57-15, ITF-8-12, J1'-20-4, J1-20-C, J2'-20-6, J2-20-E, J3'-20-8, J3-20-H, JTFa-9-24, JTPCa-9-7, LTG1-57-8, LTGa-9-25, M11-7-21, M12-6-W, M13-7-6, M18-7-9, MTFa-8-30, MTI-5-17, MTPa-9-22, OTMa-9-23, PTG1-a-9-6, PTG2-a-9-12, QTFa-9-30, RTG1-57-6, RTGa-9-14, SFD-6-R, SFDm-19-V, VTGa-8-7, WTMa-8-21, X0-57-5, X1-57-11, t1-5-27, t2-2-5-20, t3-2-5-29, t4-5-26, t5-5-25, ~ETJ2~-6-27, ~ETJ3~-6-28, ~IIG~, ~I~1-22-E, ~I~2-22-H, ~I~3-22-K, ~I~4-22-M, ~J~1'-20-3, ~J~14-22-28, ~J~15-22-29, ~J~16-22-26, ~J~2'-20-5, ~J~3'-20-7, ~J~4-23-27, ~J~5-24-3, ~J~6-24-8, ~J~7-24-19, ~J~8-24-27, ~J~9-25-3, ~KTJ1~-6-21, ~KTJ5~-6-22, ~M~12-6-Y, ~M~13-6-18, ~M~18-7-11, ~M~TFa-9-13, ~OTA~'-5-7, ~OTG1~-57-M, ~OTI~-5-18, ~OTJ~'-5-11, ~Q~1-7-15, ~RESET~2-2-Y
- wire segments 9 -> 150
- no-connect marks 13 -> 0
