File: KiCad/Real903/Backplane2/Drivers.sch (KiCad schematic (older format))
At the start: 11 parts

Commit message: July 20th
Connections:
- net labels added: SFD-6-R
Changed lines of the file:
@@
 Text GLabel 925  1525 0    50   Input ~ 0
 ~SFD
-Text GLabel 1825 2425 2    50   Input ~ 0
-SFD
+Text GLabel 1825 2425 2    32   UnSpc ~ 0
+SFD-6-R
 Text GLabel 1825 3225 2    50   Input ~ 0
 t2-1

Commit message: August 2
Parts:
- removed J106: ~, ELLIOTT:TerminalBlock-5.08_1x10, symbol Connector_Generic:Conn_01x10
- removed J107: ~, ELLIOTT:TerminalBlock_5.08_1x08, symbol Connector_Generic:Conn_01x08
- removed J108, J109, J157: ~, ELLIOTT:TerminalBlock-5.08_1x16, symbol Connector_Generic:Conn_01x16
- removed J209: ~, ELLIOTT:TerminalBlock_5.08_1x03, symbol Connector_Generic:Conn_01x03
Connections:
- net labels added: #C-6-N, #CA-7-Z, #CB-7-V, #CD-6-V, #FD-6-S, #X-57-D, #Y-57-Z, -6v, ATFa-9-21, CRS-7-AF, DTF2a-8-26, F1-57-7, F18-5-K, FTG1-57-4, FTGa-8-6, GTAa-8-27, GTJa-8-28, GTMa-8-23, GTQa-8-24, IIS-57-15, ITF-8-12, JTFa-9-24, JTPCa-9-7, LTG1-57-8, LTGa-9-25, M11-7-21, M12-6-W, M13-7-6, M18-7-9, MTFa-8-30, MTPa-9-22, OTMa-9-23, PTG1-a-9-6, PTG2-a-9-12, QTFa-9-30, RTG1-57-6, RTGa-9-14, SZ1-9-15, VTGa-8-7, WTMa-8-21, X0-57-5, X1-57-11, t4, ~ETJ2~-6-27, ~ETJ3~-6-28, ~KTJ1~-6-21, ~KTJ5~-6-22, ~M~12-6-Y, ~M~13-6-18, ~M~18-7-11, ~M~TFa-9-13, ~OTG1~-57-M, ~Q~1-7-15, ~SAO~, ~SB~, ~SFD~, ~TEST~-1-5, ~WGS~, ~X~
- net labels removed: 1TF, ATFa, CRS, CRSm, DTF2a, F1, F18, FTG1, FTGa, GTAa, GTJa, GTMa, GTQa, IIS, JTFa, JTPC, JTPCa, LTG1, LTGa, M11, M18, MTFa, MTPa, Neg6v, OTA-', OTJ-', OTMa, PTG1a, PTG2a, Q1-, QTFa, RTG1, RTGa, SFDm, SKT1JJ, SKT1KK, SKT3DD, SKT3EE, SKT3FF, SKT3GG, SKT3q, SKT5D, SZ1, TW, VTGa, X0, X1, t3-2, t4-5, ~ETJ~2, ~ETJ~3, ~KTJ~1, ~KTJ~5, ~M12, ~M13, ~M18, ~M~TFa, ~OTG~1, ~RESET~2, ~SAO, ~SB, ~SFD, ~SSI, ~TR, ~TW, ~WGS, ~X
- wire segments 324 -> 171
- no-connect marks 65 -> 68
Other:
- moved on the sheet: J57, J6, J7, J8, J9
