File: KiCad/Real903/Backplane2/FunctionsB.sch (KiCad schematic (older format))
At the start: 5 parts

Commit message: August 2
Connections:
- net Neg6v: no longer J15.AK (Pin_AK), J16.31 (Pin_31)
- net DA renamed D1
- net DB renamed D2
- net D2: now also J17.8 (Pin_8)
- net DC renamed D3
- net DD renamed D4
- net DF renamed D6
- net DG renamed D7
- net D7: no longer J17.8 (Pin_8)
- net DH renamed D8
- net S0a renamed S1
- net S0b renamed S2
- net S1a renamed S4
- net S1b renamed S5
- net S2a renamed S7
- net S2b renamed S8
- net S3a renamed S10
- net S4a renamed S12
- net SFDm renamed SFDm-19-V
- net ~S4~a renamed S14
- net ~S4~b renamed S15
- new net -6v: J15.AK (Pin_AK), J16.31 (Pin_31)
