File: KiCad/Real903/Backplane2/Matrix and Logic.sch (KiCad schematic (older format))
At the start: 13 parts

Commit message: August 2
Parts:
- removed J120, J121, J123, J124, J125, J220: ~, ELLIOTT:TerminalBlock_5.08_1x08, symbol Connector_Generic:Conn_01x08
- removed J122: ~, ELLIOTT:TerminalBlock-5.08_1x16, symbol Connector_Generic:Conn_01x16
Connections:
- net labels added: #AA1'-21-K, #AA1-21-M, #AA2'-21-U, #AA2-21-X, #AA3'-21-AF, #AA3-21-AA, #PC1, #PC10, #PC11, #PC12, #PC2, #PC3, #PC4, #PC5, #PC6, #PC7, #PC8, #PC9, #PC[1..12], -6v, D1, D2, D3, D4, D5, D6, D7, D8, D[1..8], I1-22-D, I2-22-F, I3-22-J, I4-22-L, J1'-20-4, J1-20-C, J2'-20-6, J2-20-E, J3'-20-8, J3-20-H, JTPC-23-L, PC1-4=1-22-AC, PC5-12, PC5-12=0-25-20, S1, S10, S11, S12, S13, S14, S15, S16, S17, S2, S3, S4, S5, S6, S7, S8, S9, S[1..17], ~1TPC~, ~CS~-1-H, ~I~1-22-E, ~I~2-22-H, ~I~3-22-K, ~I~4-22-M, ~J~1'-20-3, ~J~10-25-8, ~J~11-25-19, ~J~12-25-27, ~J~14-22-28, ~J~15-22-29, ~J~16-22-26, ~J~2'-20-5, ~J~3'-20-7, ~J~4-23-27, ~J~5-24-3, ~J~6-24-8, ~J~7-24-19, ~J~8-24-27, ~J~9-25-3, ~PC3~, ~PC4~, ~PC8~, ~RESET~2-2-Y, ~SAO~
- net labels removed: 1TPC-, DA, DB, DC, DD, DE, DF, DG, DH, I1, I2, I3, I4, J1, J1', J14-, J15-, J16-, J2, J2', J3, J3', Neg6v, PC1-4=1, PC3-, PC4-, PC5-12=0, PC8-, S0a, S0b, S0c, S1a, S1b, S1c, S2a, S2b, S2c, S3a, S3b, S4a, S4b, SIS1, SIS2, SKT2AA, SKT2CC, SKT2DD, SKT2EE, SKT2FF, SKT2GG, SKT2HH, SKT2JJ, SKT2KK, SKT2LL, SKT2z, SKT3AA, SKT3BB, SKT3v, SKT3w, SKT3x, SKT3z, SKT5e, STK2BB, ~I1~, ~I2~, ~I3~, ~I4~, ~J10~, ~J11~, ~J12~, ~J1~', ~J2~', ~J3~', ~J4~, ~J5~, ~J6~, ~J7~, ~J8~, ~J9~, ~RESET~2, ~S4~a, ~S4~b, ~S4~c, ~S4~d, ~SAO
- wire segments 246 -> 98
- no-connect marks 202 -> 192
Other:
- note added: "S0a"
- note added: "S0b"
- note added: "S0c"
- note added: "S1a"
- note added: "S1b"
- note added: "S1c"
- note added: "S2a"
- note added: "S2b"
- note added: "S2c"
- note added: "S3a"
- note added: "S3b"
- note added: "S4a"
- note added: "S4b"
- note added: "~S4~a"
- note added: "~S4~b"
- note added: "~S4~c"
- note added: "~S4~d"
