File: KiCad/Real903/Backplane2/Connections.sch (KiCad schematic (older format))
At the start: 9 parts

Commit message: New Backplanes
Parts:
- added BP2-DSP-4: ~, Connector_IDC:IDC-Header_2x10_P2.54mm_Horizontal_Lock, symbol Backplane2-rescue:Conn_01x20-Connector_Generic
- renumbered JBP1-BP2-1 to BP2-BP1-1, JBP1-BP2-2 to BP2-BP1-2, JBP1-BP2-3 to BP2-BP1-3, JBP1-BP2-4 to BP2-BP1-4, JBP1-BP2-5 to BP2-BP1-5, JBP3-BP2-1 to BP2-BP3-1, JSKT2-4 to BP2-DSP-1, JSKT3-3-1 to BP2-DSP-2, JSKT3-1 to BP2-DSP-3
Connections:
- net #AA1'-21-K: now also BP2-DSP-2.6 (Pin_6); no longer BP2-DSP-2.15 (Pin_15)
- net #AA1-21-M: now also BP2-DSP-2.10 (Pin_10); no longer BP2-DSP-2.18 (Pin_18)
- net #AA2'-21-U: now also BP2-DSP-2.7 (Pin_7); no longer BP2-DSP-2.16 (Pin_16)
- net #AA2-21-X: now also BP2-DSP-2.11 (Pin_11); no longer BP2-DSP-2.19 (Pin_19)
- net #AA3'-21-AF: now also BP2-DSP-2.8 (Pin_8); no longer BP2-DSP-2.17 (Pin_17)
- net #AA3-21-AA: now also BP2-DSP-2.12 (Pin_12); no longer BP2-DSP-2.20 (Pin_20)
- net #ACTIVE1-1-Y: now also BP2-DSP-3.9 (Pin_9); no longer BP2-DSP-3.13 (Pin_13)
- net #ACTIVE2-1-V: now also BP2-DSP-3.11 (Pin_11); no longer BP2-DSP-2.1 (Pin_1)
- net #ACTIVE3-1-S: now also BP2-DSP-3.18 (Pin_18); no longer BP2-DSP-2.8 (Pin_8)
- net #C-6-N: now also BP2-DSP-2.16 (Pin_16); no longer BP2-DSP-1.3 (Pin_3)
- net #CA-7-Z: now also BP2-DSP-2.14 (Pin_14); no longer BP2-DSP-1.4 (Pin_4)
- net #CB-7-V: now also BP2-DSP-2.15 (Pin_15); no longer BP2-DSP-1.5 (Pin_5)
- net #CD-6-V: now also BP2-DSP-2.17 (Pin_17); no longer BP2-DSP-1.2 (Pin_2)
- net #FD-6-S: now also BP2-DSP-2.1 (Pin_1); no longer BP2-DSP-1.6 (Pin_6)
- net #INT1-3-F: now also BP2-DSP-3.10 (Pin_10); no longer BP2-DSP-3.20 (Pin_20)
- net #INT2-3-W: now also BP2-DSP-3.12 (Pin_12); no longer BP2-DSP-2.2 (Pin_2)
- net #INT3-3-AD: now also BP2-DSP-3.19 (Pin_19); no longer BP2-DSP-2.9 (Pin_9)
- net #NOTRDY-2-AC: now also BP2-DSP-2.20 (Pin_20); no longer BP2-DSP-2.14 (Pin_14)
- net #PC1: now also BP2-DSP-1.1 (Pin_1); no longer BP2-DSP-1.9 (Pin_9)
- net #PC10: now also BP2-DSP-1.10 (Pin_10); no longer BP2-DSP-1.18 (Pin_18)
- net #PC11: now also BP2-DSP-1.11 (Pin_11); no longer BP2-DSP-1.19 (Pin_19)
- net #PC12: now also BP2-DSP-1.12 (Pin_12); no longer BP2-DSP-1.20 (Pin_20)
- net #PC2: now also BP2-DSP-1.2 (Pin_2); no longer BP2-DSP-1.10 (Pin_10)
- net #PC3: now also BP2-DSP-1.3 (Pin_3); no longer BP2-DSP-1.11 (Pin_11)
- net #PC4: now also BP2-DSP-1.4 (Pin_4); no longer BP2-DSP-1.12 (Pin_12)
- net #PC5: now also BP2-DSP-1.5 (Pin_5); no longer BP2-DSP-1.13 (Pin_13)
- net #PC6: now also BP2-DSP-1.6 (Pin_6); no longer BP2-DSP-1.14 (Pin_14)
- net #PC7: now also BP2-DSP-1.7 (Pin_7); no longer BP2-DSP-1.15 (Pin_15)
- net #PC8: now also BP2-DSP-1.8 (Pin_8); no longer BP2-DSP-1.16 (Pin_16)
- net #PC9: now also BP2-DSP-1.9 (Pin_9); no longer BP2-DSP-1.17 (Pin_17)
- net #RESET-2-Z: now also BP2-DSP-2.18 (Pin_18), BP2-DSP-4.1 (Pin_1); no longer BP2-DSP-2.12 (Pin_12), BP2-DSP-3.11 (Pin_11)
- net #STOP-2-E: now also BP2-DSP-3.4 (Pin_4); no longer BP2-DSP-3.18 (Pin_18)
- net #STOP-2-T: now also BP2-DSP-2.19 (Pin_19); no longer BP2-DSP-2.13 (Pin_13)
- net #X-57-D: now also BP2-DSP-1.14 (Pin_14); no longer BP2-DSP-1.7 (Pin_7)
- net #Y-57-Z: now also BP2-DSP-1.13 (Pin_13); no longer BP2-DSP-1.8 (Pin_8)
- net AUTO-1-L: now also BP2-DSP-4.12 (Pin_12); no longer BP2-DSP-2.11 (Pin_11)
- net CINS-1-J: now also BP2-DSP-3.13 (Pin_13); no longer BP2-DSP-2.3 (Pin_3)
- net ENG-1-6: now also BP2-DSP-4.8 (Pin_8); no longer BP2-DSP-3.4 (Pin_4)
- net INT1-3-9: now also BP2-DSP-4.11 (Pin_11); no longer BP2-DSP-3.1 (Pin_1)
- net JUMP-1-M: now also BP2-DSP-3.7 (Pin_7); no longer BP2-DSP-3.15 (Pin_15)
- net MARGIN-4-3: now also BP2-DSP-4.2 (Pin_2); no longer BP2-DSP-3.10 (Pin_10)
- net ONG-1-7: now also BP2-DSP-4.10 (Pin_10); no longer BP2-DSP-3.2 (Pin_2)
- net PS1-3-E: now also BP2-DSP-4.5 (Pin_5); no longer BP2-DSP-3.7 (Pin_7)
- net PS2-3-L: now also BP2-DSP-4.4 (Pin_4); no longer BP2-DSP-3.8 (Pin_8)
- net PS3-3-S: now also BP2-DSP-4.3 (Pin_3); no longer BP2-DSP-3.9 (Pin_9)
- net RESET-1-24: now also BP2-DSP-4.6 (Pin_6); no longer BP2-DSP-3.6 (Pin_6)
- net RESTART-1-C: now also BP2-DSP-3.5 (Pin_5); no longer BP2-DSP-3.17 (Pin_17)
- net ~CINS~-1-8: now also BP2-DSP-3.14 (Pin_14); no longer BP2-DSP-2.4 (Pin_4)
- net ~CS~-1-H: now also BP2-DSP-3.16 (Pin_16); no longer BP2-DSP-2.6 (Pin_6)
- net ~ENG~-1-4: now also BP2-DSP-4.7 (Pin_7); no longer BP2-DSP-3.5 (Pin_5)
- net ~JUMP~-1-11: now also BP2-DSP-3.8 (Pin_8); no longer BP2-DSP-3.14 (Pin_14)
- net ~ONG~-1-F: now also BP2-DSP-4.9 (Pin_9); no longer BP2-DSP-3.3 (Pin_3)
- net ~OS~-1-19: now also BP2-DSP-3.17 (Pin_17); no longer BP2-DSP-2.7 (Pin_7)
- net ~RESTART~-1-3: now also BP2-DSP-3.6 (Pin_6); no longer BP2-DSP-3.16 (Pin_16)
- net ~SMN~-4-7: now also BP2-DSP-3.20 (Pin_20); no longer BP2-DSP-2.10 (Pin_10)
- net ~STOP~-1-25: now also BP2-DSP-3.3 (Pin_3); no longer BP2-DSP-3.19 (Pin_19)
- net ~TCS~-1-AB: now also BP2-DSP-3.15 (Pin_15); no longer BP2-DSP-2.5 (Pin_5)
- net ~TEST~-1-5: now also BP2-DSP-3.1 (Pin_1); no longer BP2-DSP-3.12 (Pin_12)
- no-connect marks 10 -> 30
Other:
- moved on the sheet: BP2-BP1-1, BP2-BP1-2, BP2-BP1-3, BP2-BP1-4, BP2-BP1-5, BP2-BP3-1, BP2-DSP-1, BP2-DSP-2, BP2-DSP-3

Commit message: BP2 and 3
Parts:
- renumbered BP2-DSP-3 to BP2-CNT-1, BP2-DSP-4 to BP2-CNT-2
Connections:
- net RESET-2-U: now reaches BP2-CNT-1.2 (Pin_2)
- net MARGINS renamed MARGIN-30-16
- no-connect marks 30 -> 29
Changed lines of the file:
@@
 #INT1-3-F
 $Comp
-L Backplane2-rescue:Conn_01x20-Connector_Generic BP2-DSP-3
+L Backplane2-rescue:Conn_01x20-Connector_Generic BP2-CNT-1
 U 1 1 5F1ECBC3
 P 3125 2800
-F 0 "BP2-DSP-3" H 3125 3825 50  0000 C CNN
+F 0 "BP2-CNT-1" H 3125 3825 50  0000 C CNN
 F 1 "~" H 3045 3826 50  0000 C CNN
 F 2 "Connector_IDC:IDC-Header_2x10_P2.54mm_Horizontal_Lock" H 3125 2800 50  0001 C CNN
@@
 IIG If we need it
 Text HLabel 1700 10175 2    40   UnSpc ~ 0
-MARGINS
+MARGIN-30-16
 Text GLabel 4225 7000 2    32   UnSpc ~ 0
 W17-1-W
@@
 NoConn ~ 1700 3700
 $Comp
-L Backplane2-rescue:Conn_01x20-Connector_Generic BP2-DSP-4
+L Backplane2-rescue:Conn_01x20-Connector_Generic BP2-CNT-2
 U 1 1 63E324D9
 P 4025 2800
-F 0 "BP2-DSP-4" H 4025 3825 50  0000 C CNN
+F 0 "BP2-CNT-2" H 4025 3825 50  0000 C CNN
 F 1 "~" H 3945 3826 50  0000 C CNN
 F 2 "Connector_IDC:IDC-Header_2x10_P2.54mm_Horizontal_Lock" H 4025 2800 50  0001 C CNN
@@
 NoConn ~ 4225 3700
 NoConn ~ 4225 3800
-NoConn ~ 3325 2000
+Text GLabel 3325 2000 2    32   UnSpc ~ 0
+RESET-2-U
 $EndSCHEMATC
