File: KiCad/Real903/Backplane3/Backplane3.sch (KiCad schematic (older format))
At the start: 19 parts

Commit message: July 20th
Parts:
- removed J128, J131, J228, J231, J232: ~, ELLIOTT:TerminalBlock-5.08_1x18, symbol Connector_Generic:Conn_01x18
- removed J129, J130, J229, J230: ~, ELLIOTT:TerminalBlock-5.08_1x20, symbol Connector_Generic:Conn_01x20
- removed J132, J328: ~, ELLIOTT:TerminalBlock_5.08_1x06, symbol Connector_Generic:Conn_01x06
- removed J28, J29, J30, J31, J32: ~, ELLIOTT:DIN41612_B_2x32_Vertical, symbol LSA:Conn_02x32
- removed J331: ~, ELLIOTT:TerminalBlock_5.08_1x08, symbol Connector_Generic:Conn_01x08
Connections:
- net labels removed: IIS(TR), INT1, INT2, INT3, IP1, IP1', IP10, IP11, IP12, IP13, IP14, IP15, IP16, IP17, IP18, IP2, IP2', IP3, IP3', IP4, IP4', IP5, IP5', IP6, IP6', IP7, IP7', IP8, IP8', IP9, MARGIN, P12, P13, PC1-4=1, PC5-12=0, RBT, RBTm, SBT, SBTm, SKT10A, SKT10B, SKT10C, SKT10D, SKT10E, SKT10F, SKT10G, SKT10H, SKT10J, SKT10K, SKT10L, SKT10M, SKT10N, SKT10P, SKT10R, SKT10S, SKT10U, SKT10V, SKT10W, SKT10X, SKT10Y, SKT10~b, SKT10~d, SKT10~h, SKT10~j, SKT11C, SKT11D, SKT11E, SKT11R, SKT11S, SKT11T, SKT11V, SKT13A, SKT13C, SKT13E, SKT13G, SKT13J, SKT13L, SKT13N, SKT13R, SKT14~x, SKT14~z, SKT1LL, SKT1MM, SKT1NN, SKT1PP, SKT4AA, SKT4B, SKT4BB, SKT4C, SKT4CC, SKT4D, SKT4DD, SKT4E, SKT4EE, SKT4F, SKT4FF, SKT4G, SKT4GG, SKT4H, SKT4HH, SKT4J, SKT4K, SKT4L, SKT4M, SKT4N, SKT4P, SKT4PP, SKT4R, SKT4S, SKT4T, SKT4U, SKT4W, SKT4X, SKT4Y, SKT4Z, SKT4~a, SKT4~b, SKT4~c, SKT4~d, SKT4~e, SKT4~f, SKT4~g, SKT4~q, SKT4~r, SKT4~s, SKT4~t, SKT4~u, SKT4~v, SKT4~w, SKT4~x, SKT4~y, SKT4~z, SKT5~p, STK4V, SZ1, TRD, TZ1, W14, W15, W16, W18, W2, W3, W4, t4-2, ~A1, ~A10, ~A11, ~A12, ~A13, ~A14, ~A15, ~A16, ~A17, ~A18, ~A2, ~A3, ~A4, ~A5, ~A6, ~A7, ~A8, ~A9, ~P1, ~P10, ~P11, ~P12, ~P13, ~P2, ~P3, ~P4, ~P5, ~P6, ~P7, ~P8, ~P9, ~RESET~2, ~RGS~x, ~VTG, ~WGS~x, ~Z2
- wire segments 430 -> 6
- no-connect marks 86 -> 0

Commit message: August 2
Changed lines of the file:
@@
 encoding utf-8
 Sheet 1 3
-Title ""
+Title "Backplane 3"
 Date ""
 Rev ""
@@
 F1 "Drivers.sch" 200
 F2 "OS[1..11]" I L 6075 2850 100
-F3 "-6v" I L 6075 2600 50
-F4 "GND" I L 6075 2700 50
+F3 "-6v" I R 9625 2700 50
+F4 "GND" I R 9625 2800 50
 F5 "OA[1..18]" I L 6075 3150 100
 F6 "~A~[1..18]" I L 6075 3500 100
 F7 "IP[1..18]" I L 6075 3800 100
 F8 "IG[1..18]" I L 6075 4100 100
+F9 "6v" I R 9625 2600 50
+F10 "OP[1..8]" I L 6075 4425 100
+F11 "IR[1..8]" I L 6075 4775 100
+F12 "W[1..18]" U L 6075 5300 100
+F13 "~NG~[1..18]" U L 6075 5125 100
+F14 "~P~[1..13]" U L 6075 5800 100
+F15 "IP'[1..8]" U L 6075 6275 100
 $EndSheet
 $Sheet
@@
 F3 "~A~[1..18]" I R 4525 3500 100
 F4 "OS[1..11]" I R 4525 2850 100
+F5 "IP[1..18]" I R 4525 3800 100
+F6 "IG[1..18]" I R 4525 4100 100
+F7 "IR[1..8]" I R 4525 4775 100
+F8 "OP[1..8]" I R 4525 4425 100
+F9 "~NG~[1..18]" U R 4525 5125 100
+F10 "W[1..18]" U R 4525 5300 100
+F11 "IP'[1..8]" U R 4525 6275 100
+F12 "~P~[1..13]" U R 4525 5800 100
 $EndSheet
 Wire Bus Line
@@
 Wire Bus Line
 	6075 3500 4525 3500
+Wire Bus Line
+	6075 3800 4525 3800
+Wire Bus Line
+	4525 4100 6075 4100
+Text GLabel 9775 2800 2    40   Input ~ 0
+GND
+Wire Wire Line
+	9775 2800 9625 2800
+Wire Bus Line
+	4525 4775 6075 4775
+Wire Bus Line
+	6075 4425 4525 4425
+Wire Bus Line
+	6075 5125 4525 5125
+Wire Bus Line
+	4525 5300 6075 5300
+Wire Bus Line
+	6075 5800 4525 5800
+Wire Bus Line
+	6075 6275 4525 6275
 $EndSCHEMATC
