File: KiCad/Real903/Backplane3/Backplane3.kicad_sch (KiCad schematic)
At the start: 2 parts

Commit message: Update to design
Other:
- sheet Connections ports: added J[1..16], M[1..18], ~{STORE}[1..18]; removed none
- sheet Drivers ports: added J[1..16], M[1..18], ~{STORE}[1..18]; removed none
Changed lines of the file:
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@@
+    (stroke (width 0) (type default) (color 0 0 0 0))
+  )
+  (bus (pts (xy 114.935 163.83) (xy 154.305 163.83))
     (stroke (width 0) (type default) (color 0 0 0 0))
   )
@@
     (stroke (width 0) (type default) (color 0 0 0 0))
   )
+  (bus (pts (xy 114.935 178.435) (xy 154.305 178.435))
+    (stroke (width 0) (type default) (color 0 0 0 0))
+  )
   (bus (pts (xy 154.305 112.395) (xy 114.935 112.395))
     (stroke (width 0) (type default) (color 0 0 0 0))
@@
   )
   (wire (pts (xy 248.285 71.12) (xy 244.475 71.12))
+    (stroke (width 0) (type default) (color 0 0 0 0))
+  )
+  (bus (pts (xy 114.935 170.815) (xy 154.305 170.815))
     (stroke (width 0) (type default) (color 0 0 0 0))
   )
@@
       (effects (font (size 2.54 2.54)) (justify right))
     )
+    (pin "M[1..18]" passive (at 114.935 170.815 0)
+      (effects (font (size 2.54 2.54)) (justify right))
+    )
+    (pin "J[1..16]" passive (at 114.935 178.435 0)
+      (effects (font (size 2.54 2.54)) (justify right))
+    )
+    (pin "~{STORE}[1..18]" passive (at 114.935 163.83 0)
+      (effects (font (size 2.54 2.54)) (justify right))
+    )
   )
   (sheet (at 154.305 63.5) (size 90.17 168.91) (fields_autoplaced)
@@
       (effects (font (size 2.54 2.54)) (justify left))
     )
+    (pin "~{STORE}[1..18]" passive (at 154.305 163.83 180)
+      (effects (font (size 2.54 2.54)) (justify left))
+    )
+    (pin "M[1..18]" passive (at 154.305 170.815 180)
+      (effects (font (size 2.54 2.54)) (justify left))
+    )
+    (pin "J[1..16]" passive (at 154.305 178.435 180)
+      (effects (font (size 2.54 2.54)) (justify left))
+    )
   )
   (sheet_instances
@@
       (reference "BP3-BP1-2") (unit 1) (value "~") (footprint "Connector_IDC:IDC-Header_2x10_P2.54mm_Latch_Vertical")
     )
+    (path "/00000000-0000-0000-0000-00005f16162d/2346bf62-a68c-4a01-a775-d5b75df51457"
+      (reference "BP3-BP1-3") (unit 1) (value "~") (footprint "Connector_IDC:IDC-Header_2x10_P2.54mm_Latch_Vertical")
+    )
+    (path "/00000000-0000-0000-0000-00005f16162d/d04269ed-8493-45e5-b8a2-a5829a5edbbd"
+      (reference "BP3-BP1-4") (unit 1) (value "~") (footprint "Connector_IDC:IDC-Header_2x10_P2.54mm_Latch_Vertical")
+    )
+    (path "/00000000-0000-0000-0000-00005f16162d/3adf18cf-2357-4c2b-9807-f685e59e5621"
+      (reference "BP3-BP1-5") (unit 1) (value "~") (footprint "Connector_IDC:IDC-Header_2x10_P2.54mm_Latch_Vertical")
+    )
     (path "/00000000-0000-0000-0000-00005f16162d/00000000-0000-0000-0000-00005f16bb1b"
       (reference "BP3-BP1-6") (unit 1) (value "~") (footprint "Connector_IDC:IDC-Header_2x10_P2.54mm_Latch_Vertical")
@@
       (reference "J32") (unit 1) (value "~") (footprint "ELLIOTT:DIN41612_B_2x32_Vertical")
     )
-  )
+    (path "/00000000-0000-0000-0000-00005f184515/d5afabfc-157f-4899-bb8b-51f579ea4a07"
+      (reference "J33") (unit 1) (value "~") (footprint "ELLIOTT:DIN41612_B_2x32_Vertical")
+    )
+  )
