File: KiCad/Real903/Backplane3/Connections.kicad_sch (KiCad schematic)
At the start: 11 parts

Commit message: Start new layout with IDC connectors
Parts:
- BP3-BP1-1, BP3-BP1-2, BP3-BP1-6, BP3-BP1-7, BP3-BP2-1, BP3-CNT-1, BP3-IO-1, BP3-IO-2, BP3-IO-3, BP3-IO-4, BP3-IO-5: footprint Connector_IDC:IDC-Header_2x10_P2.54mm_Horizontal_Lock -> Connector_IDC:IDC-Header_2x10_P2.54mm_Latch_Vertical
Changed lines of the file:
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@@
     (property "Reference" "BP3-BP1-6" (id 0) (at 65.405 95.885 0))
     (property "Value" "~" (id 1) (at 63.373 98.3996 0))
-    (property "Footprint" "Connector_IDC:IDC-Header_2x10_P2.54mm_Horizontal_Lock" (id 2) (at 65.405 121.92 0)
+    (property "Footprint" "Connector_IDC:IDC-Header_2x10_P2.54mm_Latch_Vertical" (id 2) (at 65.405 121.92 0)
       (effects (font (size 1.27 1.27)) hide)
     )
@@
     (property "Reference" "BP3-IO-2" (id 0) (at 65.405 20.32 0))
     (property "Value" "~" (id 1) (at 63.373 22.8346 0))
-    (property "Footprint" "Connector_IDC:IDC-Header_2x10_P2.54mm_Horizontal_Lock" (id 2) (at 65.405 46.355 0)
+    (property "Footprint" "Connector_IDC:IDC-Header_2x10_P2.54mm_Latch_Vertical" (id 2) (at 65.405 46.355 0)
       (effects (font (size 1.27 1.27)) hide)
     )
@@
     (property "Reference" "BP3-IO-3" (id 0) (at 85.725 20.32 0))
     (property "Value" "~" (id 1) (at 83.693 22.8346 0))
-    (property "Footprint" "Connector_IDC:IDC-Header_2x10_P2.54mm_Horizontal_Lock" (id 2) (at 85.725 46.355 0)
+    (property "Footprint" "Connector_IDC:IDC-Header_2x10_P2.54mm_Latch_Vertical" (id 2) (at 85.725 46.355 0)
       (effects (font (size 1.27 1.27)) hide)
     )
@@
     (property "Reference" "BP3-IO-4" (id 0) (at 104.775 20.32 0))
     (property "Value" "~" (id 1) (at 102.743 22.8346 0))
-    (property "Footprint" "Connector_IDC:IDC-Header_2x10_P2.54mm_Horizontal_Lock" (id 2) (at 104.775 46.355 0)
+    (property "Footprint" "Connector_IDC:IDC-Header_2x10_P2.54mm_Latch_Vertical" (id 2) (at 104.775 46.355 0)
       (effects (font (size 1.27 1.27)) hide)
     )
@@
     (property "Reference" "BP3-BP1-7" (id 0) (at 85.725 95.885 0))
     (property "Value" "~" (id 1) (at 83.693 98.3996 0))
-    (property "Footprint" "Connector_IDC:IDC-Header_2x10_P2.54mm_Horizontal_Lock" (id 2) (at 85.725 121.92 0)
+    (property "Footprint" "Connector_IDC:IDC-Header_2x10_P2.54mm_Latch_Vertical" (id 2) (at 85.725 121.92 0)
       (effects (font (size 1.27 1.27)) hide)
     )
@@
     (property "Reference" "BP3-BP2-1" (id 0) (at 27.305 160.655 0))
     (property "Value" "~" (id 1) (at 27.178 163.1696 0))
-    (property "Footprint" "Connector_IDC:IDC-Header_2x10_P2.54mm_Horizontal_Lock" (id 2) (at 29.21 186.69 0)
+    (property "Footprint" "Connector_IDC:IDC-Header_2x10_P2.54mm_Latch_Vertical" (id 2) (at 29.21 186.69 0)
       (effects (font (size 1.27 1.27)) hide)
     )
@@
     (property "Reference" "BP3-IO-1" (id 0) (at 27.305 20.32 0))
     (property "Value" "~" (id 1) (at 27.178 22.8346 0))
-    (property "Footprint" "Connector_IDC:IDC-Header_2x10_P2.54mm_Horizontal_Lock" (id 2) (at 29.21 46.355 0)
+    (property "Footprint" "Connector_IDC:IDC-Header_2x10_P2.54mm_Latch_Vertical" (id 2) (at 29.21 46.355 0)
       (effects (font (size 1.27 1.27)) hide)
     )
@@
     )
     (property "Value" "~" (id 1) (at 121.793 22.8346 0))
-    (property "Footprint" "Connector_IDC:IDC-Header_2x10_P2.54mm_Horizontal_Lock" (id 2) (at 123.825 46.355 0)
+    (property "Footprint" "Connector_IDC:IDC-Header_2x10_P2.54mm_Latch_Vertical" (id 2) (at 123.825 46.355 0)
       (effects (font (size 1.27 1.27)) hide)
     )
@@
     )
     (property "Value" "~" (id 1) (at 43.688 22.8346 0))
-    (property "Footprint" "Connector_IDC:IDC-Header_2x10_P2.54mm_Horizontal_Lock" (id 2) (at 45.72 46.355 0)
+    (property "Footprint" "Connector_IDC:IDC-Header_2x10_P2.54mm_Latch_Vertical" (id 2) (at 45.72 46.355 0)
       (effects (font (size 1.27 1.27)) hide)
     )
@@
     (property "Reference" "BP3-BP1-2" (id 0) (at 43.815 95.885 0))
     (property "Value" "~" (id 1) (at 43.688 98.3996 0))
-    (property "Footprint" "Connector_IDC:IDC-Header_2x10_P2.54mm_Horizontal_Lock" (id 2) (at 45.72 121.92 0)
+    (property "Footprint" "Connector_IDC:IDC-Header_2x10_P2.54mm_Latch_Vertical" (id 2) (at 45.72 121.92 0)
       (effects (font (size 1.27 1.27)) hide)
     )
@@
     (property "Reference" "BP3-BP1-1" (id 0) (at 27.305 95.885 0))
     (property "Value" "~" (id 1) (at 27.178 98.3996 0))
-    (property "Footprint" "Connector_IDC:IDC-Header_2x10_P2.54mm_Horizontal_Lock" (id 2) (at 29.21 121.92 0)
-      (effects (font (size 1.27 1.27)) hide)
-    )
+    (property "Footprint" "Connector_IDC:IDC-Header_2x10_P2.54mm_Latch_Vertical" (id 2) (at 29.21 121.92 0)
+      (effects (font (size 1.27 1.27)) hide)
+    )

Commit message: Update to design
Parts:
- added BP3-BP1-3, BP3-BP1-4, BP3-BP1-5: ~, Connector_IDC:IDC-Header_2x10_P2.54mm_Latch_Vertical, symbol Connector_Generic:Conn_01x20
Connections:
- new net J1: BP3-BP1-5.1 (Pin_1)
- new net J10: BP3-BP1-5.10 (Pin_10)
- new net J11: BP3-BP1-5.11 (Pin_11)
- new net J12: BP3-BP1-5.12 (Pin_12)
- new net J13: BP3-BP1-5.13 (Pin_13)
- new net J14: BP3-BP1-5.14 (Pin_14)
- new net J15: BP3-BP1-5.15 (Pin_15)
- new net J16: BP3-BP1-5.16 (Pin_16)
- new net J2: BP3-BP1-5.2 (Pin_2)
- new net J3: BP3-BP1-5.3 (Pin_3)
- new net J4: BP3-BP1-5.4 (Pin_4)
- new net J5: BP3-BP1-5.5 (Pin_5)
- new net J6: BP3-BP1-5.6 (Pin_6)
- new net J7: BP3-BP1-5.7 (Pin_7)
- new net J8: BP3-BP1-5.8 (Pin_8)
- new net J9: BP3-BP1-5.9 (Pin_9)
- new net M1: BP3-BP1-4.1 (Pin_1)
- new net M10: BP3-BP1-4.10 (Pin_10)
- new net M11: BP3-BP1-4.11 (Pin_11)
- new net M12: BP3-BP1-4.12 (Pin_12)
- new net M13: BP3-BP1-4.13 (Pin_13)
- new net M14: BP3-BP1-4.14 (Pin_14)
- new net M15: BP3-BP1-4.15 (Pin_15)
- new net M16: BP3-BP1-4.16 (Pin_16)
- new net M17: BP3-BP1-4.17 (Pin_17)
- new net M18: BP3-BP1-4.18 (Pin_18)
- new net M2: BP3-BP1-4.2 (Pin_2)
- new net M3: BP3-BP1-4.3 (Pin_3)
- new net M4: BP3-BP1-4.4 (Pin_4)
- new net M5: BP3-BP1-4.5 (Pin_5)
- new net M6: BP3-BP1-4.6 (Pin_6)
- new net M7: BP3-BP1-4.7 (Pin_7)
- new net M8: BP3-BP1-4.8 (Pin_8)
- new net M9: BP3-BP1-4.9 (Pin_9)
- new net ~{STORE}1: BP3-BP1-3.1 (Pin_1)
- new net ~{STORE}10: BP3-BP1-3.10 (Pin_10)
- new net ~{STORE}11: BP3-BP1-3.11 (Pin_11)
- new net ~{STORE}12: BP3-BP1-3.12 (Pin_12)
- new net ~{STORE}13: BP3-BP1-3.13 (Pin_13)
- new net ~{STORE}14: BP3-BP1-3.14 (Pin_14)
- new net ~{STORE}15: BP3-BP1-3.15 (Pin_15)
- new net ~{STORE}16: BP3-BP1-3.16 (Pin_16)
- new net ~{STORE}17: BP3-BP1-3.17 (Pin_17)
- new net ~{STORE}18: BP3-BP1-3.18 (Pin_18)
- new net ~{STORE}2: BP3-BP1-3.2 (Pin_2)
- new net ~{STORE}3: BP3-BP1-3.3 (Pin_3)
- new net ~{STORE}4: BP3-BP1-3.4 (Pin_4)
- new net ~{STORE}5: BP3-BP1-3.5 (Pin_5)
- new net ~{STORE}6: BP3-BP1-3.6 (Pin_6)
- new net ~{STORE}7: BP3-BP1-3.7 (Pin_7)
- new net ~{STORE}8: BP3-BP1-3.8 (Pin_8)
- new net ~{STORE}9: BP3-BP1-3.9 (Pin_9)
- no-connect marks 34 -> 42
