File: KiCad/KIT88/KIT88 - IP.kicad_pcb (KiCad board)
At the start: 2 copper layers, 108 x 71.1 mm, 35 parts

Commit message: November
Parts:
- removed R9: ~, Resistor_THT:R_Axial_DIN0204_L3.6mm_D1.6mm_P7.62mm_Horizontal
- K1, K2, K3, K4: value ~ -> FINDER-30.22; footprint Relay_THT:Relay_DPDT_Kemet_EC2 -> Relay_THT:Relay_DPDT_Finder_30.22
- moved J9 71.9 mm to (68.2, 82.5), turned to 0 degrees
- moved R5 43.8 mm to (96.1, 82.7), turned to 180 degrees
- moved R6 31.2 mm to (111.9, 82.7), turned to 180 degrees
- moved D1 26.4 mm to (87.0, 69.6), turned to 270 degrees
- moved D2 20.9 mm to (104.4, 69.7), turned to 270 degrees
- moved R7 18.0 mm to (129.7, 82.5), turned to 180 degrees
- moved J4 16.1 mm to (132.5, 49.5)
- moved R8 15.9 mm to (135.1, 82.4), turned to 0 degrees
- moved D3 15.8 mm to (122.0, 69.8), turned to 270 degrees
- moved Q1 14.8 mm to (88.3, 76.2), turned to 180 degrees
- moved K4 14.2 mm to (134.6, 76.2), turned to 90 degrees
- moved R1 13.6 mm to (74.5, 79.8)
- moved D4 10.7 mm to (139.6, 69.8), turned to 270 degrees
- moved J3 10.7 mm to (115.0, 49.5)
- moved Q2 10.0 mm to (105.5, 76.2), turned to 180 degrees
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Connections:
- J0 pad 1: Net-(J0-Pad1) -> 0v
- J1 pad 2: Net-(J0-Pad1) -> 0v
- J2 pad 2: Net-(J0-Pad1) -> 0v
- J3 pad 2: Net-(J0-Pad1) -> 0v
- J4 pad 2: Net-(J0-Pad1) -> 0v
- K1 pad 12: (no net) -> Net-(K1-Pad12)
- K2 pad 12: (no net) -> Net-(K2-Pad12)
- K3 pad 12: (no net) -> Net-(K3-Pad12)
- K4 pad 12: (no net) -> Net-(K4-Pad12)
- Q1 pad 3: Net-(K1-Pad10) -> /K1
- Q2 pad 3: Net-(K2-Pad10) -> /K2
- Q3 pad 3: Net-(K3-Pad10) -> /K3
- Q4 pad 3: Net-(K4-Pad10) -> /K4
- R1 pad 2: Net-(K1-Pad10) -> /K1
- R2 pad 2: Net-(K2-Pad10) -> /K2
- R3 pad 2: Net-(K3-Pad10) -> /K3
- R4 pad 2: Net-(K4-Pad10) -> /K4
Routing:
- net 0v: track 0.00 -> 232.6 mm
- net +12v: track 0.00 -> 97.8 mm
- net Net-(J0-Pad3): track 0.00 -> 85.0 mm
- net Net-(J0-Pad2): track 0.00 -> 73.0 mm
- net Net-(J9-Pad4): track 0.00 -> 70.1 mm
- net Net-(J9-Pad3): track 0.00 -> 63.6 mm
- net Net-(J9-Pad2): track 0.00 -> 44.7 mm
- net Net-(J9-Pad1): track 0.00 -> 28.8 mm
- net Net-(J2-Pad3): track 0.00 -> 27.3 mm
- net Net-(J3-Pad3): track 0.00 -> 27.3 mm
- net Net-(J4-Pad3): track 0.00 -> 27.3 mm
- net Net-(J1-Pad3): track 0.00 -> 27.3 mm
- net Net-(J1-Pad1): track 0.00 -> 19.9 mm
- net Net-(J4-Pad1): track 0.00 -> 19.9 mm
- net Net-(J3-Pad1): track 0.00 -> 19.9 mm
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