File: KiCad/KIT88/KIT88 - IP.sch (KiCad schematic (older format))
At the start: 35 parts

Commit message: November
Parts:
- removed K1, K2, K3, K4: ~, Relay_THT:Relay_DPDT_Kemet_EC2, symbol Relay:FRT5_separated
- removed R9: ~, Resistor_THT:R_Axial_DIN0204_L3.6mm_D1.6mm_P7.62mm_Horizontal, symbol Device:R_Small
- added K1, K2, K3, K4: FINDER-30.22, Relay_THT:Relay_DPDT_Finder_30.22, symbol Relay:FINDER-30.22
Connections:
- net labels added: K1, K2, K3, K4
- wire segments 116 -> 97
Other:
- moved on the sheet: J0, J2, J3, J4
