File: KiCad/Quad/QuadNew.sch (KiCad schematic (older format))
At the start: 0 parts

Commit message: November
Parts:
- added H1, H10, H2, H3, H4, H5, H6, H7, H8, H9: ~, MountingHole:MountingHole_2.2mm_M2_ISO7380, symbol Mechanical:MountingHole
- added TP0: GROUND, Connector_Pin:Pin_D1.0mm_L10.0mm, symbol Connector:TestPoint
Connections:
- net 0v: now also TP0.1
