File: KiCad/Quad/QuadSignal.kicad_pcb (KiCad board)
At the start: 2 copper layers, 75 x 80 mm, 25 parts, among them M1 MountingHole_2mm, M2 MountingHole_2mm, M3 MountingHole_2mm, M4 MountingHole_2mm

Commit message: November
Parts:
- J0, J1, J2, J3, J4: footprint Connector_PinHeader_2.54mm:PinHeader_1x02_P2.54mm_Vertical -> Connector_Molex:Molex_KK-396_A-41791-0002_1x02_P3.96mm_Vertical
- moved J0 37.5 mm to (96.5, 133.3), turned to 180 degrees
- moved J4 28.1 mm to (132.1, 91.4), turned to 180 degrees
- moved C3 3.81 mm to (104.1, 132.1)
- moved J1 3.59 mm to (66.0, 90.2), turned to 90 degrees
- moved J3 2.84 mm to (128.3, 114.3), turned to 270 degrees
- moved C2 2.54 mm to (62.2, 132.1)
- turned J2 to 270 degrees
Routing:
- net /-6.3v: track 53.1 -> 77.7 mm
- net /0v: track 105.9 -> 127.7 mm
- net /OPT/Q: track 10.5 -> 24.9 mm
- net /+6.3v: track 90.6 -> 100.5 mm, vias 0 -> 1
- net /V4: track 37.4 -> 29.9 mm
- net Net-(J1-Pad1): track 70.0 -> 76.9 mm
- net Net-(C2-Pad1): track 72.9 -> 75.5 mm
- net Net-(C3-Pad2): track 71.1 -> 72.7 mm
- net /+330v: track 29.2 -> 30.4 mm
- net /V3: track 55.2 -> 55.7 mm
