File: KiCad/Quad/KT66New.sch (KiCad schematic (older format))
At the start: 13 parts

Commit message: New Backplanes
Parts:
- V3, V4: symbol kit88:KT66 -> QuadNew-rescue:KT66-kit88
Changed lines of the file:
@@
 $EndDescr
 $Comp
-L kit88:KT66 V?
+L QuadNew-rescue:KT66-kit88 V?
 U 1 1 5F7CA359
 P 2350 2000
@@
 $EndComp
 $Comp
-L kit88:KT66 V?
+L QuadNew-rescue:KT66-kit88 V?
 U 1 1 5F7CA35F
 P 3200 2000
@@
 W
 $Comp
-L kit88:KT66 V?
+L QuadNew-rescue:KT66-kit88 V?
 U 2 1 5F7F1688
 P 4500 2000
@@
 $EndComp
 $Comp
-L kit88:KT66 V?
+L QuadNew-rescue:KT66-kit88 V?
 U 2 1 5F7F168E
 P 5275 2000
