File: KiCad/Quad/PowerSupplyNew.sch (KiCad schematic (older format))
At the start: 41 parts, among them K1 ADW11, Q1 TIC106

Commit message: New Backplanes
Parts:
- TR2: symbol kit88:QuadPwrTrf -> QuadNew-rescue:QuadPwrTrf-kit88
Changed lines of the file:
@@
 $EndComp
 $Comp
-L kit88:QuadPwrTrf TR?
+L QuadNew-rescue:QuadPwrTrf-kit88 TR?
 U 1 1 5F7830F5
 P 6925 1275
